File: uprojects/Tommi Savikko/extension/extension.kicad_sch (KiCad schematic)
At the start: 8 parts, among them J1 2.0 mm SMD Socket, J2 Screw, J3 Screw, J4 Screw, J5 Screw, U1 AMS1117 5.0

Commit message: Updates 17Feb24
Connections:
- net at C1.2, C2.2, J1.3 (Pin_3)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: now also J1.1 (Pin_1), J4.2 (Pin_2)
Changed lines of the file:
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@@
   (junction (at 100.33 102.87) (diameter 0) (color 0 0 0 0)
   )
+  (junction (at 90.17 58.42) (diameter 0) (color 0 0 0 0)
+  )
   (junction (at 110.49 91.44) (diameter 0) (color 0 0 0 0)
+  )
+  (junction (at 90.17 63.5) (diameter 0) (color 0 0 0 0)
   )
   (junction (at 90.17 91.44) (diameter 0) (color 0 0 0 0)
@@
     (stroke (width 0) (type default))
   )
-  (wire (pts (xy 87.63 63.5) (xy 91.44 63.5))
+  (wire (pts (xy 87.63 63.5) (xy 90.17 63.5))
     (stroke (width 0) (type default))
   )
@@
   )
   (wire (pts (xy 85.09 71.12) (xy 91.44 71.12))
+    (stroke (width 0) (type default))
+  )
+  (wire (pts (xy 90.17 58.42) (xy 88.9 58.42))
     (stroke (width 0) (type default))
   )
@@
     (stroke (width 0) (type default))
   )
-  (wire (pts (xy 119.38 58.42) (xy 88.9 58.42))
+  (wire (pts (xy 119.38 58.42) (xy 90.17 58.42))
     (stroke (width 0) (type default))
   )
@@
     (stroke (width 0) (type default))
   )
+  (wire (pts (xy 90.17 63.5) (xy 91.44 63.5))
+    (stroke (width 0) (type default))
+  )
   (wire (pts (xy 76.2 74.93) (xy 82.55 74.93))
     (stroke (width 0) (type default))
@@
     (stroke (width 0) (type default))
   )
+  (wire (pts (xy 90.17 58.42) (xy 90.17 63.5))
+    (stroke (width 0) (type default))
+  )
