File: uprojects/Tommi Savikko/extension/extension.kicad_pcb (KiCad board)
At the start: 2 copper layers, 45.7 x 38.1 mm, 8 parts, among them J1 2.0 mm SMD Socket, J2 Screw, J3 Screw, J4 Screw, J5 Screw, U1 AMS1117 5.0

Commit message: Tommi PCB Updates
Other:
- board text added: "GND"
- board text removed: "0V"
Changed lines of the file:
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@@
         (effects (font (size 1 1) (thickness 0.15)))
     )
-    (fp_text value "100n" (at 0 1.43) (layer "F.Fab")
+    (fp_text value "100n" (at 0 1.43) (layer "F.SilkS")
         (effects (font (size 1 1) (thickness 0.15)))
     )
@@
         (effects (font (size 1 1) (thickness 0.15)))
     )
-    (fp_text value "100n" (at 0 1.43) (layer "F.Fab")
+    (fp_text value "100n" (at 0 1.43) (layer "F.SilkS")
         (effects (font (size 1 1) (thickness 0.15)))
     )
@@
         (effects (font (size 1 1) (thickness 0.15)))
     )
-    (fp_text value "2.0 mm SMD Socket" (at 0 5.5 90) (layer "F.Fab")
+    (fp_text value "2.0 mm SMD Socket" (at 0 5.5 90) (layer "F.SilkS")
         (effects (font (size 1 1) (thickness 0.15)))
     )
@@
         (effects (font (size 1 1) (thickness 0.15)))
     )
-    (fp_text value "AMS1117 5.0" (at 0 4.5) (layer "F.Fab")
+    (fp_text value "AMS1117 5.0" (at 0 4.5) (layer "F.SilkS")
         (effects (font (size 1 1) (thickness 0.15)))
     )
@@
   (gr_line (start 129.54 88.9) (end 83.82 88.9)
     (stroke (width 0.1) (type default)) (layer "Edge.Cuts"))
-  (gr_text "5V" (at 107.188 72.136) (layer "Edge.Cuts")
+  (gr_text "GND" (at 91.948 52.832 90) (layer "F.SilkS")
+    (effects (font (size 0.7 0.7) (thickness 0.15)) (justify left bottom))
+  )
+  (gr_text "5V" (at 107.188 72.136) (layer "F.SilkS")
     (effects (font (size 1 1) (thickness 0.15)) (justify left bottom))
   )
-  (gr_text "0V" (at 123.698 72.39 90) (layer "Edge.Cuts")
+  (gr_text "5V" (at 93.98 54.864 90) (layer "F.SilkS")
+    (effects (font (size 0.7 0.7) (thickness 0.15)) (justify left bottom))
+  )
+  (gr_text "GND" (at 89.662 54.864 90) (layer "F.SilkS")
+    (effects (font (size 0.7 0.7) (thickness 0.15)) (justify left bottom))
+  )
+  (gr_text "5V" (at 96.012 54.864 90) (layer "F.SilkS")
+    (effects (font (size 0.7 0.7) (thickness 0.15)) (justify left bottom))
+  )
+  (gr_text "GND" (at 125.222 72.39 90) (layer "F.SilkS")
     (effects (font (size 1 1) (thickness 0.15)) (justify left bottom))
   )
-  (gr_text "12V" (at 116.332 72.136) (layer "Edge.Cuts")
+  (gr_text "12V" (at 116.332 72.136) (layer "F.SilkS")
     (effects (font (size 1 1) (thickness 0.15)) (justify left bottom))
   )
-  (gr_text "0V" (at 113.792 72.136 90) (layer "Edge.Cuts")
+  (gr_text "GND" (at 113.792 72.136 90) (layer "F.SilkS")
     (effects (font (size 1 1) (thickness 0.15)) (justify left bottom))
   )

Commit message: Updates 17Feb24
Connections:
- C1 pad 2: Net-(J1-Pin_3) -> Net-(J1-Pin_1)
- C2 pad 2: Net-(J1-Pin_3) -> Net-(J1-Pin_1)
- J1 pad 3: Net-(J1-Pin_3) -> Net-(J1-Pin_1)
- J5 pad 2: Net-(J1-Pin_3) -> Net-(J1-Pin_1)
- U1 pad 1: Net-(J1-Pin_3) -> Net-(J1-Pin_1)
Routing:
- net Net-(J1-Pin_1): track 47.5 -> 139.6 mm, vias 0 -> 2
- net Net-(J1-Pin_3): track 90.1 -> 0.00 mm, vias 2 -> 0
Other:
- board text added: "GPIO"
