File: uprojects/Sufyan Mukadam/controllinoA/controllinoA.kicad_sch (KiCad schematic)
At the start: 4 parts, among them U1 ATmega2560-16A, Y1 16MHz

Commit message: Feb 5 commit
Connections:
- net +5V: now also U1.100 (AVCC)
Changed lines of the file:
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@@
   (junction (at 82.55 40.64) (diameter 0) (color 0 0 0 0)
+  )
+  (junction (at 123.19 27.94) (diameter 0) (color 0 0 0 0)
   )
   (wire (pts (xy 82.55 40.64) (xy 82.55 41.91))
@@
     (stroke (width 0) (type default))
   )
+  (wire (pts (xy 125.73 27.94) (xy 123.19 27.94))
+    (stroke (width 0) (type default))
+  )
   (wire (pts (xy 62.23 43.18) (xy 66.04 43.18))
     (stroke (width 0) (type default))
@@
     (stroke (width 0) (type default))
   )
-  (wire (pts (xy 123.19 25.4) (xy 123.19 30.48))
+  (wire (pts (xy 123.19 25.4) (xy 123.19 27.94))
     (stroke (width 0) (type default))
   )
@@
     (stroke (width 0) (type default))
   )
+  (wire (pts (xy 123.19 27.94) (xy 123.19 30.48))
+    (stroke (width 0) (type default))
+  )
   (wire (pts (xy 54.61 41.91) (xy 54.61 40.64))
     (stroke (width 0) (type default))
@@
     (stroke (width 0) (type default))
   )
+  (wire (pts (xy 125.73 30.48) (xy 125.73 27.94))
+    (stroke (width 0) (type default))
+  )

Commit message: Feb 6 commit
Parts:
- added C3: 100n, symbol Device:C_Small
- added J1: AVR-ISP-6, symbol Connector:AVR-ISP-6
- added R1: 10E, symbol Device:R_Small
Connections:
- net +5V: now also J1.2 (VCC), R1.1; no longer U1.100 (AVCC)
- net GND: now also C3.1, J1.6 (GND)
- net at U1.30 (~{RESET}): now also J1.5 (~{RST})
- net at U1.98 (AREF): now also C3.2
- new net: R1.2, U1.100 (AVCC)
Other:
- moved on the sheet: C1, C2, U1, Y1

Commit message: Feb 6 commit
Parts:
- added C4, C5: 100n, symbol Device:C_Small
Connections:
- net +5V: now also C4.2
- net GND: now also C4.1, C5.2
- net at R1.2, U1.100 (AVCC): now also C5.1
Changed lines of the file:
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@@
   (junction (at 158.75 87.63) (diameter 0) (color 0 0 0 0)
   )
+  (junction (at 218.44 62.23) (diameter 0) (color 0 0 0 0)
+  )
+  (junction (at 215.9 53.34) (diameter 0) (color 0 0 0 0)
+  )
   (junction (at 158.75 83.82) (diameter 0) (color 0 0 0 0)
   )
@@
   (junction (at 175.26 81.28) (diameter 0) (color 0 0 0 0)
   )
+  (wire (pts (xy 215.9 53.34) (xy 215.9 71.12))
+    (stroke (width 0) (type default))
+  )
   (wire (pts (xy 175.26 81.28) (xy 175.26 82.55))
     (stroke (width 0) (type default))
   )
-  (wire (pts (xy 218.44 60.96) (xy 218.44 71.12))
+  (wire (pts (xy 218.44 60.96) (xy 218.44 62.23))
     (stroke (width 0) (type default))
   )
@@
     (stroke (width 0) (type default))
   )
+  (wire (pts (xy 207.01 53.34) (xy 201.93 53.34))
+    (stroke (width 0) (type default))
+  )
   (wire (pts (xy 181.61 81.28) (xy 175.26 81.28))
     (stroke (width 0) (type default))
@@
     (stroke (width 0) (type default))
   )
+  (wire (pts (xy 218.44 62.23) (xy 229.87 62.23))
+    (stroke (width 0) (type default))
+  )
+  (wire (pts (xy 234.95 62.23) (xy 240.03 62.23))
+    (stroke (width 0) (type default))
+  )
   (wire (pts (xy 218.44 55.88) (xy 218.44 45.72))
     (stroke (width 0) (type default))
@@
     (stroke (width 0) (type default))
   )
+  (wire (pts (xy 240.03 62.23) (xy 240.03 67.31))
+    (stroke (width 0) (type default))
+  )
   (wire (pts (xy 158.75 81.28) (xy 158.75 83.82))
     (stroke (width 0) (type default))
   )
+  (wire (pts (xy 212.09 53.34) (xy 215.9 53.34))
+    (stroke (width 0) (type default))
+  )
+  (wire (pts (xy 201.93 53.34) (xy 201.93 58.42))
+    (stroke (width 0) (type default))
+  )
   (wire (pts (xy 165.1 39.37) (xy 165.1 43.18))
     (stroke (width 0) (type default))
@@
     (stroke (width 0) (type default))
   )
+  (wire (pts (xy 218.44 62.23) (xy 218.44 71.12))
+    (stroke (width 0) (type default))
+  )
   (wire (pts (xy 189.23 58.42) (xy 189.23 78.74))
     (stroke (width 0) (type default))
@@
     (stroke (width 0) (type default))
   )
-  (wire (pts (xy 215.9 45.72) (xy 215.9 71.12))
+  (wire (pts (xy 215.9 45.72) (xy 215.9 53.34))
     (stroke (width 0) (type default))
   )
@@
         (path "/cbf855aa-4ce6-42b1-9e73-b0ae89d280ce"
           (reference "Y1") (unit 1)
+        )
+      )
+    )
+  )
+  (symbol (lib_id "power:GND") (at 201.93 58.42 0) (unit 1)
+    (in_bom yes) (on_board yes) (dnp no) (fields_autoplaced)
+    (property "Reference" "#PWR05" (at 201.93 64.77 0)
+      (effects (font (size 1.27 1.27)) hide)
+    )
+    (property "Value" "GND" (at 201.93 63.5 0)
+      (effects (font (size 1.27 1.27)))
+    )
+    (property "Footprint" "" (at 201.93 58.42 0)
+      (effects (font (size 1.27 1.27)) hide)
+    )
+    (property "Datasheet" "" (at 201.93 58.42 0)
+      (effects (font (size 1.27 1.27)) hide)
+    )
+    (pin "1")
+    (instances
+      (project "controllinoA"
+        (path "/cbf855aa-4ce6-42b1-9e73-b0ae89d280ce"
+          (reference "#PWR05") (unit 1)
         )
       )
@@
     )
   )
+  (symbol (lib_id "Device:C_Small") (at 232.41 62.23 90) (unit 1)
+    (in_bom yes) (on_board yes) (dnp no)
+    (property "Reference" "C5" (at 234.95 59.69 90)
+      (effects (font (size 1.27 1.27)))
+    )
+    (property "Value" "100n" (at 229.87 59.69 90)
+      (effects (font (size 1.27 1.27)))
+    )
+    (property "Footprint" "" (at 232.41 62.23 0)
+      (effects (font (size 1.27 1.27)) hide)
+    )
+    (property "Datasheet" "~" (at 232.41 62.23 0)
+      (effects (font (size 1.27 1.27)) hide)
+    )
+    (pin "2")
+    (pin "1")
+    (instances
+      (project "controllinoA"
+        (path "/cbf855aa-4ce6-42b1-9e73-b0ae89d280ce"
+          (reference "C5") (unit 1)
+        )
+      )
+    )
+  )
   (symbol (lib_id "power:+5V") (at 165.1 39.37 0) (unit 1)
     (in_bom yes) (on_board yes) (dnp no) (fields_autoplaced)
@@
         )
       )
+    )
+  )
+  (symbol (lib_id "Device:C_Small") (at 209.55 53.34 90) (unit 1)
+    (in_bom yes) (on_board yes) (dnp no)
+    (property "Reference" "C4" (at 212.09 50.8 90)
+      (effects (font (size 1.27 1.27)))
+    )
+    (property "Value" "100n" (at 207.01 50.8 90)
+      (effects (font (size 1.27 1.27)))
+    )
+    (property "Footprint" "" (at 209.55 53.34 0)
+      (effects (font (size 1.27 1.27)) hide)
+    )
+    (property "Datasheet" "~" (at 209.55 53.34 0)
+      (effects (font (size 1.27 1.27)) hide)
+    )
+    (pin "2")
+    (pin "1")
+    (instances
+      (project "controllinoA"
+        (path "/cbf855aa-4ce6-42b1-9e73-b0ae89d280ce"
+          (reference "C4") (unit 1)
+        )
+      )
+    )
+  )
+  (symbol (lib_id "power:GND") (at 240.03 67.31 0) (unit 1)
+    (in_bom yes) (on_board yes) (dnp no) (fields_autoplaced)
+    (property "Reference" "#PWR06" (at 240.03 73.66 0)
+      (effects (font (size 1.27 1.27)) hide)
+    )
+    (property "Value" "GND" (at 240.03 72.39 0)
+      (effects (font (size 1.27 1.27)))
+    )
+    (property "Footprint" "" (at 240.03 67.31 0)
+      (effects (font (size 1.27 1.27)) hide)
+    )
+    (property "Datasheet" "" (at 240.03 67.31 0)
+      (effects (font (size 1.27 1.27)) hide)
+    )
+    (pin "1")
+    (instances
+      (project "controllinoA"
+        (path "/cbf855aa-4ce6-42b1-9e73-b0ae89d280ce"
+          (reference "#PWR06") (unit 1)
+        )
+      )

Commit message: Updates 17Feb24
Parts:
- added C10, C8, C9: 100n, Capacitor_SMD:C_0805_2012Metric_Pad1.18x1.45mm_HandSolder, symbol Device:C_Small
- added C6, C7: 100uF/35V, Capacitor_SMD:CP_Elec_6.3x7.7, symbol Device:C_Polarized_Small
- added D1, D19, D20, D21, D22, D23, D24, D25, D26, D3, D4, D5, D6, D7, D8, D9: LED, LED_SMD:LED_0805_2012Metric_Pad1.15x1.40mm_HandSolder, symbol Device:LED_Small
- added D10: SS14, Diode_SMD:D_SOD-128, symbol Device:D_Schottky
- added D11, D12, D13, D14, D15, D16, D17, D2: sch, Diode_SMD:D_SOD-128, symbol Device:D_Schottky
- added D18: ESDLC5V0PB8, Package_DFN_QFN:UDFN-9_1.0x3.8mm_P0.5mm, symbol Power_Protection:ESDLC5V0PB8
- added K1, K2, K3, K4, K5, K6, K7, K8: G5LE-1, Relay_THT:Relay_SPDT_Omron-G5LE-1, symbol Relay:G5LE-1
- added L1: 33uH, Inductor_SMD:L_Bourns_SRR1210A, symbol Device:L_Small
- added L10: L_Small, Inductor_SMD:L_1206_3216Metric, symbol Device:L_Small
- added L2, L3, L4, L5, L6, L7, L8, L9: bead, Inductor_SMD:L_1206_3216Metric, symbol Device:L_Small
- added R10: 4K7, Resistor_SMD:R_0805_2012Metric_Pad1.20x1.40mm_HandSolder, symbol Device:R_Small
- added R18, R28, R30, R32, R34, R36, R38, R40: 68K, Resistor_SMD:R_0805_2012Metric_Pad1.20x1.40mm_HandSolder, symbol Device:R_Small
- added R19, R29, R31, R33, R35, R37, R39, R41: 33K, Resistor_SMD:R_0805_2012Metric_Pad1.20x1.40mm_HandSolder, symbol Device:R_Small
- added R2, R20, R21, R22, R23, R24, R25, R26, R27, R3, R4, R5, R6, R7, R8, R9: 1K, Resistor_SMD:R_0805_2012Metric_Pad1.20x1.40mm_HandSolder, symbol Device:R_Small
- added U10, U11, U2, U4: ULN2003A, Package_SO:SOIC-16_3.9x9.9mm_P1.27mm, symbol Transistor_Array:ULN2003A
- added U3: LM2596S-5, Package_TO_SOT_SMD:TO-263-5_TabPin3, symbol Regulator_Switching:LM2596S-5
- C1, C2, C3, C4, C5: footprint (none) -> Capacitor_SMD:C_0805_2012Metric_Pad1.18x1.45mm_HandSolder
- J1: footprint (none) -> Connector_IDC:IDC-Header_2x03_P2.54mm_Vertical
- R1: footprint (none) -> Resistor_SMD:R_0805_2012Metric_Pad1.20x1.40mm_HandSolder
- Y1: footprint (none) -> Crystal:Crystal_HC49-U_Vertical
Connections:
- net +5V: now also C7.1, D11.1 (K), D12.1 (K), D13.1 (K), D14.1 (K), D15.1 (K), D16.1 (K), D17.1 (K), D2.1 (K), K1.5, K2.5, K3.5, K4.5, K5.5, K6.5, K7.5, K8.5, L1.2, R20.1, R21.1, R22.1, R23.1, R24.1, R25.1, R26.1, R27.1, U10.9 (COM), U11.9 (COM), U2.9 (COM), U3.4 (FB), U4.9 (COM)
- net GND: now also C6.2, C7.2, D10.2 (A), D18.3 (A), R19.1, R29.1, R31.1, R33.1, R35.1, R37.1, R39.1, R41.1, U10.8 (GND), U11.8 (GND), U2.8 (GND), U3.3 (GND), U3.5 (~{ON}/OFF), U4.8 (GND)
- net SCK: now reaches U1.20 (PB1)
- net SCK: now also J1.3 (SCK)
- net MOSI: now reaches U1.21 (PB2)
- net MOSI: now also J1.4 (MOSI)
- net MISO: now reaches U1.22 (PB3)
- net MISO: now also J1.1 (MISO)
- net at U1.71 (PA7): now also R9.1
- net at U1.72 (PA6): now also R8.1
- net at U1.73 (PA5): now also R7.1
- net at U1.74 (PA4): now also R6.1
- net at U1.75 (PA3): now also R5.1
- net at U1.76 (PA2): now also R4.1
- net at U1.77 (PA1): now also R3.1
- net at U1.78 (PA0): now also R2.1
- net IO07: now reaches U1.90 (PF7)
- net IO07: now also D18.9 (K8), R40.2, R41.2, U11.1 (I1)
- net IO06: now reaches U1.91 (PF6)
- net IO06: now also D18.8 (K7), R38.2, R39.2, U10.7 (I7)
- net IO05: now reaches U1.92 (PF5)
- net IO05: now also D18.7 (K6), R36.2, R37.2, U10.6 (I6)
- net IO04: now reaches U1.93 (PF4)
- net IO04: now also D18.6 (K5), R34.2, R35.2, U10.5 (I5)
- net IO03: now reaches U1.94 (PF3)
- net IO03: now also D18.5 (K4), R32.2, R33.2, U10.4 (I4)
- net IO02: now reaches U1.95 (PF2)
- net IO02: now also D18.4 (K3), R30.2, R31.2, U10.3 (I3)
- net IO01: now reaches U1.96 (PF1)
- net IO01: now also D18.2 (K2), R28.2, R29.2, U10.2 (I2)
- net IO00: now reaches U1.97 (PF0)
- net IO00: now also D18.1 (K1), R18.2, R19.2, U10.1 (I1)
- new net: D25.1 (K), U10.10 (O7)
- new net: D25.2 (A), R26.2
- new net: D3.2 (A), R3.2
- new net: D11.2 (A), K2.2, U2.15 (O2)
- new net: D9.2 (A), R9.2
- new net: D26.1 (K), U11.16 (O1)
- new net: D26.2 (A), R27.2
- new net: D5.2 (A), R5.2
- new net: D22.1 (K), U10.13 (O4)
- new net: D22.2 (A), R23.2
- new net: D20.1 (K), U10.15 (O2)
- new net: D20.2 (A), R21.2
- new net: L3.2, R28.1
- new net: D14.2 (A), K5.2, U2.12 (O5)
- new net: D10.1 (K), L1.1, U3.2 (OUT)
- new net: D24.2 (A), R25.2
- new net: D13.2 (A), K4.2, U2.13 (O4)
- new net: C10.1, C8.1, C9.1
- new net: C9.2, L10.1, R10.2
- new net: D1.2 (A), R2.2
- new net: L6.2, R34.1
- new net: D6.1 (K), U2.5 (I5)
- new net: D6.2 (A), R6.2
- new net: D7.2 (A), R7.2
- new net: D9.1 (K), U4.1 (I1)
- new net: D16.2 (A), K7.2, U2.10 (O7)
- new net: C8.2, R10.1
- new net: D3.1 (K), U2.2 (I2)
- new net: D4.2 (A), R4.2
- new net: D23.1 (K), U10.12 (O5)
- new net: D23.2 (A), R24.2
- new net: D2.2 (A), K1.2, U2.16 (O1)
- new net: D17.2 (A), K8.2, U4.16 (O1)
- new net: D21.1 (K), U10.14 (O3)
- new net: D21.2 (A), R22.2
- new net: L4.2, R30.1
- new net: D12.2 (A), K3.2, U2.14 (O3)
- new net: D4.1 (K), U2.3 (I3)
- new net: D24.1 (K), U10.11 (O6)
- new net: D19.1 (K), U10.16 (O1)
- new net: C6.1, U3.1 (VIN)
- new net: D1.1 (K), U2.1 (I1)
- new net: L7.2, R36.1
- new net: D19.2 (A), R20.2
- new net: L2.2, R18.1
- new net: L8.2, R38.1
- new net: C10.2, L10.2
- new net: D8.2 (A), R8.2
- new net: L5.2, R32.1
- new net: D8.1 (K), U2.7 (I7)
- new net: L9.2, R40.1
- new net: D15.2 (A), K6.2, U2.11 (O6)
- new net: D7.1 (K), U2.6 (I6)
- new net: D5.1 (K), U2.4 (I4)

Commit message: Updates 17Feb24
Parts:
- added J2: Conn_01x10, Connector_PinHeader_2.54mm:PinHeader_1x10_P2.54mm_Vertical, symbol Connector_Generic:Conn_01x10
Connections:
- net OC3A: now reaches U1.5 (PE3)
- net OC3A: now also C8.2, R10.1
- net OC3B: now reaches U1.6 (PE4)
- net OC3C: now reaches U1.7 (PE5)
- net at L2.1: now also J2.1 (Pin_1)
Other:
- moved on the sheet: C10, C8, C9, L10, R10

Commit message: Updates 22Feb24
Parts:
- removed D18: ESDLC5V0PB8, Package_DFN_QFN:UDFN-9_1.0x3.8mm_P0.5mm, symbol Power_Protection:ESDLC5V0PB8
- added C11: 100n, Capacitor_SMD:C_0805_2012Metric_Pad1.18x1.45mm_HandSolder, symbol Device:C_Small
- added C12, C13, C14, C15, C16, C17, C18, C19: 220n, Capacitor_SMD:C_0805_2012Metric_Pad1.18x1.45mm_HandSolder, symbol Device:C_Small
- added J3: Conn_01x05, Connector_PinHeader_2.54mm:PinHeader_1x05_P2.54mm_Vertical, symbol Connector_Generic:Conn_01x05
- added J4, J5: Conn_01x10, Connector_Phoenix_MC:PhoenixContact_MCV_1,5_10-G-3.5_1x10_P3.50mm_Vertical, symbol Connector_Generic:Conn_01x10
- added J6: Conn_01x03, Connector_Phoenix_MC_HighVoltage:PhoenixContact_MCV_1,5_3-G-5.08_1x03_P5.08mm_Vertical, symbol Connector_Generic:Conn_01x03
- added U5: TPD8F003, Package_SON:WSON-16_3.3x1.35_P0.4mm, symbol Power_Protection:TPD8F003
Connections:
- net +5V: now also C11.2
- net GND: now also C10.1, C8.1, C9.1, U1.11 (GND), U1.32 (GND), U1.62 (GND), U1.81 (GND), U1.99 (GND), C11.1, C12.1, C13.1, C14.1, C15.1, C16.1, C17.1, C18.1, C19.1, J6.2 (Pin_2), U5.17 (GND)
- net IO00: now also C12.2, U5.16 (Ch1_Out); no longer R18.2, R19.2
- net IO01: now also C13.2, U5.15 (Ch2_Out); no longer R28.2, R29.2
- net IO02: now also C14.2, U5.14 (Ch3_Out); no longer R30.2, R31.2
- net IO03: now also C15.2, U5.13 (Ch4_Out); no longer R32.2, R33.2
- net IO04: now also C16.2, U5.12 (Ch5_Out); no longer R34.2, R35.2
- net IO05: now also C17.2, U5.11 (Ch6_Out); no longer R36.2, R37.2
- net IO06: now also C18.2, U5.10 (Ch7_Out); no longer R38.2, R39.2
- net IO07: now also C19.2, U5.9 (Ch8_Out); no longer R40.2, R41.2
- net at K2.1: now also J4.4 (Pin_4)
- net at K2.3: now also J4.3 (Pin_3)
- net at K5.1: now also J5.2 (Pin_2)
- net at K5.3: now also J5.1 (Pin_1)
- net at K7.1: now also J5.6 (Pin_6)
- net at K7.3: now also J5.5 (Pin_5)
- net at K4.1: now also J4.8 (Pin_8)
- net at K4.3: now also J4.7 (Pin_7)
- net at J2.2 (Pin_2): now also L3.1
- net at J2.3 (Pin_3): now also L4.1
- net at J2.4 (Pin_4): now also L5.1
- net at J2.5 (Pin_5): now also L6.1
- net at J2.6 (Pin_6): now also L7.1
- net at J2.7 (Pin_7): now also L8.1
- net at J2.8 (Pin_8): now also L9.1
- net at C6.1, U3.1 (VIN): now also J6.1 (Pin_1)
- net at C10.2, L10.2: now also J3.1 (Pin_1)
- net at K6.1: now also J5.4 (Pin_4)
- net at K6.3: now also J5.3 (Pin_3)
- net at K1.1: now also J4.2 (Pin_2)
- net at K1.3: now also J4.1 (Pin_1)
- net at K8.1: now also J5.8 (Pin_8)
- net at K8.3: now also J5.7 (Pin_7)
- net at K3.1: now also J4.6 (Pin_6)
- net at K3.3: now also J4.5 (Pin_5)
- new net A0: R18.2, R19.2, U5.1 (Ch1_In)
- new net A1: R28.2, R29.2, U5.2 (Ch2_In)
- new net A2: R30.2, R31.2, U5.3 (Ch3_In)
- new net A3: R32.2, R33.2, U5.4 (Ch4_In)
- new net A4: R34.2, R35.2, U5.5 (Ch5_In)
- new net A5: R36.2, R37.2, U5.6 (Ch6_In)
- new net A6: R38.2, R39.2, U5.7 (Ch7_In)
- new net A7: R40.2, R41.2, U5.8 (Ch8_In)

Commit message: Feb 22 commit
Other:
- added sheet Ethernet (untitled.kicad_sch)
Changed lines of the file:
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@@
   )
   (symbol (lib_id "Device:L_Small") (at 86.36 91.44 90) (unit 1)
-    (in_bom yes) (on_board yes) (dnp no) (fields_autoplaced)
-    (property "Reference" "L1" (at 86.36 86.36 90)
+    (in_bom yes) (on_board yes) (dnp no)
+    (property "Reference" "L1" (at 81.28 88.9 90)
       (effects (font (size 1.27 1.27)))
     )
@@
       )
     )
+  )
+  (sheet (at 189.23 254) (size 78.74 21.59) (fields_autoplaced)
+    (stroke (width 0.1524) (type solid))
+    (fill (color 0 0 0 0.0000))
+    (property "Sheetname" "Ethernet" (at 189.23 253.2884 0)
+      (effects (font (size 1.27 1.27)) (justify left bottom))
+    )
+    (property "Sheetfile" "untitled.kicad_sch" (at 189.23 276.1746 0)
+      (effects (font (size 1.27 1.27)) (justify left top))
+    )
+    (instances
+      (project "controllinoA"
+        (path "/cbf855aa-4ce6-42b1-9e73-b0ae89d280ce" (page "2"))
+      )
+    )
