File: uprojects/Sufyan Mukadam/controllinoA/controllinoA.kicad_sch (KiCad schematic)
At the start: 156 parts, among them J1 AVR-ISP-6, J2 Conn_01x10, J3 Conn_01x05, J4 Conn_01x10, J5 Conn_01x10, J6 Conn_01x03, J7 Conn_01x10, J8 USB_C_Receptacle_USB2.0, K1 G5LE-1, K2 G5LE-1, K3 G5LE-1, K4 G5LE-1, K5 G5LE-1, K6 G5LE-1, K7 G5LE-1, K8 G5LE-1, U1 ATmega2560-16A, U10 ULN2003A, U11 ULN2003A, U12 CH340G, U13 TLP250, U2 ULN2003A, U3 LM2596S-5, U4 ULN2003A, U5 TPD8F003, U7 TPD8F003, U8 TPD8F003, U9 ULN2003A, Y1 16MHz, Y2 12MHz

Commit message: Feb 26 commit
Parts:
- added C9: 100n, Capacitor_SMD:C_0805_2012Metric_Pad1.18x1.45mm_HandSolder, symbol Device:C_Small
- added J9: Conn_01x02, Connector_PinHeader_2.54mm:PinHeader_1x02_P2.54mm_Vertical, symbol Connector_Generic:Conn_01x02
- added R59, R60: 5.1K, Resistor_SMD:R_0805_2012Metric_Pad1.20x1.40mm_HandSolder, symbol Device:R_Small
Connections:
- net +5V: now also C18.2, J9.1 (Pin_1)
- net GND: now also C18.1, J8.A1 (GND), J8.A12 (GND), J8.B1 (GND), J8.B12 (GND), C9.1, R59.1, R60.1; no longer C18.2
- net DO0: now reaches J3.1 (Pin_1)
- net DO0: now also U13.6 (VO), U13.7 (VO)
- net at J8.A4 (VBUS), J8.A9 (VBUS), J8.B4 (VBUS)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: now also J9.2 (Pin_2)
- net at J8.A5 (CC1): now also R59.2
- net USBDP: now reaches J8.A6 (D+)
- net USBDP: now also J8.B6 (D+), U12.5 (UD+)
- net USBDN: now reaches J8.A7 (D-)
- net USBDN: now also J8.B7 (D-), U12.6 (UD-)
- net at J8.B5 (CC2): now also R60.2
- net at U12.4 (V3): now also C9.2; no longer C18.1
Other:
- moved on the sheet: C18, C19, C20, U12, Y2

Commit message: Updates 27Feb24
Parts:
- added C10: 100n, Capacitor_SMD:C_0805_2012Metric_Pad1.18x1.45mm_HandSolder, symbol Device:C_Small
- added D34, D35, D36, D37, D38, D39: LED, LED_SMD:LED_0805_2012Metric_Pad1.15x1.40mm_HandSolder, symbol Device:LED_Small
- added J10: Conn_01x06, Connector_PinHeader_2.54mm:PinHeader_1x06_P2.54mm_Vertical, symbol Connector_Generic:Conn_01x06
- added J11: Conn_02x08_Odd_Even, Connector_PinHeader_2.54mm:PinHeader_2x08_P2.54mm_Vertical, symbol Connector_Generic:Conn_02x08_Odd_Even
- added R61, R62, R63, R64, R65, R66: 1K, Resistor_SMD:R_0805_2012Metric_Pad1.20x1.40mm_HandSolder, symbol Device:R_Small
- added R67, R69, R71, R73, R75: 68K, Resistor_SMD:R_0805_2012Metric_Pad1.20x1.40mm_HandSolder, symbol Device:R_Small
- added R68, R70, R72, R74, R76: 33K, Resistor_SMD:R_0805_2012Metric_Pad1.20x1.40mm_HandSolder, symbol Device:R_Small
- added R77: 100E, Resistor_SMD:R_0805_2012Metric_Pad1.20x1.40mm_HandSolder, symbol Device:R_Small
- added U6: TLP250, Package_DIP:DIP-8_W7.62mm, symbol Driver_FET:TLP250
Connections:
- net +5V: now also R61.1, R62.1, R63.1, R64.1, R65.1, R66.1
- net GND: now also C10.2, R68.1, R70.1, R72.1, R74.1, R76.1, U6.3 (C), U6.5 (VEE)
- net I16: now also R67.2, R68.2
- net I17: now also R69.2, R70.2
- net I18: now also R71.2, R72.2
- net IN0: now also R73.2, R74.2
- net IN1: now also R75.2, R76.2
- net IO08: now also U11.2 (I2)
- net IO09: now also U11.3 (I3)
- net IO10: now also U11.4 (I4)
- net IO11: now also U11.5 (I5)
- net IO12: now also U11.6 (I6)
- net IO13: now also U11.7 (I7)
- net OC3C: now also R77.1
- net DO2: now reaches U1.1 (PG5)
- net at U11.10 (O7): now also D39.1 (K)
- net at U11.11 (O6): now also D38.1 (K)
- net at U11.12 (O5): now also D37.1 (K)
- net at U11.13 (O4): now also D36.1 (K)
- net at U11.14 (O3): now also D35.1 (K)
- net at U11.15 (O2): now also D34.1 (K)
- new net: R77.2, U6.2 (A)
- new net: J10.5 (Pin_5), R75.1
- new net: D35.2 (A), R62.2
- new net: D37.2 (A), R64.2
- new net: D36.2 (A), R63.2
- new net: D34.2 (A), R61.2
- new net: J10.4 (Pin_4), R73.1
- new net: D39.2 (A), R66.2
- new net: J10.1 (Pin_1), R67.1
- new net: J10.2 (Pin_2), R69.1
- new net: J10.3 (Pin_3), R71.1
- new net: C10.1, U6.8 (VCC)
- new net: D38.2 (A), R65.2
- new net DO1: U6.6 (VO), U6.7 (VO)

Commit message: Feb 27 commit
Parts:
- added C21, C22: 100n, Capacitor_SMD:C_0805_2012Metric_Pad1.18x1.45mm_HandSolder, symbol Device:C_Small
- added C23: 100uF/35V, Capacitor_SMD:CP_Elec_6.3x7.7, symbol Device:C_Polarized_Small
- added J12: Conn_01x08, Connector_PinHeader_2.54mm:PinHeader_1x08_P2.54mm_Vertical, symbol Connector_Generic:Conn_01x08
- added J13: Conn_01x10, Connector_JST:JST_XH_B10B-XH-A_1x10_P2.50mm_Vertical, symbol Connector_Generic:Conn_01x10
- added R78, R79: 100E, Resistor_SMD:R_0805_2012Metric_Pad1.20x1.40mm_HandSolder, symbol Device:R_Small
- added U14, U15: TLP250, Package_DIP:DIP-8_W7.62mm, symbol Driver_FET:TLP250
- C12, C13, C14, C15, C16, C17: footprint Capacitor_SMD:C_0805_2012Metric_Pad1.18x1.45mm_HandSolder -> Capacitor_SMD:C_0603_1608Metric
- J11: value Conn_02x08_Odd_Even -> DO1
Connections:
- net +5V: now also U9.9 (COM), C23.1, J13.9 (Pin_9)
- net DO1: now also J3.2 (Pin_2)
- net DO2: now also J11.3 (Pin_3)
- net GND: now also U9.8 (GND), C21.2, C22.2, C23.2, J13.10 (Pin_10), U14.3 (C), U14.5 (VEE), U15.3 (C), U15.5 (VEE)
- net OC3A: now also J11.4 (Pin_4)
- net DO22: now reaches J3.3 (Pin_3)
- net DO22: now also U14.6 (VO), U14.7 (VO)
- net DO23: now reaches J3.4 (Pin_4)
- net DO23: now also U15.6 (VO), U15.7 (VO)
- net DO4: now reaches U1.15 (PH3)
- net DO4: now also J11.5 (Pin_5)
- net DO5: now reaches U1.16 (PH4)
- net DO5: now also J11.6 (Pin_6)
- net DO6: now reaches U1.17 (PH5)
- net DO6: now also J11.7 (Pin_7)
- net DO7: now reaches U1.18 (PH6)
- net DO7: now also J11.8 (Pin_8)
- net RX0: now reaches U1.2 (PE0)
- net RX0: now also U12.2 (TXD)
- net DO8: now reaches U1.23 (PB4)
- net DO8: now also J11.9 (Pin_9)
- net DO9: now reaches U1.24 (PB5)
- net DO9: now also J11.10 (Pin_10)
- net DO10: now reaches U1.25 (PB6)
- net DO10: now also J11.11 (Pin_11)
- net DO11: now reaches U1.26 (PB7)
- net DO11: now also J11.12 (Pin_12)
- net TX0: now reaches U1.3 (PE1)
- net TX0: now also U12.3 (RXD)
- net DO19: now reaches U1.35 (PL0)
- net DO19: now also J12.4 (Pin_4)
- net DO18: now reaches U1.36 (PL1)
- net DO18: now also J12.3 (Pin_3)
- net DO17: now reaches U1.37 (PL2)
- net DO17: now also J12.2 (Pin_2)
- net DO16: now reaches U1.38 (PL3)
- net DO16: now also J12.1 (Pin_1)
- net DO15: now reaches U1.39 (PL4)
- net DO15: now also J11.16 (Pin_16)
- net DO14: now reaches U1.40 (PL5)
- net DO14: now also J11.15 (Pin_15)
- net DO13: now reaches U1.41 (PL6)
- net DO13: now also J11.14 (Pin_14)
- net DO12: now reaches U1.42 (PL7)
- net DO12: now also J11.13 (Pin_13)
- net DO20: now reaches U1.47 (PD4)
- net DO20: now also J12.5 (Pin_5)
- net DO21: now reaches U1.48 (PD5)
- net DO21: now also J12.6 (Pin_6)
- net PD6: now reaches U1.49 (PD6)
- net PD6: now also R78.1
- net PJ4: now reaches U1.67 (PJ4)
- net PJ4: now also R79.1
- net at U9.15 (O2): now also J13.8 (Pin_8)
- net at U9.16 (O1): now also J13.7 (Pin_7)
- net at U4.10 (O7): now also J13.6 (Pin_6)
- net at U4.11 (O6): now also J13.5 (Pin_5)
- net at U4.12 (O5): now also J13.4 (Pin_4)
- net at U4.13 (O4): now also J13.3 (Pin_3)
- net at U4.14 (O3): now also J13.2 (Pin_2)
- net at U4.15 (O2): now also J13.1 (Pin_1)
- new net: C21.1, U14.8 (VCC)
- new net: R78.2, U14.2 (A)
- new net: C22.1, U15.8 (VCC)
- new net: R79.2, U15.2 (A)

Commit message: Updates 28Feb24
Parts:
- added D40: LED, LED_SMD:LED_0805_2012Metric_Pad1.15x1.40mm_HandSolder, symbol Device:LED_Small
- added D41, D42, D43, D44, D45, D46, D47, D48: sch, Diode_SMD:D_SOD-128, symbol Device:D_Schottky
- added J14: Conn_01x02, Connector_JST:JST_XH_B2B-XH-A_1x02_P2.50mm_Vertical, symbol Connector_Generic:Conn_01x02
- added J15: Conn_01x10, Connector_JST:JST_XH_B10B-XH-A_1x10_P2.50mm_Vertical, symbol Connector_Generic:Conn_01x10
- added J16, J17: Conn_01x10, Connector_Phoenix_MC:PhoenixContact_MCV_1,5_10-G-3.5_1x10_P3.50mm_Vertical, symbol Connector_Generic:Conn_01x10
- added K10, K11, K12, K13, K14, K15, K16, K9: G5LE-1, Relay_THT:Relay_SPDT_Omron-G5LE-1, symbol Relay:G5LE-1
- added R80, R81: 4K7, Resistor_SMD:R_0805_2012Metric_Pad1.20x1.40mm_HandSolder, symbol Device:R_Small
- added R82: 2K2, Resistor_SMD:R_0805_2012Metric_Pad1.20x1.40mm_HandSolder, symbol Device:R_Small
- added U16: DS3231M, Package_SO:SOIC-16W_7.5x10.3mm_P1.27mm, symbol Timer_RTC:DS3231M
Connections:
- net +5V: now also R80.2, R81.2, R82.1, U16.2 (VCC)
- net GND: now also J2.9 (Pin_9), J7.9 (Pin_9), D40.1 (K), J14.2 (Pin_2), J15.10 (Pin_10), U16.10 (GND), U16.11 (GND), U16.12 (GND), U16.13 (GND), U16.5 (GND), U16.6 (GND), U16.7 (GND), U16.8 (GND), U16.9 (GND)
- net 24V: now reaches C21.1, U14.8 (VCC)
- net 24V: now also C10.1, C22.1, C6.1, C8.1, J6.1 (Pin_1), U13.8 (VCC), U15.8 (VCC), U3.1 (VIN), U6.8 (VCC)
- net SCL: now reaches U1.43 (PD0)
- net SCL: now also R80.1, U16.16 (SCL)
- net SDA: now reaches U1.44 (PD1)
- net SDA: now also R81.1, U16.15 (SDA)
- new net: D40.2 (A), R82.2
- new net: J17.8 (Pin_8), K15.1
- new net: D47.2 (A), J15.8 (Pin_8), K15.2
- new net: J17.7 (Pin_7), K15.3
- new net: D41.1 (K), D42.1 (K), D43.1 (K), D44.1 (K), D45.1 (K), D46.1 (K), D47.1 (K), D48.1 (K), J15.9 (Pin_9), K10.5, K11.5, K12.5, K13.5, K14.5, K15.5, K16.5, K9.5
- new net: D41.2 (A), J15.2 (Pin_2), K9.2
- new net: J16.6 (Pin_6), K10.1
- new net: D42.2 (A), J15.3 (Pin_3), K10.2
- new net: J16.5 (Pin_5), K10.3
- new net: D46.2 (A), J15.7 (Pin_7), K14.2
- new net: J17.4 (Pin_4), K13.1
- new net: D45.2 (A), J15.6 (Pin_6), K13.2
- new net: J17.3 (Pin_3), K13.3
- new net: J16.4 (Pin_4), K9.1
- new net: J16.3 (Pin_3), K9.3
- new net: D44.2 (A), J15.5 (Pin_5), K12.2
- new net: J16.1 (Pin_1), K16.3
- new net: J16.2 (Pin_2), K16.1
- new net: J16.7 (Pin_7), K11.3
- new net: J16.8 (Pin_8), K11.1
- new net: D48.2 (A), J15.1 (Pin_1), K16.2
- new net: D43.2 (A), J15.4 (Pin_4), K11.2
- new net: J17.6 (Pin_6), K14.1
- new net: J17.5 (Pin_5), K14.3
- new net: J17.2 (Pin_2), K12.1
- new net: J17.1 (Pin_1), K12.3
- new net: J14.1 (Pin_1), U16.14 (VBAT)

Commit message: Feb 28 office commit
Parts:
- added U17: TLP2748, Package_SO:SO-6L_10x3.84mm_P1.27mm, symbol Isolator:TLP2748
Other:
- moved on the sheet: D41, D42, D43, D44, D45, D46, D47, D48, J15, J16, J17, K10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

Commit message: 11March24
Parts:
- added C24: 3.3uF / 16v, Capacitor_SMD:C_0805_2012Metric_Pad1.18x1.45mm_HandSolder, symbol Device:C_Small
- added C25, C26: 10uF / 16v, Capacitor_SMD:C_0805_2012Metric_Pad1.18x1.45mm_HandSolder, symbol Device:C_Small
- added L10: bead, Inductor_SMD:L_1206_3216Metric, symbol Device:L_Small
- added R83, R84: 4K7, Resistor_SMD:R_0805_2012Metric_Pad1.20x1.40mm_HandSolder, symbol Device:R_Small
- added U18: W5100, Package_QFP:LQFP-80_10x10mm_P0.4mm, symbol Interface_Ethernet:W5100
Connections:
- net GND: now also C24.1, C25.1, C26.1, R83.1, R84.1
- new net: U18.10 (GNDA), U18.4 (GNDA), U18.77 (GNDA)
- new net: C24.2, C25.2, L10.1, U18.11 (1V8_OUT), U18.15 (VCC1V8D), U18.16 (VCC1V8D), U18.33 (VCC1V8D), U18.69 (VCC1V8D)
- new net: U18.12 (VCC3V3D), U18.18 (VCC3V3D), U18.44 (VCC3V3D)
- new net: U18.13 (GNDD), U18.14 (GNDD), U18.17 (GNDD), U18.32 (GNDD), U18.43 (GNDD), U18.68 (GNDD)
- new net: R84.2, U18.19 (DATA7), U18.20 (DATA6), U18.21 (DATA5), U18.22 (DATA4), U18.23 (DATA3), U18.24 (DATA2), U18.25 (DATA1), U18.26 (DATA0)
- new net: R83.2, U18.38 (ADDR14), U18.39 (ADDR13), U18.40 (ADDR12), U18.41 (ADDR11), U18.42 (ADDR10), U18.45 (ADDR9), U18.46 (ADDR8), U18.47 (ADDR7), U18.48 (ADDR6), U18.49 (ADDR5), U18.50 (ADDR4), U18.51 (ADDR3), U18.52 (ADDR2), U18.53 (ADDR1), U18.54 (ADDR0)
- new net: C26.2, L10.2, U18.7 (VCC1V8A), U18.74 (VCC1V8A)

Commit message: March 11 office commit 1
Parts:
- added C27, C28: 13, Capacitor_SMD:C_0805_2012Metric_Pad1.18x1.45mm_HandSolder, symbol Device:C_Small
- added C29, C30: 100n, Capacitor_SMD:C_0805_2012Metric_Pad1.18x1.45mm_HandSolder, symbol Device:C_Small
- added C31: 10uF / 16v, Capacitor_SMD:C_0805_2012Metric_Pad1.18x1.45mm_HandSolder, symbol Device:C_Small
- added D49, D50, D51, D52, D53, D54: LED, LED_SMD:LED_0805_2012Metric_Pad1.15x1.40mm_HandSolder, symbol Device:LED_Small
- added L19, L20: bead, Inductor_SMD:L_1206_3216Metric, symbol Device:L_Small
- added R85: 12K, Resistor_SMD:R_0805_2012Metric_Pad1.20x1.40mm_HandSolder, symbol Device:R_Small
- added R86: 330, Resistor_SMD:R_0805_2012Metric_Pad1.20x1.40mm_HandSolder, symbol Device:R_Small
- added R87: 1M, Resistor_SMD:R_0805_2012Metric_Pad1.20x1.40mm_HandSolder, symbol Device:R_Small
- added R88, R89, R90, R91, R92, R93: 470, Resistor_SMD:R_0805_2012Metric_Pad1.20x1.40mm_HandSolder, symbol Device:R_Small
- added U19: LM1117MP-3.3, Package_TO_SOT_SMD:SOT-223-3_TabPin2, symbol Regulator_Linear:LM1117MP-3.3
- added Y3: 25MHz, Crystal:Crystal_SMD_ECS_CSM3X-2Pin_7.6x4.1mm, symbol Device:Crystal_Small
Connections:
- net +5V: now also C30.2, U19.3 (VI)
- net GND: now also U18.13 (GNDD), U18.14 (GNDD), U18.17 (GNDD), U18.32 (GNDD), U18.43 (GNDD), U18.68 (GNDD), C27.1, C28.1, C29.1, C30.1, C31.1, L20.2, R86.2, U19.1 (GND)
- net at U18.1 (RSET_BG): now also R85.1
- net GNDA: now reaches U18.10 (GNDA), U18.4 (GNDA), U18.77 (GNDA)
- net GNDA: now also L20.1
- net 3V3: now reaches U18.12 (VCC3V3D), U18.18 (VCC3V3D), U18.44 (VCC3V3D)
- net 3V3: now also C29.2, L19.1, R88.1, R89.1, R90.1, R91.1, R92.1, R93.1, U19.2 (VO)
- net at U18.2 (VCC3V3A): now also C31.2, L19.2
- net at U18.66 (LINKLED): now also D54.1 (K)
- net at U18.67 (SPDLED): now also D53.1 (K)
- net at U18.70 (FDXLED): now also D52.1 (K)
- net at U18.71 (COLLED): now also D51.1 (K)
- net at U18.72 (RXLED): now also D50.1 (K)
- net at U18.73 (TXLED): now also D49.1 (K)
- net XTLN: now reaches U18.75 (XTLN)
- net XTLN: now also C28.2, R87.1, Y3.1
- net XTLP: now reaches U18.76 (XTLP)
- net XTLP: now also C27.2, R87.2, Y3.2
- new net: D52.2 (A), R91.2
- new net: D54.2 (A), R93.2
- new net: D50.2 (A), R89.2
- new net: D53.2 (A), R92.2
- new net: D49.2 (A), R88.2
- new net: D51.2 (A), R90.2
- new net: R85.2, R86.1
