File: uprojects/Sufyan Mukadam/controllinoA/controllinoA.kicad_pcb (KiCad board)
At the start: 2 copper layers, 168.9 x 149.7 mm, 156 parts, among them J1 AVR-ISP-6, J2 Conn_01x10, J3 Conn_01x05, J4 Conn_01x10, J5 Conn_01x10, J6 Conn_01x03, J7 Conn_01x10, J8 USB_C_Receptacle_USB2.0, K1 G5LE-1, K2 G5LE-1, K3 G5LE-1, K4 G5LE-1, K5 G5LE-1, K6 G5LE-1, K7 G5LE-1, K8 G5LE-1, U1 ATmega2560-16A, U10 ULN2003A, U11 ULN2003A, U12 CH340G, U13 TLP250, U2 ULN2003A, U3 LM2596S-5, U4 ULN2003A, U5 TPD8F003, U7 TPD8F003, U8 TPD8F003, U9 ULN2003A, Y1 16MHz, Y2 12MHz

Commit message: Feb 26 commit
Parts:
- added C9: 100n, Capacitor_SMD:C_0805_2012Metric_Pad1.18x1.45mm_HandSolder, F.Cu at (144.6, 148.8)
- added J9: Conn_01x02, Connector_PinHeader_2.54mm:PinHeader_1x02_P2.54mm_Vertical, F.Cu at (94.5, 140.5)
- added R59: 5.1K, Resistor_SMD:R_0805_2012Metric_Pad1.20x1.40mm_HandSolder, F.Cu at (86.6, 143.5)
- added R60: 5.1K, Resistor_SMD:R_0805_2012Metric_Pad1.20x1.40mm_HandSolder, F.Cu at (86.6, 141.5)
- moved R58 115.9 mm to (146.9, 123.3)
- moved D33 114.4 mm to (150.8, 123.4)
- moved R51 113.7 mm to (147.0, 111.5)
- moved D27 112.4 mm to (150.9, 113.6), turned to 180 degrees
- moved D18 112.2 mm to (150.9, 111.5), turned to 180 degrees
- moved D28 111.6 mm to (151.7, 127.9)
- moved D29 111.6 mm to (151.7, 131.0)
- moved D30 111.6 mm to (151.7, 134.0)
- moved D31 111.6 mm to (151.7, 137.1)
- moved D32 111.6 mm to (151.7, 140.1)
- moved R52 111.6 mm to (147.0, 127.7)
- moved R53 111.6 mm to (147.0, 130.7)
- moved R54 111.6 mm to (147.0, 133.6)
- moved R55 111.6 mm to (147.0, 136.6)
- moved R56 111.6 mm to (147.0, 139.5)
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Connections:
- C18 pad 1: Net-(U12-V3) -> GND
- C18 pad 2: GND -> +5V
- J3 pad 1: unconnected-(J3-Pin_1-Pad1) -> DO0
- J8 pad A1: Net-(J8-GND-PadA1) -> GND
- J8 pad A12: Net-(J8-GND-PadA1) -> GND
- J8 pad A5: unconnected-(J8-CC1-PadA5) -> Net-(J8-CC1)
- J8 pad A6: unconnected-(J8-D+-PadA6) -> USBDP
- J8 pad A7: unconnected-(J8-D--PadA7) -> USBDN
- J8 pad B1: Net-(J8-GND-PadA1) -> GND
- J8 pad B12: Net-(J8-GND-PadA1) -> GND
- J8 pad B5: unconnected-(J8-CC2-PadB5) -> Net-(J8-CC2)
- J8 pad B6: unconnected-(J8-D+-PadB6) -> USBDP
- J8 pad B7: unconnected-(J8-D--PadB7) -> USBDN
- U12 pad 5: unconnected-(U12-UD+-Pad5) -> USBDP
- U12 pad 6: unconnected-(U12-UD--Pad6) -> USBDN
- U13 pad 6: Net-(U13-VO-Pad6) -> DO0
- U13 pad 7: Net-(U13-VO-Pad6) -> DO0
Routing:
- net GND: track 121.7 -> 161.9 mm, vias 0 -> 2
- net Net-(J9-Pin_2): track 0.00 -> 19.4 mm, vias 0 -> 2
- net Net-(J8-CC2): track 0.00 -> 18.3 mm, vias 0 -> 2
- net A7: track 22.0 -> 4.60 mm
- net A6: track 20.0 -> 4.09 mm
- net Net-(U12-XI): track 0.00 -> 13.9 mm
- net Net-(U12-XO): track 0.00 -> 12.5 mm
- net A5: track 17.4 -> 5.10 mm
- net Net-(J8-CC1): track 0.00 -> 11.1 mm
- net A4: track 16.3 -> 5.60 mm
- net USBDN: track 0.00 -> 7.72 mm
- net USBDP: track 0.00 -> 7.43 mm

Commit message: Updates 27Feb24
Parts:
- added C10: 100n, Capacitor_SMD:C_0805_2012Metric_Pad1.18x1.45mm_HandSolder, F.Cu at (145.1, 66.5)
- added D34: LED, LED_SMD:LED_0805_2012Metric_Pad1.15x1.40mm_HandSolder, F.Cu at (117.0, 69.3)
- added D35: LED, LED_SMD:LED_0805_2012Metric_Pad1.15x1.40mm_HandSolder, F.Cu at (117.0, 66.2)
- added D36: LED, LED_SMD:LED_0805_2012Metric_Pad1.15x1.40mm_HandSolder, F.Cu at (117.0, 63.2)
- added D37: LED, LED_SMD:LED_0805_2012Metric_Pad1.15x1.40mm_HandSolder, F.Cu at (117.0, 60.1)
- added D38: LED, LED_SMD:LED_0805_2012Metric_Pad1.15x1.40mm_HandSolder, F.Cu at (117.0, 57.1)
- added D39: LED, LED_SMD:LED_0805_2012Metric_Pad1.15x1.40mm_HandSolder, F.Cu at (117.0, 54.1)
- added J10: Conn_01x06, Connector_PinHeader_2.54mm:PinHeader_1x06_P2.54mm_Vertical, F.Cu at (73.1, 119.4)
- added J11: Conn_02x08_Odd_Even, Connector_PinHeader_2.54mm:PinHeader_2x08_P2.54mm_Vertical, F.Cu at (137.8, 55.5)
- added R61: 1K, Resistor_SMD:R_0805_2012Metric_Pad1.20x1.40mm_HandSolder, F.Cu at (108.3, 72.3)
- added R62: 1K, Resistor_SMD:R_0805_2012Metric_Pad1.20x1.40mm_HandSolder, F.Cu at (108.3, 70.2)
- added R63: 1K, Resistor_SMD:R_0805_2012Metric_Pad1.20x1.40mm_HandSolder, F.Cu at (112.3, 63.4)
- added R64: 1K, Resistor_SMD:R_0805_2012Metric_Pad1.20x1.40mm_HandSolder, F.Cu at (112.3, 60.5)
- added R65: 1K, Resistor_SMD:R_0805_2012Metric_Pad1.20x1.40mm_HandSolder, F.Cu at (112.3, 57.5)
- added R66: 1K, Resistor_SMD:R_0805_2012Metric_Pad1.20x1.40mm_HandSolder, F.Cu at (112.3, 54.6)
- added R67: 68K, Resistor_SMD:R_0805_2012Metric_Pad1.20x1.40mm_HandSolder, F.Cu at (87.5, 119.4)
- added R68: 33K, Resistor_SMD:R_0805_2012Metric_Pad1.20x1.40mm_HandSolder, F.Cu at (87.5, 121.6)
- added R69: 68K, Resistor_SMD:R_0805_2012Metric_Pad1.20x1.40mm_HandSolder, F.Cu at (87.5, 123.7)
- added R70: 33K, Resistor_SMD:R_0805_2012Metric_Pad1.20x1.40mm_HandSolder, F.Cu at (87.5, 125.9)
- added R71: 68K, Resistor_SMD:R_0805_2012Metric_Pad1.20x1.40mm_HandSolder, F.Cu at (87.5, 128.0)
- added R72: 33K, Resistor_SMD:R_0805_2012Metric_Pad1.20x1.40mm_HandSolder, F.Cu at (87.5, 130.0)
- added R73: 68K, Resistor_SMD:R_0805_2012Metric_Pad1.20x1.40mm_HandSolder, F.Cu at (87.5, 132.1)
- added R74: 33K, Resistor_SMD:R_0805_2012Metric_Pad1.20x1.40mm_HandSolder, F.Cu at (87.5, 134.3)
- added R75: 68K, Resistor_SMD:R_0805_2012Metric_Pad1.20x1.40mm_HandSolder, F.Cu at (107.0, 131.3)
- added R76: 33K, Resistor_SMD:R_0805_2012Metric_Pad1.20x1.40mm_HandSolder, F.Cu at (107.0, 134.3)
- added R77: 100E, Resistor_SMD:R_0805_2012Metric_Pad1.20x1.40mm_HandSolder, F.Cu at (149.9, 66.4)
- added U6: TLP250, Package_DIP:DIP-8_W7.62mm, F.Cu at (124.1, 136.8)
- moved C9 51.7 mm to (93.2, 143.5)
- moved C13 36.7 mm to (105.0, 100.6), turned to -90 degrees
- moved C14 36.1 mm to (102.8, 100.6), turned to -90 degrees
- moved C5 23.4 mm to (121.2, 96.8)
- moved C3 23.2 mm to (123.4, 96.9)
- moved U7 21.8 mm to (99.2, 69.5)
- moved C12 20.6 mm to (101.8, 96.0), turned to -90 degrees
- moved C16 19.0 mm to (99.7, 96.0), turned to -90 degrees
- moved R57 18.5 mm to (147.0, 124.0)
- moved R56 17.6 mm to (147.0, 121.9)
- moved R55 16.7 mm to (147.0, 119.8)
- moved C17 16.3 mm to (103.2, 90.6), turned to -90 degrees
- moved D32 16.1 mm to (150.8, 124.0), turned to 180 degrees
- moved R54 15.9 mm to (147.0, 117.8)
- moved D31 15.2 mm to (150.8, 121.9), turned to 180 degrees
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Connections:
- U1 pad 1: unconnected-(U1-PG5-Pad1) -> DO2
- U11 pad 10: unconnected-(U11-O7-Pad10) -> Net-(D39-K)
- U11 pad 11: unconnected-(U11-O6-Pad11) -> Net-(D38-K)
- U11 pad 12: unconnected-(U11-O5-Pad12) -> Net-(D37-K)
- U11 pad 13: unconnected-(U11-O4-Pad13) -> Net-(D36-K)
- U11 pad 14: unconnected-(U11-O3-Pad14) -> Net-(D35-K)
- U11 pad 15: unconnected-(U11-O2-Pad15) -> Net-(D34-K)
- U11 pad 2: unconnected-(U11-I2-Pad2) -> IO08
- U11 pad 3: unconnected-(U11-I3-Pad3) -> IO09
- U11 pad 4: unconnected-(U11-I4-Pad4) -> IO10
- U11 pad 5: unconnected-(U11-I5-Pad5) -> IO11
- U11 pad 6: unconnected-(U11-I6-Pad6) -> IO12
- U11 pad 7: unconnected-(U11-I7-Pad7) -> IO13
Routing:
- net Net-(U12-V3): track 0.00 -> 5.81 mm
- net GND: track 161.9 -> 157.1 mm
- net +5V: track 401.8 -> 398.0 mm, vias 12 -> 11
- net Net-(D14-A): track 26.4 -> 23.4 mm
- net IO07: track 6.29 -> 4.62 mm
- net Net-(D17-A): track 70.8 -> 72.2 mm
- net IO06: track 5.66 -> 4.40 mm

Commit message: Feb 27 commit
Parts:
- added C21: 100n, Capacitor_SMD:C_0805_2012Metric_Pad1.18x1.45mm_HandSolder, F.Cu at (149.0, 147.3)
- added C22: 100n, Capacitor_SMD:C_0805_2012Metric_Pad1.18x1.45mm_HandSolder, F.Cu at (164.2, 146.9)
- added C23: 100uF/35V, Capacitor_SMD:CP_Elec_6.3x7.7, F.Cu at (103.7, 52.9)
- added J12: Conn_01x08, Connector_PinHeader_2.54mm:PinHeader_1x08_P2.54mm_Vertical, F.Cu at (135.2, 141.2)
- added J13: Conn_01x10, Connector_JST:JST_XH_B10B-XH-A_1x10_P2.50mm_Vertical, F.Cu at (171.2, 110.6)
- added R78: 100E, Resistor_SMD:R_0805_2012Metric_Pad1.20x1.40mm_HandSolder, F.Cu at (138.9, 152.6)
- added R79: 100E, Resistor_SMD:R_0805_2012Metric_Pad1.20x1.40mm_HandSolder, F.Cu at (153.9, 152.3)
- added U14: TLP250, Package_DIP:DIP-8_W7.62mm, F.Cu at (142.1, 150.1)
- added U15: TLP250, Package_DIP:DIP-8_W7.62mm, F.Cu at (157.3, 149.8)
- C12, C13, C14, C15, C16, C17: footprint Capacitor_SMD:C_0805_2012Metric_Pad1.18x1.45mm_HandSolder -> Capacitor_SMD:C_0603_1608Metric
- J11: value Conn_02x08_Odd_Even -> DO1
- moved R77 91.0 mm to (120.9, 152.7)
- moved C10 82.1 mm to (130.7, 147.3), turned to 180 degrees
- moved J11 61.7 mm to (102.8, 106.3)
- moved C16 38.4 mm to (137.8, 91.9), turned to 180 degrees
- moved C12 36.5 mm to (137.8, 90.3), turned to 180 degrees
- moved C17 34.7 mm to (137.8, 93.6), turned to 180 degrees
- moved C15 34.6 mm to (137.8, 88.7), turned to 180 degrees
- moved R75 27.0 mm to (80.0, 132.1)
- moved R76 26.9 mm to (80.0, 134.3)
- moved C14 18.6 mm to (119.3, 92.1), turned to 0 degrees
- moved C13 17.7 mm to (119.3, 90.0), turned to 0 degrees
- moved C8 17.7 mm to (113.2, 147.5)
- moved U13 17.7 mm to (106.6, 150.2)
- moved R10 17.0 mm to (103.2, 152.7)
- moved U8 15.6 mm to (99.1, 130.1)
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Connections:
- J11 pad 10: unconnected-(J11-Pin_10-Pad10) -> DO9
- J11 pad 11: unconnected-(J11-Pin_11-Pad11) -> DO10
- J11 pad 12: unconnected-(J11-Pin_12-Pad12) -> DO11
- J11 pad 13: unconnected-(J11-Pin_13-Pad13) -> DO12
- J11 pad 14: unconnected-(J11-Pin_14-Pad14) -> DO13
- J11 pad 15: unconnected-(J11-Pin_15-Pad15) -> DO14
- J11 pad 16: unconnected-(J11-Pin_16-Pad16) -> DO15
- J11 pad 3: unconnected-(J11-Pin_3-Pad3) -> DO2
- J11 pad 4: unconnected-(J11-Pin_4-Pad4) -> OC3A
- J11 pad 5: unconnected-(J11-Pin_5-Pad5) -> DO4
- J11 pad 6: unconnected-(J11-Pin_6-Pad6) -> DO5
- J11 pad 7: unconnected-(J11-Pin_7-Pad7) -> DO6
- J11 pad 8: unconnected-(J11-Pin_8-Pad8) -> DO7
- J11 pad 9: unconnected-(J11-Pin_9-Pad9) -> DO8
- J3 pad 2: unconnected-(J3-Pin_2-Pad2) -> DO1
- J3 pad 3: unconnected-(J3-Pin_3-Pad3) -> DO22
- J3 pad 4: unconnected-(J3-Pin_4-Pad4) -> DO23
- U1 pad 15: unconnected-(U1-PH3-Pad15) -> DO4
- U1 pad 16: unconnected-(U1-PH4-Pad16) -> DO5
- U1 pad 17: unconnected-(U1-PH5-Pad17) -> DO6
- U1 pad 18: unconnected-(U1-PH6-Pad18) -> DO7
- U1 pad 2: unconnected-(U1-PE0-Pad2) -> RX0
- U1 pad 23: unconnected-(U1-PB4-Pad23) -> DO8
- U1 pad 24: unconnected-(U1-PB5-Pad24) -> DO9
- U1 pad 25: unconnected-(U1-PB6-Pad25) -> DO10
- U1 pad 26: unconnected-(U1-PB7-Pad26) -> DO11
- U1 pad 3: unconnected-(U1-PE1-Pad3) -> TX0
- U1 pad 35: unconnected-(U1-PL0-Pad35) -> DO19
- U1 pad 36: unconnected-(U1-PL1-Pad36) -> DO18
- U1 pad 37: unconnected-(U1-PL2-Pad37) -> DO17
- U1 pad 38: unconnected-(U1-PL3-Pad38) -> DO16
- U1 pad 39: unconnected-(U1-PL4-Pad39) -> DO15
- U1 pad 40: unconnected-(U1-PL5-Pad40) -> DO14
- U1 pad 41: unconnected-(U1-PL6-Pad41) -> DO13
- U1 pad 42: unconnected-(U1-PL7-Pad42) -> DO12
- U1 pad 47: unconnected-(U1-PD4-Pad47) -> DO20
- U1 pad 48: unconnected-(U1-PD5-Pad48) -> DO21
- U1 pad 49: unconnected-(U1-PD6-Pad49) -> PD6
- U1 pad 67: unconnected-(U1-PJ4-Pad67) -> PJ4
- U12 pad 2: unconnected-(U12-TXD-Pad2) -> RX0
- U12 pad 3: unconnected-(U12-RXD-Pad3) -> TX0
- U4 pad 10: unconnected-(U4-O7-Pad10) -> Net-(J13-Pin_6)
- U4 pad 11: unconnected-(U4-O6-Pad11) -> Net-(J13-Pin_5)
- U4 pad 12: unconnected-(U4-O5-Pad12) -> Net-(J13-Pin_4)
- U4 pad 13: unconnected-(U4-O4-Pad13) -> Net-(J13-Pin_3)
- U4 pad 14: unconnected-(U4-O3-Pad14) -> Net-(J13-Pin_2)
- U4 pad 15: unconnected-(U4-O2-Pad15) -> Net-(J13-Pin_1)
- U9 pad 15: unconnected-(U9-O2-Pad15) -> Net-(J13-Pin_8)
- U9 pad 16: unconnected-(U9-O1-Pad16) -> Net-(J13-Pin_7)
- U9 pad 8: unconnected-(U9-GND-Pad8) -> GND
- U9 pad 9: unconnected-(U9-COM-Pad9) -> +5V
Routing:
- net GND: track 157.1 -> 889.4 mm, vias 2 -> 32
- net +5V: track 398.0 -> 641.9 mm, vias 11 -> 19
- net IO12: track 0.00 -> 73.7 mm, vias 0 -> 2
- net IO08: track 0.00 -> 73.1 mm, vias 0 -> 2
- net RX0: track 0.00 -> 71.4 mm, vias 0 -> 2
- net IO13: track 0.00 -> 71.3 mm, vias 0 -> 3
- net IO09: track 0.00 -> 71.1 mm, vias 0 -> 2
- net IO10: track 0.00 -> 70.4 mm, vias 0 -> 2
- net IO15: track 0.00 -> 69.9 mm, vias 0 -> 2
- net IO11: track 0.00 -> 69.8 mm, vias 0 -> 2
- net IO14: track 0.00 -> 69.3 mm, vias 0 -> 2
- net IO17: track 0.00 -> 68.1 mm, vias 0 -> 2
- net OC3C: track 0.00 -> 66.9 mm, vias 0 -> 2
- net IO20: track 0.00 -> 65.2 mm, vias 0 -> 2
- net IO19: track 0.00 -> 63.8 mm, vias 0 -> 2
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Other:
- board text removed: "Analog Out"
- board text removed: "Digital/Analog In"

Commit message: Updates 28Feb24
Parts:
- added D40: LED, LED_SMD:LED_0805_2012Metric_Pad1.15x1.40mm_HandSolder, F.Cu at (89.5, 36.7)
- added D41: sch, Diode_SMD:D_SOD-128, F.Cu at (205.1, 142.0)
- added D42: sch, Diode_SMD:D_SOD-128, F.Cu at (205.1, 124.2)
- added D43: sch, Diode_SMD:D_SOD-128, F.Cu at (205.1, 106.4)
- added D44: sch, Diode_SMD:D_SOD-128, F.Cu at (205.1, 87.9)
- added D45: sch, Diode_SMD:D_SOD-128, F.Cu at (205.1, 70.0)
- added D46: sch, Diode_SMD:D_SOD-128, F.Cu at (205.2, 51.9)
- added D47: sch, Diode_SMD:D_SOD-128, F.Cu at (205.2, 33.3)
- added D48: sch, Diode_SMD:D_SOD-128, F.Cu at (205.2, 160.6)
- added J14: Conn_01x02, Connector_JST:JST_XH_B2B-XH-A_1x02_P2.50mm_Vertical, F.Cu at (108.6, 81.6)
- added J15: Conn_01x10, Connector_JST:JST_XH_B10B-XH-A_1x10_P2.50mm_Vertical, F.Cu at (190.7, 104.8)
- added J16: Conn_01x10, Connector_Phoenix_MC:PhoenixContact_MCV_1,5_10-G-3.5_1x10_P3.50mm_Vertical, F.Cu at (243.4, 143.3)
- added J17: Conn_01x10, Connector_Phoenix_MC:PhoenixContact_MCV_1,5_10-G-3.5_1x10_P3.50mm_Vertical, F.Cu at (243.3, 73.8)
- added K10: G5LE-1, Relay_THT:Relay_SPDT_Omron-G5LE-1, F.Cu at (210.0, 124.1)
- added K11: G5LE-1, Relay_THT:Relay_SPDT_Omron-G5LE-1, F.Cu at (210.0, 106.0)
- added K12: G5LE-1, Relay_THT:Relay_SPDT_Omron-G5LE-1, F.Cu at (210.0, 88.0)
- added K13: G5LE-1, Relay_THT:Relay_SPDT_Omron-G5LE-1, F.Cu at (210.0, 69.9)
- added K14: G5LE-1, Relay_THT:Relay_SPDT_Omron-G5LE-1, F.Cu at (210.0, 51.9)
- added K15: G5LE-1, Relay_THT:Relay_SPDT_Omron-G5LE-1, F.Cu at (210.0, 33.8)
- added K16: G5LE-1, Relay_THT:Relay_SPDT_Omron-G5LE-1, F.Cu at (210.1, 159.8)
- added K9: G5LE-1, Relay_THT:Relay_SPDT_Omron-G5LE-1, F.Cu at (210.0, 142.1)
- added R80: 4K7, Resistor_SMD:R_0805_2012Metric_Pad1.20x1.40mm_HandSolder, F.Cu at (103.4, 72.7)
- added R81: 4K7, Resistor_SMD:R_0805_2012Metric_Pad1.20x1.40mm_HandSolder, F.Cu at (103.4, 75.7)
- added R82: 2K2, Resistor_SMD:R_0805_2012Metric_Pad1.20x1.40mm_HandSolder, F.Cu at (85.7, 36.7)
- added U16: DS3231M, Package_SO:SOIC-16W_7.5x10.3mm_P1.27mm, F.Cu at (94.5, 78.8)
- moved C11 53.8 mm to (65.2, 111.8)
- moved C13 53.8 mm to (65.6, 93.6)
- moved C14 53.8 mm to (65.6, 95.6)
- moved C17 53.8 mm to (84.2, 97.1)
- moved C18 53.8 mm to (39.6, 142.9)
- moved C19 53.8 mm to (37.5, 167.6)
- moved C20 53.8 mm to (41.8, 167.7)
- moved C21 53.8 mm to (95.3, 150.9)
- moved C22 53.8 mm to (110.6, 150.5)
- moved C4 53.8 mm to (65.7, 129.5)
- moved C5 53.8 mm to (67.6, 100.4)
- moved C7 53.8 mm to (77.8, 37.9)
- moved C9 53.8 mm to (39.6, 145.2)
- moved D14 53.8 mm to (123.6, 107.2)
- moved D16 53.8 mm to (123.6, 142.9)
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Connections:
- C10 pad 1: Net-(U6-VCC) -> 24V
- C21 pad 1: Net-(U14-VCC) -> 24V
- C22 pad 1: Net-(U15-VCC) -> 24V
- C6 pad 1: Net-(J6-Pin_1) -> 24V
- C8 pad 1: Net-(U13-VCC) -> 24V
- J2 pad 9: unconnected-(J2-Pin_9-Pad9) -> GND
- J6 pad 1: Net-(J6-Pin_1) -> 24V
- J7 pad 9: unconnected-(J7-Pin_9-Pad9) -> GND
- U1 pad 43: unconnected-(U1-PD0-Pad43) -> SCL
- U1 pad 44: unconnected-(U1-PD1-Pad44) -> SDA
- U13 pad 8: Net-(U13-VCC) -> 24V
- U14 pad 8: Net-(U14-VCC) -> 24V
- U15 pad 8: Net-(U15-VCC) -> 24V
- U3 pad 1: Net-(J6-Pin_1) -> 24V
- U6 pad 8: Net-(U6-VCC) -> 24V
Routing:
- net 24V: track 0.00 -> 327.0 mm, vias 0 -> 3
- net Net-(D41-K): track 0.00 -> 241.4 mm, vias 0 -> 7
- net GND: track 889.4 -> 1037.1 mm
- net Net-(D48-A): track 0.00 -> 76.1 mm
- net +5V: track 641.9 -> 709.9 mm
- net Net-(D47-A): track 0.00 -> 67.3 mm
- net SDA: track 0.00 -> 63.3 mm, vias 0 -> 2
- net Net-(D41-A): track 0.00 -> 62.1 mm
- net SCL: track 0.00 -> 60.0 mm, vias 0 -> 2
- net Net-(D46-A): track 0.00 -> 52.7 mm
- net Net-(D42-A): track 0.00 -> 46.2 mm
- net Net-(J16-Pin_2): track 0.00 -> 46.0 mm
- net Net-(J17-Pin_2): track 0.00 -> 45.2 mm
- net Net-(J17-Pin_8): track 0.00 -> 44.0 mm
- net Net-(J16-Pin_8): track 0.00 -> 41.2 mm
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Other:
- board size 168.9 x 149.7 mm -> 236.7 x 149.7 mm
- board text added: "DI"
- board text added: "DO"
- board text added: "PWM"

Commit message: Feb 28 office commit
Parts:
- added U17: TLP2748, Package_SO:SO-6L_10x3.84mm_P1.27mm, F.Cu at (64.7, 176.5)
Changed lines of the file:
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@@
   (net 357 "unconnected-(K15-Pad4)")
   (net 358 "unconnected-(K16-Pad4)")
+  (net 359 "unconnected-(U17-A-Pad1)")
+  (net 360 "unconnected-(U17-NC-Pad2)")
+  (net 361 "unconnected-(U17-K-Pad3)")
+  (net 362 "unconnected-(U17-GND-Pad4)")
+  (net 363 "unconnected-(U17-VO-Pad5)")
+  (net 364 "unconnected-(U17-VDD-Pad6)")
   (footprint "Diode_SMD:D_SOD-128" (layer "F.Cu")
     (at 123.6237 54.418 -90)
@@
       (offset (xyz 0 0 0))
       (scale (xyz 1 1 1))
+      (rotate (xyz 0 0 0))
+    )
+  )
+  (footprint "Package_SO:SO-6L_10x3.84mm_P1.27mm" (layer "F.Cu")
+    (at 64.719 176.4792)
+    (descr "6-pin plasic small outline 7,5mm long https://toshiba.semicon-storage.com/info/docget.jsp?did=53548&prodName=TLP2770")
+    (tags "SO-6L")
+    (property "Sheetfile" "controllinoA.kicad_sch")
+    (property "Sheetname" "")
+    (property "ki_description" "10-Mbps inverting photocouple,5 kVrms, 4.5 - 30 Vdd, push-pull output, SO-6L")
+    (property "ki_keywords" "Photocouple highspeed inverting push-pull output")
+    (attr smd)
+    (fp_text reference "U17" (at -3.7 -2.9) (layer "F.SilkS")
+        (effects (font (size 1 1) (thickness 0.15)))
+    )
+    (fp_text value "TLP2748" (at 0.1 3.2) (layer "F.Fab")
+        (effects (font (size 1 1) (thickness 0.15)))
+    )
+    (fp_text user "${REFERENCE}" (at 0.3 0 180) (layer "F.Fab")
+        (effects (font (size 0.5 0.5) (thickness 0.05)))
+    )
+    (fp_line (start -5.5 -2.05) (end 3.7 -2.05)
+      (stroke (width 0.12) (type solid)) (layer "F.SilkS"))
+    (fp_line (start -3.7 2.05) (end 3.7 2.05)
+      (stroke (width 0.12) (type solid)) (layer "F.SilkS"))
+    (fp_line (start -5.65 -2.17) (end -5.65 2.17)
+      (stroke (width 0.05) (type solid)) (layer "F.CrtYd"))
+    (fp_line (start -5.65 2.17) (end 5.65 2.17)
+      (stroke (width 0.05) (type solid)) (layer "F.CrtYd"))
+    (fp_line (start 5.65 -2.17) (end -5.65 -2.17)
+      (stroke (width 0.05) (type solid)) (layer "F.CrtYd"))
+    (fp_line (start 5.65 2.17) (end 5.65 -2.17)
+      (stroke (width 0.05) (type solid)) (layer "F.CrtYd"))
+    (fp_line (start -3.75 -0.9) (end -3 -1.92)
+      (stroke (width 0.1) (type solid)) (layer "F.Fab"))
+    (fp_line (start -3.75 1.92) (end -3.75 -0.9)
+      (stroke (width 0.1) (type solid)) (layer "F.Fab"))
+    (fp_line (start -3.75 1.92) (end 3.75 1.92)
+      (stroke (width 0.1) (type solid)) (layer "F.Fab"))
+    (fp_line (start -3 -1.92) (end 3.75 -1.92)
+      (stroke (width 0.1) (type solid)) (layer "F.Fab"))
+    (fp_line (start 3.75 1.92) (end 3.75 -1.92)
+      (stroke (width 0.1) (type solid)) (layer "F.Fab"))
+    (pad "1" smd rect (at -4.75 -1.27 90) (size 0.8 1.3) (layers "F.Cu" "F.Paste" "F.Mask")
+      (net 359 "unconnected-(U17-A-Pad1)") (pinfunction "A") (pintype "passive"))
+    (pad "2" smd rect (at -4.75 0 90) (size 0.8 1.3) (layers "F.Cu" "F.Paste" "F.Mask")
+      (net 360 "unconnected-(U17-NC-Pad2)") (pinfunction "NC") (pintype "no_connect"))
+    (pad "3" smd rect (at -4.75 1.27 90) (size 0.8 1.3) (layers "F.Cu" "F.Paste" "F.Mask")
+      (net 361 "unconnected-(U17-K-Pad3)") (pinfunction "K") (pintype "passive"))
+    (pad "4" smd rect (at 4.75 1.27 90) (size 0.8 1.3) (layers "F.Cu" "F.Paste" "F.Mask")
+      (net 362 "unconnected-(U17-GND-Pad4)") (pinfunction "GND") (pintype "power_in"))
+    (pad "5" smd rect (at 4.75 0 90) (size 0.8 1.3) (layers "F.Cu" "F.Paste" "F.Mask")
+      (net 363 "unconnected-(U17-VO-Pad5)") (pinfunction "VO") (pintype "output"))
+    (pad "6" smd rect (at 4.75 -1.27 90) (size 0.8 1.3) (layers "F.Cu" "F.Paste" "F.Mask")
+      (net 364 "unconnected-(U17-VDD-Pad6)") (pinfunction "VDD") (pintype "power_in"))
+    (model "${KICAD6_3DMODEL_DIR}/Package_SO.3dshapes/SO-6L_10x3.84mm_P1.27mm.wrl"
+      (offset (xyz 0 0 0))
+      (scale (xyz 1 1 1))

Commit message: 11March24
Parts:
- added C24: 3.3uF / 16v, Capacitor_SMD:C_0805_2012Metric_Pad1.18x1.45mm_HandSolder, F.Cu at (77.4, 59.2)
- added C25: 10uF / 16v, Capacitor_SMD:C_0805_2012Metric_Pad1.18x1.45mm_HandSolder, F.Cu at (77.4, 61.3)
- added C26: 10uF / 16v, Capacitor_SMD:C_0805_2012Metric_Pad1.18x1.45mm_HandSolder, F.Cu at (108.2, 56.5)
- added L10: bead, Inductor_SMD:L_1206_3216Metric, F.Cu at (78.0, 55.7)
- added R83: 4K7, Resistor_SMD:R_0805_2012Metric_Pad1.20x1.40mm_HandSolder, F.Cu at (108.1, 59.4)
- added R84: 4K7, Resistor_SMD:R_0805_2012Metric_Pad1.20x1.40mm_HandSolder, F.Cu at (77.3, 63.4)
- added U18: W5100, Package_QFP:LQFP-80_10x10mm_P0.4mm, F.Cu at (91.6, 56.6)
Routing:
- net Net-(U18-ADDR0): track 0.00 -> 29.4 mm
- net Net-(U18-DATA0): track 0.00 -> 20.6 mm
