File: uprojects/Sufyan Mukadam/controllinoA/controllinoA.kicad_pcb (KiCad board)
At the start: 2 copper layers, 236.7 x 149.7 mm, 229 parts, among them J1 AVR-ISP-6, J10 Conn_01x06, J11 DO1, J12 Conn_01x08, J13 Conn_01x10, J14 Conn_01x02, J15 Conn_01x10, J16 Conn_01x10, J17 Conn_01x10, J2 Conn_01x10, J3 Conn_01x05, J4 Conn_01x10, J5 Conn_01x10, J6 Conn_01x03, J7 Conn_01x10, J8 USB_C_Receptacle_USB2.0, J9 Conn_01x02, K1 G5LE-1, K10 G5LE-1, K11 G5LE-1, K12 G5LE-1, K13 G5LE-1, K14 G5LE-1, K15 G5LE-1, K16 G5LE-1, K2 G5LE-1, K3 G5LE-1, K4 G5LE-1, K5 G5LE-1, K6 G5LE-1, K7 G5LE-1, K8 G5LE-1, K9 G5LE-1, U1 ATmega2560-16A, U10 ULN2003A, U11 ULN2003A, U12 CH340G, U13 TLP250, U14 TLP250, U15 TLP250, U16 DS3231M, U17 TLP2748, U18 W5100, U2 ULN2003A, U3 LM2596S-5, U4 ULN2003A, U5 TPD8F003, U6 TLP250, U7 TPD8F003, U8 TPD8F003, U9 ULN2003A, Y1 16MHz, Y2 12MHz

Commit message: March 11 office commit 1
Parts:
- added C27: 13, Capacitor_SMD:C_0805_2012Metric_Pad1.18x1.45mm_HandSolder, F.Cu at (84.5, 43.9)
- added C28: 13, Capacitor_SMD:C_0805_2012Metric_Pad1.18x1.45mm_HandSolder, F.Cu at (92.0, 43.9)
- added C29: 100n, Capacitor_SMD:C_0805_2012Metric_Pad1.18x1.45mm_HandSolder, F.Cu at (60.8, 52.1)
- added C30: 100n, Capacitor_SMD:C_0805_2012Metric_Pad1.18x1.45mm_HandSolder, F.Cu at (60.8, 57.1)
- added C31: 10uF / 16v, Capacitor_SMD:C_0805_2012Metric_Pad1.18x1.45mm_HandSolder, F.Cu at (82.1, 55.4)
- added D49: LED, LED_SMD:LED_0805_2012Metric_Pad1.15x1.40mm_HandSolder, F.Cu at (97.0, 49.0)
- added D50: LED, LED_SMD:LED_0805_2012Metric_Pad1.15x1.40mm_HandSolder, F.Cu at (100.1, 49.0)
- added D51: LED, LED_SMD:LED_0805_2012Metric_Pad1.15x1.40mm_HandSolder, F.Cu at (103.1, 49.0)
- added D52: LED, LED_SMD:LED_0805_2012Metric_Pad1.15x1.40mm_HandSolder, F.Cu at (106.1, 49.0)
- added D53: LED, LED_SMD:LED_0805_2012Metric_Pad1.15x1.40mm_HandSolder, F.Cu at (109.2, 49.0)
- added D54: LED, LED_SMD:LED_0805_2012Metric_Pad1.15x1.40mm_HandSolder, F.Cu at (112.2, 49.0)
- added L19: bead, Inductor_SMD:L_1206_3216Metric, F.Cu at (82.5, 52.9)
- added L20: bead, Inductor_SMD:L_1206_3216Metric, F.Cu at (90.3, 71.4)
- added R85: 12K, Resistor_SMD:R_0805_2012Metric_Pad1.20x1.40mm_HandSolder, F.Cu at (77.9, 57.6)
- added R86: 330, Resistor_SMD:R_0805_2012Metric_Pad1.20x1.40mm_HandSolder, F.Cu at (77.9, 55.4)
- added R87: 1M, Resistor_SMD:R_0805_2012Metric_Pad1.20x1.40mm_HandSolder, F.Cu at (88.3, 44.9)
- added R88: 470, Resistor_SMD:R_0805_2012Metric_Pad1.20x1.40mm_HandSolder, F.Cu at (97.0, 44.2)
- added R89: 470, Resistor_SMD:R_0805_2012Metric_Pad1.20x1.40mm_HandSolder, F.Cu at (99.9, 44.2)
- added R90: 470, Resistor_SMD:R_0805_2012Metric_Pad1.20x1.40mm_HandSolder, F.Cu at (102.9, 44.2)
- added R91: 470, Resistor_SMD:R_0805_2012Metric_Pad1.20x1.40mm_HandSolder, F.Cu at (105.8, 44.2)
- added R92: 470, Resistor_SMD:R_0805_2012Metric_Pad1.20x1.40mm_HandSolder, F.Cu at (108.8, 44.2)
- added R93: 470, Resistor_SMD:R_0805_2012Metric_Pad1.20x1.40mm_HandSolder, F.Cu at (111.7, 44.2)
- added U19: LM1117MP-3.3, Package_TO_SOT_SMD:SOT-223-3_TabPin2, F.Cu at (68.1, 54.7)
- added Y3: 25MHz, Crystal:Crystal_SMD_ECS_CSM3X-2Pin_7.6x4.1mm, F.Cu at (88.3, 48.4)
- moved C26 30.5 mm to (77.9, 53.1), turned to 180 degrees
- moved R83 7.63 mm to (101.4, 63.0), turned to 180 degrees
- moved L10 4.57 mm to (77.7, 60.2), turned to 180 degrees
- moved R84 3.40 mm to (77.6, 66.8)
- moved C24 3.40 mm to (77.6, 62.6)
- moved U18 3.40 mm to (91.8, 60.0)
- moved C25 3.40 mm to (77.6, 64.7)
Connections:
- net Net-(U18-GNDA-Pad10) renamed GNDA
- net Net-(U18-VCC3V3D-Pad12) renamed 3V3
- U18 pad 1: unconnected-(U18-RSET_BG-Pad1) -> Net-(U18-RSET_BG)
- U18 pad 13: Net-(U18-GNDD-Pad13) -> GND
- U18 pad 14: Net-(U18-GNDD-Pad13) -> GND
- U18 pad 17: Net-(U18-GNDD-Pad13) -> GND
- U18 pad 2: unconnected-(U18-VCC3V3A-Pad2) -> Net-(U18-VCC3V3A)
- U18 pad 32: Net-(U18-GNDD-Pad13) -> GND
- U18 pad 43: Net-(U18-GNDD-Pad13) -> GND
- U18 pad 66: unconnected-(U18-LINKLED-Pad66) -> Net-(D54-K)
- U18 pad 67: unconnected-(U18-SPDLED-Pad67) -> Net-(D53-K)
- U18 pad 68: Net-(U18-GNDD-Pad13) -> GND
- U18 pad 70: unconnected-(U18-FDXLED-Pad70) -> Net-(D52-K)
- U18 pad 71: unconnected-(U18-COLLED-Pad71) -> Net-(D51-K)
- U18 pad 72: unconnected-(U18-RXLED-Pad72) -> Net-(D50-K)
- U18 pad 73: unconnected-(U18-TXLED-Pad73) -> Net-(D49-K)
- U18 pad 75: unconnected-(U18-XTLN-Pad75) -> XTLN
- U18 pad 76: unconnected-(U18-XTLP-Pad76) -> XTLP
Routing:
- net GND: track 1037.1 -> 1105.5 mm, vias 32 -> 36
- net Net-(D2-A): track 76.2 -> 9.20 mm
- net 3V3: track 0.00 -> 53.3 mm, vias 0 -> 3
- net Net-(U18-1V8_OUT): track 0.00 -> 38.4 mm
- net Net-(D54-K): track 0.00 -> 22.3 mm
- net Net-(D53-K): track 0.00 -> 19.9 mm
- net Net-(D52-K): track 0.00 -> 17.8 mm
- net Net-(D51-K): track 0.00 -> 15.1 mm
- net Net-(D50-K): track 0.00 -> 12.4 mm
- net +5V: track 709.9 -> 719.5 mm, vias 19 -> 21
- net GNDA: track 0.00 -> 9.38 mm, vias 0 -> 2
- net Net-(D49-K): track 0.00 -> 9.33 mm
- net Net-(U18-RSET_BG): track 0.00 -> 8.70 mm, vias 0 -> 2
- net Net-(C26-Pad2): track 0.00 -> 6.86 mm
- net Net-(U18-VCC3V3A): track 0.00 -> 6.51 mm
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