File: uprojects/Sufyan Mukadam/controllinoA/controllinoA.kicad_pcb (KiCad board)
At the start: 2 copper layers, 236.7 x 149.7 mm, 261 parts, among them J1 AVR-ISP-6, J10 Conn_01x06, J11 DO1, J12 Conn_01x08, J13 Conn_01x10, J14 Conn_01x02, J15 Conn_01x10, J16 Conn_01x10, J17 Conn_01x10, J18 RJ45, J2 Conn_01x10, J3 Conn_01x05, J4 Conn_01x10, J5 Conn_01x10, J6 Conn_01x03, J7 Conn_01x10, J8 USB_C_Receptacle_USB2.0, J9 Conn_01x02, K1 G5LE-1, K10 G5LE-1, K11 G5LE-1, K12 G5LE-1, K13 G5LE-1, K14 G5LE-1, K15 G5LE-1, K16 G5LE-1, K2 G5LE-1, K3 G5LE-1, K4 G5LE-1, K5 G5LE-1, K6 G5LE-1, K7 G5LE-1, K8 G5LE-1, K9 G5LE-1, U1 ATmega2560-16A, U10 ULN2003A, U11 ULN2003A, U12 CH340G, U13 TLP250, U14 TLP250, U15 TLP250, U16 DS3231M, U18 W5100, U19 LM1117MP-3.3, U2 ULN2003A, U3 LM2596S-5, U4 ULN2003A, U5 TPD8F003, U6 TLP250, U7 TPD8F003, U8 TPD8F003, U9 ULN2003A, Y1 16MHz, Y2 12MHz, Y3 25MHz

Commit message: April 1 commit
Parts:
- added SW1: RESET, Button_Switch_SMD:SW_SPST_PTS810, F.Cu at (63.7, 122.0)
- added U17: ULN2803ADWR, ULN2803ADWR:SOIC127P1030X265-18N, F.Cu at (2.20, 117.0)
- added U20: ULN2803A, Package_SO:SOIC-18W_7.5x11.6mm_P1.27mm, F.Cu at (2.28, 130.4)
- moved J11 7.11 mm to (42.1, 110.3)
Routing:
- net GND: track 1184.0 -> 1207.2 mm, vias 38 -> 40
- net DO12: track 39.0 -> 17.8 mm
- net DO5: track 19.3 -> 0.11 mm
- net DO14: track 36.7 -> 18.5 mm
- net Net-(J1-~{RST}): track 31.2 -> 46.4 mm
- net DO4: track 22.7 -> 9.58 mm
- net DO15: track 31.8 -> 19.9 mm
- net DO8: track 22.4 -> 14.9 mm
- net DO10: track 23.1 -> 15.5 mm
- net DO6: track 22.6 -> 15.6 mm
- net DO11: track 21.5 -> 14.7 mm
- net DO2: track 23.8 -> 18.1 mm
- net DO9: track 19.7 -> 15.5 mm
- net DO7: track 19.9 -> 16.0 mm
- net OC3A: track 21.1 -> 18.0 mm
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
Commit message: April 4 commit
Parts:
- removed U20: ULN2803A, Package_SO:SOIC-18W_7.5x11.6mm_P1.27mm
- U17: value ULN2803ADWR -> TBD62783AFNG_EL; footprint ULN2803ADWR:SOIC127P1030X265-18N -> TBD62783AFNG-EL:SSOP18-P-225-0p65_TOS
- moved U17 49.7 mm to (51.7, 112.5), turned to 180 degrees
Connections:
- J11 pad 3: DO2 -> _DO2
- J11 pad 5: DO4 -> _DO4
- U17 pad 1: unconnected-(U17-1B-Pad1) -> DO2
- U17 pad 17: unconnected-(U17-2C-Pad17) -> _DO4
- U17 pad 18: unconnected-(U17-1C-Pad18) -> _DO2
- U17 pad 2: unconnected-(U17-2B-Pad2) -> DO4
Routing:
- net DO6: track 15.6 -> 6.61 mm
- net DO7: track 16.0 -> 7.20 mm
- net OC3A: track 18.0 -> 12.8 mm
- net DO2: track 18.1 -> 13.0 mm
- net DO10: track 15.5 -> 13.0 mm
- net DO9: track 15.5 -> 14.1 mm

Commit message: April 5 commit
Parts:
- added U20: TBD62783AFNG_EL, TBD62783AFNG-EL:SSOP18-P-225-0p65_TOS, F.Cu at (51.8, 120.8)
Connections:
- J11 pad 10: DO9 -> unconnected-(J11-Pin_10-Pad10)
- J11 pad 11: DO10 -> unconnected-(J11-Pin_11-Pad11)
- J11 pad 12: DO11 -> unconnected-(J11-Pin_12-Pad12)
- J11 pad 13: DO12 -> unconnected-(J11-Pin_13-Pad13)
- J11 pad 14: DO13 -> unconnected-(J11-Pin_14-Pad14)
- J11 pad 15: DO14 -> unconnected-(J11-Pin_15-Pad15)
- J11 pad 16: DO15 -> unconnected-(J11-Pin_16-Pad16)
- J11 pad 4: OC3A -> _DO3
- J11 pad 6: DO5 -> _DO5
- J11 pad 7: DO6 -> unconnected-(J11-Pin_7-Pad7)
- J11 pad 8: DO7 -> unconnected-(J11-Pin_8-Pad8)
- J11 pad 9: DO8 -> unconnected-(J11-Pin_9-Pad9)
- U17 pad 1: DO2 -> DO9
- U17 pad 10: unconnected-(U17-GND-Pad10) -> GND
- U17 pad 11: unconnected-(U17-O8-Pad11) -> _DO2
- U17 pad 12: unconnected-(U17-O7-Pad12) -> _DO3
- U17 pad 13: unconnected-(U17-O6-Pad13) -> _DO4
- U17 pad 14: unconnected-(U17-O5-Pad14) -> _DO5
- U17 pad 15: unconnected-(U17-O4-Pad15) -> _DO6
- U17 pad 16: unconnected-(U17-O3-Pad16) -> _DO7
- U17 pad 17: _DO4 -> _DO8
- U17 pad 18: _DO2 -> _DO9
- U17 pad 2: DO4 -> DO8
- U17 pad 3: unconnected-(U17-I3-Pad3) -> DO7
- U17 pad 4: unconnected-(U17-I4-Pad4) -> DO6
- U17 pad 5: unconnected-(U17-I5-Pad5) -> DO5
- U17 pad 6: unconnected-(U17-I6-Pad6) -> DO4
- U17 pad 7: unconnected-(U17-I7-Pad7) -> OC3A
- U17 pad 8: unconnected-(U17-I8-Pad8) -> DO2
- U17 pad 9: unconnected-(U17-VCC-Pad9) -> 24V
Routing:
- net DO8: track 14.5 -> 10.5 mm

Commit message: 15 April 24
Parts:
- added U21: TBD62783AFNG_EL, TBD62783AFNG-EL:SSOP18-P-225-0p65_TOS, F.Cu at (84.9, 135.8)
- moved U17 2.23 mm to (51.7, 114.8)
- moved U20 2.23 mm to (51.7, 123.0)
Connections:
- J11 pad 10: unconnected-(J11-Pin_10-Pad10) -> _DO9
- J11 pad 11: unconnected-(J11-Pin_11-Pad11) -> _DO10
- J11 pad 12: unconnected-(J11-Pin_12-Pad12) -> _DO11
- J11 pad 13: unconnected-(J11-Pin_13-Pad13) -> _DO12
- J11 pad 14: unconnected-(J11-Pin_14-Pad14) -> _DO13
- J11 pad 15: unconnected-(J11-Pin_15-Pad15) -> _DO14
- J11 pad 16: unconnected-(J11-Pin_16-Pad16) -> _DO15
- J11 pad 7: unconnected-(J11-Pin_7-Pad7) -> _DO6
- J11 pad 8: unconnected-(J11-Pin_8-Pad8) -> _DO7
- J11 pad 9: unconnected-(J11-Pin_9-Pad9) -> _DO8
- J12 pad 1: DO16 -> _DO16
- J12 pad 2: DO17 -> _DO17
- J12 pad 3: DO18 -> _DO18
- J12 pad 4: DO19 -> _DO19
- J12 pad 5: DO20 -> _DO20
- J12 pad 6: DO21 -> _DO21
- U20 pad 12: unconnected-(U20-O7-Pad12) -> _DO11
- U20 pad 13: unconnected-(U20-O6-Pad13) -> _DO12
- U20 pad 14: unconnected-(U20-O5-Pad14) -> _DO13
- U20 pad 15: unconnected-(U20-O4-Pad15) -> _DO14
- U20 pad 16: unconnected-(U20-O3-Pad16) -> _DO15
Routing:
- net 24V: track 327.0 -> 402.4 mm
- net GND: track 1207.2 -> 1233.5 mm, vias 40 -> 44
- net DO5: track 0.00 -> 16.4 mm
- net DO12: track 17.8 -> 33.8 mm
- net DO20: track 28.2 -> 13.2 mm
- net DO21: track 28.1 -> 13.4 mm
- net DO19: track 31.1 -> 17.4 mm
- net DO18: track 28.4 -> 15.5 mm
- net DO14: track 18.5 -> 31.2 mm
- net DO17: track 31.6 -> 19.3 mm
- net _DO21: track 0.00 -> 11.7 mm
- net DO16: track 31.5 -> 20.2 mm
- net DO15: track 19.9 -> 29.8 mm
- net DO6: track 6.61 -> 16.5 mm
- net _DO20: track 0.00 -> 9.74 mm
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