File: uprojects/Sufyan Mukadam/controllinoAA/controllinoA.kicad_pcb (KiCad board)
At the start: 2 copper layers, 168.9 x 149.7 mm, 156 parts, among them J1 AVR-ISP-6, J2 Conn_01x10, J3 Conn_01x05, J4 Conn_01x10, J5 Conn_01x10, J6 Conn_01x03, J7 Conn_01x10, J8 USB_C_Receptacle_USB2.0, K1 G5LE-1, K2 G5LE-1, K3 G5LE-1, K4 G5LE-1, K5 G5LE-1, K6 G5LE-1, K7 G5LE-1, K8 G5LE-1, U1 ATmega2560-16A, U10 ULN2003A, U11 ULN2003A, U12 CH340G, U13 TLP250, U2 ULN2003A, U3 LM2596S-5, U4 ULN2003A, U5 TPD8F003, U7 TPD8F003, U8 TPD8F003, U9 ULN2003A, Y1 16MHz, Y2 12MHz

Commit message: Updates 25Feb24
Parts:
- removed C18: 100n, Capacitor_SMD:C_0805_2012Metric_Pad1.18x1.45mm_HandSolder
- removed C19, C20: 15, Capacitor_SMD:C_0805_2012Metric_Pad1.18x1.45mm_HandSolder
- removed D18, D27, D28, D29, D30, D31, D32, D33: LED, LED_SMD:LED_0805_2012Metric_Pad1.15x1.40mm_HandSolder
- removed J8: USB_C_Receptacle_USB2.0, Connector_USB:USB_C_Receptacle_HCTL_HC-TYPE-C-16P-01A
- removed R51, R52, R53, R54, R55, R56, R57, R58: 1K, Resistor_SMD:R_0805_2012Metric_Pad1.20x1.40mm_HandSolder
- removed U12: CH340G, Package_SO:SOIC-16_3.9x9.9mm_P1.27mm
- removed U13: TLP250, Package_DIP:DIP-8_W7.62mm
- removed U9: ULN2003A, Package_SO:SOIC-16_3.9x9.9mm_P1.27mm
- removed Y2: 12MHz, Crystal:Crystal_HC49-U_Vertical
- added C10: 100n, Capacitor_SMD:C_0805_2012Metric_Pad1.18x1.45mm_HandSolder, F.Cu at (91.2, 152.6)
- added C9: 100n, Capacitor_SMD:C_0805_2012Metric_Pad1.18x1.45mm_HandSolder, F.Cu at (91.2, 143.5)
- added L10: L_Small, Inductor_SMD:L_1206_3216Metric, F.Cu at (91.3, 147.5)
- added U6: W5100, Package_QFP:LQFP-80_10x10mm_P0.4mm, F.Cu at (153.7, 146.1)
- R10: value 100E -> 4K7
- moved C8 41.9 mm to (91.1, 136.1), turned to 0 degrees
- moved R10 31.3 mm to (92.2, 140.5), turned to -90 degrees
- moved D10 23.6 mm to (123.0, 61.7)
- moved J6 23.6 mm to (80.5, 56.8)
- moved L1 23.6 mm to (123.7, 52.5)
- moved C6 23.6 mm to (93.3, 51.5)
- moved C7 23.6 mm to (136.5, 57.4)
- moved U3 23.6 mm to (106.3, 52.5)
- moved L15 10.6 mm to (83.7, 73.4)
- moved L16 10.6 mm to (83.7, 70.8)
- moved L17 10.6 mm to (83.7, 65.6)
- moved L18 10.6 mm to (83.7, 68.2)
- moved J7 4.37 mm to (76.9, 68.5)
- moved C13 3.68 mm to (128.0, 69.8)
- moved C3 3.68 mm to (122.0, 70.3)
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Connections:
- C8 pad 1: Net-(U13-VCC) -> GND
- C8 pad 2: GND -> OC3A
- J3 pad 1: unconnected-(J3-Pin_1-Pad1) -> Net-(J3-Pin_1)
- R10 pad 1: OC3B -> OC3A
- U1 pad 53: Net-(U1-PC0) -> unconnected-(U1-PC0-Pad53)
- U1 pad 54: Net-(U1-PC1) -> unconnected-(U1-PC1-Pad54)
- U1 pad 55: Net-(U1-PC2) -> unconnected-(U1-PC2-Pad55)
- U1 pad 56: Net-(U1-PC3) -> unconnected-(U1-PC3-Pad56)
- U1 pad 57: Net-(U1-PC4) -> unconnected-(U1-PC4-Pad57)
- U1 pad 58: Net-(U1-PC5) -> unconnected-(U1-PC5-Pad58)
- U1 pad 59: Net-(U1-PC6) -> unconnected-(U1-PC6-Pad59)
- U1 pad 60: Net-(U1-PC7) -> unconnected-(U1-PC7-Pad60)
- U4 pad 2: Net-(D18-K) -> unconnected-(U4-I2-Pad2)
- U4 pad 3: Net-(D27-K) -> unconnected-(U4-I3-Pad3)
- U4 pad 4: Net-(D28-K) -> unconnected-(U4-I4-Pad4)
- U4 pad 5: Net-(D29-K) -> unconnected-(U4-I5-Pad5)
- U4 pad 6: Net-(D30-K) -> unconnected-(U4-I6-Pad6)
- U4 pad 7: Net-(D31-K) -> unconnected-(U4-I7-Pad7)
Routing:
- net +5V: track 401.8 -> 431.8 mm
- net GND: track 121.7 -> 104.9 mm
- net Net-(C9-Pad2): track 3.17 -> 0.00 mm
- net Net-(U13-VCC): track 2.70 -> 0.00 mm

Commit message: Feb 27 commit
Parts:
- removed L10: L_Small, Inductor_SMD:L_1206_3216Metric
- added C18: 100n, Capacitor_SMD:C_0805_2012Metric_Pad1.18x1.45mm_HandSolder, F.Cu at (93.2, 139.4)
- added C19: 15, Capacitor_SMD:C_0805_2012Metric_Pad1.18x1.45mm_HandSolder, F.Cu at (91.2, 164.1)
- added C20: 15, Capacitor_SMD:C_0805_2012Metric_Pad1.18x1.45mm_HandSolder, F.Cu at (95.5, 164.1)
- added C21: 100n, Capacitor_SMD:C_0805_2012Metric_Pad1.18x1.45mm_HandSolder, F.Cu at (149.0, 147.3)
- added C22: 100n, Capacitor_SMD:C_0805_2012Metric_Pad1.18x1.45mm_HandSolder, F.Cu at (164.2, 146.9)
- added C23: 100uF/35V, Capacitor_SMD:CP_Elec_6.3x7.7, F.Cu at (103.7, 52.9)
- added D18: LED, LED_SMD:LED_0805_2012Metric_Pad1.15x1.40mm_HandSolder, F.Cu at (150.9, 111.5)
- added D27: LED, LED_SMD:LED_0805_2012Metric_Pad1.15x1.40mm_HandSolder, F.Cu at (150.9, 113.6)
- added D28: LED, LED_SMD:LED_0805_2012Metric_Pad1.15x1.40mm_HandSolder, F.Cu at (150.8, 115.7)
- added D29: LED, LED_SMD:LED_0805_2012Metric_Pad1.15x1.40mm_HandSolder, F.Cu at (150.8, 117.8)
- added D30: LED, LED_SMD:LED_0805_2012Metric_Pad1.15x1.40mm_HandSolder, F.Cu at (150.8, 119.8)
- added D31: LED, LED_SMD:LED_0805_2012Metric_Pad1.15x1.40mm_HandSolder, F.Cu at (150.8, 121.9)
- added D32: LED, LED_SMD:LED_0805_2012Metric_Pad1.15x1.40mm_HandSolder, F.Cu at (150.8, 124.0)
- added D33: LED, LED_SMD:LED_0805_2012Metric_Pad1.15x1.40mm_HandSolder, F.Cu at (150.8, 126.1)
- added D34: LED, LED_SMD:LED_0805_2012Metric_Pad1.15x1.40mm_HandSolder, F.Cu at (112.2, 72.3)
- added D35: LED, LED_SMD:LED_0805_2012Metric_Pad1.15x1.40mm_HandSolder, F.Cu at (112.2, 70.2)
- added D36: LED, LED_SMD:LED_0805_2012Metric_Pad1.15x1.40mm_HandSolder, F.Cu at (112.2, 67.9)
- added D37: LED, LED_SMD:LED_0805_2012Metric_Pad1.15x1.40mm_HandSolder, F.Cu at (112.2, 65.7)
- added D38: LED, LED_SMD:LED_0805_2012Metric_Pad1.15x1.40mm_HandSolder, F.Cu at (112.2, 63.6)
- added D39: LED, LED_SMD:LED_0805_2012Metric_Pad1.15x1.40mm_HandSolder, F.Cu at (112.2, 61.4)
- added J10: Conn_01x06, Connector_PinHeader_2.54mm:PinHeader_1x06_P2.54mm_Vertical, F.Cu at (73.1, 119.4)
- added J11: DO1, Connector_PinHeader_2.54mm:PinHeader_2x08_P2.54mm_Vertical, F.Cu at (102.8, 106.3)
- added J12: Conn_01x08, Connector_PinHeader_2.54mm:PinHeader_1x08_P2.54mm_Vertical, F.Cu at (135.2, 141.2)
- added J13: Conn_01x10, Connector_JST:JST_XH_B10B-XH-A_1x10_P2.50mm_Vertical, F.Cu at (171.2, 110.6)
- added J8: USB_C_Receptacle_USB2.0, Connector_USB:USB_C_Receptacle_HCTL_HC-TYPE-C-16P-01A, F.Cu at (79.6, 151.2)
- added J9: Conn_01x02, Connector_PinHeader_2.54mm:PinHeader_1x02_P2.54mm_Vertical, F.Cu at (94.5, 136.3)
- added R51: 1K, Resistor_SMD:R_0805_2012Metric_Pad1.20x1.40mm_HandSolder, F.Cu at (147.0, 111.5)
- added R52: 1K, Resistor_SMD:R_0805_2012Metric_Pad1.20x1.40mm_HandSolder, F.Cu at (147.0, 113.6)
- added R53: 1K, Resistor_SMD:R_0805_2012Metric_Pad1.20x1.40mm_HandSolder, F.Cu at (147.0, 115.7)
- added R54: 1K, Resistor_SMD:R_0805_2012Metric_Pad1.20x1.40mm_HandSolder, F.Cu at (147.0, 117.8)
- added R55: 1K, Resistor_SMD:R_0805_2012Metric_Pad1.20x1.40mm_HandSolder, F.Cu at (147.0, 119.8)
- added R56: 1K, Resistor_SMD:R_0805_2012Metric_Pad1.20x1.40mm_HandSolder, F.Cu at (147.0, 121.9)
- added R57: 1K, Resistor_SMD:R_0805_2012Metric_Pad1.20x1.40mm_HandSolder, F.Cu at (147.0, 124.0)
- added R58: 1K, Resistor_SMD:R_0805_2012Metric_Pad1.20x1.40mm_HandSolder, F.Cu at (147.0, 126.1)
- added R59: 5.1K, Resistor_SMD:R_0805_2012Metric_Pad1.20x1.40mm_HandSolder, F.Cu at (86.6, 143.5)
- added R60: 5.1K, Resistor_SMD:R_0805_2012Metric_Pad1.20x1.40mm_HandSolder, F.Cu at (86.6, 141.5)
- added R61: 1K, Resistor_SMD:R_0805_2012Metric_Pad1.20x1.40mm_HandSolder, F.Cu at (108.3, 72.3)
- added R62: 1K, Resistor_SMD:R_0805_2012Metric_Pad1.20x1.40mm_HandSolder, F.Cu at (108.3, 70.2)
- added R63: 1K, Resistor_SMD:R_0805_2012Metric_Pad1.20x1.40mm_HandSolder, F.Cu at (108.2, 67.9)
- added R64: 1K, Resistor_SMD:R_0805_2012Metric_Pad1.20x1.40mm_HandSolder, F.Cu at (108.2, 65.7)
- added R65: 1K, Resistor_SMD:R_0805_2012Metric_Pad1.20x1.40mm_HandSolder, F.Cu at (108.2, 63.6)
- added R66: 1K, Resistor_SMD:R_0805_2012Metric_Pad1.20x1.40mm_HandSolder, F.Cu at (108.2, 61.4)
- added R67: 68K, Resistor_SMD:R_0805_2012Metric_Pad1.20x1.40mm_HandSolder, F.Cu at (87.5, 119.4)
- added R68: 33K, Resistor_SMD:R_0805_2012Metric_Pad1.20x1.40mm_HandSolder, F.Cu at (87.5, 121.6)
- added R69: 68K, Resistor_SMD:R_0805_2012Metric_Pad1.20x1.40mm_HandSolder, F.Cu at (87.5, 123.7)
- added R70: 33K, Resistor_SMD:R_0805_2012Metric_Pad1.20x1.40mm_HandSolder, F.Cu at (87.5, 125.9)
- added R71: 68K, Resistor_SMD:R_0805_2012Metric_Pad1.20x1.40mm_HandSolder, F.Cu at (87.5, 128.0)
- added R72: 33K, Resistor_SMD:R_0805_2012Metric_Pad1.20x1.40mm_HandSolder, F.Cu at (87.5, 130.0)
- added R73: 68K, Resistor_SMD:R_0805_2012Metric_Pad1.20x1.40mm_HandSolder, F.Cu at (87.5, 132.1)
- added R74: 33K, Resistor_SMD:R_0805_2012Metric_Pad1.20x1.40mm_HandSolder, F.Cu at (87.5, 134.3)
- added R75: 68K, Resistor_SMD:R_0805_2012Metric_Pad1.20x1.40mm_HandSolder, F.Cu at (80.0, 132.1)
- added R76: 33K, Resistor_SMD:R_0805_2012Metric_Pad1.20x1.40mm_HandSolder, F.Cu at (80.0, 134.3)
- added R77: 100E, Resistor_SMD:R_0805_2012Metric_Pad1.20x1.40mm_HandSolder, F.Cu at (120.9, 152.7)
- added R78: 100E, Resistor_SMD:R_0805_2012Metric_Pad1.20x1.40mm_HandSolder, F.Cu at (138.9, 152.6)
- added R79: 100E, Resistor_SMD:R_0805_2012Metric_Pad1.20x1.40mm_HandSolder, F.Cu at (153.9, 152.3)
- added U12: CH340G, Package_SO:SOIC-16_3.9x9.9mm_P1.27mm, F.Cu at (93.2, 150.1)
- added U13: TLP250, Package_DIP:DIP-8_W7.62mm, F.Cu at (106.6, 150.2)
- added U14: TLP250, Package_DIP:DIP-8_W7.62mm, F.Cu at (142.1, 150.1)
- added U15: TLP250, Package_DIP:DIP-8_W7.62mm, F.Cu at (157.3, 149.8)
- added U9: ULN2003A, Package_SO:SOIC-16_3.9x9.9mm_P1.27mm, F.Cu at (160.3, 126.7)
- added Y2: 12MHz, Crystal:Crystal_HC49-U_Vertical, F.Cu at (95.7, 160.0)
- C12, C13, C14, C15, C16, C17: footprint Capacitor_SMD:C_0805_2012Metric_Pad1.18x1.45mm_HandSolder -> Capacitor_SMD:C_0603_1608Metric
- R10: value 4K7 -> 100E
- U6: value W5100 -> TLP250; footprint Package_QFP:LQFP-80_10x10mm_P0.4mm -> Package_DIP:DIP-8_W7.62mm
- moved C12 75.8 mm to (137.8, 90.3), turned to 180 degrees
- moved C16 75.6 mm to (137.8, 91.9), turned to 180 degrees
- moved C15 75.6 mm to (137.8, 88.7), turned to 180 degrees
- moved C17 75.5 mm to (137.8, 93.6), turned to 180 degrees
- moved U7 61.3 mm to (99.2, 69.5)
- moved U8 56.0 mm to (99.1, 130.1)
- moved R16 53.7 mm to (87.5, 61.8)
- moved R15 53.1 mm to (87.5, 59.8)
- moved R14 52.5 mm to (87.5, 57.7)
- moved R13 51.9 mm to (87.5, 55.6)
- moved R12 51.4 mm to (87.5, 53.5)
- moved R11 50.8 mm to (87.5, 51.5)
- moved L14 48.3 mm to (80.0, 69.9)
- moved L13 45.2 mm to (79.9, 73.6)
- moved L12 43.0 mm to (80.0, 77.3)
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Connections:
- C10 pad 1: GND -> Net-(U6-VCC)
- C10 pad 2: Net-(J3-Pin_1) -> GND
- C8 pad 1: GND -> Net-(U13-VCC)
- C8 pad 2: OC3A -> GND
- C9 pad 2: Net-(C9-Pad2) -> Net-(U12-V3)
- J3 pad 1: Net-(J3-Pin_1) -> DO0
- J3 pad 2: unconnected-(J3-Pin_2-Pad2) -> DO1
- J3 pad 3: unconnected-(J3-Pin_3-Pad3) -> DO22
- J3 pad 4: unconnected-(J3-Pin_4-Pad4) -> DO23
- R10 pad 1: OC3A -> OC3B
- R10 pad 2: Net-(C9-Pad2) -> Net-(U13-A)
- U1 pad 1: unconnected-(U1-PG5-Pad1) -> DO2
- U1 pad 15: unconnected-(U1-PH3-Pad15) -> DO4
- U1 pad 16: unconnected-(U1-PH4-Pad16) -> DO5
- U1 pad 17: unconnected-(U1-PH5-Pad17) -> DO6
- U1 pad 18: unconnected-(U1-PH6-Pad18) -> DO7
- U1 pad 2: unconnected-(U1-PE0-Pad2) -> RX0
- U1 pad 23: unconnected-(U1-PB4-Pad23) -> DO8
- U1 pad 24: unconnected-(U1-PB5-Pad24) -> DO9
- U1 pad 25: unconnected-(U1-PB6-Pad25) -> DO10
- U1 pad 26: unconnected-(U1-PB7-Pad26) -> DO11
- U1 pad 3: unconnected-(U1-PE1-Pad3) -> TX0
- U1 pad 35: unconnected-(U1-PL0-Pad35) -> DO19
- U1 pad 36: unconnected-(U1-PL1-Pad36) -> DO18
- U1 pad 37: unconnected-(U1-PL2-Pad37) -> DO17
- U1 pad 38: unconnected-(U1-PL3-Pad38) -> DO16
- U1 pad 39: unconnected-(U1-PL4-Pad39) -> DO15
- U1 pad 40: unconnected-(U1-PL5-Pad40) -> DO14
- U1 pad 41: unconnected-(U1-PL6-Pad41) -> DO13
- U1 pad 42: unconnected-(U1-PL7-Pad42) -> DO12
- U1 pad 47: unconnected-(U1-PD4-Pad47) -> DO20
- U1 pad 48: unconnected-(U1-PD5-Pad48) -> DO21
- U1 pad 49: unconnected-(U1-PD6-Pad49) -> PD6
- U1 pad 53: unconnected-(U1-PC0-Pad53) -> Net-(U1-PC0)
- U1 pad 54: unconnected-(U1-PC1-Pad54) -> Net-(U1-PC1)
- U1 pad 55: unconnected-(U1-PC2-Pad55) -> Net-(U1-PC2)
- U1 pad 56: unconnected-(U1-PC3-Pad56) -> Net-(U1-PC3)
- U1 pad 57: unconnected-(U1-PC4-Pad57) -> Net-(U1-PC4)
- U1 pad 58: unconnected-(U1-PC5-Pad58) -> Net-(U1-PC5)
- U1 pad 59: unconnected-(U1-PC6-Pad59) -> Net-(U1-PC6)
- U1 pad 60: unconnected-(U1-PC7-Pad60) -> Net-(U1-PC7)
- U1 pad 67: unconnected-(U1-PJ4-Pad67) -> PJ4
- U11 pad 10: unconnected-(U11-O7-Pad10) -> Net-(D39-K)
- U11 pad 11: unconnected-(U11-O6-Pad11) -> Net-(D38-K)
- U11 pad 12: unconnected-(U11-O5-Pad12) -> Net-(D37-K)
- U11 pad 13: unconnected-(U11-O4-Pad13) -> Net-(D36-K)
- U11 pad 14: unconnected-(U11-O3-Pad14) -> Net-(D35-K)
- U11 pad 15: unconnected-(U11-O2-Pad15) -> Net-(D34-K)
- U11 pad 2: unconnected-(U11-I2-Pad2) -> IO08
- U11 pad 3: unconnected-(U11-I3-Pad3) -> IO09
- U11 pad 4: unconnected-(U11-I4-Pad4) -> IO10
- U11 pad 5: unconnected-(U11-I5-Pad5) -> IO11
- U11 pad 6: unconnected-(U11-I6-Pad6) -> IO12
- U11 pad 7: unconnected-(U11-I7-Pad7) -> IO13
- U4 pad 10: unconnected-(U4-O7-Pad10) -> Net-(J13-Pin_6)
- U4 pad 11: unconnected-(U4-O6-Pad11) -> Net-(J13-Pin_5)
- U4 pad 12: unconnected-(U4-O5-Pad12) -> Net-(J13-Pin_4)
- U4 pad 13: unconnected-(U4-O4-Pad13) -> Net-(J13-Pin_3)
- U4 pad 14: unconnected-(U4-O3-Pad14) -> Net-(J13-Pin_2)
- U4 pad 15: unconnected-(U4-O2-Pad15) -> Net-(J13-Pin_1)
- U4 pad 2: unconnected-(U4-I2-Pad2) -> Net-(D18-K)
- U4 pad 3: unconnected-(U4-I3-Pad3) -> Net-(D27-K)
- U4 pad 4: unconnected-(U4-I4-Pad4) -> Net-(D28-K)
- U4 pad 5: unconnected-(U4-I5-Pad5) -> Net-(D29-K)
- U4 pad 6: unconnected-(U4-I6-Pad6) -> Net-(D30-K)
- U4 pad 7: unconnected-(U4-I7-Pad7) -> Net-(D31-K)
- U6 pad 2: unconnected-(U6-VCC3V3A-Pad2) -> Net-(U6-A)
- U6 pad 3: unconnected-(U6-NC-Pad3) -> GND
- U6 pad 4: Net-(U6-GNDA-Pad10) -> unconnected-(U6-NC-Pad4)
- U6 pad 5: unconnected-(U6-RXIP-Pad5) -> GND
- U6 pad 6: unconnected-(U6-RXIN-Pad6) -> DO1
- U6 pad 7: Net-(U6-VCC1V8A-Pad7) -> DO1
- U6 pad 8: unconnected-(U6-TXOP-Pad8) -> Net-(U6-VCC)
Routing:
- net GND: track 104.9 -> 889.4 mm, vias 0 -> 32
- net +5V: track 431.8 -> 641.9 mm, vias 12 -> 19
- net IO12: track 0.00 -> 73.7 mm, vias 0 -> 2
- net IO08: track 0.00 -> 73.1 mm, vias 0 -> 2
- net RX0: track 0.00 -> 71.4 mm, vias 0 -> 2
- net IO13: track 0.00 -> 71.3 mm, vias 0 -> 3
- net IO09: track 0.00 -> 71.1 mm, vias 0 -> 2
- net IO10: track 0.00 -> 70.4 mm, vias 0 -> 2
- net IO15: track 0.00 -> 69.9 mm, vias 0 -> 2
- net IO11: track 0.00 -> 69.8 mm, vias 0 -> 2
- net IO14: track 0.00 -> 69.3 mm, vias 0 -> 2
- net IO17: track 0.00 -> 68.1 mm, vias 0 -> 2
- net OC3C: track 0.00 -> 66.9 mm, vias 0 -> 2
- net IO20: track 0.00 -> 65.2 mm, vias 0 -> 2
- net IO19: track 0.00 -> 63.8 mm, vias 0 -> 2
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Other:
- board text removed: "Analog Out"
- board text removed: "Digital/Analog In"
