File: uprojects/Sufyan Mukadam/controllinoAA/controllinoA.kicad_pcb (KiCad board)
At the start: 2 copper layers, 236.7 x 149.7 mm, 261 parts, among them J1 AVR-ISP-6, J10 Conn_01x06, J11 DO1, J12 Conn_01x08, J13 Conn_01x10, J14 Conn_01x02, J15 Conn_01x10, J16 Conn_01x10, J17 Conn_01x10, J18 RJ45, J2 Conn_01x10, J3 Conn_01x05, J4 Conn_01x10, J5 Conn_01x10, J6 Conn_01x03, J7 Conn_01x10, J8 USB_C_Receptacle_USB2.0, J9 Conn_01x02, K1 G5LE-1, K10 G5LE-1, K11 G5LE-1, K12 G5LE-1, K13 G5LE-1, K14 G5LE-1, K15 G5LE-1, K16 G5LE-1, K2 G5LE-1, K3 G5LE-1, K4 G5LE-1, K5 G5LE-1, K6 G5LE-1, K7 G5LE-1, K8 G5LE-1, K9 G5LE-1, U1 ATmega2560-16A, U10 ULN2003A, U11 ULN2003A, U12 CH340G, U13 TLP250, U14 TLP250, U15 TLP250, U16 DS3231M, U18 W5100, U19 LM1117MP-3.3, U2 ULN2003A, U3 LM2596S-5, U4 ULN2003A, U5 TPD8F003, U6 TLP250, U7 TPD8F003, U8 TPD8F003, U9 ULN2003A, Y1 16MHz, Y2 12MHz, Y3 25MHz

Commit message: 15 April 24
Parts:
- added SW1: RESET, Button_Switch_SMD:SW_SPST_PTS810, F.Cu at (63.7, 122.0)
- added U17: TBD62783AFNG_EL, TBD62783AFNG-EL:SSOP18-P-225-0p65_TOS, F.Cu at (51.7, 114.8)
- added U20: TBD62783AFNG_EL, TBD62783AFNG-EL:SSOP18-P-225-0p65_TOS, F.Cu at (51.7, 123.0)
- added U21: TBD62783AFNG_EL, TBD62783AFNG-EL:SSOP18-P-225-0p65_TOS, F.Cu at (84.9, 135.8)
- moved J11 7.11 mm to (42.1, 110.3)
Connections:
- J11 pad 10: DO9 -> _DO9
- J11 pad 11: DO10 -> _DO10
- J11 pad 12: DO11 -> _DO11
- J11 pad 13: DO12 -> _DO12
- J11 pad 14: DO13 -> _DO13
- J11 pad 15: DO14 -> _DO14
- J11 pad 16: DO15 -> _DO15
- J11 pad 3: DO2 -> _DO2
- J11 pad 4: OC3A -> _DO3
- J11 pad 5: DO4 -> _DO4
- J11 pad 6: DO5 -> _DO5
- J11 pad 7: DO6 -> _DO6
- J11 pad 8: DO7 -> _DO7
- J11 pad 9: DO8 -> _DO8
- J12 pad 1: DO16 -> _DO16
- J12 pad 2: DO17 -> _DO17
- J12 pad 3: DO18 -> _DO18
- J12 pad 4: DO19 -> _DO19
- J12 pad 5: DO20 -> _DO20
- J12 pad 6: DO21 -> _DO21
Routing:
- net 24V: track 327.0 -> 402.4 mm
- net GND: track 1184.0 -> 1233.5 mm, vias 38 -> 44
- net Net-(J1-~{RST}): track 31.2 -> 46.4 mm
- net DO20: track 28.2 -> 13.2 mm
- net DO21: track 28.1 -> 13.4 mm
- net DO19: track 31.1 -> 17.4 mm
- net DO18: track 28.4 -> 15.5 mm
- net DO17: track 31.6 -> 19.3 mm
- net _DO21: track 0.00 -> 11.7 mm
- net DO16: track 31.5 -> 20.2 mm
- net _DO20: track 0.00 -> 9.74 mm
- net _DO14: track 0.00 -> 9.07 mm
- net _DO8: track 0.00 -> 8.21 mm
- net _DO12: track 0.00 -> 7.99 mm
- net _DO19: track 0.00 -> 7.71 mm
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