File: uprojects/Sufyan Mukadam/controllinoAA/controllinoA.kicad_sch (KiCad schematic)
At the start: 156 parts, among them J1 AVR-ISP-6, J2 Conn_01x10, J3 Conn_01x05, J4 Conn_01x10, J5 Conn_01x10, J6 Conn_01x03, J7 Conn_01x10, J8 USB_C_Receptacle_USB2.0, K1 G5LE-1, K2 G5LE-1, K3 G5LE-1, K4 G5LE-1, K5 G5LE-1, K6 G5LE-1, K7 G5LE-1, K8 G5LE-1, U1 ATmega2560-16A, U10 ULN2003A, U11 ULN2003A, U12 CH340G, U13 TLP250, U2 ULN2003A, U3 LM2596S-5, U4 ULN2003A, U5 TPD8F003, U7 TPD8F003, U8 TPD8F003, U9 ULN2003A, Y1 16MHz, Y2 12MHz

Commit message: Updates 25Feb24
Parts:
- removed U13: TLP250, Package_DIP:DIP-8_W7.62mm, symbol Driver_FET:TLP250
- added C10, C9: 100n, Capacitor_SMD:C_0805_2012Metric_Pad1.18x1.45mm_HandSolder, symbol Device:C_Small
- added L10: L_Small, Inductor_SMD:L_1206_3216Metric, symbol Device:L_Small
- J8: footprint Connector_USB:USB_C_Receptacle_HCTL_HC-TYPE-C-16P-01A -> (none)
- R10: value 100E -> 4K7
Connections:
- net GND: now also C8.1, C10.1, C9.1; no longer C8.2
- net OC3A: now also C8.2, R10.1
- net OC3B: no longer R10.1
- net at R10.2: now also C9.2, L10.1
- new net: C10.2, L10.2
Other:
- added sheet Ethernet (untitled.kicad_sch)
- moved on the sheet: C12, C13, C14, C15, C16, C17, J3

Commit message: Feb 27 commit
Parts:
- removed L10: L_Small, Inductor_SMD:L_1206_3216Metric, symbol Device:L_Small
- added C21, C22: 100n, Capacitor_SMD:C_0805_2012Metric_Pad1.18x1.45mm_HandSolder, symbol Device:C_Small
- added C23: 100uF/35V, Capacitor_SMD:CP_Elec_6.3x7.7, symbol Device:C_Polarized_Small
- added D34, D35, D36, D37, D38, D39: LED, LED_SMD:LED_0805_2012Metric_Pad1.15x1.40mm_HandSolder, symbol Device:LED_Small
- added J10: Conn_01x06, Connector_PinHeader_2.54mm:PinHeader_1x06_P2.54mm_Vertical, symbol Connector_Generic:Conn_01x06
- added J11: DO1, Connector_PinHeader_2.54mm:PinHeader_2x08_P2.54mm_Vertical, symbol Connector_Generic:Conn_02x08_Odd_Even
- added J12: Conn_01x08, Connector_PinHeader_2.54mm:PinHeader_1x08_P2.54mm_Vertical, symbol Connector_Generic:Conn_01x08
- added J13: Conn_01x10, Connector_JST:JST_XH_B10B-XH-A_1x10_P2.50mm_Vertical, symbol Connector_Generic:Conn_01x10
- added J9: Conn_01x02, Connector_PinHeader_2.54mm:PinHeader_1x02_P2.54mm_Vertical, symbol Connector_Generic:Conn_01x02
- added R59, R60: 5.1K, Resistor_SMD:R_0805_2012Metric_Pad1.20x1.40mm_HandSolder, symbol Device:R_Small
- added R61, R62, R63, R64, R65, R66: 1K, Resistor_SMD:R_0805_2012Metric_Pad1.20x1.40mm_HandSolder, symbol Device:R_Small
- added R67, R69, R71, R73, R75: 68K, Resistor_SMD:R_0805_2012Metric_Pad1.20x1.40mm_HandSolder, symbol Device:R_Small
- added R68, R70, R72, R74, R76: 33K, Resistor_SMD:R_0805_2012Metric_Pad1.20x1.40mm_HandSolder, symbol Device:R_Small
- added R77, R78, R79: 100E, Resistor_SMD:R_0805_2012Metric_Pad1.20x1.40mm_HandSolder, symbol Device:R_Small
- added U13, U14, U15, U6: TLP250, Package_DIP:DIP-8_W7.62mm, symbol Driver_FET:TLP250
- C12, C13, C14, C15, C16, C17: footprint Capacitor_SMD:C_0805_2012Metric_Pad1.18x1.45mm_HandSolder -> Capacitor_SMD:C_0603_1608Metric
- J8: footprint (none) -> Connector_USB:USB_C_Receptacle_HCTL_HC-TYPE-C-16P-01A
- R10: value 4K7 -> 100E
Connections:
- net +5V: now also C18.2, U9.9 (COM), C23.1, J13.9 (Pin_9), J9.1 (Pin_1), R61.1, R62.1, R63.1, R64.1, R65.1, R66.1
- net GND: now also C10.2, C18.1, C8.2, J8.A1 (GND), J8.A12 (GND), J8.B1 (GND), J8.B12 (GND), U9.8 (GND), C21.2, C22.2, C23.2, J13.10 (Pin_10), R59.1, R60.1, R68.1, R70.1, R72.1, R74.1, R76.1, U13.3 (C), U13.5 (VEE), U14.3 (C), U14.5 (VEE), U15.3 (C), U15.5 (VEE), U6.3 (C), U6.5 (VEE); no longer C10.1, C18.2, C8.1
- net I16: now also R67.2, R68.2
- net I17: now also R69.2, R70.2
- net I18: now also R71.2, R72.2
- net IN0: now also R73.2, R74.2
- net IN1: now also R75.2, R76.2
- net IO08: now also U11.2 (I2)
- net IO09: now also U11.3 (I3)
- net IO10: now also U11.4 (I4)
- net IO11: now also U11.5 (I5)
- net IO12: now also U11.6 (I6)
- net IO13: now also U11.7 (I7)
- net OC3A: now also J11.4 (Pin_4); no longer C8.2, R10.1
- net OC3B: now also R10.1
- net OC3C: now also R77.1
- net DO0: now reaches J3.1 (Pin_1)
- net DO0: now also U13.6 (VO), U13.7 (VO)
- net DO1: now reaches J3.2 (Pin_2)
- net DO1: now also U6.6 (VO), U6.7 (VO)
- net DO22: now reaches J3.3 (Pin_3)
- net DO22: now also U14.6 (VO), U14.7 (VO)
- net DO23: now reaches J3.4 (Pin_4)
- net DO23: now also U15.6 (VO), U15.7 (VO)
- net at J8.A4 (VBUS), J8.A9 (VBUS), J8.B4 (VBUS)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: now also J9.2 (Pin_2)
- net at J8.A5 (CC1): now also R59.2
- net USBDP: now reaches J8.A6 (D+)
- net USBDP: now also J8.B6 (D+), U12.5 (UD+)
- net USBDN: now reaches J8.A7 (D-)
- net USBDN: now also J8.B7 (D-), U12.6 (UD-)
- net at J8.B5 (CC2): now also R60.2
- net at R10.2: now also U13.2 (A); no longer C9.2
- net DO2: now reaches U1.1 (PG5)
- net DO2: now also J11.3 (Pin_3)
- net DO4: now reaches U1.15 (PH3)
- net DO4: now also J11.5 (Pin_5)
- net DO5: now reaches U1.16 (PH4)
- net DO5: now also J11.6 (Pin_6)
- net DO6: now reaches U1.17 (PH5)
- net DO6: now also J11.7 (Pin_7)
- net DO7: now reaches U1.18 (PH6)
- net DO7: now also J11.8 (Pin_8)
- net RX0: now reaches U1.2 (PE0)
- net RX0: now also U12.2 (TXD)
- net DO8: now reaches U1.23 (PB4)
- net DO8: now also J11.9 (Pin_9)
- net DO9: now reaches U1.24 (PB5)
- net DO9: now also J11.10 (Pin_10)
- net DO10: now reaches U1.25 (PB6)
- net DO10: now also J11.11 (Pin_11)
- net DO11: now reaches U1.26 (PB7)
- net DO11: now also J11.12 (Pin_12)
- net TX0: now reaches U1.3 (PE1)
- net TX0: now also U12.3 (RXD)
- net DO19: now reaches U1.35 (PL0)
- net DO19: now also J12.4 (Pin_4)
- net DO18: now reaches U1.36 (PL1)
- net DO18: now also J12.3 (Pin_3)
- net DO17: now reaches U1.37 (PL2)
- net DO17: now also J12.2 (Pin_2)
- net DO16: now reaches U1.38 (PL3)
- net DO16: now also J12.1 (Pin_1)
- net DO15: now reaches U1.39 (PL4)
- net DO15: now also J11.16 (Pin_16)
- net DO14: now reaches U1.40 (PL5)
- net DO14: now also J11.15 (Pin_15)
- net DO13: now reaches U1.41 (PL6)
- net DO13: now also J11.14 (Pin_14)
- net DO12: now reaches U1.42 (PL7)
- net DO12: now also J11.13 (Pin_13)
- net DO20: now reaches U1.47 (PD4)
- net DO20: now also J12.5 (Pin_5)
- net DO21: now reaches U1.48 (PD5)
- net DO21: now also J12.6 (Pin_6)
- net PD6: now reaches U1.49 (PD6)
- net PD6: now also R78.1
- net PJ4: now reaches U1.67 (PJ4)
- net PJ4: now also R79.1
- net at U9.15 (O2): now also J13.8 (Pin_8)
- net at U9.16 (O1): now also J13.7 (Pin_7)
- net at U4.10 (O7): now also J13.6 (Pin_6)
- net at U4.11 (O6): now also J13.5 (Pin_5)
- net at U4.12 (O5): now also J13.4 (Pin_4)
- net at U4.13 (O4): now also J13.3 (Pin_3)
- net at U4.14 (O3): now also J13.2 (Pin_2)
- net at U4.15 (O2): now also J13.1 (Pin_1)
- net at U12.4 (V3): now also C9.2; no longer C18.1
- net at U11.10 (O7): now also D39.1 (K)
- net at U11.11 (O6): now also D38.1 (K)
- net at U11.12 (O5): now also D37.1 (K)
- net at U11.13 (O4): now also D36.1 (K)
- net at U11.14 (O3): now also D35.1 (K)
- net at U11.15 (O2): now also D34.1 (K)
- new net: C21.1, U14.8 (VCC)
- new net: R77.2, U6.2 (A)
- new net: J10.5 (Pin_5), R75.1
- new net: D35.2 (A), R62.2
- new net: R78.2, U14.2 (A)
- new net: C22.1, U15.8 (VCC)
- new net: D37.2 (A), R64.2
- new net: D36.2 (A), R63.2
- new net: C8.1, U13.8 (VCC)
- new net: D34.2 (A), R61.2
- new net: R79.2, U15.2 (A)
- new net: J10.4 (Pin_4), R73.1
- new net: D39.2 (A), R66.2
- new net: J10.1 (Pin_1), R67.1
- new net: J10.2 (Pin_2), R69.1
- new net: J10.3 (Pin_3), R71.1
- new net: C10.1, U6.8 (VCC)
- new net: D38.2 (A), R65.2
Other:
- removed sheet Ethernet
- moved on the sheet: C12, C13, C14, C15, C16, C17, C18, C19, C20, J3, U12, Y2
