File: uprojects/Sufyan Mukadam/controllinoAA/controllinoA.kicad_sch (KiCad schematic)
At the start: 261 parts, among them J1 AVR-ISP-6, J10 Conn_01x06, J11 DO1, J12 Conn_01x08, J13 Conn_01x10, J14 Conn_01x02, J15 Conn_01x10, J16 Conn_01x10, J17 Conn_01x10, J2 Conn_01x10, J3 Conn_01x05, J4 Conn_01x10, J5 Conn_01x10, J6 Conn_01x03, J7 Conn_01x10, J8 USB_C_Receptacle_USB2.0, J9 Conn_01x02, K1 G5LE-1, K10 G5LE-1, K11 G5LE-1, K12 G5LE-1, K13 G5LE-1, K14 G5LE-1, K15 G5LE-1, K16 G5LE-1, K2 G5LE-1, K3 G5LE-1, K4 G5LE-1, K5 G5LE-1, K6 G5LE-1, K7 G5LE-1, K8 G5LE-1, K9 G5LE-1, U1 ATmega2560-16A, U10 ULN2003A, U11 ULN2003A, U12 CH340G, U13 TLP250, U14 TLP250, U15 TLP250, U16 DS3231M, U18 W5100, U19 LM1117MP-3.3, U2 ULN2003A, U3 LM2596S-5, U4 ULN2003A, U5 TPD8F003, U6 TLP250, U7 TPD8F003, U8 TPD8F003, U9 ULN2003A, Y1 16MHz, Y2 12MHz, Y3 25MHz

Commit message: 15 April 24
Parts:
- added SW1: RESET, Button_Switch_SMD:SW_SPST_PTS810, symbol Switch:SW_Push
- added U17, U20, U21: TBD62783AFNG_EL, TBD62783AFNG-EL:SSOP18-P-225-0p65_TOS, symbol TBD62783AFNG-EL:TBD62783AFNG_EL
Connections:
- net 24V: now also U17.9 (VCC), U20.9 (VCC), U21.9 (VCC)
- net DO10: now also U20.8 (I8); no longer J11.11 (Pin_11)
- net DO11: now also U20.7 (I7); no longer J11.12 (Pin_12)
- net DO12: now also U20.6 (I6); no longer J11.13 (Pin_13)
- net DO13: now also U20.5 (I5); no longer J11.14 (Pin_14)
- net DO14: now also U20.4 (I4); no longer J11.15 (Pin_15)
- net DO15: now also U20.3 (I3); no longer J11.16 (Pin_16)
- net DO16: now also U21.8 (I8); no longer J12.1 (Pin_1)
- net DO17: now also U21.7 (I7); no longer J12.2 (Pin_2)
- net DO18: now also U21.6 (I6); no longer J12.3 (Pin_3)
- net DO19: now also U21.5 (I5); no longer J12.4 (Pin_4)
- net DO2: now also U17.8 (I8); no longer J11.3 (Pin_3)
- net DO20: now also U21.4 (I4); no longer J12.5 (Pin_5)
- net DO21: now also U21.3 (I3); no longer J12.6 (Pin_6)
- net DO4: now also U17.6 (I6); no longer J11.5 (Pin_5)
- net DO5: now also U17.5 (I5); no longer J11.6 (Pin_6)
- net DO6: now also U17.4 (I4); no longer J11.7 (Pin_7)
- net DO7: now also U17.3 (I3); no longer J11.8 (Pin_8)
- net DO8: now also U17.2 (I2); no longer J11.9 (Pin_9)
- net DO9: now also U17.1 (I1); no longer J11.10 (Pin_10)
- net GND: now also SW1.2, U17.10 (GND), U20.10 (GND), U21.10 (GND)
- net OC3A: now also U17.7 (I7); no longer J11.4 (Pin_4)
- net at J1.5 (~{RST}), U1.30 (~{RESET}): now also SW1.1
- new net _DO10: J11.11 (Pin_11), U20.11 (O8)
- new net _DO11: J11.12 (Pin_12), U20.12 (O7)
- new net _DO12: J11.13 (Pin_13), U20.13 (O6)
- new net _DO13: J11.14 (Pin_14), U20.14 (O5)
- new net _DO14: J11.15 (Pin_15), U20.15 (O4)
- new net _DO15: J11.16 (Pin_16), U20.16 (O3)
- new net _DO16: J12.1 (Pin_1), U21.11 (O8)
- new net _DO17: J12.2 (Pin_2), U21.12 (O7)
- new net _DO18: J12.3 (Pin_3), U21.13 (O6)
- new net _DO19: J12.4 (Pin_4), U21.14 (O5)
- new net _DO2: J11.3 (Pin_3), U17.11 (O8)
- new net _DO20: J12.5 (Pin_5), U21.15 (O4)
- new net _DO21: J12.6 (Pin_6), U21.16 (O3)
- new net _DO3: J11.4 (Pin_4), U17.12 (O7)
- new net _DO4: J11.5 (Pin_5), U17.13 (O6)
- new net _DO5: J11.6 (Pin_6), U17.14 (O5)
- new net _DO6: J11.7 (Pin_7), U17.15 (O4)
- new net _DO7: J11.8 (Pin_8), U17.16 (O3)
- new net _DO8: J11.9 (Pin_9), U17.17 (O2)
- new net _DO9: J11.10 (Pin_10), U17.18 (O1)
Other:
- moved on the sheet: C4, C?, J?, R14, R15, R?
