File: uprojects/ESP32-S3-Basic/ESP32-S3-BasicA/ESP32-S3-BasicA.kicad_pcb (KiCad board)
At the start: 2 copper layers, 5 parts, among them U1 ESP32-S3-WROOM-1x-N8R8

Commit message: March 27 commit
Parts:
- moved R1 0.18 mm to (134.9, 65.5)
- turned C1 to 180 degrees
- turned C2 to 0 degrees
- turned C3 to 180 degrees
Changed lines of the file:
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@@
   (net 39 "ESP_EN")
   (footprint "Resistor_SMD:R_0805_2012Metric" (layer "F.Cu")
-    (at 134.8994 65.6336)
+    (at 134.874 65.4558)
     (descr "Resistor SMD 0805 (2012 Metric), square (rectangular) end terminal, IPC_7351 nominal, (Body size source: IPC-SM-782 page 72, https://www.pcb-3d.com/wordpress/wp-content/uploads/ipc-sm-782a_amendment_1_and_2.pdf), generated with kicad-footprint-generator")
     (tags "resistor")
@@
     (property "Sheetname" "")
     (attr smd)
-    (fp_text reference "R1" (at 0 -1.65) (layer "F.SilkS")
-        (effects (font (size 1 1) (thickness 0.15)))
-    )
-    (fp_text value "10k/R0402" (at 0 1.65) (layer "F.Fab")
+    (fp_text reference "R1" (at -2.6416 0.0254) (layer "F.SilkS")
+        (effects (font (size 1 1) (thickness 0.15)))
+    )
+    (fp_text value "10k/R0402" (at -7.8994 -8.255) (layer "F.Fab")
         (effects (font (size 1 1) (thickness 0.15)))
     )
@@
   )
   (footprint "Capacitor_SMD:C_0805_2012Metric" (layer "F.Cu")
-    (at 134.9248 61.0616 180)
+    (at 134.9248 61.0616)
     (descr "Capacitor SMD 0805 (2012 Metric), square (rectangular) end terminal, IPC_7351 nominal, (Body size source: IPC-SM-782 page 76, https://www.pcb-3d.com/wordpress/wp-content/uploads/ipc-sm-782a_amendment_1_and_2.pdf, https://docs.google.com/spreadsheets/d/1BsfQQcO9C6DZCsRaXUlFlo91Tg2WpOkGARC1WS5S8t0/edit?usp=sharing), generated with kicad-footprint-generator")
     (tags "capacitor")
@@
     (property "Sheetname" "")
     (attr smd)
-    (fp_text reference "C2" (at 0 -1.68 180) (layer "F.SilkS")
-        (effects (font (size 1 1) (thickness 0.15)))
-    )
-    (fp_text value "100nF/10V/10%/X7R/C0402" (at 6.1214 2.3368 180) (layer "F.Fab")
-        (effects (font (size 1 1) (thickness 0.15)))
-    )
-    (fp_text user "${REFERENCE}" (at 0 0 180) (layer "F.Fab")
+    (fp_text reference "C2" (at -2.9464 0.0254) (layer "F.SilkS")
+        (effects (font (size 1 1) (thickness 0.15)))
+    )
+    (fp_text value "100nF/10V/10%/X7R/C0402" (at -0.889 -7.366) (layer "F.Fab")
+        (effects (font (size 1 1) (thickness 0.15)))
+    )
+    (fp_text user "${REFERENCE}" (at 0 0) (layer "F.Fab")
         (effects (font (size 0.5 0.5) (thickness 0.08)))
     )
@@
     (fp_line (start 1 0.625) (end -1 0.625)
       (stroke (width 0.1) (type solid)) (layer "F.Fab"))
-    (pad "1" smd roundrect (at -0.95 0 180) (size 1 1.45) (layers "F.Cu" "F.Paste" "F.Mask") (roundrect_rratio 0.25)
+    (pad "1" smd roundrect (at -0.95 0) (size 1 1.45) (layers "F.Cu" "F.Paste" "F.Mask") (roundrect_rratio 0.25)
       (net 38 "GND") (pintype "passive"))
-    (pad "2" smd roundrect (at 0.95 0 180) (size 1 1.45) (layers "F.Cu" "F.Paste" "F.Mask") (roundrect_rratio 0.25)
+    (pad "2" smd roundrect (at 0.95 0) (size 1 1.45) (layers "F.Cu" "F.Paste" "F.Mask") (roundrect_rratio 0.25)
       (net 37 "+3.3V") (pintype "passive"))
     (model "${KICAD6_3DMODEL_DIR}/Capacitor_SMD.3dshapes/C_0805_2012Metric.wrl"
@@
   )
   (footprint "Capacitor_SMD:C_0805_2012Metric" (layer "F.Cu")
-    (at 134.9248 63.2714)
+    (at 134.9248 63.2714 180)
     (descr "Capacitor SMD 0805 (2012 Metric), square (rectangular) end terminal, IPC_7351 nominal, (Body size source: IPC-SM-782 page 76, https://www.pcb-3d.com/wordpress/wp-content/uploads/ipc-sm-782a_amendment_1_and_2.pdf, https://docs.google.com/spreadsheets/d/1BsfQQcO9C6DZCsRaXUlFlo91Tg2WpOkGARC1WS5S8t0/edit?usp=sharing), generated with kicad-footprint-generator")
     (tags "capacitor")
@@
     (property "Sheetname" "")
     (attr smd)
-    (fp_text reference "C3" (at 0 -1.68) (layer "F.SilkS")
-        (effects (font (size 1 1) (thickness 0.15)))
-    )
-    (fp_text value "1uF/10V/10%/X5R/C0603" (at 0 1.68) (layer "F.Fab")
+    (fp_text reference "C3" (at 2.794 -0.127) (layer "F.SilkS")
+        (effects (font (size 1 1) (thickness 0.15)))
+    )
+    (fp_text value "1uF/10V/10%/X5R/C0603" (at 1.8034 7.8486) (layer "F.Fab")
         (effects (font (size 1 1) (thickness 0.15)))
     )
@@
     (fp_line (start 1 0.625) (end -1 0.625)
       (stroke (width 0.1) (type solid)) (layer "F.Fab"))
-    (pad "1" smd roundrect (at -0.95 0) (size 1 1.45) (layers "F.Cu" "F.Paste" "F.Mask") (roundrect_rratio 0.25)
+    (pad "1" smd roundrect (at -0.95 0 180) (size 1 1.45) (layers "F.Cu" "F.Paste" "F.Mask") (roundrect_rratio 0.25)
       (net 39 "ESP_EN") (pintype "passive"))
-    (pad "2" smd roundrect (at 0.95 0) (size 1 1.45) (layers "F.Cu" "F.Paste" "F.Mask") (roundrect_rratio 0.25)
+    (pad "2" smd roundrect (at 0.95 0 180) (size 1 1.45) (layers "F.Cu" "F.Paste" "F.Mask") (roundrect_rratio 0.25)
       (net 38 "GND") (pintype "passive"))
     (model "${KICAD6_3DMODEL_DIR}/Capacitor_SMD.3dshapes/C_0805_2012Metric.wrl"
@@
   )
   (footprint "Capacitor_SMD:C_0805_2012Metric" (layer "F.Cu")
-    (at 134.9248 58.9026)
+    (at 134.9248 58.9026 180)
     (descr "Capacitor SMD 0805 (2012 Metric), square (rectangular) end terminal, IPC_7351 nominal, (Body size source: IPC-SM-782 page 76, https://www.pcb-3d.com/wordpress/wp-content/uploads/ipc-sm-782a_amendment_1_and_2.pdf, https://docs.google.com/spreadsheets/d/1BsfQQcO9C6DZCsRaXUlFlo91Tg2WpOkGARC1WS5S8t0/edit?usp=sharing), generated with kicad-footprint-generator")
     (tags "capacitor")
@@
     (property "Sheetname" "")
     (attr smd)
-    (fp_text reference "C1" (at 0 -1.68) (layer "F.SilkS")
-        (effects (font (size 1 1) (thickness 0.15)))
-    )
-    (fp_text value "22uF/6.3V/20%/X5R/C0603" (at -4.6482 -2.4638) (layer "F.Fab")
+    (fp_text reference "C1" (at 2.7432 0.0762) (layer "F.SilkS")
+        (effects (font (size 1 1) (thickness 0.15)))
+    )
+    (fp_text value "22uF/6.3V/20%/X5R/C0603" (at 1.2954 7.2136) (layer "F.Fab")
         (effects (font (size 1 1) (thickness 0.15)))
     )
@@
     (fp_line (start 1 0.625) (end -1 0.625)
       (stroke (width 0.1) (type solid)) (layer "F.Fab"))
-    (pad "1" smd roundrect (at -0.95 0) (size 1 1.45) (layers "F.Cu" "F.Paste" "F.Mask") (roundrect_rratio 0.25)
+    (pad "1" smd roundrect (at -0.95 0 180) (size 1 1.45) (layers "F.Cu" "F.Paste" "F.Mask") (roundrect_rratio 0.25)
       (net 37 "+3.3V") (pintype "passive"))
-    (pad "2" smd roundrect (at 0.95 0) (size 1 1.45) (layers "F.Cu" "F.Paste" "F.Mask") (roundrect_rratio 0.25)
+    (pad "2" smd roundrect (at 0.95 0 180) (size 1 1.45) (layers "F.Cu" "F.Paste" "F.Mask") (roundrect_rratio 0.25)
       (net 38 "GND") (pintype "passive"))
     (model "${KICAD6_3DMODEL_DIR}/Capacitor_SMD.3dshapes/C_0805_2012Metric.wrl"

Commit message: April 1 commit
Parts:
- added C4: 15, Capacitor_SMD:C_0805_2012Metric_Pad1.18x1.45mm_HandSolder, F.Cu at (121.3, 67.9)
- added C5: 15, Capacitor_SMD:C_0805_2012Metric_Pad1.18x1.45mm_HandSolder, F.Cu at (121.3, 70.9)
- added D1: 1N5819WS, Diode_SMD:D_SOD-323, F.Cu at (120.6, 86.0)
- added J1: USB_C_Receptacle, Connector_USB:USB_C_Receptacle_Amphenol_12401610E4-2A_CircularHoles, F.Cu at (110.9, 79.0)
- added U2: CH340G, Package_SO:SOIC-16_3.9x9.9mm_P1.27mm, F.Cu at (122.6, 78.8)
- added Y1: 12MHz, Crystal:Crystal_HC49-U_Vertical, F.Cu at (110.0, 69.7)

Commit message: April 1 commit
Parts:
- removed Y1: 12MHz, Crystal:Crystal_HC49-U_Vertical
- added Y2: 12MHz, Crystal:Crystal_SMD_3225-4Pin_3.2x2.5mm, F.Cu at (121.1, 80.3)
- moved C5 14.5 mm to (121.0, 85.4)
- moved D1 7.70 mm to (113.3, 88.4)
- moved U2 5.68 mm to (128.3, 79.1)
Changed lines of the file:
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@@
   (net 69 "unconnected-(U2-R232-Pad15)")
   (net 70 "unconnected-(U2-VCC-Pad16)")
+  (net 71 "unconnected-(Y2-Pad2)")
   (footprint "Capacitor_SMD:C_0805_2012Metric_Pad1.18x1.45mm_HandSolder" (layer "F.Cu")
-    (at 121.3454 70.9054)
+    (at 120.9802 85.4456)
     (descr "Capacitor SMD 0805 (2012 Metric), square (rectangular) end terminal, IPC_7351 nominal with elongated pad for handsoldering. (Body size source: IPC-SM-782 page 76, https://www.pcb-3d.com/wordpress/wp-content/uploads/ipc-sm-782a_amendment_1_and_2.pdf, https://docs.google.com/spreadsheets/d/1BsfQQcO9C6DZCsRaXUlFlo91Tg2WpOkGARC1WS5S8t0/edit?usp=sharing), generated with kicad-footprint-generator")
     (tags "capacitor handsolder")
@@
       (net 41 "Net-(U2-XO)") (pintype "passive"))
     (model "${KICAD6_3DMODEL_DIR}/Capacitor_SMD.3dshapes/C_0805_2012Metric.wrl"
+      (offset (xyz 0 0 0))
+      (scale (xyz 1 1 1))
+      (rotate (xyz 0 0 0))
+    )
+  )
+  (footprint "Crystal:Crystal_SMD_3225-4Pin_3.2x2.5mm" (layer "F.Cu")
+    (at 121.1248 80.2504 180)
+    (descr "SMD Crystal SERIES SMD3225/4 http://www.txccrystal.com/images/pdf/7m-accuracy.pdf, 3.2x2.5mm^2 package")
+    (tags "SMD SMT crystal")
+    (property "Sheetfile" "ESP32-S3-BasicA.kicad_sch")
+    (property "Sheetname" "")
+    (property "ki_description" "Four pin crystal, GND on pins 2 and 3, small symbol")
+    (property "ki_keywords" "quartz ceramic resonator oscillator")
+    (attr smd)
+    (fp_text reference "Y2" (at 0 -2.45) (layer "F.SilkS")
+        (effects (font (size 1 1) (thickness 0.15)))
+    )
+    (fp_text value "12MHz" (at 0 2.45) (layer "F.Fab")
+        (effects (font (size 1 1) (thickness 0.15)))
+    )
+    (fp_text user "${REFERENCE}" (at 0 0) (layer "F.Fab")
+        (effects (font (size 0.7 0.7) (thickness 0.105)))
+    )
+    (fp_line (start -2 -1.65) (end -2 1.65)
+      (stroke (width 0.12) (type solid)) (layer "F.SilkS"))
+    (fp_line (start -2 1.65) (end 2 1.65)
+      (stroke (width 0.12) (type solid)) (layer "F.SilkS"))
+    (fp_line (start -2.1 -1.7) (end -2.1 1.7)
+      (stroke (width 0.05) (type solid)) (layer "F.CrtYd"))
+    (fp_line (start -2.1 1.7) (end 2.1 1.7)
+      (stroke (width 0.05) (type solid)) (layer "F.CrtYd"))
+    (fp_line (start 2.1 -1.7) (end -2.1 -1.7)
+      (stroke (width 0.05) (type solid)) (layer "F.CrtYd"))
+    (fp_line (start 2.1 1.7) (end 2.1 -1.7)
+      (stroke (width 0.05) (type solid)) (layer "F.CrtYd"))
+    (fp_line (start -1.6 -1.25) (end -1.6 1.25)
+      (stroke (width 0.1) (type solid)) (layer "F.Fab"))
+    (fp_line (start -1.6 0.25) (end -0.6 1.25)
+      (stroke (width 0.1) (type solid)) (layer "F.Fab"))
+    (fp_line (start -1.6 1.25) (end 1.6 1.25)
+      (stroke (width 0.1) (type solid)) (layer "F.Fab"))
+    (fp_line (start 1.6 -1.25) (end -1.6 -1.25)
+      (stroke (width 0.1) (type solid)) (layer "F.Fab"))
+    (fp_line (start 1.6 1.25) (end 1.6 -1.25)
+      (stroke (width 0.1) (type solid)) (layer "F.Fab"))
+    (pad "1" smd rect (at -1.1 0.85 180) (size 1.4 1.2) (layers "F.Cu" "F.Paste" "F.Mask")
+      (net 41 "Net-(U2-XO)") (pinfunction "1") (pintype "passive"))
+    (pad "2" smd rect (at 1.1 0.85 180) (size 1.4 1.2) (layers "F.Cu" "F.Paste" "F.Mask")
+      (net 71 "unconnected-(Y2-Pad2)") (pinfunction "2") (pintype "passive"))
+    (pad "3" smd rect (at 1.1 -0.85 180) (size 1.4 1.2) (layers "F.Cu" "F.Paste" "F.Mask")
+      (net 38 "GND") (pinfunction "3") (pintype "passive"))
+    (pad "4" smd rect (at -1.1 -0.85 180) (size 1.4 1.2) (layers "F.Cu" "F.Paste" "F.Mask")
+      (net 40 "Net-(U2-XI)") (pinfunction "4") (pintype "passive"))
+    (model "${KICAD6_3DMODEL_DIR}/Crystal.3dshapes/Crystal_SMD_3225-4Pin_3.2x2.5mm.wrl"
       (offset (xyz 0 0 0))
       (scale (xyz 1 1 1))
@@
   )
   (footprint "Diode_SMD:D_SOD-323" (layer "F.Cu")
-    (at 120.5904 85.9654)
+    (at 113.284 88.392)
     (descr "SOD-323")
     (tags "SOD-323")
@@
       (net 43 "Net-(D1-A)") (pinfunction "A") (pintype "passive"))
     (model "${KICAD6_3DMODEL_DIR}/Diode_SMD.3dshapes/D_SOD-323.wrl"
-      (offset (xyz 0 0 0))
-      (scale (xyz 1 1 1))
-      (rotate (xyz 0 0 0))
-    )
-  )
-  (footprint "Crystal:Crystal_HC49-U_Vertical" (layer "F.Cu")
-    (at 110.0154 69.7154)
-    (descr "Crystal THT HC-49/U http://5hertz.com/pdfs/04404_D.pdf")
-    (tags "THT crystalHC-49/U")
-    (property "Sheetfile" "ESP32-S3-BasicA.kicad_sch")
-    (property "Sheetname" "")
-    (property "ki_description" "Two pin crystal, small symbol")
-    (property "ki_keywords" "quartz ceramic resonator oscillator")
-    (attr through_hole)
-    (fp_text reference "Y1" (at 2.44 -3.525) (layer "F.SilkS")
-        (effects (font (size 1 1) (thickness 0.15)))
-    )
-    (fp_text value "12MHz" (at 2.44 3.525) (layer "F.Fab")
-        (effects (font (size 1 1) (thickness 0.15)))
-    )
-    (fp_text user "${REFERENCE}" (at 2.44 0) (layer "F.Fab")
-        (effects (font (size 1 1) (thickness 0.15)))
-    )
-    (fp_line (start -0.685 -2.525) (end 5.565 -2.525)
-      (stroke (width 0.12) (type solid)) (layer "F.SilkS"))
-    (fp_line (start -0.685 2.525) (end 5.565 2.525)
-      (stroke (width 0.12) (type solid)) (layer "F.SilkS"))
-    (fp_arc (start -0.685 2.525) (mid -3.21 0) (end -0.685 -2.525)
-      (stroke (width 0.12) (type solid)) (layer "F.SilkS"))
-    (fp_arc (start 5.565 -2.525) (mid 8.09 0) (end 5.565 2.525)
-      (stroke (width 0.12) (type solid)) (layer "F.SilkS"))
-    (fp_line (start -3.5 -2.8) (end -3.5 2.8)
-      (stroke (width 0.05) (type solid)) (layer "F.CrtYd"))
-    (fp_line (start -3.5 2.8) (end 8.4 2.8)
-      (stroke (width 0.05) (type solid)) (layer "F.CrtYd"))
-    (fp_line (start 8.4 -2.8) (end -3.5 -2.8)
-      (stroke (width 0.05) (type solid)) (layer "F.CrtYd"))
-    (fp_line (start 8.4 2.8) (end 8.4 -2.8)
-      (stroke (width 0.05) (type solid)) (layer "F.CrtYd"))
-    (fp_line (start -0.685 -2.325) (end 5.565 -2.325)
-      (stroke (width 0.1) (type solid)) (layer "F.Fab"))
-    (fp_line (start -0.685 2.325) (end 5.565 2.325)
-      (stroke (width 0.1) (type solid)) (layer "F.Fab"))
-    (fp_line (start -0.56 -2) (end 5.44 -2)
-      (stroke (width 0.1) (type solid)) (layer "F.Fab"))
-    (fp_line (start -0.56 2) (end 5.44 2)
-      (stroke (width 0.1) (type solid)) (layer "F.Fab"))
-    (fp_arc (start -0.685 2.325) (mid -3.01 0) (end -0.685 -2.325)
-      (stroke (width 0.1) (type solid)) (layer "F.Fab"))
-    (fp_arc (start -0.56 2) (mid -2.56 0) (end -0.56 -2)
-      (stroke (width 0.1) (type solid)) (layer "F.Fab"))
-    (fp_arc (start 5.44 -2) (mid 7.44 0) (end 5.44 2)
-      (stroke (width 0.1) (type solid)) (layer "F.Fab"))
-    (fp_arc (start 5.565 -2.325) (mid 7.89 0) (end 5.565 2.325)
-      (stroke (width 0.1) (type solid)) (layer "F.Fab"))
-    (pad "1" thru_hole circle (at 0 0) (size 1.5 1.5) (drill 0.8) (layers "*.Cu" "*.Mask")
-      (net 41 "Net-(U2-XO)") (pinfunction "1") (pintype "passive"))
-    (pad "2" thru_hole circle (at 4.88 0) (size 1.5 1.5) (drill 0.8) (layers "*.Cu" "*.Mask")
-      (net 40 "Net-(U2-XI)") (pinfunction "2") (pintype "passive"))
-    (model "${KICAD6_3DMODEL_DIR}/Crystal.3dshapes/Crystal_HC49-U_Vertical.wrl"
       (offset (xyz 0 0 0))
       (scale (xyz 1 1 1))
@@
   )
   (footprint "Package_SO:SOIC-16_3.9x9.9mm_P1.27mm" (layer "F.Cu")
-    (at 122.6454 78.7654)
+    (at 128.3208 79.0956)
     (descr "SOIC, 16 Pin (JEDEC MS-012AC, https://www.analog.com/media/en/package-pcb-resources/package/pkg_pdf/soic_narrow-r/r_16.pdf), generated with kicad-footprint-generator ipc_gullwing_generator.py")
     (tags "SOIC SO")

Commit message: April 2 commit
Parts:
- removed Y2: 12MHz, Crystal:Crystal_SMD_3225-4Pin_3.2x2.5mm
- added Q1: BC817, Package_TO_SOT_SMD:SOT-23, F.Cu at (128.4, 78.1)
- added Q2: BC817, Package_TO_SOT_SMD:SOT-23, F.Cu at (128.4, 82.5)
- added R2: 4k7/R0402, Resistor_SMD:R_0805_2012Metric, F.Cu at (128.1, 86.2)
- added R3: 4k7/R0402, Resistor_SMD:R_0805_2012Metric, F.Cu at (128.1, 89.2)
- added R4: 4k7/R0402, Resistor_SMD:R_0805_2012Metric, F.Cu at (128.1, 92.1)
- added SW1: ESP32_EN, Button_Switch_SMD:SW_SPST_EVQPE1, F.Cu at (121.4, 78.4)
- added SW2: ESP32_EN, Button_Switch_SMD:SW_SPST_EVQPE1, F.Cu at (121.4, 83.4)
- added Y1: 12MHz, Crystal:Crystal_SMD_3225-4Pin_3.2x2.5mm, F.Cu at (153.1, 104.9)
- C4, C5: footprint Capacitor_SMD:C_0805_2012Metric_Pad1.18x1.45mm_HandSolder -> Capacitor_SMD:C_0402_1005Metric
- J1: footprint Connector_USB:USB_C_Receptacle_Amphenol_12401610E4-2A_CircularHoles -> Connector_USB:USB_C_Receptacle_Amphenol_12401548E4-2A_CircularHoles
- moved J1 53.5 mm to (149.6, 116.1), turned to 0 degrees
- moved C4 47.4 mm to (150.8, 105.0), turned to 90 degrees
- moved C5 39.6 mm to (155.5, 104.9), turned to 90 degrees
- moved D1 37.9 mm to (146.7, 106.4), turned to -90 degrees
- moved U2 29.0 mm to (149.6, 98.7), turned to 90 degrees
Connections:
- U1 pad 27: unconnected-(U1-IO0/RTC_GPIO0/GPIO0-Pad27) -> GPIO00\BUT1
- U2 pad 13: unconnected-(U2-~{DTR}-Pad13) -> Net-(Q2-E)
- U2 pad 14: unconnected-(U2-~{RTS}-Pad14) -> Net-(Q1-E)
- U2 pad 9: unconnected-(U2-~{CTS}-Pad9) -> Net-(U2-~{CTS})

Commit message: April 3 commit
Parts:
- removed D1: 1N5819WS, Diode_SMD:D_SOD-323
- removed J1: USB_C_Receptacle, Connector_USB:USB_C_Receptacle_Amphenol_12401548E4-2A_CircularHoles
- added D2: 1N5819WS, Diode_SMD:D_SOD-323, F.Cu at (125.6, 109.7)
- added USB-C1: USB2.0_TYPE-C(A40-00119-A52-12), Connector_USB:USB_C_Receptacle_HRO_TYPE-C-31-M-12, F.Cu at (136.9, 116.3)
