File: uprojects/ESP32-S3-Basic/ESP32-S3-BasicA/ESP32-S3-BasicA.kicad_sch (KiCad schematic)
At the start: 5 parts, among them U1 ESP32-S3-WROOM-1x-N8R8

Commit message: April 1 commit
Parts:
- added C4, C5: 15, Capacitor_SMD:C_0805_2012Metric_Pad1.18x1.45mm_HandSolder, symbol Device:C_Small
- added D1: 1N5819WS, Diode_SMD:D_SOD-323, symbol Diode:1N5819WS
- added J1: USB_C_Receptacle, Connector_USB:USB_C_Receptacle_Amphenol_12401610E4-2A_CircularHoles, symbol Connector:USB_C_Receptacle
- added U2: CH340G, Package_SO:SOIC-16_3.9x9.9mm_P1.27mm, symbol Interface_USB:CH340G
- added Y1: 12MHz, Crystal:Crystal_HC49-U_Vertical, symbol Device:Crystal_Small
Connections:
- net GND: now also C4.1, C5.1, U2.1 (GND)
- new net: C5.2, U2.8 (XO), Y1.1
- new net: C4.2, U2.7 (XI), Y1.2
- new net: J1.A1 (GND), J1.A12 (GND), J1.B1 (GND), J1.B12 (GND)
- new net: D1.2 (A), J1.A4 (VBUS), J1.A9 (VBUS), J1.B4 (VBUS), J1.B9 (VBUS)
- new net: J1.A6 (D+), J1.B6 (D+), U2.5 (UD+)
- new net: J1.A7 (D-), J1.B7 (D-), U2.6 (UD-)
- new net +5V: D1.1 (K)
Other:
- moved on the sheet: C1, C2, C3, R1, U1

Commit message: April 1 commit
Parts:
- removed Y1: 12MHz, Crystal:Crystal_HC49-U_Vertical, symbol Device:Crystal_Small
- added Y1: 12MHz, symbol Device:Crystal_GND24_Small
Connections:
- net GND: now also Y1.4
- net at C5.2, U2.8 (XO): now also Y1.1
- net at C4.2, U2.7 (XI): now also Y1.3
Changed lines of the file:
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@@
 (kicad_sch (version 20230121) (generator eeschema)
   (paper "A3")
+  (junction (at 64.77 140.97) (diameter 0) (color 0 0 0 0)
+  )
   (junction (at 52.07 132.08) (diameter 0) (color 0 0 0 0)
   )
-  (junction (at 62.23 146.05) (diameter 0) (color 0 0 0 0)
-  )
   (junction (at 55.88 146.05) (diameter 0) (color 0 0 0 0)
   )
@@
   (junction (at 217.805 146.05) (diameter 0) (color 0 0 0 0)
   )
+  (junction (at 55.88 143.51) (diameter 0) (color 0 0 0 0)
+  )
   (junction (at 194.945 102.87) (diameter 0) (color 0 0 0 0)
   )
@@
   (junction (at 215.265 102.87) (diameter 0) (color 0 0 0 0)
   )
-  (junction (at 62.23 140.97) (diameter 0) (color 0 0 0 0)
+  (junction (at 64.77 146.05) (diameter 0) (color 0 0 0 0)
   )
   (junction (at 215.265 118.11) (diameter 0) (color 0 0 0 0)
@@
     (stroke (width 0) (type default))
   )
-  (wire (pts (xy 62.23 140.97) (xy 67.31 140.97))
-    (stroke (width 0) (type default))
-  )
   (wire (pts (xy 46.355 113.03) (xy 51.435 113.03))
     (stroke (width 0) (type default))
@@
     (stroke (width 0) (type default))
   )
-  (wire (pts (xy 55.88 140.97) (xy 55.88 146.05))
+  (wire (pts (xy 55.88 140.97) (xy 55.88 143.51))
     (stroke (width 0) (type default))
   )
@@
     (stroke (width 0) (type default))
   )
-  (wire (pts (xy 62.23 146.05) (xy 67.31 146.05))
-    (stroke (width 0) (type default))
-  )
   (wire (pts (xy 52.07 125.73) (xy 52.07 127))
     (stroke (width 0) (type default))
@@
     (stroke (width 0) (type default))
   )
-  (wire (pts (xy 60.96 140.97) (xy 62.23 140.97))
+  (wire (pts (xy 60.96 140.97) (xy 64.77 140.97))
     (stroke (width 0) (type default))
   )
@@
     (stroke (width 0) (type default))
   )
+  (wire (pts (xy 55.88 143.51) (xy 62.23 143.51))
+    (stroke (width 0) (type default))
+  )
+  (wire (pts (xy 55.88 143.51) (xy 55.88 146.05))
+    (stroke (width 0) (type default))
+  )
   (wire (pts (xy 57.15 132.08) (xy 52.07 132.08))
     (stroke (width 0) (type default))
@@
     (stroke (width 0) (type default))
   )
-  (wire (pts (xy 60.96 146.05) (xy 62.23 146.05))
+  (wire (pts (xy 60.96 146.05) (xy 64.77 146.05))
     (stroke (width 0) (type default))
   )
@@
     (stroke (width 0) (type default))
   )
+  (wire (pts (xy 64.77 140.97) (xy 67.31 140.97))
+    (stroke (width 0) (type default))
+  )
   (wire (pts (xy 67.31 133.35) (xy 57.15 133.35))
     (stroke (width 0) (type default))
   )
   (wire (pts (xy 52.07 127) (xy 52.07 128.27))
+    (stroke (width 0) (type default))
+  )
+  (wire (pts (xy 64.77 146.05) (xy 67.31 146.05))
     (stroke (width 0) (type default))
   )
@@
     (property "Intersheetrefs" "${INTERSHEET_REFS}" (at 199.4892 153.67 0)
       (effects (font (size 1.27 1.27)) (justify right) hide)
-    )
-  )
-  (symbol (lib_id "Device:Crystal_Small") (at 62.23 143.51 90) (unit 1)
-    (in_bom yes) (on_board yes) (dnp no) (fields_autoplaced)
-    (property "Reference" "Y1" (at 65.405 142.24 90)
-      (effects (font (size 1.27 1.27)) (justify right))
-    )
-    (property "Value" "12MHz" (at 65.405 144.78 90)
-      (effects (font (size 1.27 1.27)) (justify right))
-    )
-    (property "Footprint" "Crystal:Crystal_HC49-U_Vertical" (at 62.23 143.51 0)
-      (effects (font (size 1.27 1.27)) hide)
-    )
-    (property "Datasheet" "~" (at 62.23 143.51 0)
-      (effects (font (size 1.27 1.27)) hide)
-    )
-    (pin "1")
-    (pin "2")
-    (instances
-      (project "ESP32-S3-BasicA"
-        (path "/161e3938-9168-4147-870e-90c69eac8c76"
-          (reference "Y1") (unit 1)
-        )
-      )
-      (project "controllinoA"
-        (path "/cbf855aa-4ce6-42b1-9e73-b0ae89d280ce"
-          (reference "Y2") (unit 1)
-        )
-      )
     )
   )
@@
         )
       )
+    )
+  )
+  (symbol (lib_id "Device:Crystal_GND24_Small") (at 64.77 143.51 90) (unit 1)
+    (in_bom yes) (on_board yes) (dnp no)
+    (property "Reference" "Y1" (at 78.74 140.5957 90)
+      (effects (font (size 1.27 1.27)))
+    )
+    (property "Value" "12MHz" (at 64.77 147.955 90)
+      (effects (font (size 1.27 1.27)))
+    )
+    (property "Footprint" "" (at 64.77 143.51 0)
+      (effects (font (size 1.27 1.27)) hide)
+    )
+    (property "Datasheet" "~" (at 64.77 143.51 0)
+      (effects (font (size 1.27 1.27)) hide)
+    )
+    (pin "1")
+    (pin "3")
+    (pin "2")
+    (pin "4")
+    (instances
+      (project "ESP32-S3-BasicA"
+        (path "/161e3938-9168-4147-870e-90c69eac8c76"
+          (reference "Y1") (unit 1)
+        )
+      )

Commit message: April 2 commit
Parts:
- added Q1, Q2: BC817, Package_TO_SOT_SMD:SOT-23, symbol Transistor_BJT:BC817
- added R2, R3, R4: 4k7/R0402, Resistor_SMD:R_0805_2012Metric, symbol ESP32-S3-DevKit-LiPo_Rev_B:R
- added SW1, SW2: ESP32_EN, Button_Switch_SMD:SW_SPST_EVQPE1, symbol Switch:SW_Push
- C4, C5: footprint Capacitor_SMD:C_0805_2012Metric_Pad1.18x1.45mm_HandSolder -> Capacitor_SMD:C_0402_1005Metric
- J1: footprint Connector_USB:USB_C_Receptacle_Amphenol_12401610E4-2A_CircularHoles -> Connector_USB:USB_C_Receptacle_Amphenol_12401548E4-2A_CircularHoles
- Y1: footprint (none) -> Crystal:Crystal_SMD_3225-4Pin_3.2x2.5mm
Connections:
- net ESP_EN: now also Q1.3 (C), SW1.2
- net GND: now also SW1.1, SW2.1
- net GPIO00\BUT1: now reaches U1.27 (IO0/RTC_GPIO0/GPIO0)
- net GPIO00\BUT1: now also Q2.3 (C), SW2.2
- net at U2.13 (~{DTR}): now also Q2.2 (E), R2.1, R3.2
- net at U2.14 (~{RTS}): now also Q1.2 (E), R4.2
- net at U2.9 (~{CTS}): now also R2.2
- new net: Q2.1 (B), R4.1
- new net: Q1.1 (B), R3.1

Commit message: April 3 commit
Parts:
- removed D1: 1N5819WS, Diode_SMD:D_SOD-323, symbol Diode:1N5819WS
- removed J1: USB_C_Receptacle, Connector_USB:USB_C_Receptacle_Amphenol_12401548E4-2A_CircularHoles, symbol Connector:USB_C_Receptacle
- added D2: 1N5819WS, Diode_SMD:D_SOD-323, symbol Diode:1N5819WS
- added USB-C1: USB2.0_TYPE-C(A40-00119-A52-12), Connector_USB:USB_C_Receptacle_HRO_TYPE-C-31-M-12, symbol ESP32-S3-DevKit-LiPo_Rev_B:USB2.0_TYPE-C(A40-00119-A52-12)
Connections:
- net +5V: now also D2.1 (K)
- net GND: now also USB-C1.A1 (GND), USB-C1.A12 (GND), USB-C1.B1 (GND), USB-C1.B12 (GND)
- net at U2.5 (UD+): now also USB-C1.A6 (DP1), USB-C1.B6 (DP2)
- net at U2.6 (UD-): now also USB-C1.A7 (DN1), USB-C1.B7 (DN2)
- new net: D2.2 (A), USB-C1.A4 (VBUS), USB-C1.A9 (VBUS), USB-C1.B4 (VBUS), USB-C1.B9 (VBUS)
