File: uprojects/WiznetW5100S/TPIA/TPIA.kicad_sch (KiCad schematic)
At the start: 5 parts

Commit message: 13 May 24 Office
Parts:
- added C5, C6: 100n, Capacitor_SMD:C_1206_3216Metric, symbol Device:C_Small
- added D1: MMSZ4680T1G CE, Diode_SMD:D_SOD-123, symbol Device:D_Zener_Small
- added D2, D3: S2, Diode_SMD:D_SOD-323, symbol Device:D_Schottky_Small
- added D4: SS14, Diode_SMD:D_SMA, symbol Device:D_Small
- added J1: Conn_01x06, Connector_Phoenix_MC_HighVoltage:PhoenixContact_MC_1,5_6-G-5.08_1x06_P5.08mm_Horizontal, symbol Connector_Generic:Conn_01x06
- added R1, R2, R3, R4: 10K, Resistor_SMD:R_1206_3216Metric, symbol Device:R_Small
- added R5: 1K, Resistor_SMD:R_1206_3216Metric, symbol Device:R_Small
- added SW1, SW2, SW3: SW_Push, Button_Switch_SMD:SW_SPST_PTS810, symbol Switch:SW_Push
- added U2: buck2596, DC_DC_LM2596_small:DC_DC_LM2596_small, symbol Buck2596:buck2596
Connections:
- net GND: now also C5.2, C6.2, D1.2 (A), D2.2 (A), D3.2 (A), J1.3 (Pin_3), R2.2, R4.2, U2.4 (out-)
- net at U1.17 (GP13): now also SW1.2
- net at U1.19 (GP14): now also SW2.2
- net at U1.20 (GP15): now also SW3.2
- net ADC0: now reaches U1.31 (GP26)
- net ADC0: now also C5.1, D2.1 (K), R1.2, R2.1
- net ADC1: now reaches U1.32 (GP27)
- net ADC1: now also C6.1, D3.1 (K), R3.2, R4.1
- net ADC2: now reaches U1.34 (GP28)
- net at C3.1, U1.36 (3V3): now also R5.1
- net Vin: now reaches C1.1, U1.39 (VSYS)
- net Vin: now also U2.3 (out+)
- new net: J1.5 (Pin_5), U2.2 (in-)
- new net: D4.2 (A), J1.6 (Pin_6)
- new net: D4.1 (K), U2.1 (in+)
- new net AIN0: J1.2 (Pin_2), R1.1
- new net AIN1: R3.1
- new net Top: D1.1 (K), J1.1 (Pin_1), R5.2
