File: uprojects/WiznetW5100S/TPIA/TPIA.kicad_pcb (KiCad board)
At the start: 2 copper layers, 5 parts

Commit message: 13 May 24 Office
Connections:
- C3 pad 1: unconnected-(C3-Pad1) -> Net-(U1-3V3)
- U1 pad 36: unconnected-(U1-3V3-Pad36) -> Net-(U1-3V3)

Commit message: 14 May 24 Office
Parts:
- added C5: 100n, Capacitor_SMD:C_1206_3216Metric, F.Cu at (172.0, 81.7)
- added C6: 100n, Capacitor_SMD:C_1206_3216Metric, F.Cu at (196.1, 117.7)
- added D1: MMSZ4680T1G CE, Diode_SMD:D_SOD-123, F.Cu at (172.1, 58.3)
- added D2: S2, Diode_SMD:D_SOD-323, F.Cu at (171.6, 79.4)
- added D3: S2, Diode_SMD:D_SOD-323, F.Cu at (195.5, 123.8)
- added D4: SS14, Diode_SMD:D_SMA, F.Cu at (216.1, 79.0)
- added J1: Conn_01x06, Connector_Phoenix_MC_HighVoltage:PhoenixContact_MC_1,5_6-G-5.08_1x06_P5.08mm_Horizontal, F.Cu at (222.5, 104.5)
- added R1: 10K, Resistor_SMD:R_1206_3216Metric, F.Cu at (172.0, 84.2)
- added R2: 10K, Resistor_SMD:R_1206_3216Metric, F.Cu at (172.0, 77.1)
- added R3: 10K, Resistor_SMD:R_1206_3216Metric, F.Cu at (183.8, 120.9)
- added R4: 10K, Resistor_SMD:R_1206_3216Metric, F.Cu at (183.8, 124.2)
- added R5: 1K, Resistor_SMD:R_1206_3216Metric, F.Cu at (172.0, 60.7)
- added SW1: SW_Push, Button_Switch_SMD:SW_SPST_PTS810, F.Cu at (127.7, 85.9)
- added SW2: SW_Push, Button_Switch_SMD:SW_SPST_PTS810, F.Cu at (127.6, 92.9)
- added SW3: SW_Push, Button_Switch_SMD:SW_SPST_PTS810, F.Cu at (127.6, 100.2)
- added U2: buck2596, DC_DC_LM2596_small:DC_DC_LM2596_small, F.Cu at (205.9, 59.8)
- moved C1 40.7 mm to (172.1, 55.3), turned to 0 degrees
- moved C4 1.27 mm to (172.1, 52.7)
- moved C3 1.18 mm to (172.0, 63.2)
- moved C2 1.17 mm to (172.0, 65.7)
Connections:
- C1 pad 1: unconnected-(C1-Pad1) -> Vin
- C1 pad 2: GND -> Bottom
- C2 pad 1: unconnected-(C2-Pad1) -> Net-(U1-ADC_REF)
- C2 pad 2: GND -> Bottom
- C3 pad 2: GND -> Bottom
- C4 pad 1: unconnected-(C4-Pad1) -> Net-(U1-VBUS)
- C4 pad 2: GND -> Bottom
- U1 pad 17: unconnected-(U1-GP13-Pad17) -> Net-(U1-GP13)
- U1 pad 19: unconnected-(U1-GP14-Pad19) -> Net-(U1-GP14)
- U1 pad 20: unconnected-(U1-GP15-Pad20) -> Net-(U1-GP15)
- U1 pad 3: GND -> Bottom
- U1 pad 31: unconnected-(U1-GP26-Pad31) -> ADC0
- U1 pad 32: unconnected-(U1-GP27-Pad32) -> ADC1
- U1 pad 33: unconnected-(U1-GND-Pad33) -> Bottom
- U1 pad 34: unconnected-(U1-GP28-Pad34) -> ADC2
- U1 pad 35: unconnected-(U1-ADC_REF-Pad35) -> Net-(U1-ADC_REF)
- U1 pad 38: unconnected-(U1-GND-Pad38) -> Bottom
- U1 pad 39: unconnected-(U1-VSYS-Pad39) -> Vin
- U1 pad 40: unconnected-(U1-VBUS-Pad40) -> Net-(U1-VBUS)
Routing:
- net ADC0: track 0.00 -> 7.10 mm
- net Bottom: track 0.00 -> 5.29 mm
Other:
- rule pad_to_mask_clearance: 0 -> 0.2
