File: uprojects/WiznetW5100S/TPIA/TPIA.kicad_pcb (KiCad board)
At the start: 2 copper layers, 21 parts, among them J1 Conn_01x06, SW1 SW_Push, SW2 SW_Push, SW3 SW_Push, U2 buck2596

Commit message: 17 May 24
Parts:
- moved D3 39.8 mm to (172.1, 91.6)
- moved C6 39.3 mm to (172.0, 86.7)
Changed lines of the file:
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@@
   )
   (footprint "Capacitor_SMD:C_1206_3216Metric" (layer "F.Cu")
-    (at 196.137 117.729)
+    (at 171.9834 86.6648)
     (descr "Capacitor SMD 1206 (3216 Metric), square (rectangular) end terminal, IPC_7351 nominal, (Body size source: IPC-SM-782 page 76, https://www.pcb-3d.com/wordpress/wp-content/uploads/ipc-sm-782a_amendment_1_and_2.pdf), generated with kicad-footprint-generator")
     (tags "capacitor")
@@
   )
   (footprint "Diode_SMD:D_SOD-323" (layer "F.Cu")
-    (at 195.482 123.829)
+    (at 172.0596 91.5924)
     (descr "SOD-323")
     (tags "SOD-323")
