File: uprojects/Laurent ESP Mesh/meshlite/meshlite/meshlite.kicad_pcb (KiCad board)
At the start: 2 copper layers, 55.3 x 53.8 mm, 13 parts, among them J1 Conn_01x02, J2 Conn_01x02, J3 Conn_01x06, K1 CPC1916Y, U1 MOUDLE-SEEEDUINO-XIAO-ESP32C3

Commit message: 1 July 24
Parts:
- J1, J2: footprint Connector_PinHeader_2.54mm:PinHeader_1x02_P2.54mm_Vertical -> Connector_Phoenix_MC_HighVoltage:PhoenixContact_MC_1,5_2-G-5.08_1x02_P5.08mm_Horizontal
- R1: value 3K3 -> R_Small
- moved J1 35.5 mm to (126.2, 127.0)
- moved J2 14.8 mm to (167.4, 127.1), turned to 0 degrees
Other:
- board text added: "SENSOR"
