File: uprojects/Laurent ESP Mesh/meshlite/meshlite/meshlite.kicad_sch (KiCad schematic)
At the start: 3 parts, among them J1 Conn_01x02, U1 MOUDLE-SEEEDUINO-XIAO-ESP32C3

Commit message: 30 June 24
Parts:
- added D1, D2, D3: LED, LED_SMD:LED_0603_1608Metric, symbol Device:LED_Small
- added J2: Conn_01x02, Connector_PinHeader_2.54mm:PinHeader_1x02_P2.54mm_Vertical, symbol Connector_Generic:Conn_01x02
- added J3: Conn_01x06, Connector_PinHeader_2.54mm:PinHeader_1x06_P2.54mm_Vertical, symbol Connector_Generic:Conn_01x06
- added K1: CPC1916Y, CPC1916Y:CPC1916Y, symbol CPC1916Y:CPC1916Y
- added R2: R_Small, Resistor_SMD:R_0603_1608Metric, symbol Device:R_Small
- added R3, R4, R5: 470E, Resistor_SMD:R_0603_1608Metric, symbol Device:R_Small
- J1: footprint (none) -> Connector_PinHeader_2.54mm:PinHeader_1x02_P2.54mm_Vertical
- R1: footprint (none) -> Resistor_SMD:R_0603_1608Metric
- U1: footprint MOUDLE14P-SMD-2.54-21X17.8MM -> xiao ESP32C3_PCB:MOUDLE14P-SMD-2.54-21X17.8MM
Connections:
- net A0: now also U1.1 (PA02_A0_D0)
- net GND: now also D1.1 (K), D2.1 (K), D3.1 (K), K1.2
- net at U1.11 (PA6_A10_D10_MOSI): now also R2.1
- net at U1.2 (PA4_A1_D1): now also R3.2
- net at U1.3 (PA10_A2_D2): now also R4.2
- net at U1.4 (PA11_A3_D3): now also R5.2
- new net: D1.2 (A), R3.1
- new net: K1.1, R2.2
- new net: D3.2 (A), R5.1
- new net: J2.2 (Pin_2), K1.3
- new net: J2.1 (Pin_1), K1.4
- new net: D2.2 (A), R4.1

Commit message: 1 July 24
Parts:
- J1, J2: footprint Connector_PinHeader_2.54mm:PinHeader_1x02_P2.54mm_Vertical -> Connector_Phoenix_MC_HighVoltage:PhoenixContact_MC_1,5_2-G-5.08_1x02_P5.08mm_Horizontal
Changed lines of the file:
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@@
       (effects (font (size 1.27 1.27)))
     )
-    (property "Footprint" "Connector_PinHeader_2.54mm:PinHeader_1x02_P2.54mm_Vertical" (at 41.91 82.55 0)
+    (property "Footprint" "Connector_Phoenix_MC_HighVoltage:PhoenixContact_MC_1,5_2-G-5.08_1x02_P5.08mm_Horizontal" (at 41.91 82.55 0)
       (effects (font (size 1.27 1.27)) hide)
     )
@@
       (effects (font (size 1.27 1.27)) (justify left))
     )
-    (property "Footprint" "Connector_PinHeader_2.54mm:PinHeader_1x02_P2.54mm_Vertical" (at 239.395 86.995 0)
+    (property "Footprint" "Connector_Phoenix_MC_HighVoltage:PhoenixContact_MC_1,5_2-G-5.08_1x02_P5.08mm_Horizontal" (at 239.395 86.995 0)
       (effects (font (size 1.27 1.27)) hide)
     )

Commit message: 7 August Office 001
Parts:
- removed J3: Conn_01x06, Connector_PinHeader_2.54mm:PinHeader_1x06_P2.54mm_Vertical, symbol Connector_Generic:Conn_01x06
- added J3, J4: Conn_02x05_Odd_Even, Connector_IDC:IDC-Header_2x05_P2.54mm_Vertical, symbol Connector_Generic:Conn_02x05_Odd_Even
Changed lines of the file:
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@@
+    )
+  )
+  (symbol (lib_id "Connector_Generic:Conn_02x05_Odd_Even") (at 182.88 136.525 0) (unit 1)
+    (in_bom yes) (on_board yes) (dnp no) (fields_autoplaced)
+    (property "Reference" "J4" (at 184.15 125.73 0)
+      (effects (font (size 1.27 1.27)))
+    )
+    (property "Value" "Conn_02x05_Odd_Even" (at 184.15 128.27 0)
+      (effects (font (size 1.27 1.27)))
+    )
+    (property "Footprint" "Connector_IDC:IDC-Header_2x05_P2.54mm_Vertical" (at 182.88 136.525 0)
+      (effects (font (size 1.27 1.27)) hide)
+    )
+    (property "Datasheet" "~" (at 182.88 136.525 0)
+      (effects (font (size 1.27 1.27)) hide)
+    )
+    (pin "10")
+    (pin "6")
+    (pin "5")
+    (pin "3")
+    (pin "2")
+    (pin "4")
+    (pin "1")
+    (pin "8")
+    (pin "7")
+    (pin "9")
+    (instances
+      (project "meshlite"
+        (path "/5228a7f0-3f2c-4c1e-8386-5ebdfda02c7b"
+          (reference "J4") (unit 1)
+        )
+      )
     )
   )
@@
     )
   )
-  (symbol (lib_id "Connector_Generic:Conn_01x06") (at 89.535 130.81 180) (unit 1)
+  (symbol (lib_id "Connector_Generic:Conn_02x05_Odd_Even") (at 83.82 136.525 0) (unit 1)
     (in_bom yes) (on_board yes) (dnp no) (fields_autoplaced)
-    (property "Reference" "J3" (at 89.535 116.84 0)
+    (property "Reference" "J3" (at 85.09 125.73 0)
       (effects (font (size 1.27 1.27)))
     )
-    (property "Value" "Conn_01x06" (at 89.535 119.38 0)
+    (property "Value" "Conn_02x05_Odd_Even" (at 85.09 128.27 0)
       (effects (font (size 1.27 1.27)))
     )
-    (property "Footprint" "Connector_PinHeader_2.54mm:PinHeader_1x06_P2.54mm_Vertical" (at 89.535 130.81 0)
+    (property "Footprint" "Connector_IDC:IDC-Header_2x05_P2.54mm_Vertical" (at 83.82 136.525 0)
       (effects (font (size 1.27 1.27)) hide)
     )
-    (property "Datasheet" "~" (at 89.535 130.81 0)
+    (property "Datasheet" "~" (at 83.82 136.525 0)
       (effects (font (size 1.27 1.27)) hide)
     )
+    (pin "10")
     (pin "6")
-    (pin "1")
+    (pin "5")
+    (pin "3")
     (pin "2")
     (pin "4")
-    (pin "3")
-    (pin "5")
+    (pin "1")
+    (pin "8")
+    (pin "7")
+    (pin "9")
     (instances
       (project "meshlite"

Commit message: 8-august 24
Parts:
- removed J1, J2: Conn_01x02, Connector_Phoenix_MC_HighVoltage:PhoenixContact_MC_1,5_2-G-5.08_1x02_P5.08mm_Horizontal, symbol Connector_Generic:Conn_01x02
- J3, J4: footprint Connector_IDC:IDC-Header_2x05_P2.54mm_Vertical -> Connector_PinSocket_2.54mm:PinSocket_2x05_P2.54mm_Vertical
Changed lines of the file:
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@@
-    (stroke (width 0) (type default))
-  )
-  (wire (pts (xy 51.435 82.55) (xy 51.435 87.63))
     (stroke (width 0) (type default))
   )
@@
     (stroke (width 0) (type default))
   )
-  (wire (pts (xy 48.26 72.39) (xy 53.34 72.39))
-    (stroke (width 0) (type default))
-  )
   (wire (pts (xy 94.615 94.615) (xy 97.155 94.615))
     (stroke (width 0) (type default))
@@
     (stroke (width 0) (type default))
   )
-  (wire (pts (xy 215.9 86.995) (xy 234.315 86.995))
-    (stroke (width 0) (type default))
-  )
-  (wire (pts (xy 53.34 72.39) (xy 53.34 74.295))
-    (stroke (width 0) (type default))
-  )
   (wire (pts (xy 105.41 86.995) (xy 117.475 86.995))
     (stroke (width 0) (type default))
@@
     (stroke (width 0) (type default))
   )
-  (wire (pts (xy 215.9 89.535) (xy 234.315 89.535))
-    (stroke (width 0) (type default))
-  )
-  (wire (pts (xy 48.26 80.01) (xy 48.26 72.39))
-    (stroke (width 0) (type default))
-  )
   (wire (pts (xy 86.36 85.725) (xy 86.36 90.17))
     (stroke (width 0) (type default))
@@
     (stroke (width 0) (type default))
   )
-  (wire (pts (xy 46.99 82.55) (xy 51.435 82.55))
-    (stroke (width 0) (type default))
-  )
   (wire (pts (xy 81.28 90.17) (xy 86.36 90.17))
     (stroke (width 0) (type default))
@@
   )
   (wire (pts (xy 105.41 85.725) (xy 105.41 86.995))
-    (stroke (width 0) (type default))
-  )
-  (wire (pts (xy 46.99 80.01) (xy 48.26 80.01))
     (stroke (width 0) (type default))
   )
@@
     )
   )
-  (symbol (lib_id "Connector_Generic:Conn_01x02") (at 41.91 82.55 180) (unit 1)
-    (in_bom yes) (on_board yes) (dnp no) (fields_autoplaced)
-    (property "Reference" "J1" (at 41.91 73.66 0)
-      (effects (font (size 1.27 1.27)))
-    )
-    (property "Value" "Conn_01x02" (at 41.91 76.2 0)
-      (effects (font (size 1.27 1.27)))
-    )
-    (property "Footprint" "Connector_Phoenix_MC_HighVoltage:PhoenixContact_MC_1,5_2-G-5.08_1x02_P5.08mm_Horizontal" (at 41.91 82.55 0)
-      (effects (font (size 1.27 1.27)) hide)
-    )
-    (property "Datasheet" "~" (at 41.91 82.55 0)
-      (effects (font (size 1.27 1.27)) hide)
-    )
-    (pin "1")
-    (pin "2")
-    (instances
-      (project "meshlite"
-        (path "/5228a7f0-3f2c-4c1e-8386-5ebdfda02c7b"
-          (reference "J1") (unit 1)
-        )
-      )
-    )
-  )
   (symbol (lib_id "CPC1916Y:CPC1916Y") (at 187.96 86.995 0) (unit 1)
     (in_bom yes) (on_board yes) (dnp no) (fields_autoplaced)
@@
       (effects (font (size 1.27 1.27)))
     )
-    (property "Footprint" "Connector_IDC:IDC-Header_2x05_P2.54mm_Vertical" (at 182.88 136.525 0)
+    (property "Footprint" "Connector_PinSocket_2.54mm:PinSocket_2x05_P2.54mm_Vertical" (at 182.88 136.525 0)
       (effects (font (size 1.27 1.27)) hide)
     )
@@
         (path "/5228a7f0-3f2c-4c1e-8386-5ebdfda02c7b"
           (reference "D2") (unit 1)
-        )
-      )
-    )
-  )
-  (symbol (lib_id "Connector_Generic:Conn_01x02") (at 239.395 86.995 0) (unit 1)
-    (in_bom yes) (on_board yes) (dnp no) (fields_autoplaced)
-    (property "Reference" "J2" (at 241.935 86.995 0)
-      (effects (font (size 1.27 1.27)) (justify left))
-    )
-    (property "Value" "Conn_01x02" (at 241.935 89.535 0)
-      (effects (font (size 1.27 1.27)) (justify left))
-    )
-    (property "Footprint" "Connector_Phoenix_MC_HighVoltage:PhoenixContact_MC_1,5_2-G-5.08_1x02_P5.08mm_Horizontal" (at 239.395 86.995 0)
-      (effects (font (size 1.27 1.27)) hide)
-    )
-    (property "Datasheet" "~" (at 239.395 86.995 0)
-      (effects (font (size 1.27 1.27)) hide)
-    )
-    (pin "1")
-    (pin "2")
-    (instances
-      (project "meshlite"
-        (path "/5228a7f0-3f2c-4c1e-8386-5ebdfda02c7b"
-          (reference "J2") (unit 1)
         )
       )
@@
       (effects (font (size 1.27 1.27)))
     )
-    (property "Footprint" "Connector_IDC:IDC-Header_2x05_P2.54mm_Vertical" (at 83.82 136.525 0)
-      (effects (font (size 1.27 1.27)) hide)
-    )
+    (property "Footprint" "Connector_PinSocket_2.54mm:PinSocket_2x05_P2.54mm_Vertical" (at 83.82 136.525 0)
+      (effects (font (size 1.27 1.27)) hide)
+    )
