File: uprojects/Adee/PCB/STA5635/STA5635.kicad_sch (KiCad schematic)
At the start: 1 part, among them U1 STA5635A

Commit message: 1-august 24
Parts:
- added C1, C2: 1uF, symbol Device:C_Small
- added J1: USB_C_Receptacle_USB2.0, symbol Connector:USB_C_Receptacle_USB2.0
- added R1, R2: 5.1K, symbol Device:R_Small
- added U2: AP2127K-1.8, Package_TO_SOT_SMD:SOT-23-5, symbol Regulator_Linear:AP2127K-1.8
Connections:
- new net: J1.A5 (CC1), R1.1
- new net: C1.1, J1.A4 (VBUS), J1.A9 (VBUS), J1.B4 (VBUS), J1.B9 (VBUS), U2.1 (VIN), U2.3 (EN)
- new net: J1.B5 (CC2), R2.1
- new net GND: C1.2, C2.2, J1.A1 (GND), J1.A12 (GND), J1.B1 (GND), J1.B12 (GND), J1.S1 (SHIELD), R1.2, R2.2, U2.2 (GND)
- new net VCC: C2.1, U2.5 (VOUT)

Commit message: 3-august 24
Parts:
- removed J1: USB_C_Receptacle_USB2.0, symbol Connector:USB_C_Receptacle_USB2.0
- removed R2: 5.1K, symbol Device:R_Small
- added C3, C4, C5, C6: 104, Capacitor_SMD:C_1206_3216Metric, symbol Device:C_Small
- added J1: Conn_01x20, Connector_PinHeader_2.54mm:PinHeader_1x20_P2.54mm_Vertical, symbol Connector_Generic:Conn_01x20
- C1, C2: footprint (none) -> Capacitor_SMD:C_1206_3216Metric
- R1: value 5.1K -> R_Small
- U1: footprint VFQPN_A5635A_STM -> VFQPN_A5635A_STM:VFQPN_A5635A_STM
Connections:
- net GND: now also U1.14 (GND_DIG), C3.2, C4.2, C5.2, C6.2; no longer R1.2
- net VCC: now also R1.1
- net CHIP_EN: now reaches U1.12 (CHIP_EN)
- net CHIP_EN: now also R1.2, C3.1
- net at U1.13 (V11_OUT_DIG): now also C6.1
- net at U1.15 (VCC_IO): now also C5.1
- net at U1.16 (V18_OUT): now also C4.1
- net at U1.17 (TCXO_CLK): now also J1.20 (Pin_20)
- net at U1.18 (GND_IO): now also J1.19 (Pin_19)
- net at U1.19 (Q-sign2): now also J1.18 (Pin_18)
- net at U1.20 (I-mag2): now also J1.17 (Pin_17)
- net at U1.21 (I-sign2): now also J1.16 (Pin_16)
- net at U1.22 (Q-mag2): now also J1.15 (Pin_15)
- net at U1.23 (I-mag1): now also J1.14 (Pin_14)
- net at U1.24 (I-sign1): now also J1.13 (Pin_13)
- net at U1.25 (Q-sign1): now also J1.12 (Pin_12)
- net at U1.26 (Q-mag1): now also J1.11 (Pin_11)
- net at U1.27 (SPI_CLK): now also J1.10 (Pin_10)
- net at U1.28 (SPI_DI): now also J1.9 (Pin_9)
- net at U1.29 (SPI_DO): now also J1.8 (Pin_8)
- net at U1.30 (SPI_NCS): now also J1.7 (Pin_7)
- net at U1.31 (LNA_IN): now also J1.6 (Pin_6)
- net at U1.32 (LNA_GND): now also J1.5 (Pin_5)

Commit message: 4-august 24
Parts:
- added C7, C8, C9: 104, Capacitor_SMD:C_1206_3216Metric, symbol Device:C_Small
- added J2: SMA_CONNECTOR, SMA_CONNECTOR:LPRS_SMA_CONNECTOR, symbol SMA_CONNECTOR:SMA_CONNECTOR
- added L1, L2: L_Small, Inductor_SMD:L_1206_3216Metric_Pad1.22x1.90mm_HandSolder, symbol Device:L_Small
- added R2: 1K, Resistor_SMD:R_1206_3216Metric, symbol Device:R_Small
- R1: value R_Small -> 1K; footprint (none) -> Resistor_SMD:R_1206_3216Metric
Connections:
- net GND: now also C7.2, C8.2, J2.G1, J2.G2, J2.G3, J2.G4
- net VCC: now also U1.8 (VCC_RF), C8.1, R2.1
- net VDD: now reaches C1.1, U2.1 (VIN), U2.3 (EN)
- net at U1.1 (V11_LNA): now also U1.3 (V11_CHAIN), U1.7 (V11_OUT_RF), U1.9 (V11_PLL), C7.1
- net at U1.5 (TP_IF_P/Sense1(1)): now also L1.1, R2.2
- net at U1.6 (TP_IF_N/Sense2(1)): now also L1.2, L2.1
- new net: C9.2, L2.2
- new net: C9.1, J2.1
Other:
- moved on the sheet: C3, R1

Commit message: 36 July Office 001
Parts:
- removed J1: Conn_01x20, Connector_PinHeader_2.54mm:PinHeader_1x20_P2.54mm_Vertical, symbol Connector_Generic:Conn_01x20
- added J1: Conn_02x20_Odd_Even, Connector_PinHeader_2.54mm:PinHeader_2x20_P2.54mm_Vertical, symbol Connector_Generic:Conn_02x20_Odd_Even
- added J3, J4: Conn_01x02, Connector_PinHeader_2.54mm:PinHeader_1x02_P2.54mm_Vertical, symbol Connector_Generic:Conn_01x02
Connections:
- net CHIP_EN: now also J1.1 (Pin_1), J3.2 (Pin_2); no longer C3.1, R1.2
- net GND: now also U1.18 (GND_IO), U1.33 (GND), J1.12 (Pin_12), J1.30 (Pin_30)
- net VCC: now also U1.5 (TP_IF_P/Sense1(1))
- net VDD: now also J1.29 (Pin_29), J4.2 (Pin_2); no longer U2.3 (EN)
- net LNA_IN: now reaches L1.2, L2.1
- net LNA_IN: now also U1.31 (LNA_IN); no longer U1.6 (TP_IF_N/Sense2(1))
- net at L1.1, R2.2: now also U1.6 (TP_IF_N/Sense2(1)); no longer U1.5 (TP_IF_P/Sense1(1))
- net at U1.27 (SPI_CLK): now also J1.19 (Pin_19)
- net at U1.26 (Q-mag1): now also J1.21 (Pin_21)
- net at U1.25 (Q-sign1): now also J1.23 (Pin_23)
- net at U1.24 (I-sign1): now also J1.25 (Pin_25)
- net at U1.23 (I-mag1): now also J1.27 (Pin_27)
- net at U1.22 (Q-mag2): now also J1.37 (Pin_37)
- net at U1.21 (I-sign2): now also J1.31 (Pin_31)
- net at U1.20 (I-mag2): now also J1.33 (Pin_33)
- net at U1.19 (Q-sign2): now also J1.35 (Pin_35)
- net at U1.17 (TCXO_CLK): now also J1.39 (Pin_39)
- net GNDA: now reaches U1.32 (LNA_GND)
- net at U1.30 (SPI_NCS): now also J1.13 (Pin_13)
- net at U1.29 (SPI_DO): now also J1.15 (Pin_15)
- net at U1.28 (SPI_DI): now also J1.17 (Pin_17)
- new net: C3.1, J3.1 (Pin_1), R1.2
- new net: J4.1 (Pin_1), U2.3 (EN)
- new net 5V: J1.11 (Pin_11)
Other:
- moved on the sheet: C1

Commit message: 6 August Office 001
Parts:
- added TP1, TP2: TP, symbol Connector:TestPoint_Small
Connections:
- net at U1.2 (LNA_OUT): now also TP2.1
- net at U1.4 (RFA_IN): now also TP1.1
Changed lines of the file:
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@@
+    (stroke (width 0) (type default))
+  )
+  (wire (pts (xy 103.505 80.645) (xy 103.505 65.405))
     (stroke (width 0) (type default))
   )
@@
     (stroke (width 0) (type default))
   )
+  (wire (pts (xy 105.41 75.565) (xy 105.41 65.405))
+    (stroke (width 0) (type default))
+  )
   (wire (pts (xy 86.995 45.085) (xy 81.915 45.085))
     (stroke (width 0) (type default))
   )
+  (wire (pts (xy 107.95 75.565) (xy 105.41 75.565))
+    (stroke (width 0) (type default))
+  )
   (wire (pts (xy 19.05 83.82) (xy 19.05 85.725))
     (stroke (width 0) (type default))
@@
   )
   (wire (pts (xy 184.15 73.025) (xy 191.77 73.025))
+    (stroke (width 0) (type default))
+  )
+  (wire (pts (xy 107.95 80.645) (xy 103.505 80.645))
     (stroke (width 0) (type default))
   )
@@
     )
   )
+  (symbol (lib_id "Connector:TestPoint_Small") (at 105.41 65.405 90) (unit 1)
+    (in_bom yes) (on_board yes) (dnp no)
+    (property "Reference" "TP2" (at 105.41 63.5 0)
+      (effects (font (face "KiCad Font") (size 0.8 0.8)) (justify left))
+    )
+    (property "Value" "TP" (at 105.41 64.77 0)
+      (effects (font (face "KiCad Font") (size 0.8 0.8)) (justify left))
+    )
+    (property "Footprint" "" (at 105.41 60.325 0)
+      (effects (font (size 1.27 1.27)) hide)
+    )
+    (property "Datasheet" "~" (at 105.41 60.325 0)
+      (effects (font (size 1.27 1.27)) hide)
+    )
+    (pin "1")
+    (instances
+      (project "STA5635"
+        (path "/8189ff51-b9c1-4db5-b4d6-e4c84473a181"
+          (reference "TP2") (unit 1)
+        )
+      )
+    )
+  )
   (symbol (lib_id "power:VCC") (at 81.915 68.58 0) (unit 1)
     (in_bom yes) (on_board yes) (dnp no) (fields_autoplaced)
@@
         )
       )
+    )
+  )
+  (symbol (lib_id "Connector:TestPoint_Small") (at 103.505 65.405 90) (unit 1)
+    (in_bom yes) (on_board yes) (dnp no)
+    (property "Reference" "TP1" (at 103.505 63.5 0)
+      (effects (font (face "KiCad Font") (size 0.8 0.8)) (justify left))
+    )
+    (property "Value" "TP" (at 103.505 64.77 0)
+      (effects (font (face "KiCad Font") (size 0.8 0.8)) (justify left))
+    )
+    (property "Footprint" "" (at 103.505 60.325 0)
+      (effects (font (size 1.27 1.27)) hide)
+    )
+    (property "Datasheet" "~" (at 103.505 60.325 0)
+      (effects (font (size 1.27 1.27)) hide)
+    )
+    (pin "1")
+    (instances
+      (project "STA5635"
+        (path "/8189ff51-b9c1-4db5-b4d6-e4c84473a181"
+          (reference "TP1") (unit 1)
+        )
+      )

Commit message: 6 August Office 001
Parts:
- added TP10, TP3, TP4, TP5, TP6, TP7, TP8, TP9: TP, Connector_PinHeader_2.54mm:PinHeader_1x01_P2.54mm_Vertical, symbol Connector:TestPoint_Small
- TP1, TP2: footprint (none) -> Connector_PinHeader_2.54mm:PinHeader_1x01_P2.54mm_Vertical
Connections:
- net GND: now also TP10.1
- net VCC: now also TP6.1, TP9.1
- net at C5.1, U1.15 (VCC_IO): now also TP3.1
- net 1.1V: now reaches C7.1, U1.1 (V11_LNA), U1.3 (V11_CHAIN), U1.7 (V11_OUT_RF), U1.9 (V11_PLL)
- net 1.1V: now also TP5.1, TP7.1
- net at L1.1, R2.2, U1.6 (TP_IF_N/Sense2(1)): now also TP8.1
- net at C6.1, U1.13 (V11_OUT_DIG): now also TP4.1

Commit message: 27 August Office 001
Other:
- note added: "D10 COMPATIBLE GPIO0 HEADER"
Changed lines of the file:
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@@
     (stroke (width 0) (type default))
+  )
+  (text "D10 COMPATIBLE GPIO0 HEADER" (at 242.57 57.785 0)
+    (effects (font (size 1.27 1.27)) (justify left bottom))
   )
   (global_label "CHIP_EN" (shape input) (at 104.775 100.965 180) (fields_autoplaced)

Commit message: 29 August Office 001
Parts:
- J3: value Conn_01x02 -> EN
Changed lines of the file:
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@@
       (effects (font (size 1.27 1.27)) (justify left))
     )
-    (property "Value" "Conn_01x02" (at 34.29 81.915 0)
+    (property "Value" "EN" (at 34.29 81.915 0)
       (effects (font (size 1.27 1.27)) (justify left))
     )
