File: uprojects/Adee/PCB/STA5635/STA5635.kicad_sch (KiCad schematic)
At the start: 29 parts, among them J1 Conn_02x20_Odd_Even, J2 SMA_CONNECTOR, J3 EN, J4 Conn_01x02, U1 STA5635A, U2 AP2127K-1.8

Commit message: update from home 30-8-2024
Parts:
- removed TP6, TP7: TP, Connector_PinHeader_2.54mm:PinHeader_1x01_P2.54mm_Vertical, symbol Connector:TestPoint_Small
Changed lines of the file:
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@@
   (junction (at 48.26 73.025) (diameter 0) (color 0 0 0 0)
   )
-  (junction (at 104.14 88.265) (diameter 0) (color 0 0 0 0)
-  )
   (junction (at 49.53 46.355) (diameter 0) (color 0 0 0 0)
   )
@@
   (junction (at 97.155 88.265) (diameter 0) (color 0 0 0 0)
   )
-  (junction (at 93.345 90.805) (diameter 0) (color 0 0 0 0)
-  )
   (junction (at 74.93 114.935) (diameter 0) (color 0 0 0 0)
   )
@@
     (stroke (width 0) (type default))
   )
-  (wire (pts (xy 107.95 88.265) (xy 104.14 88.265))
+  (wire (pts (xy 97.155 88.265) (xy 107.95 88.265))
     (stroke (width 0) (type default))
   )
@@
     (stroke (width 0) (type default))
   )
-  (wire (pts (xy 89.535 90.805) (xy 93.345 90.805))
-    (stroke (width 0) (type default))
-  )
   (wire (pts (xy 184.15 103.505) (xy 250.19 103.505))
     (stroke (width 0) (type default))
@@
     (stroke (width 0) (type default))
   )
-  (wire (pts (xy 104.14 86.995) (xy 104.14 88.265))
-    (stroke (width 0) (type default))
-  )
   (wire (pts (xy 262.89 100.965) (xy 266.065 100.965))
     (stroke (width 0) (type default))
@@
     (stroke (width 0) (type default))
   )
-  (wire (pts (xy 104.14 88.265) (xy 97.155 88.265))
-    (stroke (width 0) (type default))
-  )
   (wire (pts (xy 24.765 79.375) (xy 24.765 85.725))
     (stroke (width 0) (type default))
@@
     (stroke (width 0) (type default))
   )
-  (wire (pts (xy 93.345 89.535) (xy 93.345 90.805))
-    (stroke (width 0) (type default))
-  )
   (wire (pts (xy 102.87 81.915) (xy 102.87 83.185))
     (stroke (width 0) (type default))
@@
     (stroke (width 0) (type default))
   )
-  (wire (pts (xy 93.345 90.805) (xy 107.95 90.805))
+  (wire (pts (xy 89.535 90.805) (xy 107.95 90.805))
     (stroke (width 0) (type default))
   )
@@
         (path "/8189ff51-b9c1-4db5-b4d6-e4c84473a181"
           (reference "J4") (unit 1)
-        )
-      )
-    )
-  )
-  (symbol (lib_id "Connector:TestPoint_Small") (at 93.345 89.535 180) (unit 1)
-    (in_bom yes) (on_board yes) (dnp no)
-    (property "Reference" "TP6" (at 91.44 89.535 0)
-      (effects (font (face "KiCad Font") (size 0.8 0.8)) (justify left))
-    )
-    (property "Value" "TP" (at 92.71 89.535 0)
-      (effects (font (face "KiCad Font") (size 0.8 0.8)) (justify left))
-    )
-    (property "Footprint" "Connector_PinHeader_2.54mm:PinHeader_1x01_P2.54mm_Vertical" (at 88.265 89.535 0)
-      (effects (font (size 1.27 1.27)) hide)
-    )
-    (property "Datasheet" "~" (at 88.265 89.535 0)
-      (effects (font (size 1.27 1.27)) hide)
-    )
-    (pin "1")
-    (instances
-      (project "STA5635"
-        (path "/8189ff51-b9c1-4db5-b4d6-e4c84473a181"
-          (reference "TP6") (unit 1)
         )
       )
@@
         )
       )
-    )
-  )
-  (symbol (lib_id "Connector:TestPoint_Small") (at 104.14 86.995 180) (unit 1)
-    (in_bom yes) (on_board yes) (dnp no)
-    (property "Reference" "TP7" (at 102.235 86.995 0)
-      (effects (font (face "KiCad Font") (size 0.8 0.8)) (justify left))
-    )
-    (property "Value" "TP" (at 103.505 86.995 0)
-      (effects (font (face "KiCad Font") (size 0.8 0.8)) (justify left))
-    )
-    (property "Footprint" "Connector_PinHeader_2.54mm:PinHeader_1x01_P2.54mm_Vertical" (at 99.06 86.995 0)
-      (effects (font (size 1.27 1.27)) hide)
-    )
-    (property "Datasheet" "~" (at 99.06 86.995 0)
-      (effects (font (size 1.27 1.27)) hide)
-    )
-    (pin "1")
-    (instances
-      (project "STA5635"
-        (path "/8189ff51-b9c1-4db5-b4d6-e4c84473a181"
-          (reference "TP7") (unit 1)
-        )
-      )

Commit message: 30 August Office 001
Parts:
- added TP6: TP, Connector_PinHeader_2.54mm:PinHeader_1x01_P2.54mm_Vertical, symbol Connector:TestPoint_Small
Connections:
- net at U1.10 (TCXO_IN): now also TP6.1
Changed lines of the file:
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@@
+    (stroke (width 0) (type default))
+  )
+  (wire (pts (xy 103.505 95.885) (xy 103.505 97.155))
     (stroke (width 0) (type default))
   )
@@
     (stroke (width 0) (type default))
   )
+  (wire (pts (xy 107.95 95.885) (xy 103.505 95.885))
+    (stroke (width 0) (type default))
+  )
   (wire (pts (xy 70.485 94.615) (xy 70.485 92.075))
     (stroke (width 0) (type default))
@@
   )
   (wire (pts (xy 72.39 114.935) (xy 74.93 114.935))
+    (stroke (width 0) (type default))
+  )
+  (wire (pts (xy 103.505 97.155) (xy 102.235 97.155))
     (stroke (width 0) (type default))
   )
@@
         )
       )
+    )
+  )
+  (symbol (lib_id "Connector:TestPoint_Small") (at 102.235 97.155 180) (unit 1)
+    (in_bom yes) (on_board yes) (dnp no)
+    (property "Reference" "TP6" (at 100.33 97.155 0)
+      (effects (font (face "KiCad Font") (size 0.8 0.8)) (justify left))
+    )
+    (property "Value" "TP" (at 101.6 97.155 0)
+      (effects (font (face "KiCad Font") (size 0.8 0.8)) (justify left))
+    )
+    (property "Footprint" "Connector_PinHeader_2.54mm:PinHeader_1x01_P2.54mm_Vertical" (at 97.155 97.155 0)
+      (effects (font (size 1.27 1.27)) hide)
+    )
+    (property "Datasheet" "~" (at 97.155 97.155 0)
+      (effects (font (size 1.27 1.27)) hide)
+    )
+    (pin "1")
+    (instances
+      (project "STA5635"
+        (path "/8189ff51-b9c1-4db5-b4d6-e4c84473a181"
+          (reference "TP6") (unit 1)
+        )
+      )

Commit message: for push
Connections:
- net LNA_IN: no longer L1.2
- net at C9.1, J2.1: now also L1.2
Changed lines of the file:
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@@
   (junction (at 85.725 114.935) (diameter 0) (color 0 0 0 0)
   )
-  (junction (at 81.915 89.535) (diameter 0) (color 0 0 0 0)
-  )
   (junction (at 19.05 85.725) (diameter 0) (color 0 0 0 0)
   )
   (junction (at 97.155 88.265) (diameter 0) (color 0 0 0 0)
   )
+  (junction (at 59.055 89.535) (diameter 0) (color 0 0 0 0)
+  )
   (junction (at 74.93 114.935) (diameter 0) (color 0 0 0 0)
   )
@@
     (stroke (width 0) (type default))
   )
+  (wire (pts (xy 81.915 89.535) (xy 76.835 89.535))
+    (stroke (width 0) (type default))
+  )
   (wire (pts (xy 30.48 46.355) (xy 49.53 46.355))
     (stroke (width 0) (type default))
@@
     (stroke (width 0) (type default))
   )
+  (wire (pts (xy 74.295 89.535) (xy 75.565 89.535))
+    (stroke (width 0) (type default))
+  )
   (wire (pts (xy 85.725 95.25) (xy 85.725 90.805))
     (stroke (width 0) (type default))
   )
+  (wire (pts (xy 59.055 80.01) (xy 59.055 89.535))
+    (stroke (width 0) (type default))
+  )
+  (wire (pts (xy 81.915 88.9) (xy 81.915 89.535))
+    (stroke (width 0) (type default))
+  )
   (wire (pts (xy 103.505 80.645) (xy 103.505 65.405))
     (stroke (width 0) (type default))
@@
     (stroke (width 0) (type default))
   )
-  (wire (pts (xy 74.295 89.535) (xy 81.915 89.535))
-    (stroke (width 0) (type default))
-  )
   (wire (pts (xy 184.15 103.505) (xy 250.19 103.505))
     (stroke (width 0) (type default))
@@
     (stroke (width 0) (type default))
   )
+  (wire (pts (xy 75.565 89.535) (xy 75.565 92.075))
+    (stroke (width 0) (type default))
+  )
   (wire (pts (xy 93.345 83.185) (xy 93.345 74.93))
     (stroke (width 0) (type default))
@@
     (stroke (width 0) (type default))
   )
-  (wire (pts (xy 60.96 89.535) (xy 45.72 89.535))
+  (wire (pts (xy 60.96 89.535) (xy 59.055 89.535))
     (stroke (width 0) (type default))
   )
@@
     (stroke (width 0) (type default))
   )
+  (wire (pts (xy 59.055 89.535) (xy 45.72 89.535))
+    (stroke (width 0) (type default))
+  )
+  (wire (pts (xy 76.835 89.535) (xy 76.835 80.01))
+    (stroke (width 0) (type default))
+  )
   (wire (pts (xy 103.505 97.155) (xy 102.235 97.155))
     (stroke (width 0) (type default))
@@
     (stroke (width 0) (type default))
   )
-  (wire (pts (xy 81.915 88.9) (xy 81.915 89.535))
-    (stroke (width 0) (type default))
-  )
   (wire (pts (xy 74.295 57.15) (xy 74.295 58.42))
     (stroke (width 0) (type default))
   )
-  (wire (pts (xy 81.915 92.075) (xy 81.915 89.535))
-    (stroke (width 0) (type default))
-  )
   (wire (pts (xy 95.25 114.935) (xy 95.25 108.585))
     (stroke (width 0) (type default))
@@
     (stroke (width 0) (type default))
   )
-  (wire (pts (xy 70.485 92.075) (xy 81.915 92.075))
+  (wire (pts (xy 70.485 92.075) (xy 75.565 92.075))
     (stroke (width 0) (type default))
   )
@@
     (stroke (width 0) (type default))
   )
+  (wire (pts (xy 76.835 80.01) (xy 59.055 80.01))
+    (stroke (width 0) (type default))
+  )

Commit message: 4 Sept Office 001
Connections:
- net LNA_IN: now also L2.2; no longer L2.1
- net at C9.2: now also J2.1, L1.2; no longer L2.2
- new net: C9.1, L2.1
Other:
- moved on the sheet: C9, L2
Changed lines of the file:
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@@
     (stroke (width 0) (type default))
   )
-  (wire (pts (xy 81.915 89.535) (xy 76.835 89.535))
+  (wire (pts (xy 59.055 89.535) (xy 81.915 89.535))
     (stroke (width 0) (type default))
   )
@@
     (stroke (width 0) (type default))
   )
-  (wire (pts (xy 74.295 89.535) (xy 75.565 89.535))
-    (stroke (width 0) (type default))
-  )
   (wire (pts (xy 85.725 95.25) (xy 85.725 90.805))
     (stroke (width 0) (type default))
   )
-  (wire (pts (xy 59.055 80.01) (xy 59.055 89.535))
-    (stroke (width 0) (type default))
-  )
   (wire (pts (xy 81.915 88.9) (xy 81.915 89.535))
     (stroke (width 0) (type default))
@@
     (stroke (width 0) (type default))
   )
+  (wire (pts (xy 59.055 105.41) (xy 59.055 107.95))
+    (stroke (width 0) (type default))
+  )
   (wire (pts (xy 95.25 122.555) (xy 95.25 125.73))
     (stroke (width 0) (type default))
@@
     (stroke (width 0) (type default))
   )
-  (wire (pts (xy 66.04 89.535) (xy 69.215 89.535))
-    (stroke (width 0) (type default))
-  )
   (wire (pts (xy 243.84 100.965) (xy 250.19 100.965))
     (stroke (width 0) (type default))
@@
     (stroke (width 0) (type default))
   )
-  (wire (pts (xy 75.565 89.535) (xy 75.565 92.075))
-    (stroke (width 0) (type default))
-  )
   (wire (pts (xy 93.345 83.185) (xy 93.345 74.93))
     (stroke (width 0) (type default))
@@
     (stroke (width 0) (type default))
   )
-  (wire (pts (xy 70.485 94.615) (xy 70.485 92.075))
-    (stroke (width 0) (type default))
-  )
   (wire (pts (xy 86.995 41.275) (xy 86.995 45.085))
     (stroke (width 0) (type default))
@@
     (stroke (width 0) (type default))
   )
-  (wire (pts (xy 60.96 94.615) (xy 70.485 94.615))
-    (stroke (width 0) (type default))
-  )
   (wire (pts (xy 26.67 79.375) (xy 24.765 79.375))
     (stroke (width 0) (type default))
@@
     (stroke (width 0) (type default))
   )
-  (wire (pts (xy 60.96 89.535) (xy 59.055 89.535))
-    (stroke (width 0) (type default))
-  )
   (wire (pts (xy 95.25 108.585) (xy 107.95 108.585))
     (stroke (width 0) (type default))
@@
     (stroke (width 0) (type default))
   )
-  (wire (pts (xy 76.835 89.535) (xy 76.835 80.01))
-    (stroke (width 0) (type default))
-  )
   (wire (pts (xy 103.505 97.155) (xy 102.235 97.155))
     (stroke (width 0) (type default))
@@
     (stroke (width 0) (type default))
   )
+  (wire (pts (xy 59.055 89.535) (xy 59.055 92.71))
+    (stroke (width 0) (type default))
+  )
   (wire (pts (xy 102.87 81.915) (xy 102.87 83.185))
     (stroke (width 0) (type default))
@@
     (stroke (width 0) (type default))
   )
+  (wire (pts (xy 59.055 97.79) (xy 59.055 100.33))
+    (stroke (width 0) (type default))
+  )
   (wire (pts (xy 104.775 111.125) (xy 107.95 111.125))
     (stroke (width 0) (type default))
@@
     (stroke (width 0) (type default))
   )
-  (wire (pts (xy 70.485 92.075) (xy 75.565 92.075))
-    (stroke (width 0) (type default))
-  )
   (wire (pts (xy 184.15 85.725) (xy 250.19 85.725))
     (stroke (width 0) (type default))
@@
   )
   (wire (pts (xy 184.15 83.185) (xy 250.19 83.185))
-    (stroke (width 0) (type default))
-  )
-  (wire (pts (xy 76.835 80.01) (xy 59.055 80.01))
     (stroke (width 0) (type default))
   )
@@
     )
   )
-  (global_label "LNA_IN" (shape input) (at 60.96 94.615 180) (fields_autoplaced)
+  (global_label "LNA_IN" (shape input) (at 59.055 107.95 270) (fields_autoplaced)
     (effects (font (size 1.27 1.27)) (justify right))
-    (property "Intersheetrefs" "${INTERSHEET_REFS}" (at 51.6247 94.615 0)
+    (property "Intersheetrefs" "${INTERSHEET_REFS}" (at 59.055 117.2853 90)
       (effects (font (size 1.27 1.27)) (justify right) hide)
     )
   )
-  (symbol (lib_id "Device:L_Small") (at 71.755 89.535 270) (unit 1)
-    (in_bom yes) (on_board yes) (dnp no) (fields_autoplaced)
-    (property "Reference" "L2" (at 71.755 84.455 90)
-      (effects (font (size 1.27 1.27)))
-    )
-    (property "Value" "L_Small" (at 71.755 86.995 90)
-      (effects (font (size 1.27 1.27)))
-    )
-    (property "Footprint" "Inductor_SMD:L_1206_3216Metric_Pad1.22x1.90mm_HandSolder" (at 71.755 89.535 0)
-      (effects (font (size 1.27 1.27)) hide)
-    )
-    (property "Datasheet" "~" (at 71.755 89.535 0)
+  (symbol (lib_id "Device:L_Small") (at 59.055 102.87 0) (unit 1)
+    (in_bom yes) (on_board yes) (dnp no) (fields_autoplaced)
+    (property "Reference" "L2" (at 60.96 101.6 0)
+      (effects (font (size 1.27 1.27)) (justify left))
+    )
+    (property "Value" "L_Small" (at 60.96 104.14 0)
+      (effects (font (size 1.27 1.27)) (justify left))
+    )
+    (property "Footprint" "Inductor_SMD:L_1206_3216Metric_Pad1.22x1.90mm_HandSolder" (at 59.055 102.87 0)
+      (effects (font (size 1.27 1.27)) hide)
+    )
+    (property "Datasheet" "~" (at 59.055 102.87 0)
       (effects (font (size 1.27 1.27)) hide)
     )
@@
     )
   )
-  (symbol (lib_id "Device:C_Small") (at 63.5 89.535 90) (unit 1)
-    (in_bom yes) (on_board yes) (dnp no) (fields_autoplaced)
-    (property "Reference" "C9" (at 63.5063 82.55 90)
-      (effects (font (size 1.27 1.27)))
-    )
-    (property "Value" "104" (at 63.5063 85.09 90)
-      (effects (font (size 1.27 1.27)))
-    )
-    (property "Footprint" "Capacitor_SMD:C_1206_3216Metric" (at 63.5 89.535 0)
-      (effects (font (size 1.27 1.27)) hide)
-    )
-    (property "Datasheet" "~" (at 63.5 89.535 0)
-      (effects (font (size 1.27 1.27)) hide)
-    )
+  (symbol (lib_id "Device:C_Small") (at 59.055 95.25 180) (unit 1)
+    (in_bom yes) (on_board yes) (dnp no) (fields_autoplaced)
+    (property "Reference" "C9" (at 62.23 93.9736 0)
+      (effects (font (size 1.27 1.27)) (justify right))
+    )
+    (property "Value" "104" (at 62.23 96.5136 0)
+      (effects (font (size 1.27 1.27)) (justify right))
+    )
+    (property "Footprint" "Capacitor_SMD:C_1206_3216Metric" (at 59.055 95.25 0)
+      (effects (font (size 1.27 1.27)) hide)
+    )
+    (property "Datasheet" "~" (at 59.055 95.25 0)
+      (effects (font (size 1.27 1.27)) hide)
+    )

Commit message: update from home 04-9-2024
Parts:
- added H1, H2, H3, H4: MountingHole, MountingHole:MountingHole_2.2mm_M2, symbol Mechanical:MountingHole
Changed lines of the file:
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@@
+    )
+  )
+  (symbol (lib_id "Mechanical:MountingHole") (at 135.255 21.59 0) (unit 1)
+    (in_bom yes) (on_board yes) (dnp no) (fields_autoplaced)
+    (property "Reference" "H2" (at 137.795 20.32 0)
+      (effects (font (size 1.27 1.27)) (justify left))
+    )
+    (property "Value" "MountingHole" (at 137.795 22.86 0)
+      (effects (font (size 1.27 1.27)) (justify left))
+    )
+    (property "Footprint" "MountingHole:MountingHole_2.2mm_M2" (at 135.255 21.59 0)
+      (effects (font (size 1.27 1.27)) hide)
+    )
+    (property "Datasheet" "~" (at 135.255 21.59 0)
+      (effects (font (size 1.27 1.27)) hide)
+    )
+    (instances
+      (project "STA5635"
+        (path "/8189ff51-b9c1-4db5-b4d6-e4c84473a181"
+          (reference "H2") (unit 1)
+        )
+      )
     )
   )
@@
         (path "/8189ff51-b9c1-4db5-b4d6-e4c84473a181"
           (reference "J4") (unit 1)
+        )
+      )
+    )
+  )
+  (symbol (lib_id "Mechanical:MountingHole") (at 135.89 29.21 0) (unit 1)
+    (in_bom yes) (on_board yes) (dnp no) (fields_autoplaced)
+    (property "Reference" "H4" (at 138.43 27.94 0)
+      (effects (font (size 1.27 1.27)) (justify left))
+    )
+    (property "Value" "MountingHole" (at 138.43 30.48 0)
+      (effects (font (size 1.27 1.27)) (justify left))
+    )
+    (property "Footprint" "MountingHole:MountingHole_2.2mm_M2" (at 135.89 29.21 0)
+      (effects (font (size 1.27 1.27)) hide)
+    )
+    (property "Datasheet" "~" (at 135.89 29.21 0)
+      (effects (font (size 1.27 1.27)) hide)
+    )
+    (instances
+      (project "STA5635"
+        (path "/8189ff51-b9c1-4db5-b4d6-e4c84473a181"
+          (reference "H4") (unit 1)
         )
       )
@@
     )
   )
+  (symbol (lib_id "Mechanical:MountingHole") (at 115.57 29.21 0) (unit 1)
+    (in_bom yes) (on_board yes) (dnp no) (fields_autoplaced)
+    (property "Reference" "H3" (at 118.11 27.94 0)
+      (effects (font (size 1.27 1.27)) (justify left))
+    )
+    (property "Value" "MountingHole" (at 118.11 30.48 0)
+      (effects (font (size 1.27 1.27)) (justify left))
+    )
+    (property "Footprint" "MountingHole:MountingHole_2.2mm_M2" (at 115.57 29.21 0)
+      (effects (font (size 1.27 1.27)) hide)
+    )
+    (property "Datasheet" "~" (at 115.57 29.21 0)
+      (effects (font (size 1.27 1.27)) hide)
+    )
+    (instances
+      (project "STA5635"
+        (path "/8189ff51-b9c1-4db5-b4d6-e4c84473a181"
+          (reference "H3") (unit 1)
+        )
+      )
+    )
+  )
   (symbol (lib_id "Device:C_Small") (at 74.93 120.015 0) (unit 1)
     (in_bom yes) (on_board yes) (dnp no) (fields_autoplaced)
@@
         )
       )
+    )
+  )
+  (symbol (lib_id "Mechanical:MountingHole") (at 115.57 21.59 0) (unit 1)
+    (in_bom yes) (on_board yes) (dnp no) (fields_autoplaced)
+    (property "Reference" "H1" (at 118.11 20.32 0)
+      (effects (font (size 1.27 1.27)) (justify left))
+    )
+    (property "Value" "MountingHole" (at 118.11 22.86 0)
+      (effects (font (size 1.27 1.27)) (justify left))
+    )
+    (property "Footprint" "MountingHole:MountingHole_2.2mm_M2" (at 115.57 21.59 0)
+      (effects (font (size 1.27 1.27)) hide)
+    )
+    (property "Datasheet" "~" (at 115.57 21.59 0)
+      (effects (font (size 1.27 1.27)) hide)
+    )
+    (instances
+      (project "STA5635"
+        (path "/8189ff51-b9c1-4db5-b4d6-e4c84473a181"
+          (reference "H1") (unit 1)
+        )
+      )
