File: uprojects/Adee/PCB/STA5635/STA5635.kicad_sch (KiCad schematic)
At the start: 32 parts, among them J1 Conn_02x20_Odd_Even, J2 SMA_CONNECTOR, J3 EN, J4 Conn_01x02, U1 STA5635A, U2 AP2127K-1.8

Commit message: 6 Sept Office 001
Parts:
- C9: value 104 -> 2PF
- H3, H4: footprint MountingHole:MountingHole_2.2mm_M2 -> MountingHole:MountingHole_2.2mm_M2_DIN965
- J2: value SMA_CONNECTOR -> SMA
- L1: value L_Small -> 10nH
- L2: value L_Small -> 3.6nH
- R2: value 1K -> 1E4
Connections:
- net VCC: no longer R2.1, TP9.1, U1.5 (TP_IF_P/Sense1(1))
- net VDD: now also R2.1, TP9.1, U1.5 (TP_IF_P/Sense1(1))
- net TCXO_IN: now reaches TP6.1, U1.10 (TCXO_IN)
- net TCXO_IN: now also J1.39 (Pin_39), U1.17 (TCXO_CLK)
Other:
- note added: "3V3"
- moved on the sheet: TP6
Changed lines of the file:
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@@
   (junction (at 48.26 73.025) (diameter 0) (color 0 0 0 0)
   )
+  (junction (at 202.565 113.665) (diameter 0) (color 0 0 0 0)
+  )
   (junction (at 49.53 46.355) (diameter 0) (color 0 0 0 0)
   )
@@
   (junction (at 59.055 89.535) (diameter 0) (color 0 0 0 0)
   )
+  (junction (at 199.39 113.665) (diameter 0) (color 0 0 0 0)
+  )
   (junction (at 74.93 114.935) (diameter 0) (color 0 0 0 0)
   )
@@
     (stroke (width 0) (type default))
   )
-  (wire (pts (xy 184.15 113.665) (xy 250.19 113.665))
+  (wire (pts (xy 184.15 113.665) (xy 199.39 113.665))
     (stroke (width 0) (type default))
   )
@@
     (stroke (width 0) (type default))
   )
+  (wire (pts (xy 202.565 113.665) (xy 250.19 113.665))
+    (stroke (width 0) (type default))
+  )
   (wire (pts (xy 69.85 100.33) (xy 89.535 100.33))
     (stroke (width 0) (type default))
@@
     (stroke (width 0) (type default))
   )
+  (wire (pts (xy 199.39 113.665) (xy 202.565 113.665))
+    (stroke (width 0) (type default))
+  )
   (wire (pts (xy 184.15 103.505) (xy 250.19 103.505))
     (stroke (width 0) (type default))
@@
     (stroke (width 0) (type default))
   )
+  (wire (pts (xy 196.85 118.745) (xy 199.39 118.745))
+    (stroke (width 0) (type default))
+  )
   (wire (pts (xy 85.725 114.935) (xy 85.725 106.045))
     (stroke (width 0) (type default))
@@
     (stroke (width 0) (type default))
   )
+  (wire (pts (xy 199.39 118.745) (xy 199.39 113.665))
+    (stroke (width 0) (type default))
+  )
   (wire (pts (xy 105.41 75.565) (xy 105.41 65.405))
     (stroke (width 0) (type default))
@@
     (stroke (width 0) (type default))
   )
-  (wire (pts (xy 103.505 97.155) (xy 102.235 97.155))
+  (wire (pts (xy 100.965 97.155) (xy 103.505 97.155))
     (stroke (width 0) (type default))
   )
@@
   )
   (text "D10 COMPATIBLE GPIO0 HEADER" (at 242.57 57.785 0)
+    (effects (font (size 1.27 1.27)) (justify left bottom))
+  )
+  (text "3V3" (at 47.625 36.83 0)
+    (effects (font (size 1.27 1.27)) (justify left bottom))
+  )
+  (text "3V3" (at 80.01 63.5 0)
+    (effects (font (size 1.27 1.27)) (justify left bottom))
+  )
+  (text "3V3" (at 243.84 102.87 0)
     (effects (font (size 1.27 1.27)) (justify left bottom))
   )
@@
     )
   )
+  (global_label "TCXO_IN" (shape input) (at 196.85 118.745 180) (fields_autoplaced)
+    (effects (font (size 1.27 1.27)) (justify right))
+    (property "Intersheetrefs" "${INTERSHEET_REFS}" (at 186.1843 118.745 0)
+      (effects (font (size 1.27 1.27)) (justify right) hide)
+    )
+  )
+  (global_label "TCXO_IN" (shape input) (at 100.965 97.155 180) (fields_autoplaced)
+    (effects (font (size 1.27 1.27)) (justify right))
+    (property "Intersheetrefs" "${INTERSHEET_REFS}" (at 90.2993 97.155 0)
+      (effects (font (size 1.27 1.27)) (justify right) hide)
+    )
+  )
   (global_label "CHIP_EN" (shape input) (at 238.76 65.405 180) (fields_autoplaced)
     (effects (font (size 1.27 1.27)) (justify right))
@@
       (effects (font (size 1.27 1.27)) (justify left))
     )
-    (property "Value" "L_Small" (at 60.96 104.14 0)
+    (property "Value" "3.6nH" (at 60.96 104.14 0)
       (effects (font (size 1.27 1.27)) (justify left))
     )
@@
       (effects (font (size 1.27 1.27)))
     )
-    (property "Value" "SMA_CONNECTOR" (at 37.0205 100.33 0)
+    (property "Value" "SMA" (at 37.0205 100.33 0)
       (effects (font (size 1.27 1.27)))
     )
@@
     )
   )
-  (symbol (lib_id "power:VCC") (at 81.915 68.58 0) (unit 1)
-    (in_bom yes) (on_board yes) (dnp no) (fields_autoplaced)
-    (property "Reference" "#PWR012" (at 81.915 72.39 0)
-      (effects (font (size 1.27 1.27)) hide)
-    )
-    (property "Value" "VCC" (at 81.915 64.135 0)
-      (effects (font (size 1.27 1.27)))
-    )
-    (property "Footprint" "" (at 81.915 68.58 0)
-      (effects (font (size 1.27 1.27)) hide)
-    )
-    (property "Datasheet" "" (at 81.915 68.58 0)
-      (effects (font (size 1.27 1.27)) hide)
-    )
-    (pin "1")
-    (instances
-      (project "STA5635"
-        (path "/8189ff51-b9c1-4db5-b4d6-e4c84473a181"
-          (reference "#PWR012") (unit 1)
-        )
-      )
-    )
-  )
   (symbol (lib_id "Connector_Generic:Conn_01x02") (at 31.75 79.375 0) (unit 1)
     (in_bom yes) (on_board yes) (dnp no) (fields_autoplaced)
@@
       (effects (font (size 1.27 1.27)) (justify left))
     )
-    (property "Footprint" "MountingHole:MountingHole_2.2mm_M2" (at 135.89 29.21 0)
+    (property "Footprint" "MountingHole:MountingHole_2.2mm_M2_DIN965" (at 135.89 29.21 0)
       (effects (font (size 1.27 1.27)) hide)
     )
@@
   (symbol (lib_id "Device:R_Small") (at 81.915 79.375 0) (unit 1)
     (in_bom yes) (on_board yes) (dnp no) (fields_autoplaced)
-    (property "Reference" "R2" (at 84.455 78.105 0)
-      (effects (font (size 1.27 1.27)) (justify left))
-    )
-    (property "Value" "1K" (at 84.455 80.645 0)
+    (property "Reference" "R2" (at 83.82 78.105 0)
+      (effects (font (size 1.27 1.27)) (justify left))
+    )
+    (property "Value" "1E4" (at 83.82 80.645 0)
       (effects (font (size 1.27 1.27)) (justify left))
     )
@@
   (symbol (lib_id "Device:L_Small") (at 81.915 86.36 0) (unit 1)
     (in_bom yes) (on_board yes) (dnp no) (fields_autoplaced)
-    (property "Reference" "L1" (at 83.185 85.09 0)
-      (effects (font (size 1.27 1.27)) (justify left))
-    )
-    (property "Value" "L_Small" (at 83.185 87.63 0)
+    (property "Reference" "L1" (at 83.82 85.09 0)
+      (effects (font (size 1.27 1.27)) (justify left))
+    )
+    (property "Value" "10nH" (at 83.82 87.63 0)
       (effects (font (size 1.27 1.27)) (justify left))
     )
@@
     )
   )
-  (symbol (lib_id "Connector:TestPoint_Small") (at 102.235 97.155 180) (unit 1)
+  (symbol (lib_id "power:VDD") (at 81.915 68.58 0) (unit 1)
+    (in_bom yes) (on_board yes) (dnp no) (fields_autoplaced)
+    (property "Reference" "#PWR012" (at 81.915 72.39 0)
+      (effects (font (size 1.27 1.27)) hide)
+    )
+    (property "Value" "VDD" (at 81.915 64.135 0)
+      (effects (font (size 1.27 1.27)))
+    )
+    (property "Footprint" "" (at 81.915 68.58 0)
+      (effects (font (size 1.27 1.27)) hide)
+    )
+    (property "Datasheet" "" (at 81.915 68.58 0)
+      (effects (font (size 1.27 1.27)) hide)
+    )
+    (pin "1")
+    (instances
+      (project "STA5635"
+        (path "/8189ff51-b9c1-4db5-b4d6-e4c84473a181"
+          (reference "#PWR012") (unit 1)
+        )
+      )
+    )
+  )
+  (symbol (lib_id "Connector:TestPoint_Small") (at 202.565 113.665 270) (unit 1)
     (in_bom yes) (on_board yes) (dnp no)
-    (property "Reference" "TP6" (at 100.33 97.155 0)
+    (property "Reference" "TP6" (at 202.565 115.57 0)
       (effects (font (face "KiCad Font") (size 0.8 0.8)) (justify left))
     )
-    (property "Value" "TP" (at 101.6 97.155 0)
+    (property "Value" "TP" (at 202.565 114.3 0)
       (effects (font (face "KiCad Font") (size 0.8 0.8)) (justify left))
     )
-    (property "Footprint" "Connector_PinHeader_2.54mm:PinHeader_1x01_P2.54mm_Vertical" (at 97.155 97.155 0)
-      (effects (font (size 1.27 1.27)) hide)
-    )
-    (property "Datasheet" "~" (at 97.155 97.155 0)
+    (property "Footprint" "Connector_PinHeader_2.54mm:PinHeader_1x01_P2.54mm_Vertical" (at 202.565 118.745 0)
+      (effects (font (size 1.27 1.27)) hide)
+    )
+    (property "Datasheet" "~" (at 202.565 118.745 0)
       (effects (font (size 1.27 1.27)) hide)
     )
@@
       (effects (font (size 1.27 1.27)) (justify left))
     )
-    (property "Footprint" "MountingHole:MountingHole_2.2mm_M2" (at 115.57 29.21 0)
+    (property "Footprint" "MountingHole:MountingHole_2.2mm_M2_DIN965" (at 115.57 29.21 0)
       (effects (font (size 1.27 1.27)) hide)
     )
@@
       (effects (font (size 1.27 1.27)) (justify right))
     )
-    (property "Value" "104" (at 62.23 96.5136 0)
+    (property "Value" "2PF" (at 62.23 96.5136 0)
       (effects (font (size 1.27 1.27)) (justify right))
     )
@@
   )
   (symbol (lib_id "Device:C_Small") (at 89.535 95.25 0) (unit 1)
-    (in_bom yes) (on_board yes) (dnp no) (fields_autoplaced)
+    (in_bom yes) (on_board yes) (dnp no)
     (property "Reference" "C8" (at 92.71 93.9863 0)
       (effects (font (size 1.27 1.27)) (justify left))
     )
-    (property "Value" "104" (at 92.71 96.5263 0)
-      (effects (font (size 1.27 1.27)) (justify left))
-    )
+    (property "Value" "104" (at 92.075 92.075 0)
+      (effects (font (size 1.27 1.27)) (justify left))
+    )
