File: uprojects/Adee/PCB/STA5635/STA5635.kicad_pcb (KiCad board)
At the start: 2 copper layers, 5 parts, among them J1 Conn_01x20, U1 STA5635A, U2 AP2127K-1.8

Commit message: 4-august 24
Parts:
- added C3: 104, Capacitor_SMD:C_1206_3216Metric, F.Cu at (129.7, 88.9)
- added C4: 104, Capacitor_SMD:C_1206_3216Metric, F.Cu at (129.6, 101.3)
- added C5: 104, Capacitor_SMD:C_1206_3216Metric, F.Cu at (129.6, 98.8)
- added C6: 104, Capacitor_SMD:C_1206_3216Metric, F.Cu at (129.6, 96.3)
- added C7: 104, Capacitor_SMD:C_1206_3216Metric, F.Cu at (129.6, 93.8)
- added C8: 104, Capacitor_SMD:C_1206_3216Metric, F.Cu at (129.6, 91.3)
- added C9: 104, Capacitor_SMD:C_1206_3216Metric, F.Cu at (118.4, 87.5)
- added J2: SMA_CONNECTOR, SMA_CONNECTOR:LPRS_SMA_CONNECTOR, F.Cu at (141.1, 109.9)
- added L1: L_Small, Inductor_SMD:L_1206_3216Metric_Pad1.22x1.90mm_HandSolder, F.Cu at (118.6, 80.7)
- added L2: L_Small, Inductor_SMD:L_1206_3216Metric_Pad1.22x1.90mm_HandSolder, F.Cu at (118.6, 84.1)
- added R1: 1K, Resistor_SMD:R_1206_3216Metric, F.Cu at (129.7, 86.5)
- added R2: 1K, Resistor_SMD:R_1206_3216Metric, F.Cu at (124.5, 80.6)
- moved J1 12.1 mm to (157.5, 64.5)
Connections:
- net Net-(U2-EN) renamed VDD
- J1 pad 5: unconnected-(J1-Pin_5-Pad5) -> Net-(J1-Pin_5)
- U1 pad 1: unconnected-(U1-V11_LNA-Pad1) -> Net-(U1-V11_CHAIN)
- U1 pad 12: unconnected-(U1-CHIP_EN-Pad12) -> CHIP_EN
- U1 pad 13: unconnected-(U1-V11_OUT_DIG-Pad13) -> Net-(U1-V11_OUT_DIG)
- U1 pad 14: unconnected-(U1-GND_DIG-Pad14) -> GND
- U1 pad 15: unconnected-(U1-VCC_IO-Pad15) -> Net-(U1-VCC_IO)
- U1 pad 16: unconnected-(U1-V18_OUT-Pad16) -> Net-(U1-V18_OUT)
- U1 pad 3: unconnected-(U1-V11_CHAIN-Pad3) -> Net-(U1-V11_CHAIN)
- U1 pad 32: unconnected-(U1-LNA_GND-Pad32) -> Net-(J1-Pin_5)
- U1 pad 5: unconnected-(U1-TP_IF_P/Sense1(1)-Pad5) -> Net-(U1-TP_IF_P/Sense1(1))
- U1 pad 6: unconnected-(U1-TP_IF_N/Sense2(1)-Pad6) -> Net-(U1-TP_IF_N/Sense2(1))
- U1 pad 7: unconnected-(U1-V11_OUT_RF-Pad7) -> Net-(U1-V11_CHAIN)
- U1 pad 8: unconnected-(U1-VCC_RF-Pad8) -> VCC
- U1 pad 9: unconnected-(U1-V11_PLL-Pad9) -> Net-(U1-V11_CHAIN)
Other:
- board outline added: 60.1 x 72.8 mm

Commit message: 36 July Office 001
Parts:
- added J3: Conn_01x02, Connector_PinHeader_2.54mm:PinHeader_1x02_P2.54mm_Vertical, F.Cu at (131.3, 90.6)
- J1: value Conn_01x20 -> Conn_02x20_Odd_Even; footprint Connector_PinHeader_2.54mm:PinHeader_1x20_P2.54mm_Vertical -> Connector_PinHeader_2.54mm:PinHeader_2x20_P2.54mm_Vertical
- moved C6 11.2 mm to (125.0, 106.5)
- moved C7 11.2 mm to (125.0, 104.0)
- moved C8 11.2 mm to (125.0, 101.5)
- moved C3 11.2 mm to (125.1, 99.1)
- moved C4 11.2 mm to (125.0, 111.5)
- moved C5 11.2 mm to (125.0, 109.0)
- moved R1 11.2 mm to (125.1, 96.7)
- moved L1 10.7 mm to (125.2, 89.1)
- moved L2 9.97 mm to (125.2, 91.6)
- moved C9 9.39 mm to (125.1, 94.2)
- moved R2 5.91 mm to (125.0, 86.5)
- moved J1 1.96 mm to (156.1, 63.1)
- moved J2 1.76 mm to (140.6, 108.3)
Connections:
- C3 pad 1: CHIP_EN -> Net-(J3-Pin_1)
- J1 pad 10: Net-(J1-Pin_10) -> unconnected-(J1-Pin_10-Pad10)
- J1 pad 11: Net-(J1-Pin_11) -> 5V
- J1 pad 12: Net-(J1-Pin_12) -> GND
- J1 pad 14: Net-(J1-Pin_14) -> unconnected-(J1-Pin_14-Pad14)
- J1 pad 16: Net-(J1-Pin_16) -> unconnected-(J1-Pin_16-Pad16)
- J1 pad 18: Net-(J1-Pin_18) -> unconnected-(J1-Pin_18-Pad18)
- J1 pad 20: Net-(J1-Pin_20) -> unconnected-(J1-Pin_20-Pad20)
- J1 pad 5: Net-(J1-Pin_5) -> unconnected-(J1-Pin_5-Pad5)
- J1 pad 6: Net-(J1-Pin_6) -> unconnected-(J1-Pin_6-Pad6)
- J1 pad 7: Net-(J1-Pin_7) -> unconnected-(J1-Pin_7-Pad7)
- J1 pad 8: Net-(J1-Pin_8) -> unconnected-(J1-Pin_8-Pad8)
- J1 pad 9: Net-(J1-Pin_9) -> unconnected-(J1-Pin_9-Pad9)
- L1 pad 1: Net-(U1-TP_IF_P/Sense1(1)) -> Net-(U1-TP_IF_N/Sense2(1))
- L1 pad 2: Net-(U1-TP_IF_N/Sense2(1)) -> LNA_IN
- L2 pad 1: Net-(U1-TP_IF_N/Sense2(1)) -> LNA_IN
- R1 pad 2: CHIP_EN -> Net-(J3-Pin_1)
- R2 pad 2: Net-(U1-TP_IF_P/Sense1(1)) -> Net-(U1-TP_IF_N/Sense2(1))
- U1 pad 17: Net-(J1-Pin_20) -> Net-(J1-Pin_39)
- U1 pad 18: Net-(J1-Pin_19) -> GND
- U1 pad 19: Net-(J1-Pin_18) -> Net-(J1-Pin_35)
- U1 pad 20: Net-(J1-Pin_17) -> Net-(J1-Pin_33)
- U1 pad 21: Net-(J1-Pin_16) -> Net-(J1-Pin_31)
- U1 pad 22: Net-(J1-Pin_15) -> Net-(J1-Pin_37)
- U1 pad 23: Net-(J1-Pin_14) -> Net-(J1-Pin_27)
- U1 pad 24: Net-(J1-Pin_13) -> Net-(J1-Pin_25)
- U1 pad 25: Net-(J1-Pin_12) -> Net-(J1-Pin_23)
- U1 pad 26: Net-(J1-Pin_11) -> Net-(J1-Pin_21)
- U1 pad 27: Net-(J1-Pin_10) -> Net-(J1-Pin_19)
- U1 pad 28: Net-(J1-Pin_9) -> Net-(J1-Pin_17)
- U1 pad 29: Net-(J1-Pin_8) -> Net-(J1-Pin_15)
- U1 pad 30: Net-(J1-Pin_7) -> Net-(J1-Pin_13)
- U1 pad 31: Net-(J1-Pin_6) -> LNA_IN
- U1 pad 32: Net-(J1-Pin_5) -> GNDA
- U1 pad 33: unconnected-(U1-GND-Pad33) -> GND
- U1 pad 5: Net-(U1-TP_IF_P/Sense1(1)) -> VCC
- U2 pad 3: VDD -> unconnected-(U2-EN-Pad3)

Commit message: 6 August Office 001
Parts:
- added J4: Conn_01x02, Connector_PinHeader_2.54mm:PinHeader_1x02_P2.54mm_Vertical, F.Cu at (136.9, 68.2)
- added TP1: TP, Connector_PinHeader_2.54mm:PinHeader_1x01_P2.54mm_Vertical, F.Cu at (123.0, 64.7)
- added TP10: TP, Connector_PinHeader_2.54mm:PinHeader_1x01_P2.54mm_Vertical, F.Cu at (138.5, 99.4)
- added TP2: TP, Connector_PinHeader_2.54mm:PinHeader_1x01_P2.54mm_Vertical, F.Cu at (123.0, 69.4)
- added TP3: TP, Connector_PinHeader_2.54mm:PinHeader_1x01_P2.54mm_Vertical, F.Cu at (123.0, 74.0)
- added TP4: TP, Connector_PinHeader_2.54mm:PinHeader_1x01_P2.54mm_Vertical, F.Cu at (123.0, 78.7)
- added TP5: TP, Connector_PinHeader_2.54mm:PinHeader_1x01_P2.54mm_Vertical, F.Cu at (142.5, 80.0)
- added TP6: TP, Connector_PinHeader_2.54mm:PinHeader_1x01_P2.54mm_Vertical, F.Cu at (127.6, 64.7)
- added TP7: TP, Connector_PinHeader_2.54mm:PinHeader_1x01_P2.54mm_Vertical, F.Cu at (127.6, 69.4)
- added TP8: TP, Connector_PinHeader_2.54mm:PinHeader_1x01_P2.54mm_Vertical, F.Cu at (127.6, 74.0)
- added TP9: TP, Connector_PinHeader_2.54mm:PinHeader_1x01_P2.54mm_Vertical, F.Cu at (127.6, 78.7)
- moved C2 9.65 mm to (144.5, 68.2)
- moved U2 9.65 mm to (144.5, 72.5)
- moved C1 9.65 mm to (137.9, 72.7)
Connections:
- net Net-(U1-V11_CHAIN) renamed 1.1V
- J1 pad 1: unconnected-(J1-Pin_1-Pad1) -> CHIP_EN
- U1 pad 2: unconnected-(U1-LNA_OUT-Pad2) -> Net-(U1-LNA_OUT)
- U1 pad 4: unconnected-(U1-RFA_IN-Pad4) -> Net-(U1-RFA_IN)
- U2 pad 3: unconnected-(U2-EN-Pad3) -> Net-(J4-Pin_1)

Commit message: 27 August Office 001
Parts:
- moved C7 27.3 mm to (141.2, 82.0)
- moved TP10 5.76 mm to (134.6, 103.7)
- moved TP5 2.41 mm to (142.5, 77.6)
Routing:
- net Net-(J1-Pin_35): track 0.00 -> 23.3 mm
- net Net-(J1-Pin_37): track 0.00 -> 22.4 mm, vias 0 -> 1
- net Net-(J1-Pin_13): track 0.00 -> 21.8 mm
- net Net-(J1-Pin_33): track 0.00 -> 21.7 mm
- net Net-(J1-Pin_15): track 0.00 -> 20.6 mm
- net Net-(J1-Pin_31): track 0.00 -> 20.1 mm
- net Net-(J1-Pin_17): track 0.00 -> 18.5 mm
- net Net-(J1-Pin_19): track 0.00 -> 16.8 mm
- net Net-(J1-Pin_27): track 0.00 -> 16.3 mm
- net Net-(J1-Pin_21): track 0.00 -> 15.9 mm
- net Net-(J1-Pin_23): track 0.00 -> 15.1 mm
- net Net-(J1-Pin_25): track 0.00 -> 15.0 mm
- net 1.1V: track 0.00 -> 13.1 mm, vias 0 -> 3
- net VCC: track 0.00 -> 6.27 mm, vias 0 -> 2
Changed lines of the file:
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@@
   )
   (footprint "Connector_PinHeader_2.54mm:PinHeader_1x01_P2.54mm_Vertical" (layer "F.Cu")
-    (at 138.4808 99.3902)
+    (at 134.6454 103.6828)
     (descr "Through hole straight pin header, 1x01, 2.54mm pitch, single row")
     (tags "Through hole pin header THT 1x01 2.54mm single row")
@@
   )
   (footprint "Capacitor_SMD:C_1206_3216Metric" (layer "F.Cu")
-    (at 125.046 103.9876 180)
+    (at 141.224 81.9912 180)
     (descr "Capacitor SMD 1206 (3216 Metric), square (rectangular) end terminal, IPC_7351 nominal, (Body size source: IPC-SM-782 page 76, https://www.pcb-3d.com/wordpress/wp-content/uploads/ipc-sm-782a_amendment_1_and_2.pdf), generated with kicad-footprint-generator")
     (tags "capacitor")
@@
     (property "ki_keywords" "capacitor cap")
     (attr smd)
-    (fp_text reference "C7" (at 3.38 -0.0762) (layer "F.SilkS")
-        (effects (font (size 1 1) (thickness 0.15)))
-    )
-    (fp_text value "104" (at 3.8608 -0.0254) (layer "F.Fab")
+    (fp_text reference "C7" (at 3.302 -0.1524) (layer "F.SilkS")
+        (effects (font (size 1 1) (thickness 0.15)))
+    )
+    (fp_text value "104" (at 0.1016 0) (layer "F.Fab")
         (effects (font (size 1 1) (thickness 0.15)))
     )
@@
   )
   (footprint "Connector_PinHeader_2.54mm:PinHeader_1x01_P2.54mm_Vertical" (layer "F.Cu")
-    (at 142.5194 80.0354)
+    (at 142.494 77.6224)
     (descr "Through hole straight pin header, 1x01, 2.54mm pitch, single row")
     (tags "Through hole pin header THT 1x01 2.54mm single row")
@@
     (property "ki_keywords" "test point tp")
     (attr through_hole)
-    (fp_text reference "TP5" (at 4.5102 -10.8644) (layer "F.SilkS")
+    (fp_text reference "TP5" (at 3.4036 -0.0508) (layer "F.SilkS")
         (effects (font (size 1 1) (thickness 0.15)))
     )
@@
   (gr_line (start 111.4552 126.619) (end 111.4552 53.8988)
     (stroke (width 0.1) (type default)) (layer "Edge.Cuts"))
+  (segment (start 139.475337 89.5096) (end 139.475337 87.633937) (width 0.25) (layer "F.Cu") (net 2))
+  (segment (start 137.974959 89.5096) (end 137.974959 88.343359) (width 0.25) (layer "F.Cu") (net 2))
+  (segment (start 137.974959 88.343359) (end 137.2616 87.63) (width 0.25) (layer "F.Cu") (net 2))
+  (segment (start 139.475337 87.633937) (end 139.4714 87.63) (width 0.25) (layer "F.Cu") (net 2))
+  (via (at 137.2616 87.63) (size 0.8) (drill 0.4) (layers "F.Cu" "B.Cu") (net 2))
+  (via (at 139.4714 87.63) (size 0.8) (drill 0.4) (layers "F.Cu" "B.Cu") (net 2))
+  (segment (start 137.2616 87.63) (end 139.4714 87.63) (width 0.25) (layer "B.Cu") (net 2))
+  (segment (start 148.7424 81.0514) (end 151.4856 78.3082) (width 0.25) (layer "F.Cu") (net 12))
+  (segment (start 142.796274 91.185111) (end 148.7424 85.238985) (width 0.25) (layer "F.Cu") (net 12))
+  (segment (start 148.7424 85.238985) (end 148.7424 81.0514) (width 0.25) (layer "F.Cu") (net 12))
+  (segment (start 151.4856 78.3082) (end 156.1338 78.3082) (width 0.25) (layer "F.Cu") (net 12))
+  (segment (start 142.1511 91.185111) (end 142.796274 91.185111) (width 0.25) (layer "F.Cu") (net 12))
+  (segment (start 149.2504 82.2198) (end 150.622 80.8482) (width 0.25) (layer "F.Cu") (net 14))
+  (segment (start 142.1511 91.685237) (end 143.391763 91.685237) (width 0.25) (layer "F.Cu") (net 14))
+  (segment (start 149.2504 85.8266) (end 149.2504 82.2198) (width 0.25) (layer "F.Cu") (net 14))
+  (segment (start 150.622 80.8482) (end 156.1338 80.8482) (width 0.25) (layer "F.Cu") (net 14))
+  (segment (start 143.391763 91.685237) (end 149.2504 85.8266) (width 0.25) (layer "F.Cu") (net 14))
+  (segment (start 151.1808 83.3882) (end 156.1338 83.3882) (width 0.25) (layer "F.Cu") (net 15))
+  (segment (start 142.1511 92.185363) (end 143.958437 92.185363) (width 0.25) (layer "F.Cu") (net 15))
+  (segment (start 143.958437 92.185363) (end 149.7076 86.4362) (width 0.25) (layer "F.Cu") (net 15))
+  (segment (start 149.7076 84.8614) (end 151.1808 83.3882) (width 0.25) (layer "F.Cu") (net 15))
+  (segment (start 149.7076 86.4362) (end 149.7076 84.8614) (width 0.25) (layer "F.Cu") (net 15))
+  (segment (start 144.347311 92.685489) (end 151.1046 85.9282) (width 0.25) (layer "F.Cu") (net 17))
+  (segment (start 151.1046 85.9282) (end 156.1338 85.9282) (width 0.25) (layer "F.Cu") (net 17))
+  (segment (start 142.1511 92.685489) (end 144.347311 92.685489) (width 0.25) (layer "F.Cu") (net 17))
+  (segment (start 149.4536 88.4682) (end 156.1338 88.4682) (width 0.25) (layer "F.Cu") (net 32))
+  (segment (start 142.1511 93.185615) (end 144.736185 93.185615) (width 0.25) (layer "F.Cu") (net 32))
+  (segment (start 144.736185 93.185615) (end 149.4536 88.4682) (width 0.25) (layer "F.Cu") (net 32))
+  (segment (start 147.8026 91.0082) (end 156.1338 91.0082) (width 0.25) (layer "F.Cu") (net 34))
+  (segment (start 142.1511 93.685741) (end 145.125059 93.685741) (width 0.25) (layer "F.Cu") (net 34))
+  (segment (start 145.125059 93.685741) (end 147.8026 91.0082) (width 0.25) (layer "F.Cu") (net 34))
+  (segment (start 141.475841 94.361) (end 145.923 94.361) (width 0.25) (layer "F.Cu") (net 36))
+  (segment (start 145.923 94.361) (end 146.7358 93.5482) (width 0.25) (layer "F.Cu") (net 36))
+  (segment (start 146.7358 93.5482) (end 156.1338 93.5482) (width 0.25) (layer "F.Cu") (net 36))
+  (segment (start 140.975715 94.361) (end 140.975715 95.006174) (width 0.25) (layer "F.Cu") (net 38))
+  (segment (start 142.057741 96.0882) (end 156.1338 96.0882) (width 0.25) (layer "F.Cu") (net 38))
+  (segment (start 140.975715 95.006174) (end 142.057741 96.0882) (width 0.25) (layer "F.Cu") (net 38))
+  (segment (start 140.833695 97.0788) (end 148.3614 97.0788) (width 0.25) (layer "F.Cu") (net 40))
+  (segment (start 148.3614 97.0788) (end 152.4508 101.1682) (width 0.25) (layer "F.Cu") (net 40))
+  (segment (start 152.4508 101.1682) (end 156.1338 101.1682) (width 0.25) (layer "F.Cu") (net 40))
+  (segment (start 139.975463 96.220568) (end 140.833695 97.0788) (width 0.25) (layer "F.Cu") (net 40))
+  (segment (start 139.975463 94.361) (end 139.975463 96.220568) (width 0.25) (layer "F.Cu") (net 40))
+  (segment (start 139.475337 94.361) (end 139.475337 96.356838) (width 0.25) (layer "F.Cu") (net 42))
+  (segment (start 139.475337 96.356838) (end 140.908499 97.79) (width 0.25) (layer "F.Cu") (net 42))
+  (segment (start 147.9804 97.79) (end 153.8986 103.7082) (width 0.25) (layer "F.Cu") (net 42))
+  (segment (start 140.908499 97.79) (end 147.9804 97.79) (width 0.25) (layer "F.Cu") (net 42))
+  (segment (start 153.8986 103.7082) (end 156.1338 103.7082) (width 0.25) (layer "F.Cu") (net 42))
+  (segment (start 154.9146 106.2482) (end 156.1338 106.2482) (width 0.25) (layer "F.Cu") (net 44))
+  (segment (start 147.1422 98.4758) (end 154.9146 106.2482) (width 0.25) (layer "F.Cu") (net 44))
+  (segment (start 140.957903 98.4758) (end 147.1422 98.4758) (width 0.25) (layer "F.Cu") (net 44))
+  (segment (start 138.975211 94.361) (end 138.975211 96.493108) (width 0.25) (layer "F.Cu") (net 44))
+  (segment (start 138.975211 96.493108) (end 140.957903 98.4758) (width 0.25) (layer "F.Cu") (net 44))
+  (segment (start 140.475589 94.361) (end 140.475589 95.695389) (width 0.25) (layer "F.Cu") (net 50))
+  (segment (start 140.475589 95.695389) (end 140.843 96.0628) (width 0.25) (layer "F.Cu") (net 50))
+  (via (at 140.843 96.0628) (size 0.8) (drill 0.4) (layers "F.Cu" "B.Cu") (net 50))
+  (segment (start 153.5684 108.7882) (end 156.1338 108.7882) (width 0.25) (layer "B.Cu") (net 50))
+  (segment (start 140.843 96.0628) (end 153.5684 108.7882) (width 0.25) (layer "B.Cu") (net 50))
+  (segment (start 138.475085 86.746715) (end 138.4808 86.741) (width 0.25) (layer "F.Cu") (net 56))
+  (segment (start 142.7226 86.7664) (end 142.748 86.741) (width 0.25) (layer "F.Cu") (net 56))
+  (segment (start 141.475841 88.444959) (end 142.7226 87.1982) (width 0.25) (layer "F.Cu") (net 56))
+  (segment (start 141.475841 89.5096) (end 141.475841 88.444959) (width 0.25) (layer "F.Cu") (net 56))
+  (segment (start 140.475589 86.752811) (end 140.4874 86.741) (width 0.25) (layer "F.Cu") (net 56))
+  (segment (start 138.475085 89.5096) (end 138.475085 86.746715) (width 0.25) (layer "F.Cu") (net 56))
+  (segment (start 142.7226 87.1982) (end 142.7226 86.7664) (width 0.25) (layer "F.Cu") (net 56))
+  (segment (start 140.475589 89.5096) (end 140.475589 86.752811) (width 0.25) (layer "F.Cu") (net 56))
+  (via (at 138.4808 86.741) (size 0.8) (drill 0.4) (layers "F.Cu" "B.Cu") (net 56))
+  (via (at 140.4874 86.741) (size 0.8) (drill 0.4) (layers "F.Cu" "B.Cu") (net 56))
+  (via (at 142.748 86.741) (size 0.8) (drill 0.4) (layers "F.Cu" "B.Cu") (net 56))
+  (segment (start 138.4808 86.741) (end 140.4874 86.741) (width 0.25) (layer "B.Cu") (net 56))
+  (segment (start 142.748 86.741) (end 140.4874 86.741) (width 0.25) (layer "B.Cu") (net 56))
 )

Commit message: 29 August Office 001
Parts:
- J3: value Conn_01x02 -> EN
- moved TP2 27.0 mm to (145.9, 83.8)
- moved J3 6.21 mm to (129.9, 96.7), turned to 90 degrees
Routing:
- net CHIP_EN: track 0.00 -> 47.8 mm, vias 0 -> 1
- net Net-(U1-LNA_OUT): track 0.00 -> 8.72 mm
- net Net-(J3-Pin_1): track 0.00 -> 2.41 mm
Changed lines of the file:
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@@
   )
   (footprint "Connector_PinHeader_2.54mm:PinHeader_1x02_P2.54mm_Vertical" (layer "F.Cu")
-    (at 131.318 90.6322 180)
+    (at 129.8906 96.6724 90)
     (descr "Through hole straight pin header, 1x02, 2.54mm pitch, single row")
     (tags "Through hole pin header THT 1x02 2.54mm single row")
@@
     (property "ki_keywords" "connector")
     (attr through_hole)
-    (fp_text reference "J3" (at 0 -2.33) (layer "F.SilkS")
-        (effects (font (size 1 1) (thickness 0.15)))
-    )
-    (fp_text value "Conn_01x02" (at 0 4.87) (layer "F.Fab")
-        (effects (font (size 1 1) (thickness 0.15)))
-    )
-    (fp_text user "${REFERENCE}" (at 0 1.27 90) (layer "F.Fab")
+    (fp_text reference "J3" (at 0 -2.33 90) (layer "F.SilkS")
+        (effects (font (size 1 1) (thickness 0.15)))
+    )
+    (fp_text value "EN" (at 0 4.87 90) (layer "F.Fab")
+        (effects (font (size 1 1) (thickness 0.15)))
+    )
+    (fp_text user "${REFERENCE}" (at 0 1.27) (layer "F.Fab")
         (effects (font (size 1 1) (thickness 0.15)))
     )
@@
     (fp_line (start 1.27 3.81) (end -1.27 3.81)
       (stroke (width 0.1) (type solid)) (layer "F.Fab"))
-    (pad "1" thru_hole rect (at 0 0 180) (size 1.7 1.7) (drill 1) (layers "*.Cu" "*.Mask")
+    (pad "1" thru_hole rect (at 0 0 90) (size 1.7 1.7) (drill 1) (layers "*.Cu" "*.Mask")
       (net 6 "Net-(J3-Pin_1)") (pinfunction "Pin_1") (pintype "passive"))
-    (pad "2" thru_hole oval (at 0 2.54 180) (size 1.7 1.7) (drill 1) (layers "*.Cu" "*.Mask")
+    (pad "2" thru_hole oval (at 0 2.54 90) (size 1.7 1.7) (drill 1) (layers "*.Cu" "*.Mask")
       (net 22 "CHIP_EN") (pinfunction "Pin_2") (pintype "passive"))
     (model "${KICAD6_3DMODEL_DIR}/Connector_PinHeader_2.54mm.3dshapes/PinHeader_1x02_P2.54mm_Vertical.wrl"
@@
   )
   (footprint "Connector_PinHeader_2.54mm:PinHeader_1x01_P2.54mm_Vertical" (layer "F.Cu")
-    (at 122.985 69.3656)
+    (at 145.8722 83.7692)
     (descr "Through hole straight pin header, 1x01, 2.54mm pitch, single row")
     (tags "Through hole pin header THT 1x01 2.54mm single row")
@@
   (via (at 139.4714 87.63) (size 0.8) (drill 0.4) (layers "F.Cu" "B.Cu") (net 2))
   (segment (start 137.2616 87.63) (end 139.4714 87.63) (width 0.25) (layer "B.Cu") (net 2))
+  (segment (start 126.5299 99.0854) (end 126.5299 96.6746) (width 0.25) (layer "F.Cu") (net 6))
+  (segment (start 126.5299 96.6746) (end 126.5321 96.6724) (width 0.25) (layer "F.Cu") (net 6))
   (segment (start 148.7424 81.0514) (end 151.4856 78.3082) (width 0.25) (layer "F.Cu") (net 12))
   (segment (start 142.796274 91.185111) (end 148.7424 85.238985) (width 0.25) (layer "F.Cu") (net 12))
@@
   (segment (start 151.1046 85.9282) (end 156.1338 85.9282) (width 0.25) (layer "F.Cu") (net 17))
   (segment (start 142.1511 92.685489) (end 144.347311 92.685489) (width 0.25) (layer "F.Cu") (net 17))
+  (segment (start 137.2997 91.685237) (end 134.585837 91.685237) (width 0.25) (layer "F.Cu") (net 22))
+  (segment (start 134.585837 91.685237) (end 132.9182 90.0176) (width 0.25) (layer "F.Cu") (net 22))
+  (via (at 132.9182 90.0176) (size 0.8) (drill 0.4) (layers "F.Cu" "B.Cu") (net 22))
+  (segment (start 147.3962 88.6206) (end 149.1996 86.8172) (width 0.25) (layer "B.Cu") (net 22))
+  (segment (start 149.1996 65.8622) (end 151.892 63.1698) (width 0.25) (layer "B.Cu") (net 22))
+  (segment (start 136.144 88.6206) (end 147.3962 88.6206) (width 0.25) (layer "B.Cu") (net 22))
+  (segment (start 134.7724 88.1634) (end 135.2804 88.1634) (width 0.25) (layer "B.Cu") (net 22))
+  (segment (start 135.6868 88.1634) (end 136.144 88.6206) (width 0.25) (layer "B.Cu") (net 22))
+  (segment (start 132.9182 90.0176) (end 134.7724 88.1634) (width 0.25) (layer "B.Cu") (net 22))
+  (segment (start 135.2804 88.1634) (end 135.6868 88.1634) (width 0.25) (layer "B.Cu") (net 22))
+  (segment (start 149.1996 86.8172) (end 149.1996 65.8622) (width 0.25) (layer "B.Cu") (net 22))
   (segment (start 149.4536 88.4682) (end 156.1338 88.4682) (width 0.25) (layer "F.Cu") (net 32))
   (segment (start 142.1511 93.185615) (end 144.736185 93.185615) (width 0.25) (layer "F.Cu") (net 32))
@@
   (segment (start 153.5684 108.7882) (end 156.1338 108.7882) (width 0.25) (layer "B.Cu") (net 50))
   (segment (start 140.843 96.0628) (end 153.5684 108.7882) (width 0.25) (layer "B.Cu") (net 50))
+  (segment (start 144.272 85.3948) (end 145.8722 83.7946) (width 0.25) (layer "F.Cu") (net 55))
+  (segment (start 140.975715 89.5096) (end 140.975715 88.005285) (width 0.25) (layer "F.Cu") (net 55))
+  (segment (start 141.6812 87.2998) (end 141.6812 86.36) (width 0.25) (layer "F.Cu") (net 55))
+  (segment (start 140.975715 88.005285) (end 141.6812 87.2998) (width 0.25) (layer "F.Cu") (net 55))
+  (segment (start 141.6812 86.36) (end 142.6464 85.3948) (width 0.25) (layer "F.Cu") (net 55))
+  (segment (start 142.6464 85.3948) (end 144.272 85.3948) (width 0.25) (layer "F.Cu") (net 55))
+  (segment (start 145.8722 83.7946) (end 145.8722 83.7692) (width 0.25) (layer "F.Cu") (net 55))
   (segment (start 138.475085 86.746715) (end 138.4808 86.741) (width 0.25) (layer "F.Cu") (net 56))
   (segment (start 142.7226 86.7664) (end 142.748 86.741) (width 0.25) (layer "F.Cu") (net 56))

Commit message: 29 August Office 001
Parts:
- moved TP3 19.0 mm to (130.5, 91.5)
- moved TP5 9.71 mm to (135.0, 83.8)
- moved TP10 4.80 mm to (138.0, 100.3)
- moved C1 1.56 mm to (139.5, 72.7), turned to -90 degrees
- moved C7 0.73 mm to (140.5, 82.2)
- moved C2 0.29 mm to (144.2, 68.2)
Routing:
- net GND: track 0.00 -> 46.8 mm, vias 0 -> 2
- net Net-(C9-Pad1): track 0.00 -> 28.4 mm, vias 0 -> 1
- net Net-(U1-VCC_IO): track 0.00 -> 27.4 mm, vias 0 -> 2
- net Net-(U1-V11_OUT_DIG): track 0.00 -> 20.3 mm
- net Net-(J4-Pin_1): track 0.00 -> 11.2 mm, vias 0 -> 1
- net VCC: track 6.27 -> 16.3 mm
- net 1.1V: track 13.1 -> 23.0 mm
- net VDD: track 0.00 -> 6.99 mm
- net CHIP_EN: track 47.8 -> 54.7 mm
- net LNA_IN: track 0.00 -> 4.34 mm
- net Net-(U1-TP_IF_N/Sense2(1)): track 0.00 -> 3.94 mm
- net Net-(J3-Pin_1): track 2.41 -> 5.77 mm
- net Net-(C9-Pad2): track 0.00 -> 2.73 mm

Commit message: update from home 30-8-2024
Parts:
- removed TP6, TP7: TP, Connector_PinHeader_2.54mm:PinHeader_1x01_P2.54mm_Vertical
- moved TP4 26.9 mm to (134.0, 103.1)
- moved TP1 20.7 mm to (131.0, 83.8)
- moved TP8 8.83 mm to (127.2, 82.8)
- moved TP9 6.55 mm to (122.6, 82.8)
Routing:
- net VCC: track 16.3 -> 65.3 mm, vias 2 -> 5
- net VDD: track 6.99 -> 45.4 mm, vias 0 -> 3
- net LNA_IN: track 4.34 -> 33.9 mm, vias 0 -> 2
- net Net-(U1-TP_IF_N/Sense2(1)): track 3.94 -> 24.8 mm, vias 0 -> 1
- net Net-(U1-RFA_IN): track 0.00 -> 14.3 mm
- net 1.1V: track 23.0 -> 34.7 mm, vias 3 -> 5
- net Net-(U1-V11_OUT_DIG): track 20.3 -> 31.7 mm, vias 0 -> 2
