File: uprojects/Adee/PCB/STA5635/STA5635.kicad_pcb (KiCad board)
At the start: 2 copper layers, 60.1 x 72.8 mm, 27 parts, among them J1 Conn_02x20_Odd_Even, J2 SMA_CONNECTOR, J3 EN, J4 Conn_01x02, U1 STA5635A, U2 AP2127K-1.8

Commit message: 30 August Office 001
Parts:
- added TP6: TP, Connector_PinHeader_2.54mm:PinHeader_1x01_P2.54mm_Vertical, F.Cu at (142.0, 101.5)
Connections:
- U1 pad 10: unconnected-(U1-TCXO_IN-Pad10) -> Net-(U1-TCXO_IN)
Routing:
- net GND: track 46.8 -> 154.2 mm, vias 2 -> 4
- net Net-(U1-TCXO_IN): track 0.00 -> 35.5 mm, vias 0 -> 1
- net Net-(U1-V18_OUT): track 0.00 -> 27.9 mm
- net Net-(J1-Pin_39): track 0.00 -> 27.1 mm, vias 0 -> 1
- net CHIP_EN: track 54.3 -> 58.8 mm
Other:
- rule pad_to_mask_clearance: 0 -> 0.05
