File: uprojects/Adee/PCB/STA5635/STA5635.kicad_pcb (KiCad board)
At the start: 2 copper layers, 60.1 x 72.8 mm, 28 parts, among them J1 Conn_02x20_Odd_Even, J2 SMA_CONNECTOR, J3 EN, J4 Conn_01x02, U1 STA5635A, U2 AP2127K-1.8

Commit message: for push
Parts:
- moved TP4 30.5 mm to (127.9, 73.3)
- moved TP6 27.3 mm to (127.9, 78.2)
- moved TP3 19.3 mm to (124.1, 73.3)
- moved TP1 15.5 mm to (131.7, 68.3)
- moved TP2 15.2 mm to (131.7, 78.2)
- moved TP9 14.6 mm to (124.1, 68.3)
- moved TP8 14.5 mm to (127.9, 68.3)
- moved TP5 11.0 mm to (131.7, 73.3)
- moved J4 0.08 mm to (136.9, 68.3)
Connections:
- L1 pad 2: LNA_IN -> Net-(C9-Pad1)
Routing:
- net Net-(C9-Pad1): track 28.4 -> 12.6 mm
- net LNA_IN: track 33.9 -> 27.7 mm
- net Net-(U1-TP_IF_N/Sense2(1)): track 24.8 -> 18.7 mm
- net Net-(U1-V11_OUT_DIG): track 31.7 -> 26.1 mm
- net Net-(U1-TCXO_IN): track 35.5 -> 31.7 mm
- net 1.1V: track 34.7 -> 31.1 mm
- net Net-(U1-VCC_IO): track 27.4 -> 24.6 mm
- net Net-(U1-RFA_IN): track 14.3 -> 11.6 mm
- net Net-(U1-LNA_OUT): track 8.72 -> 6.46 mm

Commit message: 4 Sept Office 001
Parts:
- moved J2 34.7 mm to (144.9, 73.8)
- moved C4 24.2 mm to (149.0, 108.1), turned to -90 degrees
- moved C9 23.8 mm to (144.5, 80.4), turned to -90 degrees
- moved C5 21.5 mm to (146.5, 108.1), turned to -90 degrees
- moved L2 20.3 mm to (144.5, 85.4), turned to 90 degrees
- moved C6 19.0 mm to (144.0, 108.1), turned to -90 degrees
- moved L1 17.9 mm to (140.4, 79.6)
- moved C8 15.5 mm to (139.0, 108.1), turned to -90 degrees
- moved C3 14.6 mm to (136.6, 108.1), turned to -90 degrees
- moved R1 14.6 mm to (134.2, 108.1), turned to 90 degrees
- moved R2 6.72 mm to (131.6, 85.8), turned to 90 degrees
- moved TP3 4.21 mm to (127.9, 75.1)
- moved TP9 4.21 mm to (127.9, 70.2)
- moved TP4 4.21 mm to (131.7, 75.1)
- moved TP6 4.21 mm to (131.7, 80.1)
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Routing:
- net VCC: track 65.3 -> 20.7 mm, vias 5 -> 3
- net GND: track 154.2 -> 110.5 mm
- net Net-(U1-TCXO_IN): track 31.7 -> 6.50 mm
- net LNA_IN: track 27.7 -> 2.49 mm, vias 2 -> 1
- net Net-(U1-V18_OUT): track 27.9 -> 9.10 mm
- net Net-(U1-VCC_IO): track 24.6 -> 9.78 mm
- net Net-(U1-V11_OUT_DIG): track 26.1 -> 11.5 mm, vias 2 -> 1
- net Net-(U1-TP_IF_N/Sense2(1)): track 18.7 -> 5.08 mm
- net Net-(C9-Pad1): track 12.6 -> 0.00 mm, vias 1 -> 0
- net CHIP_EN: track 58.8 -> 53.1 mm
- net Net-(J3-Pin_1): track 5.77 -> 2.41 mm
- net Net-(U1-LNA_OUT): track 6.46 -> 3.44 mm
- net Net-(C9-Pad2): track 2.73 -> 0.00 mm
- net VDD: track 45.4 -> 42.7 mm

Commit message: update from home 04-9-2024
Parts:
- added H1: MountingHole, MountingHole:MountingHole_2.2mm_M2, F.Cu at (128.3, 60.3)
- added H2: MountingHole, MountingHole:MountingHole_2.2mm_M2, F.Cu at (128.3, 112.8)
- added H3: MountingHole, MountingHole:MountingHole_2.2mm_M2, F.Cu at (168.9, 84.3)
- added H4: MountingHole, MountingHole:MountingHole_2.2mm_M2, F.Cu at (168.9, 92.2)
- moved TP4 29.1 mm to (142.0, 102.3)
- moved TP3 11.6 mm to (131.7, 64.1)
- moved TP9 9.75 mm to (135.5, 64.1)
- moved L1 4.34 mm to (140.5, 83.9)
- moved J1 3.10 mm to (153.0, 62.9)
- moved J4 2.96 mm to (140.0, 64.1)
- moved C2 2.85 mm to (147.1, 63.9)
- moved R2 2.50 mm to (133.7, 84.3), turned to 0 degrees
- moved TP10 2.05 mm to (138.3, 102.3)
- moved C7 0.71 mm to (140.5, 81.5)
- moved J3 0.54 mm to (131.7, 96.4)
- moved TP5 0.10 mm to (135.5, 75.2)
Connections:
- J2 pad 1: Net-(C9-Pad1) -> Net-(C9-Pad2)
- L1 pad 2: Net-(C9-Pad1) -> Net-(C9-Pad2)
- L2 pad 1: LNA_IN -> Net-(C9-Pad1)
- L2 pad 2: Net-(C9-Pad2) -> LNA_IN
Routing:
- net VCC: track 20.7 -> 103.6 mm
- net Net-(U1-VCC_IO): track 9.78 -> 60.4 mm, vias 2 -> 1
- net GND: track 110.5 -> 136.3 mm, vias 4 -> 13
- net Net-(U1-TP_IF_N/Sense2(1)): track 5.08 -> 26.6 mm
- net Net-(U1-V18_OUT): track 9.10 -> 26.0 mm
- net Net-(U1-V11_OUT_DIG): track 11.5 -> 27.4 mm, vias 1 -> 2
- net 1.1V: track 31.1 -> 44.4 mm
- net Net-(U1-RFA_IN): track 11.6 -> 24.1 mm, vias 0 -> 2
- net Net-(C9-Pad1): track 0.00 -> 11.3 mm
- net Net-(J3-Pin_1): track 2.41 -> 13.7 mm
- net Net-(U1-TCXO_IN): track 6.50 -> 15.9 mm
- net Net-(U1-LNA_OUT): track 3.44 -> 12.9 mm, vias 0 -> 1
- net VDD: track 42.7 -> 46.6 mm
- net Net-(J1-Pin_21): track 15.9 -> 12.9 mm
- net Net-(J1-Pin_25): track 15.0 -> 12.0 mm
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- added copper zone on B.Cu, net GND
Other:
- board size 60.1 x 72.8 mm -> 34.7 x 57.5 mm

Commit message: 6 Sept Office 001
Parts:
- C9: value 104 -> 2PF
- H3, H4: footprint MountingHole:MountingHole_2.2mm_M2 -> MountingHole:MountingHole_2.2mm_M2_DIN965
- J2: value SMA_CONNECTOR -> SMA
- L1: value L_Small -> 10nH
- L2: value L_Small -> 3.6nH
- R2: value 1K -> 1E4
- moved H3 25.8 mm to (159.9, 60.1), turned to 90 degrees
- moved H4 22.7 mm to (159.9, 113.0), turned to 90 degrees
- moved C9 2.52 mm to (147.0, 80.3), turned to 90 degrees
- moved L2 1.24 mm to (145.8, 85.4), turned to -90 degrees
Connections:
- J1 pad 39: Net-(J1-Pin_39) -> TCXO_IN
- R2 pad 1: VCC -> VDD
- TP6 pad 1: Net-(U1-TCXO_IN) -> TCXO_IN
- TP9 pad 1: VCC -> VDD
- U1 pad 10: Net-(U1-TCXO_IN) -> TCXO_IN
- U1 pad 17: Net-(J1-Pin_39) -> TCXO_IN
- U1 pad 5: VCC -> VDD
Routing:
- net TCXO_IN: track 0.00 -> 54.9 mm, vias 0 -> 2
- net VDD: track 46.6 -> 92.8 mm, vias 3 -> 5
- net Net-(J1-Pin_39): track 28.4 -> 0.00 mm, vias 1 -> 0
- net Net-(U1-TCXO_IN): track 15.9 -> 0.00 mm, vias 1 -> 0
- net Net-(C9-Pad2): track 1.85 -> 14.1 mm
- net VCC: track 103.6 -> 92.7 mm, vias 3 -> 1
- net Net-(C9-Pad1): track 11.3 -> 2.98 mm
- net GNDA: track 0.00 -> 4.05 mm, vias 0 -> 3
- net 1.1V: track 44.4 -> 45.3 mm
- net Net-(J1-Pin_17): track 15.5 -> 16.4 mm
- net Net-(J1-Pin_13): track 18.7 -> 19.4 mm
- net LNA_IN: track 5.18 -> 5.81 mm, vias 1 -> 0
- added copper zone on B.Cu, net GNDA
- added copper zone on F.Cu, net GNDA
Other:
- board size 34.7 x 57.5 mm -> 36.4 x 57.5 mm
