File: KiCads/kicad_upwork/jonathan/touch_switch/touch_switch.kicad_pcb (KiCad board)
At the start: 2 copper layers, 33.7 x 37.1 mm, 9 parts, among them J1 USB_B, J2 Conn_01x02, J3 Conn_01x02, U1 TTP223-BA6

Commit message: 26 Aug 2025 Dorm
Parts:
- added U2: H11F1S, H11F1SM:OPTOCOUPLER_H11F3SR2M, F.Cu at (152.7, 93.9)
- J1: footprint Connector_USB:USB_B_Amphenol_MUSB-D511_Vertical_Rugged -> Connector_USB:USB_B_Lumberg_2411_02_Horizontal
- R2: value 3K3 -> 330
- moved R2 8.89 mm to (144.5, 91.2), turned to 0 degrees
- moved J1 8.85 mm to (142.5, 87.2), turned to 90 degrees
- moved C1 4.92 mm to (144.6, 96.8)
- moved C2 4.92 mm to (134.6, 91.9)
- moved U1 4.92 mm to (139.4, 92.1)
- moved D1 4.92 mm to (140.9, 96.8)
- moved R1 4.92 mm to (137.0, 96.8)
Connections:
- J2 pad 2: GND -> Net-(J2-Pin_2)
- R2 pad 2: Net-(J2-Pin_1) -> Net-(R2-Pad2)
Routing:
- net Net-(U1-Q): track 6.26 -> 19.3 mm, vias 0 -> 2
- net Net-(J2-Pin_2): track 0.00 -> 9.28 mm
- net +5V: track 19.1 -> 10.8 mm
- net GND: track 30.6 -> 25.6 mm
- net Net-(J3-Pin_1): track 30.9 -> 27.5 mm
- net Net-(R2-Pad2): track 0.00 -> 3.14 mm
- net Net-(J2-Pin_1): track 16.1 -> 18.8 mm
Other:
- board text added: "OUT1"
- board text added: "OUT2"
- board text removed: "GND"
- board text removed: "OUT+"
