File: Trismed/HT300/Schem_PCB/HT300/HT300.kicad_sch (KiCad schematic)
At the start: 1 part, among them U1 ATSAM4S16BB-AN

Commit message: 5 Sept 25 Office
Parts:
- added C1: 0.1uF, symbol Device:C_Small
- added C2: 0.01uF, symbol Device:C_Small
Connections:
- net at U1.1 (ADVREF): now also C1.1, C2.1
- net GND: now reaches U1.2 (GND)
- net GND: now also C1.2, C2.2
