File: uprojects/Laurent ESP Mesh/meshlite.pcb/meshlite2/meshlite.kicad_pcb (KiCad board)
At the start: 2 copper layers, 89.2 x 57.1 mm, 12 parts, among them J3 Conn_02x05_Odd_Even, J4 Conn_02x05_Odd_Even, K1 CPC1916Y, U1 MOUDLE-SEEEDUINO-XIAO-ESP32C3

Commit message: Updates 19-Jan-25
Parts:
- added D4: SS14, Diode_SMD:D_SMA, F.Cu at (99.1, 67.6)
- added K2: FINDER-36.11, Relay_THT:Relay_SPDT_Finder_36.11, F.Cu at (97.5, 48.9)
- added Q1: MMBT2222A, Package_TO_SOT_SMD:SOT-23, F.Cu at (114.3, 47.4)
- added R6: 470E, Resistor_SMD:R_0603_1608Metric, F.Cu at (113.9, 50.8)
- added U2: INA219, INA219:MODULE_INA219, F.Cu at (163.5, 82.5)
Connections:
- U1 pad 10: unconnected-(U1-PA5_A9_D9_MISO-Pad10) -> /RELAY_ON
- U1 pad 14: unconnected-(U1-5V-Pad14) -> Net-(U1-5V)
- U1 pad 5: unconnected-(U1-PA8_A4_D4_SDA-Pad5) -> Net-(U1-PA8_A4_D4_SDA)
- U1 pad 6: unconnected-(U1-PA9_A5_D5_SCL-Pad6) -> Net-(U1-PA9_A5_D5_SCL)
Other:
- board text added: "INA219"
- board text removed: "SENSOR"

Commit message: 20 Jan 26 Office
Parts:
- removed J3, J4: Conn_02x05_Odd_Even, Connector_PinSocket_2.54mm:PinSocket_2x05_P2.54mm_Vertical
- added J1: DCJ200-10-A-XX-K_REVA, DCJ200-10-A-XX-K_REVA:GCT_DCJ200-10-A-XX-K_REVA, F.Cu at (105.2, 87.7)
- added J2: Conn_01x05, Connector_Wago:Wago_734-165_1x05_P3.50mm_Horizontal, F.Cu at (171.0, 60.5)
- moved U1 26.5 mm to (145.9, 56.4), turned to 180 degrees

Commit message: Updates 20-Jan-25
Parts:
- removed J2: Conn_01x05, Connector_Wago:Wago_734-165_1x05_P3.50mm_Horizontal
- added J3: B5PS-VH, footprints:CONN_B5PS-VH_JST, F.Cu at (172.7, 67.8)
- moved U1 17.2 mm to (140.9, 72.9)
- moved R2 15.3 mm to (129.5, 56.0)
- moved Q1 5.76 mm to (115.5, 53.0)
- moved R6 5.76 mm to (115.0, 56.5)
- moved D4 3.86 mm to (99.1, 71.5)
- moved K2 3.86 mm to (97.6, 52.8)
- moved U2 1.58 mm to (163.0, 84.0)
Routing:
- net (no net): vias 1 -> 3
Other:
- outline, holes or cut-outs redrawn

Commit message: 26 Jan 26 Office
Parts:
- removed K1: CPC1916Y, CPC1916Y:CPC1916Y
- removed R2: R_Small, Resistor_SMD:R_0603_1608Metric
- added U3: YAAJ_DCDC_StepDown_LM2596, KiCad:YAAJ_DCDC_StepDown_LM2596, F.Cu at (126.4, 51.7)
- moved J1 31.3 mm to (136.5, 87.0)
- moved U1 27.5 mm to (113.4, 73.9)
- moved D2 13.7 mm to (121.0, 53.0)
- moved R4 13.2 mm to (116.2, 69.0)
- moved D1 13.2 mm to (116.3, 61.0)
- moved R1 13.2 mm to (116.2, 63.9)
- moved R5 13.2 mm to (116.2, 71.5)
- moved R3 13.2 mm to (116.2, 66.4)
- moved D3 8.61 mm to (121.0, 50.5)
- moved D4 2.45 mm to (99.1, 69.0)
- moved K2 2.00 mm to (97.6, 50.8)
Connections:
- U1 pad 11: Net-(U1-PA6_A10_D10_MOSI) -> unconnected-(U1-PA6_A10_D10_MOSI-Pad11)

Commit message: Upate From Home Mac 28 Jan 2026
Parts:
- moved J1 41.1 mm to (139.0, 46.0), turned to 180 degrees
- moved U2 26.5 mm to (189.5, 84.0)
- moved U3 5.55 mm to (127.7, 57.1)
- moved J3 4.72 mm to (176.7, 65.3)
Other:
- outline, holes or cut-outs redrawn
Changed lines of the file:
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@@
 	(footprint "DCJ200-10-A-XX-K_REVA:GCT_DCJ200-10-A-XX-K_REVA"
 		(layer "F.Cu")
-		(at 136.5 87)
+		(at 139 45.95 180)
 		(property "Reference" "J1"
-			(at -1.575 -12.075 0)
+			(at -8 -6.55 0)
 			(layer "F.SilkS")
 			(effects
@@
 		)
 		(property "Value" "DCJ200-10-A-XX-K_REVA"
-			(at 0.3 -10.65 0)
+			(at -17 -3.05 0)
 			(layer "F.Fab")
 			(effects
@@
 		)
 		(property "MF" "Global Connector Technology"
-			(at 0 0 0)
+			(at 0 0 180)
 			(unlocked yes)
 			(layer "F.Fab")
@@
 		)
 		(property "MAXIMUM_PACKAGE_HEIGHT" "11 mm"
-			(at 0 0 0)
+			(at 0 0 180)
 			(unlocked yes)
 			(layer "F.Fab")
@@
 		)
 		(property "Package" "None"
-			(at 0 0 0)
+			(at 0 0 180)
 			(unlocked yes)
 			(layer "F.Fab")
@@
 		)
 		(property "Price" "None"
-			(at 0 0 0)
+			(at 0 0 180)
 			(unlocked yes)
 			(layer "F.Fab")
@@
 		)
 		(property "Check_prices" "https://www.snapeda.com/parts/DCJ200-10-A-K1-K/Global+Connector+Technology/view-part/?ref=eda"
-			(at 0 0 0)
+			(at 0 0 180)
 			(unlocked yes)
 			(layer "F.Fab")
@@
 		)
 		(property "STANDARD" "Manufacturer Recommendations"
-			(at 0 0 0)
+			(at 0 0 180)
 			(unlocked yes)
 			(layer "F.Fab")
@@
 		)
 		(property "PARTREV" "A"
-			(at 0 0 0)
+			(at 0 0 180)
 			(unlocked yes)
 			(layer "F.Fab")
@@
 		)
 		(property "SnapEDA_Link" "https://www.snapeda.com/parts/DCJ200-10-A-K1-K/Global+Connector+Technology/view-part/?ref=snap"
-			(at 0 0 0)
+			(at 0 0 180)
 			(unlocked yes)
 			(layer "F.Fab")
@@
 		)
 		(property "MP" "DCJ200-10-A-K1-K"
-			(at 0 0 0)
+			(at 0 0 180)
 			(unlocked yes)
 			(layer "F.Fab")
@@
 		)
 		(property "Description_1" "Power Barrel Connector Jack 2.05mm ID (0.081), 5.50mm OD (0.217) Through Hole, Right Angle"
-			(at 0 0 0)
+			(at 0 0 180)
 			(unlocked yes)
 			(layer "F.Fab")
@@
 		)
 		(property "MANUFACTURER" "Global Connector Technology"
-			(at 0 0 0)
+			(at 0 0 180)
 			(unlocked yes)
 			(layer "F.Fab")
@@
 		)
 		(property "Availability" "In Stock"
-			(at 0 0 0)
+			(at 0 0 180)
 			(unlocked yes)
 			(layer "F.Fab")
@@
 		)
 		(property "SNAPEDA_PN" "DCJ200-10-A-K1-K"
-			(at 0 0 0)
+			(at 0 0 180)
 			(unlocked yes)
 			(layer "F.Fab")
@@
 		(attr through_hole)
 		(fp_line
-			(start -4.5 7.15)
-			(end -4.5 -7.15)
+			(start 4.5 7.15)
+			(end 4.5 -1.4)
 			(stroke
 				(width 0.2)
@@
 		)
 		(fp_line
-			(start -4.5 7.15)
-			(end 4.5 7.15)
+			(start 4.5 -7.15)
+			(end 4.5 -5.9)
 			(stroke
 				(width 0.2)
@@
 		)
 		(fp_line
-			(start -2.45 -7.15)
-			(end -4.5 -7.15)
+			(start 2.45 -7.15)
+			(end 4.5 -7.15)
 			(stroke
 				(width 0.2)
@@
 		)
 		(fp_line
-			(start 2.45 -7.15)
-			(end 4.5 -7.15)
+			(start -2.45 -7.15)
+			(end -4.5 -7.15)
 			(stroke
 				(width 0.2)
@@
 		)
 		(fp_line
-			(start 4.5 -7.15)
-			(end 4.5 -5.9)
+			(start -4.5 7.15)
+			(end 4.5 7.15)
 			(stroke
 				(width 0.2)
@@
 		)
 		(fp_line
-			(start 4.5 7.15)
-			(end 4.5 -1.4)
+			(start -4.5 7.15)
+			(end -4.5 -7.15)
 			(stroke
 				(width 0.2)
@@
 		)
 		(fp_line
-			(start -4.75 -7.9)
-			(end -4.75 7.4)
+			(start 6.05 7.4)
+			(end 6.05 -7.9)
 			(stroke
 				(width 0.05)
@@
 		)
 		(fp_line
-			(start -4.75 7.4)
-			(end 6.05 7.4)
+			(start 6.05 -7.9)
+			(end -4.75 -7.9)
 			(stroke
 				(width 0.05)
@@
 		)
 		(fp_line
-			(start 6.05 -7.9)
-			(end -4.75 -7.9)
+			(start -4.75 7.4)
+			(end 6.05 7.4)
 			(stroke
 				(width 0.05)
@@
 		)
 		(fp_line
-			(start 6.05 7.4)
-			(end 6.05 -7.9)
+			(start -4.75 -7.9)
+			(end -4.75 7.4)
 			(stroke
 				(width 0.05)
@@
 		)
 		(fp_line
-			(start -4.5 -7.15)
+			(start 4.5 7.15)
 			(end 4.5 -7.15)
 			(stroke
@@
 		(fp_line
 			(start -4.5 7.15)
-			(end -4.5 -7.15)
+			(end 4.5 7.15)
 			(stroke
 				(width 0.1)
@@
 		(fp_line
 			(start -4.5 7.15)
-			(end 4.5 7.15)
+			(end -4.5 -7.15)
 			(stroke
 				(width 0.1)
@@
 		)
 		(fp_line
-			(start 4.5 7.15)
+			(start -4.5 -7.15)
 			(end 4.5 -7.15)
 			(stroke
@@
 		)
 		(pad "1" thru_hole oval
-			(at 0 -6.55)
+			(at 0 -6.55 180)
 			(size 4.4 2.2)
 			(drill oval 3.6 1)
@@
 		)
 		(pad "2" thru_hole oval
-			(at 0 -0.25)
+			(at 0 -0.25 180)
 			(size 4 2)
 			(drill oval 3.2 1)
@@
 		)
 		(pad "3" thru_hole oval
-			(at 4.8 -3.65)
+			(at 4.8 -3.65 180)
 			(size 2 4)
 			(drill oval 1 3.2)
@@
 	(footprint "KiCad:YAAJ_DCDC_StepDown_LM2596"
 		(layer "F.Cu")
-		(at 126.36 51.72)
+		(at 127.68 57.11)
 		(property "Reference" "U3"
 			(at 21.59 -3.81 0)
@@
 	(footprint "footprints:CONN_B5PS-VH_JST"
 		(layer "F.Cu")
-		(at 172.6556 67.8151 90)
+		(at 176.6556 65.3151 90)
 		(tags "B5PS-VH ")
 		(property "Reference" "J3"
@@
 	(footprint "INA219:MODULE_INA219"
 		(layer "F.Cu")
-		(at 163 84 180)
+		(at 189.5 84 180)
 		(property "Reference" "U2"
 			(at -9.525 -12.065 0)
@@
 		)
 		(property "Value" "FINDER-36.11"
-			(at 12.4325 16.7 0)
+			(at 5.9325 9.7 0)
 			(layer "F.Fab")
 			(effects
@@
 	)
 	(gr_line
+		(start 138.5 87)
+		(end 175.5 87)
+		(stroke
+			(width 0.1)
+			(type default)
+		)
+		(layer "Edge.Cuts")
+	)
+	(gr_line
 		(start 92.583 95.25)
 		(end 95.0595 95.25)
@@
 	)
 	(gr_line
+		(start 175.5 43)
+		(end 175.5 87)
+		(stroke
+			(width 0.1)
+			(type default)
+		)
+		(layer "Edge.Cuts")
+	)
+	(gr_line
 		(start 92.71 38.1)
 		(end 181.737 38.1)
@@
 		(layer "Edge.Cuts")
 	)
-	(gr_line
-		(start 93.5 43)
-		(end 183.5 43)
-		(stroke
-			(width 0.1)
-			(type default)
-		)
-		(layer "F.Fab")
-	)
 	(gr_text "INA219"
 		(at 155 71 0)
@@
 	(dimension
 		(type orthogonal)
-		(layer "F.Fab")
+		(layer "Edge.Cuts")
 		(pts
-			(xy 92.583 38.1) (xy 92.71 43)
+			(xy 99.5 43) (xy 175.5 43)
 		)
-		(height 13.917)
-		(orientation 1)
+		(height -2)
+		(orientation 0)
 		(format
 			(prefix "")
@@
 			(keep_text_aligned yes)
 		)
-		(gr_text "4.9"
-			(at 105.35 40.55 90)
-			(layer "F.Fab")
+		(gr_text "76"
+			(at 137.5 39.85 0)
+			(layer "Edge.Cuts")
 			(effects
 				(font
@@
 		(layer "F.Fab")
 		(pts
-			(xy 172.5 43) (xy 101.5 43)
+			(xy 92.583 38.1) (xy 92.71 43)
 		)
-		(height -13.5)
-		(orientation 0)
+		(height 13.917)
+		(orientation 1)
 		(format
 			(prefix "")
@@
 			(keep_text_aligned yes)
 		)
-		(gr_text "71"
-			(at 137 28.35 0)
+		(gr_text "4.9"
+			(at 105.35 40.55 90)
 			(layer "F.Fab")
 			(effects
@@
 	)
 	(via
-		(at 101.5 43)
+		(at 138.5 87)
 		(size 5)
 		(drill 3)
@@
 	)
 	(via
-		(at 163.449 80.518)
-		(size 3.8)
-		(drill 2.5)
+		(at 99.5 43)
+		(size 5)
+		(drill 3)
 		(layers "F.Cu" "B.Cu")
 		(net 0)
 	)
 	(via
-		(at 172.5 43)
+		(at 175.5 43)
 		(size 5)
 		(drill 3)

Commit message: update 03-Feb-2026
Parts:
- moved U2 9.14 mm to (180.6, 81.8), turned to -90 degrees
- moved U3 3.00 mm to (124.7, 57.1)
Other:
- board size 89.2 x 57.1 mm -> 109.5 x 57.2 mm

Commit message: update 03-Feb-2026
Parts:
- moved U3 40.9 mm to (147.1, 91.3), turned to 90 degrees
- moved U1 19.2 mm to (114.1, 93.1), turned to 0 degrees
- moved D4 10.4 mm to (109.5, 68.0)
- moved D1 7.83 mm to (122.7, 56.5)
- moved D2 7.83 mm to (127.4, 48.5)
- moved D3 7.83 mm to (127.4, 46.0)
- moved Q1 7.83 mm to (121.9, 48.5)
- moved R1 7.83 mm to (122.7, 59.5)
- moved R4 7.83 mm to (122.7, 64.6)
- moved R5 7.83 mm to (122.7, 67.1)
- moved R6 7.83 mm to (121.5, 52.0)
- moved R3 7.83 mm to (122.7, 62.0)
- moved K2 5.59 mm to (103.1, 49.8)
- moved J1 1.35 mm to (137.7, 46.0)
Other:
- board size 109.5 x 57.2 mm -> 109.5 x 57.1 mm

Commit message: Update 20 Feb 2026
Parts:
- added D4: LED, LED_THT:LED_D3.0mm, F.Cu at (195.2, 84.3)
- added J2: B5PS-VH, footprints:CONN_B5PS-VH_JST, F.Cu at (202.7, 86.3)
- D1, D2, D3: footprint LED_SMD:LED_0603_1608Metric -> LED_THT:LED_D3.0mm
- moved K2 109.3 mm to (211.9, 59.2), turned to 180 degrees
- moved D6 97.5 mm to (207.0, 66.0), turned to 180 degrees
- moved Q1 78.0 mm to (194.6, 77.0), turned to 180 degrees
- moved R6 76.6 mm to (195.0, 73.6), turned to 180 degrees
- moved R5 67.9 mm to (190.0, 58.5), turned to 180 degrees
- moved D2 67.8 mm to (195.3, 48.5), turned to 180 degrees
- moved R1 67.7 mm to (190.0, 66.1), turned to 180 degrees
- moved R4 67.4 mm to (190.0, 61.0), turned to 180 degrees
- moved R3 67.3 mm to (190.0, 63.6), turned to 0 degrees
- moved U1 59.5 mm to (166.6, 65.1)
- moved J3 58.1 mm to (118.8, 70.7), turned to -90 degrees
- moved J1 49.6 mm to (160.3, 90.0), turned to 0 degrees
- moved D3 38.4 mm to (123.8, 84.3)
- moved U3 37.1 mm to (150.0, 54.4), turned to -90 degrees
- moved D1 8.11 mm to (123.7, 48.5)
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- renumbered D4 to D6
Connections:
- J3 pad 1: unconnected-(J3-Pad1) -> /24VDC-IN
- J3 pad 2: unconnected-(J3-Pad2) -> GND
- J3 pad 3: unconnected-(J3-Pad3) -> /PGND
Other:
- board size 109.5 x 57.1 mm -> 109.5 x 57.2 mm
