File: uprojects/Laurent ESP Mesh/meshlite.pcb/meshlite2/meshlite.kicad_pcb (KiCad board)
At the start: 2 copper layers, 109.5 x 57.2 mm, 18 parts, among them J1 DCJ200-10-A-XX-K_REVA, J2 B5PS-VH, J3 B5PS-VH, K2 FINDER-36.11, Q1 MMBT2222A, U1 MOUDLE-SEEEDUINO-XIAO-ESP32C3, U2 INA219, U3 YAAJ_DCDC_StepDown_LM2596

Commit message: Update 23 Feb 2026
Parts:
- added J4: Conn_01x07, Connector_PinSocket_2.54mm:PinSocket_1x07_P2.54mm_Vertical, F.Cu at (167.0, 47.4)
- added J5: Conn_01x07, Connector_PinSocket_2.54mm:PinSocket_1x07_P2.54mm_Vertical, F.Cu at (183.0, 62.5)
- added J6: Conn_01x06, Connector_PinSocket_2.54mm:PinSocket_1x06_P2.54mm_Vertical, F.Cu at (171.5, 76.7)
- added R2: 1K, Resistor_SMD:R_0603_1608Metric, F.Cu at (125.5, 54.5)
- moved R5 28.0 mm to (162.2, 55.0), turned to 0 degrees
- moved R1 26.4 mm to (171.2, 47.5)
- moved U1 26.0 mm to (166.1, 39.1)
- moved R3 23.2 mm to (171.2, 50.0), turned to 180 degrees
- moved R4 20.6 mm to (171.2, 52.5)
- moved U2 3.41 mm to (179.1, 83.0)
- moved Q1 3.12 mm to (196.4, 74.5), turned to 0 degrees
- moved R6 1.99 mm to (193.2, 74.5), turned to -90 degrees
- moved D6 1.41 mm to (206.0, 65.0)
- moved J3 0.50 mm to (119.3, 70.7)
Connections:
- D2 pad 1: GND -> /LED-C-LMP1
- D2 pad 2: Net-(D2-A) -> /LED-A-LMP1
- D4 pad 1: unconnected-(D4-K-Pad1) -> /LED-C-LMP2
- D4 pad 2: unconnected-(D4-A-Pad2) -> /LED-A-LMP2
- J1 pad 1: unconnected-(J1-Pad1) -> Net-(U3-Vin)
- J1 pad 2: unconnected-(J1-Pad2) -> GND
- J1 pad 3: unconnected-(J1-Pad3) -> GND
- J2 pad 1: unconnected-(J2-Pad1) -> /24VDC-IN
- J2 pad 2: unconnected-(J2-Pad2) -> GND
- J2 pad 3: unconnected-(J2-Pad3) -> /PGND
- J2 pad 4: unconnected-(J2-Pad4) -> /LED-C-LMP2
- J2 pad 5: unconnected-(J2-Pad5) -> /LED-A-LMP2
- J3 pad 4: unconnected-(J3-Pad4) -> /LED-C-LMP1
- J3 pad 5: unconnected-(J3-Pad5) -> /LED-A-LMP1
- R3 pad 1: Net-(D1-A) -> unconnected-(R3-Pad1)
- R3 pad 2: Net-(U1-PA4_A1_D1) -> Net-(J4-Pin_2)
- R4 pad 1: Net-(D2-A) -> unconnected-(R4-Pad1)
- R4 pad 2: Net-(U1-PA10_A2_D2) -> Net-(J4-Pin_3)
- R5 pad 2: Net-(U1-PA11_A3_D3) -> Net-(J4-Pin_4)
- U1 pad 1: A0 -> unconnected-(U1-PA02_A0_D0-Pad1)
- U1 pad 10: /RELAY_ON -> unconnected-(U1-PA5_A9_D9_MISO-Pad10)
- U1 pad 14: Net-(U1-5V) -> unconnected-(U1-5V-Pad14)
- U1 pad 2: Net-(U1-PA4_A1_D1) -> unconnected-(U1-PA4_A1_D1-Pad2)
- U1 pad 3: Net-(U1-PA10_A2_D2) -> unconnected-(U1-PA10_A2_D2-Pad3)
- U1 pad 4: Net-(U1-PA11_A3_D3) -> unconnected-(U1-PA11_A3_D3-Pad4)
- U1 pad 5: Net-(U1-PA8_A4_D4_SDA) -> unconnected-(U1-PA8_A4_D4_SDA-Pad5)
- U1 pad 6: Net-(U1-PA9_A5_D5_SCL) -> unconnected-(U1-PA9_A5_D5_SCL-Pad6)
- U2 pad 1: Net-(U1-5V) -> +5V
- U2 pad 3: Net-(U1-PA9_A5_D5_SCL) -> Net-(J4-Pin_6)
- U2 pad 4: Net-(U1-PA8_A4_D4_SDA) -> Net-(J4-Pin_5)
- U3 pad 1: unconnected-(U3-Vin-Pad1) -> Net-(U3-Vin)
- U3 pad 2: unconnected-(U3-GND-Pad2) -> GND
- U3 pad 3: unconnected-(U3-GND-Pad3) -> GND
- U3 pad 4: unconnected-(U3-Vout-Pad4) -> +5V
Routing:
- net GND: track 0.00 -> 226.6 mm
- net /LED-A-LMP1: track 0.00 -> 141.6 mm
- net /LED-C-LMP1: track 0.00 -> 120.0 mm
- net +5V: track 0.00 -> 74.6 mm
- net Net-(U3-Vin): track 0.00 -> 34.8 mm
- net /RELAY_ON: track 0.00 -> 24.0 mm
- net Net-(D6-A): track 0.00 -> 23.0 mm
- net /24VDC-IN: track 0.00 -> 19.1 mm
- net Net-(J6-Pin_5): track 0.00 -> 16.3 mm
- net Net-(J6-Pin_6): track 0.00 -> 15.9 mm
- net Net-(D6-K): track 0.00 -> 7.43 mm
- net Net-(D1-A): track 0.00 -> 6.36 mm
- net A0: track 0.00 -> 3.47 mm
- net Net-(J4-Pin_2): track 0.00 -> 3.46 mm
- net Net-(J4-Pin_3): track 0.00 -> 3.44 mm
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Other:
- outline, holes or cut-outs redrawn
- board text added: "LAMP1"
- board text added: "LAMP2"
- board text added: "POWER"

Commit message: local update 23 feb 26
Parts:
- added R7: 4k7, Resistor_SMD:R_0603_1608Metric, F.Cu at (172.0, 60.0)
- added R8: 4k7, Resistor_SMD:R_0603_1608Metric, F.Cu at (172.0, 57.5)
Connections:
- J1 pad 1: Net-(U3-Vin) -> /24VDC-IN
- U3 pad 1: Net-(U3-Vin) -> /24VDC-IN
Routing:
- net Net-(J4-Pin_5): track 0.00 -> 45.3 mm
- net Net-(J4-Pin_6): track 0.00 -> 37.0 mm
- net Net-(U3-Vin): track 34.8 -> 0.00 mm
- net /24VDC-IN: track 19.1 -> 53.9 mm
- net +5V: track 74.6 -> 80.7 mm
- net Net-(J4-Pin_4): track 0.00 -> 3.93 mm

Commit message: Update 24 Feb 2026
Parts:
- removed U1: MOUDLE-SEEEDUINO-XIAO-ESP32C3, xiao ESP32C3_PCB:MOUDLE14P-SMD-2.54-21X17.8MM
- added J7: Conn_01x02, Connector_PinHeader_2.54mm:PinHeader_1x02_P2.54mm_Vertical, F.Cu at (195.5, 60.0)
Connections:
- D6 pad 1: Net-(D6-K) -> +5V
- J1 pad 1: /24VDC-IN -> Net-(J6-Pin_6)
- K2 pad 11: unconnected-(K2-Pad11) -> /24VDC-IN
- K2 pad 14: unconnected-(K2-Pad14) -> Net-(J6-Pin_5)
- K2 pad A1: Net-(D6-K) -> +5V
- U3 pad 1: /24VDC-IN -> Net-(J6-Pin_6)
Routing:
- net /24VDC-IN: track 53.9 -> 181.0 mm, vias 0 -> 1
- net +5V: track 80.7 -> 191.6 mm, vias 0 -> 1
- net Net-(D3-A): track 0.00 -> 65.6 mm, vias 0 -> 1
- net Net-(J6-Pin_5): track 16.3 -> 75.8 mm, vias 0 -> 1
- net GND: track 226.6 -> 282.4 mm
- net Net-(J6-Pin_6): track 15.9 -> 68.8 mm
- net /LED-A-LMP2: track 0.00 -> 17.9 mm
- net /LED-C-LMP2: track 0.00 -> 13.6 mm
- net Net-(D6-K): track 7.43 -> 0.00 mm
Other:
- outline, holes or cut-outs redrawn

Commit message: Update 24 Feb 2026
Routing:
- net /PGND: track 0.00 -> 240.5 mm, vias 0 -> 6
- net Net-(D3-A): track 65.6 -> 59.6 mm
- net /24VDC-IN: track 181.0 -> 186.8 mm
- net (no net): vias 3 -> 0
Changed lines of the file:
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@@
 		)
-	)
-	(via
-		(at 159.5 48.5)
-		(size 5)
-		(drill 3)
-		(layers "F.Cu" "B.Cu")
-		(net 0)
-	)
-	(via
-		(at 198.5 93)
-		(size 5)
-		(drill 3)
-		(layers "F.Cu" "B.Cu")
-		(net 0)
-	)
-	(via
-		(at 122.5 93)
-		(size 5)
-		(drill 3)
-		(layers "F.Cu" "B.Cu")
-		(net 0)
 	)
 	(segment
@@
 	)
 	(segment
+		(start 126.29 84.3)
+		(end 135.5 75.09)
+		(width 0.8)
+		(layer "B.Cu")
+		(net 4)
+	)
+	(segment
 		(start 153.25 49.75)
 		(end 158.27 54.77)
@@
 	)
 	(segment
-		(start 126.29 84.3)
-		(end 135.5 75.09)
+		(start 135.5 75.09)
+		(end 135.5 61.75)
 		(width 0.8)
 		(layer "B.Cu")
@@
 	)
 	(segment
-		(start 135.5 51.5)
-		(end 137.25 49.75)
+		(start 135.5 61.75)
+		(end 147.5 49.75)
 		(width 0.8)
 		(layer "B.Cu")
@@
 	)
 	(segment
-		(start 135.5 75.09)
-		(end 135.5 51.5)
-		(width 0.8)
-		(layer "B.Cu")
-		(net 4)
-	)
-	(segment
-		(start 137.25 49.75)
+		(start 147.5 49.75)
 		(end 153.25 49.75)
 		(width 0.8)
@@
 	)
 	(segment
-		(start 142.25 46.75)
-		(end 138 51)
-		(width 1.5)
-		(layer "F.Cu")
-		(net 22)
-	)
-	(segment
-		(start 128.25 52.5)
-		(end 128.25 64.75)
-		(width 1.5)
-		(layer "F.Cu")
-		(net 22)
-	)
-	(segment
-		(start 126.325 63.704301)
-		(end 126.325 54.5)
-		(width 0.5)
-		(layer "F.Cu")
-		(net 22)
-	)
-	(segment
-		(start 128.25 64.75)
-		(end 122.3151 70.6849)
-		(width 1.5)
-		(layer "F.Cu")
-		(net 22)
-	)
-	(segment
-		(start 129.75 51)
-		(end 128.25 52.5)
-		(width 1.5)
-		(layer "F.Cu")
-		(net 22)
-	)
-	(segment
-		(start 138 51)
-		(end 129.75 51)
-		(width 1.5)
-		(layer "F.Cu")
-		(net 22)
-	)
-	(segment
-		(start 119.344401 70.6849)
-		(end 126.325 63.704301)
-		(width 0.5)
-		(layer "F.Cu")
-		(net 22)
-	)
-	(segment
-		(start 122.3151 70.6849)
-		(end 119.344401 70.6849)
-		(width 1.5)
-		(layer "F.Cu")
-		(net 22)
+		(start 195 96.5)
+		(end 198.5 93)
+		(width 1.5)
+		(layer "F.Cu")
+		(net 21)
+	)
+	(segment
+		(start 154 92)
+		(end 158.5 96.5)
+		(width 1.5)
+		(layer "F.Cu")
+		(net 21)
+	)
+	(segment
+		(start 198.5 93)
+		(end 210.5 93)
+		(width 2.5)
+		(layer "F.Cu")
+		(net 21)
+	)
+	(segment
+		(start 212.5 91)
+		(end 212.5 78.5)
+		(width 2.5)
+		(layer "F.Cu")
+		(net 21)
+	)
+	(segment
+		(start 158.5 96.5)
+		(end 195 96.5)
+		(width 1.5)
+		(layer "F.Cu")
+		(net 21)
+	)
+	(segment
+		(start 122.5 93)
+		(end 124 91.5)
+		(width 1.5)
+		(layer "F.Cu")
+		(net 21)
+	)
+	(segment
+		(start 210.5 93)
+		(end 212.5 91)
+		(width 2.5)
+		(layer "F.Cu")
+		(net 21)
+	)
+	(segment
+		(start 212.3951 78.3951)
+		(end 202.6556 78.3951)
+		(width 2.5)
+		(layer "F.Cu")
+		(net 21)
+	)
+	(segment
+		(start 133.5 47)
+		(end 158 47)
+		(width 2.5)
+		(layer "F.Cu")
+		(net 21)
+	)
+	(segment
+		(start 212.5 78.5)
+		(end 212.3951 78.3951)
+		(width 2.5)
+		(layer "F.Cu")
+		(net 21)
+	)
+	(segment
+		(start 124 91.5)
+		(end 141.25 91.5)
+		(width 1.5)
+		(layer "F.Cu")
+		(net 21)
+	)
+	(segment
+		(start 158 47)
+		(end 159.5 48.5)
+		(width 2.5)
+		(layer "F.Cu")
+		(net 21)
 	)
 	(via
-		(at 142.25 46.75)
+		(at 159.5 48.5)
+		(size 5)
+		(drill 3)
+		(layers "F.Cu" "B.Cu")
+		(free yes)
+		(net 21)
+	)
+	(via
+		(at 154 92)
 		(size 2.5)
 		(drill 1)
 		(layers "F.Cu" "B.Cu")
-		(net 22)
-	)
-	(segment
-		(start 182 42.25)
-		(end 146.75 42.25)
-		(width 1.5)
-		(layer "B.Cu")
+		(net 21)
+	)
+	(via
+		(at 198.5 93)
+		(size 5)
+		(drill 3)
+		(layers "F.Cu" "B.Cu")
+		(free yes)
+		(net 21)
+	)
+	(via
+		(at 133.5 47)
+		(size 2.5)
+		(drill 1)
+		(layers "F.Cu" "B.Cu")
+		(net 21)
+	)
+	(via
+		(at 141.25 91.5)
+		(size 2.5)
+		(drill 1)
+		(layers "F.Cu" "B.Cu")
+		(net 21)
+	)
+	(via
+		(at 122.5 93)
+		(size 5)
+		(drill 3)
+		(layers "F.Cu" "B.Cu")
+		(free yes)
+		(net 21)
+	)
+	(segment
+		(start 109 46.25)
+		(end 111.75 43.5)
+		(width 2.5)
+		(layer "B.Cu")
+		(net 21)
+	)
+	(segment
+		(start 111.25 93)
+		(end 109 90.75)
+		(width 2.5)
+		(layer "B.Cu")
+		(net 21)
+	)
+	(segment
+		(start 111.75 43.5)
+		(end 130 43.5)
+		(width 2.5)
+		(layer "B.Cu")
+		(net 21)
+	)
+	(segment
+		(start 153.5 91.5)
+		(end 154 92)
+		(width 1.5)
+		(layer "B.Cu")
+		(net 21)
+	)
+	(segment
+		(start 109.3951 78.6049)
+		(end 119.344401 78.6049)
+		(width 2.5)
+		(layer "B.Cu")
+		(net 21)
+	)
+	(segment
+		(start 141.25 91.5)
+		(end 153.5 91.5)
+		(width 1.5)
+		(layer "B.Cu")
+		(net 21)
+	)
+	(segment
+		(start 122.5 93)
+		(end 111.25 93)
+		(width 2.5)
+		(layer "B.Cu")
+		(net 21)
+	)
+	(segment
+		(start 130 43.5)
+		(end 133.5 47)
+		(width 2.5)
+		(layer "B.Cu")
+		(net 21)
+	)
+	(segment
+		(start 109 79)
+		(end 109.3951 78.6049)
+		(width 2.5)
+		(layer "B.Cu")
+		(net 21)
+	)
+	(segment
+		(start 109 90.75)
+		(end 109 79)
+		(width 2.5)
+		(layer "B.Cu")
+		(net 21)
+	)
+	(segment
+		(start 109 79)
+		(end 109 46.25)
+		(width 2.5)
+		(layer "B.Cu")
+		(net 21)
+	)
+	(segment
+		(start 122.3151 70.6849)
+		(end 119.344401 70.6849)
+		(width 1.5)
+		(layer "F.Cu")
+		(net 22)
+	)
+	(segment
+		(start 129.75 51)
+		(end 128.25 52.5)
+		(width 1.5)
+		(layer "F.Cu")
+		(net 22)
+	)
+	(segment
+		(start 126.325 63.704301)
+		(end 126.325 54.5)
+		(width 0.5)
+		(layer "F.Cu")
+		(net 22)
+	)
+	(segment
+		(start 138 51)
+		(end 129.75 51)
+		(width 1.5)
+		(layer "F.Cu")
+		(net 22)
+	)
+	(segment
+		(start 128.25 52.5)
+		(end 128.25 64.75)
+		(width 1.5)
+		(layer "F.Cu")
+		(net 22)
+	)
+	(segment
+		(start 119.344401 70.6849)
+		(end 126.325 63.704301)
+		(width 0.5)
+		(layer "F.Cu")
+		(net 22)
+	)
+	(segment
+		(start 128.25 64.75)
+		(end 122.3151 70.6849)
+		(width 1.5)
+		(layer "F.Cu")
+		(net 22)
+	)
+	(via
+		(at 138 51)
+		(size 2.5)
+		(drill 1)
+		(layers "F.Cu" "B.Cu")
 		(net 22)
 	)
@@
 	)
 	(segment
-		(start 205.9325 44.6825)
-		(end 203.75 42.5)
-		(width 1.5)
-		(layer "B.Cu")
-		(net 22)
-	)
-	(segment
-		(start 142.25 46.75)
-		(end 142.5 46.75)
+		(start 138 51)
+		(end 146.75 42.25)
 		(width 1.5)
 		(layer "B.Cu")
@@
 	)
 	(segment
+		(start 203.5 42.25)
+		(end 205.9325 44.6825)
+		(width 1.5)
+		(layer "B.Cu")
+		(net 22)
+	)
+	(segment
 		(start 195.5 62.5)
 		(end 204.6325 62.5)
@@
 	)
 	(segment
+		(start 205.9325 44.6825)
+		(end 205.9325 61.2)
+		(width 1.5)
+		(layer "B.Cu")
+		(net 22)
+	)
+	(segment
+		(start 138 51)
+		(end 142.25 46.75)
+		(width 1.5)
+		(layer "B.Cu")
+		(net 22)
+	)
+	(segment
 		(start 146.75 42.25)
-		(end 142.25 46.75)
-		(width 1.5)
-		(layer "B.Cu")
-		(net 22)
-	)
-	(segment
-		(start 203.5 42.25)
-		(end 182 42.25)
-		(width 1.5)
-		(layer "B.Cu")
-		(net 22)
-	)
-	(segment
-		(start 203.75 42.5)
 		(end 203.5 42.25)
 		(width 1.5)
 		(layer "B.Cu")
-		(net 22)
-	)
-	(segment
-		(start 205.9325 61.2)
-		(end 205.9325 44.6825)
-		(width 1.5)
-		(layer "B.Cu")

Commit message: Update 19 mar 2026
Parts:
- removed R1: R_Small, Resistor_SMD:R_0603_1608Metric
- added S1: JCHL HL4*22C, Spacer:SPACER_01, F.Cu at (125.0, 48.5)
- added S2: JCHL HL4*22C, Spacer:SPACER_01, F.Cu at (194.0, 48.5)
- added S3: JCHL HL4*22C, Spacer:SPACER_01, F.Cu at (125.0, 84.3)
- added S4: JCHL HL4*22C, Spacer:SPACER_01, F.Cu at (194.0, 84.3)
- K2: value FINDER-36.11 -> Songle Relay SRD-05VDC-SL-C
Other:
- outline, holes or cut-outs redrawn

Commit message: Update 27 mar 2026
Connections:
- J4 pad 7: unconnected-(J4-Pin_7-Pad7) -> /RELAY_ON
- J5 pad 3: /RELAY_ON -> unconnected-(J5-Pin_3-Pad3)
Routing:
- net /RELAY_ON: track 24.0 -> 75.3 mm, vias 0 -> 1
Changed lines of the file:
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@@
 	(net 14 "Net-(J4-Pin_6)")
 	(net 15 "Net-(J4-Pin_5)")
-	(net 16 "unconnected-(J4-Pin_7-Pad7)")
+	(net 16 "unconnected-(J5-Pin_3-Pad3)")
 	(net 17 "unconnected-(J5-Pin_5-Pad5)")
 	(net 18 "unconnected-(J5-Pin_1-Pad1)")
@@
 			(layers "*.Cu" "*.Mask")
 			(remove_unused_layers no)
-			(net 12 "/RELAY_ON")
+			(net 16 "unconnected-(J5-Pin_3-Pad3)")
 			(pinfunction "Pin_3")
 			(pintype "passive")
@@
 			(layers "*.Cu" "*.Mask")
 			(remove_unused_layers no)
-			(net 16 "unconnected-(J4-Pin_7-Pad7)")
+			(net 12 "/RELAY_ON")
 			(pinfunction "Pin_7")
 			(pintype "passive")
@@
 	)
 	(segment
-		(start 183 57.46)
-		(end 188.96 57.46)
-		(width 0.8)
+		(start 193.25 73.675)
+		(end 193.25 70.695)
+		(width 0.5)
 		(layer "F.Cu")
 		(net 12)
 	)
 	(segment
-		(start 193.25 61.75)
-		(end 193.25 73.675)
-		(width 0.8)
+		(start 186.944 64.389)
+		(end 186.944 47.752)
+		(width 0.5)
 		(layer "F.Cu")
 		(net 12)
 	)
 	(segment
-		(start 188.96 57.46)
-		(end 193.25 61.75)
-		(width 0.8)
+		(start 193.25 70.695)
+		(end 188.722 66.167)
+		(width 0.5)
 		(layer "F.Cu")
 		(net 12)
 	)
+	(segment
+		(start 188.722 66.167)
+		(end 186.944 64.389)
+		(width 0.5)
+		(layer "F.Cu")
+		(net 12)
+	)
+	(via
+		(at 186.944 47.752)
+		(size 2.5)
+		(drill 1)
+		(layers "F.Cu" "B.Cu")
+		(net 12)
+	)
+	(segment
+		(start 186.944 47.752)
+		(end 186.944 45.085)
+		(width 0.5)
+		(layer "B.Cu")
+		(net 12)
+	)
+	(segment
+		(start 163.83 61.722)
+		(end 164.728 62.62)
+		(width 0.5)
+		(layer "B.Cu")
+		(net 12)
+	)
+	(segment
+		(start 186.182 44.323)
+		(end 164.338 44.323)
+		(width 0.5)
+		(layer "B.Cu")
+		(net 12)
+	)
+	(segment
+		(start 186.944 45.085)
+		(end 186.182 44.323)
+		(width 0.5)
+		(layer "B.Cu")
+		(net 12)
+	)
+	(segment
+		(start 164.338 44.323)
+		(end 163.83 44.831)
+		(width 0.5)
+		(layer "B.Cu")
+		(net 12)
+	)
+	(segment
+		(start 164.728 62.62)
+		(end 167 62.62)
+		(width 0.5)
+		(layer "B.Cu")
+		(net 12)
+	)
+	(segment
+		(start 163.83 44.831)
+		(end 163.83 61.722)
+		(width 0.5)
+		(layer "B.Cu")
+		(net 12)
+	)

Commit message: Meshlite PCB 001 Update
Parts:
- moved D1 3.29 mm to (123.0, 51.7)
- moved S1 3.29 mm to (124.2, 51.7)
- moved R2 3.20 mm to (125.5, 57.7)
- moved D2 3.15 mm to (195.3, 51.7)
- moved S2 3.15 mm to (194.0, 51.7)
- moved D3 1.04 mm to (123.0, 85.0)
- moved S3 1.04 mm to (124.2, 85.0)
- moved D4 0.70 mm to (195.2, 85.0)
- moved S4 0.70 mm to (194.0, 85.0)
Routing:
- net /24VDC-IN: track 186.8 -> 169.6 mm
- net /LED-C-LMP1: track 120.0 -> 123.0 mm
- net Net-(D3-A): track 59.6 -> 60.6 mm
- net /LED-A-LMP2: track 17.9 -> 18.6 mm

Commit message: Update 29 Apr 2026
Routing:
- net /PGND: track 240.5 -> 241.8 mm
Other:
- board text added: "12V/24V in"
- board text added: "3V3"
- board text added: "5V"
- board text added: "BYPASS JUMPER"
- board text added: "GND"
- board text added: "ReSPR REV 0.3"
- board text added: "SCL"
- board text added: "SDA"
- board text added: "VIN+"
- board text added: "VIN-"
