File: uprojects/Laurent ESP Mesh/meshlite.pcb/meshlite2/meshlite.kicad_sch (KiCad schematic)
At the start: 24 parts, among them J1 DCJ200-10-A-XX-K_REVA, J2 B5PS-VH, J3 B5PS-VH, J4 Conn_01x07, J5 Conn_01x07, J6 Conn_01x06, K2 FINDER-36.11, Q1 MMBT2222A, U1 MOUDLE-SEEEDUINO-XIAO-ESP32C3, U2 INA219, U3 YAAJ_DCDC_StepDown_LM2596

Commit message: Update 24 Feb 2026
Parts:
- added J7: Conn_01x02, Connector_PinHeader_2.54mm:PinHeader_1x02_P2.54mm_Vertical, symbol Connector_Generic:Conn_01x02
- D1, D2, D3, D4: LCSC (none) -> C473831
- D6: LCSC (none) -> C83852
- J1: LCSC (none) -> C5280493
- J2, J3: LCSC (none) -> C157989
- J4, J5: LCSC (none) -> C492406
- J6: LCSC (none) -> C42431807
- K2: value FINDER-36.11 -> Songle Relay SRD-05VDC-SL-C; LCSC (none) -> C35449
- Q1: LCSC (none) -> C82460
- R1, U3: now not fitted; now left out of the parts list
- R2: LCSC (none) -> C22548
- R3, R4, R5, R6: LCSC (none) -> C114669
- R7, R8: LCSC (none) -> C99782
Connections:
- net +5V: now also D6.1 (K), K2.A1
- net 24VDC-IN: now also K2.11, J7.2 (Pin_2); no longer J1.1, U3.1 (Vin)
- net at J6.5 (Pin_5), U2.5 (VIN-), U2.VIN-: now also K2.14, J7.1 (Pin_1)
- net at J6.6 (Pin_6), U2.6 (VIN+), U2.VIN+: now also J1.1, U3.1 (Vin)

Commit message: Update 19 mar 2026
Parts:
- added S1, S2, S3, S4: JCHL HL4*22C, Spacer:SPACER_01, symbol spacer:SPACER_LED01
- J1: Check_prices https://www.snapeda.com/parts/DCJ200-10-A-K1-K/Global+Conne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 -> (none); LCSC C5280493 -> C720557; MF Global Connector Technology -> XUNPU DC-005-A200; MP DCJ200-10-A-K1-K -> XUNPU DC-005-A200; SNAPEDA_PN DCJ200-10-A-K1-K -> XUNPU DC-005-A200; SnapEDA_Link https://www.snapeda.com/parts/DCJ200-10-A-K1-K/Global+Conne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 -> (none)

Commit message: Update 27 mar 2026
Connections:
- net RELAY_ON: now also J4.7 (Pin_7); no longer J5.3 (Pin_3)
Changed lines of the file:
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@@
+	(wire
+		(pts
+			(xy 121.92 97.79) (xy 116.84 97.79)
+		)
+		(stroke
+			(width 0)
+			(type default)
+		)
+	)
 	(wire
 		(pts
@@
 	(wire
 		(pts
+			(xy 116.84 97.79) (xy 116.84 105.41)
+		)
+		(stroke
+			(width 0)
+			(type default)
+		)
+	)
+	(wire
+		(pts
 			(xy 49.53 137.16) (xy 49.53 143.51)
 		)
@@
 	(wire
 		(pts
-			(xy 175.26 92.71) (xy 166.37 92.71)
+			(xy 116.84 105.41) (xy 125.73 105.41)
 		)
 		(stroke
@@
 	)
 	(label "RELAY_ON"
-		(at 175.26 92.71 0)
-		(effects
-			(font
+		(at 125.73 105.41 0)
+		(effects
+			(font
