File: uprojects/John Ottolenghi/kicadA/snifferA/snifferA.kicad_sch (KiCad schematic)
At the start: 1 part, among them U1 MQ-131

Commit message: Update 29 Jan 2026
Parts:
- added A1: ARDUINO_MEGA_2560_REV3_A000067, ARDUINO_MEGA_2560_REV3_A000067:ARDUINO_ARDUINO_MEGA_2560_REV3_A000067, symbol ARDUINO_MEGA_2560_REV3_A000067:ARDUINO_MEGA_2560_REV3_A000067
- added J1: DHT22, Connector_PinSocket_2.54mm:PinSocket_1x04_P2.54mm_Vertical, symbol Connector_Generic:Conn_01x04
- added J2: Conn_01x10, Connector_PinHeader_2.54mm:PinHeader_1x10_P2.54mm_Vertical, symbol Connector_Generic:Conn_01x10
- added J3: Conn_01x08, Connector_PinHeader_2.54mm:PinHeader_1x08_P2.54mm_Vertical, symbol Connector_Generic:Conn_01x08
- added U2: MQ-135, MQ-X:MQ, symbol MQ-X:MQ
- added U3: MQ-136, MQ-X:MQ, symbol MQ-X:MQ
- added U4: MQ-137, MQ-X:MQ, symbol MQ-X:MQ
- added U5: MQ-02, MQ-X:MQ, symbol MQ-X:MQ
- added U6: MQ-04, MQ-X:MQ, symbol MQ-X:MQ
- added U7: MQ-06, MQ-X:MQ, symbol MQ-X:MQ
- added U8: MQ-08, MQ-X:MQ, symbol MQ-X:MQ

Commit message: Update 30 Jan 2026
Parts:
- added U9: YAAJ_DCDC_StepDown_LM2596, symbol yaaj_dcdc_stepdown_lm2596:YAAJ_DCDC_StepDown_LM2596
Other:
- note added: "MQ-131 LOW RL - 1M"
Changed lines of the file:
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@@
 	(generator_version "9.0")
 	(paper "A4")
+	(text "MQ-131 LOW RL - 1M\n"
+		(exclude_from_sim no)
+		(at 243.078 126.238 0)
+		(effects
+			(font
+				(size 1.27 1.27)
+			)
+		)
+	)
 	(symbol
 		(lib_id "MQ-X:MQ")
@@
 					(unit 1)
 				)
+			)
+		)
+	)
+	(symbol
+		(lib_id "yaaj_dcdc_stepdown_lm2596:YAAJ_DCDC_StepDown_LM2596")
+		(at 138.43 176.53 0)
+		(unit 1)
+		(exclude_from_sim no)
+		(in_bom yes)
+		(on_board yes)
+		(dnp no)
+		(fields_autoplaced yes)
+		(property "Reference" "U9"
+			(at 138.43 166.37 0)
+			(effects
+				(font
+					(size 1.27 1.27)
+				)
+			)
+		)
+		(property "Value" "YAAJ_DCDC_StepDown_LM2596"
+			(at 138.43 168.91 0)
+			(effects
+				(font
+					(size 1.27 1.27)
+				)
+			)
+		)
+		(property "Footprint" ""
+			(at 137.16 176.53 0)
+			(effects
+				(font
+					(size 1.27 1.27)
+				)
+				(hide yes)
+			)
+		)
+		(property "Datasheet" ""
+			(at 137.16 176.53 0)
+			(effects
+				(font
+					(size 1.27 1.27)
+				)
+				(hide yes)
+			)
+		)
+		(property "Description" "module : adjustable step down module 3.2V-40V to 1.25V-35V 3A"
+			(at 138.43 176.53 0)
+			(effects
+				(font
+					(size 1.27 1.27)
+				)
+				(hide yes)
+			)
+		)
+		(pin "2"
+		)
+		(pin "1"
+		)
+		(pin "3"
+		)
+		(pin "4"
+		)
+		(instances
+			(project ""
+				(path "/15fbcfff-fd81-4c4b-9218-077244baf01d"
+					(reference "U9")
+					(unit 1)
+				)

Commit message: update 02-Feb-2026
Parts:
- U9: footprint (none) -> KiCad:YAAJ_DCDC_StepDown_LM2596
Changed lines of the file:
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@@
 			)
 		)
-		(property "Footprint" ""
+		(property "Footprint" "KiCad:YAAJ_DCDC_StepDown_LM2596"
 			(at 137.16 176.53 0)
 			(effects

Commit message: Update 10 Feb 2026
Parts:
- added J4, J5, J7, J8, J9: Conn_01x08, Connector_PinHeader_2.54mm:PinHeader_1x08_P2.54mm_Vertical, symbol Connector_Generic:Conn_01x08
- added J6: Conn_02x18_Odd_Even, Connector_PinHeader_2.54mm:PinHeader_2x18_P2.54mm_Vertical, symbol Connector_Generic:Conn_02x18_Odd_Even
- added U10: MQ-131-L, MQ-X:MQ, symbol MQ-X:MQ
- U1: value MQ-131 -> MQ-131-H
Other:
- moved on the sheet: U9

Commit message: Update 11 Feb 2026
Parts:
- added J10: ZP07, Connector_PinSocket_2.54mm:PinSocket_1x04_P2.54mm_Vertical, symbol Connector_Generic:Conn_01x04
- added U11: ~, sensors:SM4-NO2-20, symbol sensors:SM4-NO2-20
- added U12: ZE08-CH20, sensors:ZE-08, symbol sensors:ZE08-CH20
- added U13: ZP07, sensors:ZP07-FRAME, symbol sensors:ZP07
- J3: value Conn_01x08 -> CCS811_CJMCU
Other:
- moved on the sheet: U1, U10, U2, U3, U4, U5, U6, U7, U8

Commit message: Update 12 Feb 2026
Parts:
- added U14: SM4-NO2-20, sensors:SM4-NO2-20, symbol sensors:SM4-NO2-20
Changed lines of the file:
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@@
+	)
+	(symbol
+		(lib_id "sensors:SM4-NO2-20")
+		(at 212.09 77.47 0)
+		(unit 1)
+		(exclude_from_sim no)
+		(in_bom yes)
+		(on_board yes)
+		(dnp no)
+		(fields_autoplaced yes)
+		(property "Reference" "U14"
+			(at 215.9 82.55 0)
+			(effects
+				(font
+					(size 1.27 1.27)
+				)
+			)
+		)
+		(property "Value" "SM4-NO2-20"
+			(at 215.9 85.09 0)
+			(effects
+				(font
+					(size 1.27 1.27)
+				)
+			)
+		)
+		(property "Footprint" "sensors:SM4-NO2-20"
+			(at 212.09 77.47 0)
+			(effects
+				(font
+					(size 1.27 1.27)
+				)
+				(hide yes)
+			)
+		)
+		(property "Datasheet" ""
+			(at 212.09 77.47 0)
+			(effects
+				(font
+					(size 1.27 1.27)
+				)
+				(hide yes)
+			)
+		)
+		(property "Description" ""
+			(at 212.09 77.47 0)
+			(effects
+				(font
+					(size 1.27 1.27)
+				)
+				(hide yes)
+			)
+		)
+		(pin "1"
+		)
+		(pin "4"
+		)
+		(pin "2"
+		)
+		(pin "5"
+		)
+		(pin "3"
+		)
+		(instances
+			(project ""
+				(path "/15fbcfff-fd81-4c4b-9218-077244baf01d"
+					(reference "U14")
+					(unit 1)
+				)
+			)
+		)
 	)
 	(symbol

Commit message: Update 24 Feb 2026
Parts:
- added C1, C2: 0.1uF, Capacitor_SMD:C_1206_3216Metric_Pad1.33x1.80mm_HandSolder, symbol Device:C_Small
- added R1, R4: 10k, Resistor_SMD:R_1206_3216Metric, symbol Device:R_Small
- added R2, R3: 10K, Resistor_SMD:R_1206_3216Metric, symbol Device:R_Small
- added U15: MQ-07, MQ-X:MQ, symbol MQ-X:MQ
- J2: LCSC (none) -> C42431810
- J4, J5, J7, J8, J9: LCSC (none) -> C6332201
- J6: LCSC (none) -> C41376109
- U11: value ~ -> ZE-03
Connections:
- net GND: now also J2.7 (Pin_7), U1.4 (B), U1.6 (B), U10.4 (B), U10.6 (B), C1.1, C2.1, R2.2, R3.2
- net +5VP: now reaches U10.1 (A)
- net +5VP: now also U1.1 (A), U1.3 (A), U10.3 (A), U2.1 (A), U2.3 (A)
- net +5V: now reaches U10.2 (H)
- net +5V: now also U1.2 (H), U2.2 (H), U9.4 (Vout)
- net at U10.5 (H): now also R1.1, R2.1
- net at U1.5 (H): now also R3.1, R4.1
- net at J8.7 (Pin_7): now also C2.2, R4.2
- net at J8.8 (Pin_8): now also C1.2, R1.2
Other:
- moved on the sheet: J1, U1, U10, U11, U2, U3, U4, U5, U6, U7, U8

Commit message: Update 26 Feb 2026
Parts:
- added C10, C3, C4, C5, C6, C7, C8, C9: 0.1uF, Capacitor_SMD:C_1206_3216Metric_Pad1.33x1.80mm_HandSolder, symbol Device:C_Small
- added R10, R12, R14, R16, R18, R20, R6, R8: 10k, Resistor_SMD:R_1206_3216Metric, symbol Device:R_Small
- added R11, R13, R15, R17, R19, R5, R7, R9: 10K, Resistor_SMD:R_1206_3216Metric, symbol Device:R_Small
- J3: LCSC (none) -> C6332201
Connections:
- net +5V: now also U15.2 (H), U3.2 (H), U4.2 (H), U5.2 (H), U6.2 (H), U7.2 (H), U8.2 (H)
- net +5VP: now also U15.1 (A), U15.3 (A), U3.1 (A), U3.3 (A), U4.1 (A), U4.3 (A), U5.1 (A), U5.3 (A), U6.1 (A), U6.3 (A), U7.1 (A), U7.3 (A), U8.1 (A), U8.3 (A)
- net GND: now also U11.1, U14.1, U15.4 (B), U15.6 (B), U2.4 (B), U2.6 (B), U3.4 (B), U3.6 (B), U4.4 (B), U4.6 (B), U5.4 (B), U5.6 (B), U6.4 (B), U6.6 (B), U7.4 (B), U7.6 (B), U8.4 (B), U8.6 (B), C10.1, C3.1, C4.1, C5.1, C6.1, C7.1, C8.1, C9.1, R11.2, R13.2, R15.2, R17.2, R19.2, R5.2, R7.2, R9.2
- net at U3.5 (H): now also R7.1, R8.1
- net at U15.5 (H): now also R17.1, R18.1
- net at U7.5 (H): now also R15.1, R16.1
- net A15-SM4-N02: now reaches J7.1 (Pin_1)
- net A15-SM4-N02: now also U14.3
- net A14-ZE-03: now reaches J7.2 (Pin_2)
- net A14-ZE-03: now also U11.3
- net at J7.7 (Pin_7): now also C10.2, R20.2
- net at J7.8 (Pin_8): now also C9.2, R18.2
- net at U14.2: now also U11.2
- net at J8.1 (Pin_1): now also C8.2, R16.2
- net at J8.2 (Pin_2): now also C7.2, R14.2
- net at J8.3 (Pin_3): now also C6.2, R12.2
- net at J8.4 (Pin_4): now also C5.2, R10.2
- net at J8.5 (Pin_5): now also C4.2, R8.2
- net at J8.6 (Pin_6): now also C3.2, R6.2
- net at U4.5 (H): now also R10.1, R9.1
- net at U2.5 (H): now also R5.1, R6.1
- net at U5.5 (H): now also R11.1, R12.1
- net at U8.5 (H): now also R19.1, R20.1
- net at U6.5 (H): now also R13.1, R14.1
Other:
- moved on the sheet: J1, J3, U11, U12, U15, U8
