File: uprojects/John Ottolenghi/kicadA/snifferA/snifferA.kicad_sch (KiCad schematic)
At the start: 56 parts, among them J1 DHT22, J10 ZP07, J2 Conn_01x10, J3 CCS811_CJMCU, J4 Conn_01x08, J5 Conn_01x08, J6 Conn_02x18_Odd_Even, J7 Conn_01x08, J8 Conn_01x08, J9 Conn_01x08, U1 MQ-131-H, U10 MQ-131-L, U11 ZE-03, U12 ZE08-CH20, U13 ZP07, U14 SM4-NO2-20, U15 MQ-07, U2 MQ-135, U3 MQ-136, U4 MQ-137, U5 MQ-02, U6 MQ-04, U7 MQ-06, U8 MQ-08, U9 YAAJ_DCDC_StepDown_LM2596

Commit message: Update 26 Feb 2026
Parts:
- added C11, C12, C13: 0.1uF, Capacitor_SMD:C_1206_3216Metric_Pad1.33x1.80mm_HandSolder, symbol Device:C_Small
- added J11: DCJ200-10-A-XX-K_REVA, DCJ200-10-A-XX-K_REVA:GCT_DCJ200-10-A-XX-K_REVA, symbol DCJ200-10-A-XX-K_REVA:DCJ200-10-A-XX-K_REVA
- added R21, R22, R23: 10k, Resistor_SMD:R_1206_3216Metric, symbol Device:R_Small
- added U16: YAAJ_DCDC_StepDown_LM2596, KiCad:YAAJ_DCDC_StepDown_LM2596, symbol yaaj_dcdc_stepdown_lm2596:YAAJ_DCDC_StepDown_LM2596
Connections:
- net +5V: now also J10.3 (Pin_3), J3.1 (Pin_1), U11.4, U12.4, U14.4
- net +5VP: now also U16.4 (Vout)
- net A14-ZE-03: now also C11.2, R21.2; no longer U11.3
- net A15-SM4-N02: now also C12.2, R22.2; no longer U14.3
- net GND: now also J10.4 (Pin_4), J3.2 (Pin_2), U11.5, U12.3, U14.5, U9.2 (GND), U9.3 (GND), C11.1, C12.1, C13.1, J11.2, J11.3, U16.2 (GND), U16.3 (GND); no longer U11.1, U14.1
- net at J5.1 (Pin_1): now also U12.6
- net at J5.2 (Pin_2): now also U12.5
- net at J5.3 (Pin_3): now also U14.1
- net at J5.4 (Pin_4): now also U14.2
- net at J5.5 (Pin_5): now also U11.1
- net at J5.6 (Pin_6): now also U11.2
- net A12-ZP07-B: now reaches J10.1 (Pin_1)
- net A11-ZP07-A: now reaches J10.2 (Pin_2)
- net A11-ZP07-A: now also J7.5 (Pin_5)
- net at U9.1 (Vin): now also J11.1, U16.1 (Vin)
- net A13-ZE08-CH20: now reaches J7.3 (Pin_3)
- net A13-ZE08-CH20: now also C13.2, R23.2
- net A12-ZP07-A: now reaches J7.4 (Pin_4)
- net at U12.2: now also R23.1
- new net: R21.1, U11.3
- new net: R22.1, U14.3
Other:
- note added: "Rx1"
- note added: "Rx2"
- note added: "Rx3"
- note added: "Tx1"
- note added: "Tx2"
- note added: "Tx3"
- moved on the sheet: J1, J10, J3, U11, U12, U13, U9

Commit message: local update 2 Mar 26
Connections:
- net A12-ZP07-A is gone; now on net A12-ZP07-B: J7.4 (Pin_4)
- net +5V: now also J1.1 (Pin_1)
- net GND: now also J1.4 (Pin_4)
- net SCL: now also J3.3 (Pin_3)
- net SDA: now also J3.4 (Pin_4)
Other:
- note added: "SCL"
- note added: "SDA"
Changed lines of the file:
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@@
 		)
 	)
+	(text "SCL"
+		(exclude_from_sim no)
+		(at 48.7114 176.8404 0)
+		(effects
+			(font
+				(size 1.27 1.27)
+			)
+		)
+	)
 	(text "Tx1"
 		(exclude_from_sim no)
@@
 		)
 	)
+	(text "SDA"
+		(exclude_from_sim no)
+		(at 48.514 179.324 0)
+		(effects
+			(font
+				(size 1.27 1.27)
+			)
+		)
+	)
 	(text "Tx3"
 		(exclude_from_sim no)
@@
 	(wire
 		(pts
+			(xy 15.24 154.94) (xy 27.94 154.94)
+		)
+		(stroke
+			(width 0)
+			(type default)
+		)
+	)
+	(wire
+		(pts
 			(xy 73.66 68.58) (xy 71.12 68.58)
 		)
@@
 	(wire
 		(pts
+			(xy 16.51 143.51) (xy 16.51 147.32)
+		)
+		(stroke
+			(width 0)
+			(type default)
+		)
+	)
+	(wire
+		(pts
 			(xy 52.07 151.13) (xy 52.07 153.67)
 		)
@@
 	(wire
 		(pts
+			(xy 15.24 157.48) (xy 15.24 154.94)
+		)
+		(stroke
+			(width 0)
+			(type default)
+		)
+	)
+	(wire
+		(pts
 			(xy 71.12 35.56) (xy 73.66 35.56)
 		)
@@
 	(wire
 		(pts
-			(xy 16.51 154.94) (xy 27.94 154.94)
-		)
-		(stroke
-			(width 0)
-			(type default)
-		)
-	)
-	(wire
-		(pts
 			(xy 96.52 26.67) (xy 93.98 26.67)
 		)
@@
 	)
 	(label "SDA"
-		(at 46.99 180.34 0)
+		(at 21.59 179.07 0)
 		(effects
 			(font
@@
 	)
 	(label "SCL"
-		(at 46.99 177.8 0)
+		(at 21.59 176.53 0)
 		(effects
 			(font
@@
 		)
 	)
-	(label "A12-ZP07-A"
+	(label "A12-ZP07-B"
 		(at 109.22 93.98 0)
 		(effects
@@
 	)
 	(symbol
+		(lib_id "power:GND")
+		(at 15.24 157.48 0)
+		(unit 1)
+		(exclude_from_sim no)
+		(in_bom yes)
+		(on_board yes)
+		(dnp no)
+		(fields_autoplaced yes)
+		(property "Reference" "#PWR047"
+			(at 15.24 163.83 0)
+			(effects
+				(font
+					(size 1.27 1.27)
+				)
+				(hide yes)
+			)
+		)
+		(property "Value" "GND"
+			(at 17.78 158.7499 0)
+			(effects
+				(font
+					(size 1.27 1.27)
+				)
+				(justify left)
+			)
+		)
+		(property "Footprint" ""
+			(at 15.24 157.48 0)
+			(effects
+				(font
+					(size 1.27 1.27)
+				)
+				(hide yes)
+			)
+		)
+		(property "Datasheet" ""
+			(at 15.24 157.48 0)
+			(effects
+				(font
+					(size 1.27 1.27)
+				)
+				(hide yes)
+			)
+		)
+		(property "Description" "Power symbol creates a global label with name \"GND\" , ground"
+			(at 15.24 157.48 0)
+			(effects
+				(font
+					(size 1.27 1.27)
+				)
+				(hide yes)
+			)
+		)
+		(pin "1"
+		)
+		(instances
+			(project "snifferA"
+				(path "/15fbcfff-fd81-4c4b-9218-077244baf01d"
+					(reference "#PWR047")
+					(unit 1)
+				)
+			)
+		)
+	)
+	(symbol
 		(lib_id "Device:R_Small")
 		(at 78.74 80.01 90)
@@
 					(unit 1)
 				)
+			)
+		)
+	)
+	(symbol
+		(lib_id "power:+5V")
+		(at 16.51 143.51 0)
+		(unit 1)
+		(exclude_from_sim no)
+		(in_bom yes)
+		(on_board yes)
+		(dnp no)
+		(fields_autoplaced yes)
+		(property "Reference" "#PWR046"
+			(at 16.51 147.32 0)
+			(effects
+				(font
+					(size 1.27 1.27)
+				)
+				(hide yes)
+			)
+		)
+		(property "Value" "+5V"
+			(at 16.51 138.43 0)
+			(effects
+				(font
+					(size 1.27 1.27)
+				)
+			)
+		)
+		(property "Footprint" ""
+			(at 16.51 143.51 0)
+			(effects
+				(font
+					(size 1.27 1.27)
+				)
+				(hide yes)
+			)
+		)
+		(property "Datasheet" ""
+			(at 16.51 143.51 0)
+			(effects
+				(font
+					(size 1.27 1.27)
+				)
+				(hide yes)
+			)
+		)
+		(property "Description" "Power symbol creates a global label with name \"+5V\""
+			(at 16.51 143.51 0)
+			(effects
+				(font
+					(size 1.27 1.27)
+				)
+				(hide yes)
+			)
+		)
+		(pin "1"
+		)
+		(instances
+			(project "snifferA"
+				(path "/15fbcfff-fd81-4c4b-9218-077244baf01d"
+					(reference "#PWR046")
+					(unit 1)
+				)

Commit message: Update 3 mar 2026
Parts:
- A1: now not fitted; now left out of the parts list
Connections:
- net ADD: now also J3.8 (Pin_8), J6.3 (Pin_3)
- net INT: now also J3.6 (Pin_6), J6.7 (Pin_7)
- net RST: now also J3.7 (Pin_7), J6.5 (Pin_5)
- net SCL: now also J5.8 (Pin_8)
- net SDA: now also J5.7 (Pin_7)
- net WAK: now also J3.5 (Pin_5), J6.9 (Pin_9)
- net DHT22_DATA: now reaches J1.2 (Pin_2)
- net DHT22_DATA: now also J6.15 (Pin_15)
Other:
- note added: "ADD"
- note added: "INT"
- note added: "RST"
- note added: "WAK"
- moved on the sheet: J6

Commit message: Update 9 mar 2026
Parts:
- added R24, R25, R26, R27, R28, R29: 4K7, Resistor_SMD:R_0603_1608Metric, symbol Device:R_Small
Connections:
- net +5V: now also R24.1, R25.1, R26.1, R27.1, R28.1, R29.1
- net ADD: now also R29.2
- net INT: now also R27.2
- net RST: now also R28.2
- net SCL: now also R24.2
- net SDA: now also R25.2
- net WAK: now also R26.2
Other:
- moved on the sheet: J3
