File: uprojects/John Ottolenghi/kicadA/snifferA/snifferA.kicad_sch (KiCad schematic)
At the start: 67 parts, among them J1 DHT22, J10 ZP07, J11 DCJ200-10-A-XX-K_REVA, J2 Conn_01x10, J3 CCS811_CJMCU, J4 Conn_01x08, J5 Conn_01x08, J6 Conn_02x18_Odd_Even, J7 Conn_01x08, J8 Conn_01x08, J9 Conn_01x08, U1 MQ-131-H, U10 MQ-131-L, U12 ZE08-CH20, U13 ZP07, U14 SM4-NO2-20, U15 MQ-07, U16 YAAJ_DCDC_StepDown_LM2596, U2 MQ-135, U3 MQ-136, U4 MQ-137, U5 MQ-02, U6 MQ-04, U7 MQ-06, U8 MQ-08, U9 YAAJ_DCDC_StepDown_LM2596

Commit message: Update 12 mar 2026
Parts:
- removed U16, U9: YAAJ_DCDC_StepDown_LM2596, KiCad:YAAJ_DCDC_StepDown_LM2596, symbol yaaj_dcdc_stepdown_lm2596:YAAJ_DCDC_StepDown_LM2596
- added Q1: SI4403DDY-T1-GE3, MOSFET-P-20V:SO-8_MS-012_VIS, symbol MOSFET-P-20V:SI4403DDY-T1-GE3
Connections:
- net +5V: no longer J3.1 (Pin_1), R24.1, R25.1, R26.1, R27.1, R28.1, R29.1
- net GND: no longer J11.2, J11.3
- net +3.3V: now reaches J9.5 (Pin_5)
- net +3.3V: now also J3.1 (Pin_1), R24.1, R25.1, R26.1, R27.1, R28.1, R29.1

Commit message: Update 13 mar 2026
Parts:
- removed C9: 0.1uF, Capacitor_SMD:C_1206_3216Metric_Pad1.33x1.80mm_HandSolder, symbol Device:C_Small
- removed R17: 10K, Resistor_SMD:R_1206_3216Metric, symbol Device:R_Small
- removed R18: 10k, Resistor_SMD:R_1206_3216Metric, symbol Device:R_Small
- removed U15: MQ-07, MQ-X:MQ, symbol MQ-X:MQ
- added J12: MICS-6814, Connector_PinSocket_2.54mm:PinSocket_1x05_P2.54mm_Vertical, symbol Connector_Generic:Conn_01x05

Commit message: Update 17 mar 2026
Parts:
- added R17: 1M, Resistor_SMD:R_0603_1608Metric_Pad0.98x0.95mm_HandSolder, symbol Device:R_Small
- added R18, R21: 1K, Resistor_SMD:R_0603_1608Metric_Pad0.98x0.95mm_HandSolder, symbol Device:R_Small
- added RV1: 1M, Potentiometer_THT:Potentiometer_Vishay_T73YP_Vertical, symbol Device:R_Potentiometer_US
- added RV2: 500K, Potentiometer_THT:Potentiometer_Vishay_T73YP_Vertical, symbol Device:R_Potentiometer_US
- added RV3: 100K, Potentiometer_THT:Potentiometer_Vishay_T73YP_Vertical, symbol Device:R_Potentiometer_US
Connections:
- net +5V: now also R17.1, R18.1, R21.1
- net A11-ZP07-A: now also J6.29 (Pin_29); no longer J7.5 (Pin_5)
- net A12-ZP07-B: now also J6.27 (Pin_27); no longer J7.4 (Pin_4)
- net CO: now reaches J12.1 (Pin_1)
- net CO: now also RV1.2, RV1.3
- net NH3: now reaches J12.2 (Pin_2)
- net NH3: now also RV2.2, RV2.3
- net NO2: now reaches J12.3 (Pin_3)
- net NO2: now also RV3.2, RV3.3
- net A14-ZE-03: no longer names the net of J7.2 (Pin_2)
- new net: R21.2, RV3.1
- new net: R18.2, RV2.1
- new net: R17.2, RV1.1
Other:
- note added: "5V"
- note added: "CO"
- note added: "GND"
- note added: "NH3"
- note added: "NO2"
- moved on the sheet: J11, J12

Commit message: Update 18 mar 2026
Parts:
- added D1: SS14, Diode_SMD:D_SMA, symbol Diode:SS14
- added J13: Conn_01x02, Connector_PinHeader_2.54mm:PinHeader_1x02_P2.54mm_Vertical, symbol Connector_Generic:Conn_01x02
- added R30: 1K, Resistor_SMD:R_0603_1608Metric_Pad0.98x0.95mm_HandSolder, symbol Device:R_Small
- added R31: 10K, Resistor_SMD:R_1206_3216Metric, symbol Device:R_Small
Connections:
- net +5V: now also J6.1 (Pin_1), J6.2 (Pin_2), Q1.1, Q1.2, Q1.3, J13.1 (Pin_1), R31.1
- net +5VP: now also Q1.5, Q1.6, Q1.7, Q1.8
- net CO: now also J7.8 (Pin_8)
- net GND: now also J11.2, J11.3, J6.35 (Pin_35), J6.36 (Pin_36)
- net NH3: now also J7.6 (Pin_6)
- net NO2: now also J7.5 (Pin_5)
- net at J11.1: now also D1.2 (A)
- net at Q1.4: now also R30.2, R31.2
- net at J6.25 (Pin_25): now also R30.1
- new net: D1.1 (K), J13.2 (Pin_2)

Commit message: Update 19 mar 2026
Parts:
- removed R17: 1M, Resistor_SMD:R_0603_1608Metric_Pad0.98x0.95mm_HandSolder, symbol Device:R_Small
- removed R18, R21: 1K, Resistor_SMD:R_0603_1608Metric_Pad0.98x0.95mm_HandSolder, symbol Device:R_Small
- removed RV1: 1M, Potentiometer_THT:Potentiometer_Vishay_T73YP_Vertical, symbol Device:R_Potentiometer_US
- removed RV2: 500K, Potentiometer_THT:Potentiometer_Vishay_T73YP_Vertical, symbol Device:R_Potentiometer_US
- removed RV3: 100K, Potentiometer_THT:Potentiometer_Vishay_T73YP_Vertical, symbol Device:R_Potentiometer_US

Commit message: local update 22 Mar 26
Parts:
- added J14, J15: Conn_01x02, Connector_PinHeader_2.54mm:PinHeader_1x02_P2.54mm_Vertical, symbol Connector_Generic:Conn_01x02
Connections:
- net +5V: now also J15.2 (Pin_2)
- net GND: now also J15.1 (Pin_1)
- net Rx: now reaches J5.1 (Pin_1), U12.6
- net Rx: now also J14.1 (Pin_1)
- net Tx: now reaches J5.2 (Pin_2), U12.5
- net Tx: now also J14.2 (Pin_2)
Other:
- added sheet ADS1115_ADC (ADS1115_ADC.kicad_sch)
- moved on the sheet: C13, R23, U12
