File: uprojects/John Ottolenghi/kicadA/snifferA/snifferA.kicad_pcb (KiCad board)
At the start: 2 copper layers, 1 part, among them U1 MQ-X

Commit message: Update 29 Jan 2026
Parts:
- added A1: ARDUINO_MEGA_2560_REV3_A000067, ARDUINO_MEGA_2560_REV3_A000067:ARDUINO_ARDUINO_MEGA_2560_REV3_A000067, B.Cu at (156.0, 106.5)
- added J1: DHT22, Connector_PinSocket_2.54mm:PinSocket_1x04_P2.54mm_Vertical, F.Cu at (121.9, 171.0)
- added J2: Conn_01x10, Connector_PinHeader_2.54mm:PinHeader_1x10_P2.54mm_Vertical, F.Cu at (126.5, 74.6)
- added J3: Conn_01x08, Connector_PinHeader_2.54mm:PinHeader_1x08_P2.54mm_Vertical, F.Cu at (142.7, 171.0)
- added U2: MQ-135, MQ-X:MQ, F.Cu at (107.5, 48.0)
- added U3: MQ-136, MQ-X:MQ, F.Cu at (201.8, 48.5)
- added U4: MQ-137, MQ-X:MQ, F.Cu at (106.5, 154.0)
- added U5: MQ-02, MQ-X:MQ, F.Cu at (106.6, 128.9)
- added U6: MQ-04, MQ-X:MQ, F.Cu at (106.6, 101.4)
- added U7: MQ-06, MQ-X:MQ, F.Cu at (202.0, 74.5)
- added U8: MQ-08, MQ-X:MQ, F.Cu at (202.2, 101.5)
- U1: value MQ-X -> MQ-131

Commit message: Update 30 Jan 2026
Parts:
- moved A1 53.4 mm to (103.0, 100.0)
- moved J1 53.4 mm to (68.9, 164.5)
- moved J2 53.4 mm to (73.5, 68.1)
- moved J3 53.4 mm to (89.7, 164.5)
- moved U1 53.4 mm to (53.6, 68.1)
- moved U2 53.4 mm to (54.5, 41.5)
- moved U3 53.4 mm to (148.8, 42.0)
- moved U4 53.4 mm to (53.5, 147.5)
- moved U5 53.4 mm to (53.6, 122.4)
- moved U6 53.4 mm to (53.6, 94.9)
- moved U7 53.4 mm to (149.0, 68.0)
- moved U8 53.4 mm to (149.2, 95.0)
Other:
- board outline added: 139 x 174 mm
Changed lines of the file:
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@@
 	(footprint "MQ-X:MQ"
 		(layer "F.Cu")
-		(at 106.641243 101.358757)
+		(at 53.641243 94.858757)
 		(property "Reference" "U6"
 			(at 0 -9.5 0)
@@
 	(footprint "MQ-X:MQ"
 		(layer "F.Cu")
-		(at 106.641243 74.641243)
+		(at 53.641243 68.141243)
 		(property "Reference" "U1"
 			(at 0 -9.5 0)
@@
 	(footprint "Connector_PinHeader_2.54mm:PinHeader_1x08_P2.54mm_Vertical"
 		(layer "F.Cu")
-		(at 142.72 171 90)
+		(at 89.72 164.5 90)
 		(descr "Through hole straight pin header, 1x08, 2.54mm pitch, single row")
 		(tags "Through hole pin header THT 1x08 2.54mm single row")
@@
 	(footprint "Connector_PinSocket_2.54mm:PinSocket_1x04_P2.54mm_Vertical"
 		(layer "F.Cu")
-		(at 121.92 171 90)
+		(at 68.92 164.5 90)
 		(descr "Through hole straight socket strip, 1x04, 2.54mm pitch, single row (from Kicad 4.0.7), script generated")
 		(tags "Through hole socket strip THT 1x04 2.54mm single row")
@@
 	(footprint "MQ-X:MQ"
 		(layer "F.Cu")
-		(at 106.641243 128.858757)
+		(at 53.641243 122.358757)
 		(property "Reference" "U5"
 			(at 0 -9.5 0)
@@
 	(footprint "MQ-X:MQ"
 		(layer "F.Cu")
-		(at 107.5 48)
+		(at 54.5 41.5)
 		(property "Reference" "U2"
 			(at 0 -9.5 0)
@@
 	(footprint "MQ-X:MQ"
 		(layer "F.Cu")
-		(at 106.5 154)
+		(at 53.5 147.5)
 		(property "Reference" "U4"
 			(at 0 -9.5 0)
@@
 	(footprint "MQ-X:MQ"
 		(layer "F.Cu")
-		(at 202.25 101.5)
+		(at 149.25 95)
 		(property "Reference" "U8"
 			(at 0 -9.5 0)
@@
 	(footprint "MQ-X:MQ"
 		(layer "F.Cu")
-		(at 202 74.5)
+		(at 149 68)
 		(property "Reference" "U7"
 			(at 0 -9.5 0)
@@
 	(footprint "Connector_PinHeader_2.54mm:PinHeader_1x10_P2.54mm_Vertical"
 		(layer "F.Cu")
-		(at 126.5 74.64)
+		(at 73.5 68.14)
 		(descr "Through hole straight pin header, 1x10, 2.54mm pitch, single row")
 		(tags "Through hole pin header THT 1x10 2.54mm single row")
@@
 	(footprint "MQ-X:MQ"
 		(layer "F.Cu")
-		(at 201.75 48.5)
+		(at 148.75 42)
 		(property "Reference" "U3"
 			(at 0 -9.5 0)
@@
 	(footprint "ARDUINO_MEGA_2560_REV3_A000067:ARDUINO_ARDUINO_MEGA_2560_REV3_A000067"
 		(layer "B.Cu")
-		(at 156 106.5 180)
+		(at 103 100 180)
 		(property "Reference" "A1"
 			(at -23.525 53.945 0)
@@
 			)
 		)
+	)
+	(gr_line
+		(start 178.5 196)
+		(end 39.5 196)
+		(stroke
+			(width 0.05)
+			(type default)
+		)
+		(layer "Edge.Cuts")
+	)
+	(gr_line
+		(start 39.5 22)
+		(end 162 22)
+		(stroke
+			(width 0.05)
+			(type default)
+		)
+		(layer "Edge.Cuts")
+	)
+	(gr_line
+		(start 162 22)
+		(end 162 196)
+		(stroke
+			(width 0.05)
+			(type default)
+		)
+		(layer "Edge.Cuts")
+	)
+	(gr_line
+		(start 39.5 196)
+		(end 39.5 22)
+		(stroke
+			(width 0.05)
+			(type default)
+		)
+		(layer "Edge.Cuts")
+	)
+	(dimension
+		(type orthogonal)
+		(layer "F.SilkS")
+		(pts
+			(xy 39.5 22) (xy 162 22)
+		)
+		(height 5)
+		(orientation 0)
+		(format
+			(prefix "")
+			(suffix "")
+			(units 3)
+			(units_format 0)
+			(precision 4)
+			(suppress_zeroes yes)
+		)
+		(style
+			(thickness 0.1)
+			(arrow_length 1.27)
+			(text_position_mode 0)
+			(arrow_direction outward)
+			(extension_height 0.58642)
+			(extension_offset 0.5)
+			(keep_text_aligned yes)
+		)
+		(gr_text "122.5"
+			(at 100.75 25.9 0)
+			(layer "F.SilkS")
+			(effects
+				(font
+					(size 1 1)
+					(thickness 0.1)
+				)
+			)
+		)
+	)
+	(dimension
+		(type orthogonal)
+		(layer "F.SilkS")
+		(pts
+			(xy 162 22) (xy 162 196)
+		)
+		(height -25)
+		(orientation 1)
+		(format
+			(prefix "")
+			(suffix "")
+			(units 3)
+			(units_format 0)
+			(precision 4)
+			(suppress_zeroes yes)
+		)
+		(style
+			(thickness 0.1)
+			(arrow_length 1.27)
+			(text_position_mode 0)
+			(arrow_direction outward)
+			(extension_height 0.58642)
+			(extension_offset 0.5)
+			(keep_text_aligned yes)
+		)
+		(gr_text "174"
+			(at 135.9 109 90)
+			(layer "F.SilkS")
+			(effects
+				(font
+					(size 1 1)
+					(thickness 0.1)
+				)
+			)
+		)

Commit message: update 02-Feb-2026
Parts:
- added U9: YAAJ_DCDC_StepDown_LM2596, KiCad:YAAJ_DCDC_StepDown_LM2596, F.Cu at (82.4, 173.2)

Commit message: Update 10 Feb 2026
Parts:
- added J4: Conn_01x08, Connector_PinHeader_2.54mm:PinHeader_1x08_P2.54mm_Vertical, F.Cu at (73.5, 95.0)
- added J5: Conn_01x08, Connector_PinHeader_2.54mm:PinHeader_1x08_P2.54mm_Vertical, F.Cu at (73.5, 117.7)
- added J6: Conn_02x18_Odd_Even, Connector_PinHeader_2.54mm:PinHeader_2x18_P2.54mm_Vertical, F.Cu at (78.8, 156.5)
- added J7: Conn_01x08, Connector_PinHeader_2.54mm:PinHeader_1x08_P2.54mm_Vertical, F.Cu at (132.0, 140.8)
- added J8: Conn_01x08, Connector_PinHeader_2.54mm:PinHeader_1x08_P2.54mm_Vertical, F.Cu at (132.0, 117.8)
- added J9: Conn_01x08, Connector_PinHeader_2.54mm:PinHeader_1x08_P2.54mm_Vertical, F.Cu at (132.0, 94.8)
- added U10: MQ-131-L, MQ-X:MQ, F.Cu at (149.6, 122.6)
- U1: value MQ-131 -> MQ-131-H
- moved J2 0.14 mm to (73.5, 68.0)

Commit message: Update 11 Feb 2026
Parts:
- added U11: ~, sensors:SM4-NO2-20, F.Cu at (150.5, 148.0)
- added U12: ZE08-CH20, sensors:ZE-08, F.Cu at (147.5, 191.2)
- J3: value Conn_01x08 -> CCS811_CJMCU
- moved J3 42.3 mm to (53.6, 186.5)

Commit message: Update 24 Feb 2026
Parts:
- added C1: 0.1uF, Capacitor_SMD:C_1206_3216Metric_Pad1.33x1.80mm_HandSolder, F.Cu at (110.1, 67.1)
- added C2: 0.1uF, Capacitor_SMD:C_1206_3216Metric_Pad1.33x1.80mm_HandSolder, F.Cu at (110.0, 74.6)
- added J10: ZP07, Connector_PinSocket_2.54mm:PinSocket_1x04_P2.54mm_Vertical, F.Cu at (96.7, 169.9)
- added R1: 10k, Resistor_SMD:R_1206_3216Metric, F.Cu at (110.0, 64.4)
- added R2: 10K, Resistor_SMD:R_1206_3216Metric, F.Cu at (69.1, 32.8)
- added R3: 10K, Resistor_SMD:R_1206_3216Metric, F.Cu at (69.2, 57.9)
- added R4: 10k, Resistor_SMD:R_1206_3216Metric, F.Cu at (110.0, 71.9)
- added U13: ZP07, sensors:ZP07-FRAME, F.Cu at (97.9, 168.6)
- added U14: SM4-NO2-20, sensors:SM4-NO2-20, F.Cu at (77.6, 147.9)
- added U15: MQ-07, MQ-X:MQ, F.Cu at (100.4, 148.5)
- U11: value ~ -> ZE-03
- moved U10 129.0 mm to (55.4, 34.6)
- moved U9 53.9 mm to (131.0, 149.9), turned to -90 degrees
- moved U2 43.9 mm to (56.9, 85.4)
- moved J6 35.7 mm to (78.3, 120.8)
- moved J7 25.7 mm to (126.5, 115.7)
- moved J8 25.6 mm to (126.5, 92.8)
- moved J4 25.5 mm to (78.3, 69.9)
- moved J9 25.4 mm to (126.5, 70.0)
- moved J2 25.4 mm to (78.3, 43.1)
- moved J5 25.3 mm to (78.3, 92.9)
- moved A1 24.9 mm to (102.4, 75.1)
- moved U6 23.5 mm to (30.2, 92.8)
- moved J3 19.3 mm to (63.3, 169.8), turned to -90 degrees
- moved U1 8.57 mm to (55.4, 59.8)
- moved J1 5.65 mm to (71.3, 169.6)
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Connections:
- J8 pad 7: unconnected-(J8-Pin_7-Pad7) -> Net-(J8-Pin_7)
- J8 pad 8: unconnected-(J8-Pin_8-Pad8) -> Net-(J8-Pin_8)
- U1 pad 1: unconnected-(U1-A-Pad1) -> +5VP
- U1 pad 2: unconnected-(U1-H-Pad2) -> +5V
- U1 pad 3: unconnected-(U1-A-Pad3) -> +5VP
- U1 pad 4: unconnected-(U1-B-Pad4) -> GND
- U1 pad 5: unconnected-(U1-H-Pad5) -> Net-(R3-Pad1)
- U1 pad 6: unconnected-(U1-B-Pad6) -> GND
- U10 pad 1: unconnected-(U10-A-Pad1) -> +5VP
- U10 pad 2: unconnected-(U10-H-Pad2) -> +5V
- U10 pad 3: unconnected-(U10-A-Pad3) -> +5VP
- U10 pad 4: unconnected-(U10-B-Pad4) -> GND
- U10 pad 5: unconnected-(U10-H-Pad5) -> Net-(R1-Pad1)
- U10 pad 6: unconnected-(U10-B-Pad6) -> GND
- U2 pad 1: unconnected-(U2-A-Pad1) -> +5VP
- U2 pad 2: unconnected-(U2-H-Pad2) -> +5V
- U2 pad 3: unconnected-(U2-A-Pad3) -> +5VP
- U9 pad 4: unconnected-(U9-Vout-Pad4) -> +5V

Commit message: Update 26 Feb 2026
Parts:
- added C10: 0.1uF, Capacitor_SMD:C_1206_3216Metric_Pad1.33x1.80mm_HandSolder, F.Cu at (107.1, 101.9)
- added C3: 0.1uF, Capacitor_SMD:C_1206_3216Metric_Pad1.33x1.80mm_HandSolder, F.Cu at (107.4, 62.8)
- added C4: 0.1uF, Capacitor_SMD:C_1206_3216Metric_Pad1.33x1.80mm_HandSolder, F.Cu at (107.4, 68.9)
- added C5: 0.1uF, Capacitor_SMD:C_1206_3216Metric_Pad1.33x1.80mm_HandSolder, F.Cu at (107.4, 74.6)
- added C6: 0.1uF, Capacitor_SMD:C_1206_3216Metric_Pad1.33x1.80mm_HandSolder, F.Cu at (107.2, 80.4)
- added C7: 0.1uF, Capacitor_SMD:C_1206_3216Metric_Pad1.33x1.80mm_HandSolder, F.Cu at (107.0, 89.4)
- added C8: 0.1uF, Capacitor_SMD:C_1206_3216Metric_Pad1.33x1.80mm_HandSolder, F.Cu at (107.1, 92.5)
- added C9: 0.1uF, Capacitor_SMD:C_1206_3216Metric_Pad1.33x1.80mm_HandSolder, F.Cu at (107.1, 98.8)
- added R10: 10k, Resistor_SMD:R_1206_3216Metric, F.Cu at (107.4, 71.8)
- added R11: 10K, Resistor_SMD:R_1206_3216Metric, F.Cu at (61.5, 150.1)
- added R12: 10k, Resistor_SMD:R_1206_3216Metric, F.Cu at (107.2, 77.6)
- added R13: 10K, Resistor_SMD:R_1206_3216Metric, F.Cu at (78.9, 152.5)
- added R14: 10k, Resistor_SMD:R_1206_3216Metric, F.Cu at (107.1, 86.6)
- added R15: 10K, Resistor_SMD:R_1206_3216Metric, F.Cu at (157.8, 82.2)
- added R16: 10k, Resistor_SMD:R_1206_3216Metric, F.Cu at (107.1, 83.6)
- added R17: 10K, Resistor_SMD:R_1206_3216Metric, F.Cu at (85.6, 136.5)
- added R18: 10k, Resistor_SMD:R_1206_3216Metric, F.Cu at (107.1, 95.6)
- added R19: 10K, Resistor_SMD:R_1206_3216Metric, F.Cu at (158.0, 106.6)
- added R20: 10k, Resistor_SMD:R_1206_3216Metric, F.Cu at (107.1, 105.0)
- added R5: 10K, Resistor_SMD:R_1206_3216Metric, F.Cu at (66.0, 82.9)
- added R6: 10k, Resistor_SMD:R_1206_3216Metric, F.Cu at (107.4, 59.9)
- added R7: 10K, Resistor_SMD:R_1206_3216Metric, F.Cu at (66.0, 108.1)
- added R8: 10k, Resistor_SMD:R_1206_3216Metric, F.Cu at (107.5, 65.9)
- added R9: 10K, Resistor_SMD:R_1206_3216Metric, F.Cu at (59.5, 124.5)
- moved U3 118.2 mm to (52.0, 110.0)
- moved U11 110.4 mm to (148.6, 37.5), turned to 180 degrees
- moved U14 108.3 mm to (148.6, 66.1)
- moved U6 82.8 mm to (72.9, 163.8)
- moved U12 72.6 mm to (85.1, 154.1), turned to -90 degrees
- moved U5 37.8 mm to (52.0, 160.1)
- moved U15 29.0 mm to (73.0, 139.0)
- moved U7 24.3 mm to (148.9, 92.2)
- moved U9 23.0 mm to (115.8, 132.7), turned to 0 degrees
- moved U8 21.4 mm to (149.1, 116.4)
- moved C1 19.6 mm to (107.5, 47.8)
- moved C2 19.6 mm to (107.4, 55.2)
- moved R1 19.6 mm to (107.4, 45.0)
- moved R4 19.6 mm to (107.4, 52.5)
- moved U4 12.5 mm to (52.0, 135.1)
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Connections:
- J2 pad 7: unconnected-(J2-Pin_7-Pad7) -> GND
- J7 pad 7: unconnected-(J7-Pin_7-Pad7) -> Net-(J7-Pin_7)
- J7 pad 8: unconnected-(J7-Pin_8-Pad8) -> Net-(J7-Pin_8)
- J8 pad 1: unconnected-(J8-Pin_1-Pad1) -> Net-(J8-Pin_1)
- J8 pad 2: unconnected-(J8-Pin_2-Pad2) -> Net-(J8-Pin_2)
- J8 pad 3: unconnected-(J8-Pin_3-Pad3) -> Net-(J8-Pin_3)
- J8 pad 4: unconnected-(J8-Pin_4-Pad4) -> Net-(J8-Pin_4)
- J8 pad 5: unconnected-(J8-Pin_5-Pad5) -> Net-(J8-Pin_5)
- J8 pad 6: unconnected-(J8-Pin_6-Pad6) -> Net-(J8-Pin_6)
- U15 pad 1: unconnected-(U15-A-Pad1) -> +5VP
- U15 pad 2: unconnected-(U15-H-Pad2) -> +5V
- U15 pad 3: unconnected-(U15-A-Pad3) -> +5VP
- U15 pad 4: unconnected-(U15-B-Pad4) -> GND
- U15 pad 5: unconnected-(U15-H-Pad5) -> Net-(R17-Pad1)
- U15 pad 6: unconnected-(U15-B-Pad6) -> GND
- U2 pad 4: unconnected-(U2-B-Pad4) -> GND
- U2 pad 5: unconnected-(U2-H-Pad5) -> Net-(R5-Pad1)
- U2 pad 6: unconnected-(U2-B-Pad6) -> GND
- U3 pad 1: unconnected-(U3-A-Pad1) -> +5VP
- U3 pad 2: unconnected-(U3-H-Pad2) -> +5V
- U3 pad 3: unconnected-(U3-A-Pad3) -> +5VP
- U3 pad 4: unconnected-(U3-B-Pad4) -> GND
- U3 pad 5: unconnected-(U3-H-Pad5) -> Net-(R7-Pad1)
- U3 pad 6: unconnected-(U3-B-Pad6) -> GND
- U4 pad 1: unconnected-(U4-A-Pad1) -> +5VP
- U4 pad 2: unconnected-(U4-H-Pad2) -> +5V
- U4 pad 3: unconnected-(U4-A-Pad3) -> +5VP
- U4 pad 4: unconnected-(U4-B-Pad4) -> GND
- U4 pad 5: unconnected-(U4-H-Pad5) -> Net-(R10-Pad1)
- U4 pad 6: unconnected-(U4-B-Pad6) -> GND
- U5 pad 1: unconnected-(U5-A-Pad1) -> +5VP
- U5 pad 2: unconnected-(U5-H-Pad2) -> +5V
- U5 pad 3: unconnected-(U5-A-Pad3) -> +5VP
- U5 pad 4: unconnected-(U5-B-Pad4) -> GND
- U5 pad 5: unconnected-(U5-H-Pad5) -> Net-(R11-Pad1)
- U5 pad 6: unconnected-(U5-B-Pad6) -> GND
- U6 pad 1: unconnected-(U6-A-Pad1) -> +5VP
- U6 pad 2: unconnected-(U6-H-Pad2) -> +5V
- U6 pad 3: unconnected-(U6-A-Pad3) -> +5VP
- U6 pad 4: unconnected-(U6-B-Pad4) -> GND
- U6 pad 5: unconnected-(U6-H-Pad5) -> Net-(R13-Pad1)
- U6 pad 6: unconnected-(U6-B-Pad6) -> GND
- U7 pad 1: unconnected-(U7-A-Pad1) -> +5VP
- U7 pad 2: unconnected-(U7-H-Pad2) -> +5V
- U7 pad 3: unconnected-(U7-A-Pad3) -> +5VP
- U7 pad 4: unconnected-(U7-B-Pad4) -> GND
- U7 pad 5: unconnected-(U7-H-Pad5) -> Net-(R15-Pad1)
- U7 pad 6: unconnected-(U7-B-Pad6) -> GND
- U8 pad 1: unconnected-(U8-A-Pad1) -> +5VP
- U8 pad 2: unconnected-(U8-H-Pad2) -> +5V
- U8 pad 3: unconnected-(U8-A-Pad3) -> +5VP
- U8 pad 4: unconnected-(U8-B-Pad4) -> GND
- U8 pad 5: unconnected-(U8-H-Pad5) -> Net-(R19-Pad1)
- U8 pad 6: unconnected-(U8-B-Pad6) -> GND
Other:
- board size 139 x 174 mm -> 122.5 x 174 mm

Commit message: Update 26 Feb 2026
Parts:
- added C11: 0.1uF, Capacitor_SMD:C_1206_3216Metric_Pad1.33x1.80mm_HandSolder, F.Cu at (135.5, 28.8)
- added C12: 0.1uF, Capacitor_SMD:C_1206_3216Metric_Pad1.33x1.80mm_HandSolder, F.Cu at (135.1, 54.4)
- added C13: 0.1uF, Capacitor_SMD:C_1206_3216Metric_Pad1.33x1.80mm_HandSolder, F.Cu at (94.6, 155.5)
- added J11: DCJ200-10-A-XX-K_REVA, DCJ200-10-A-XX-K_REVA:GCT_DCJ200-10-A-XX-K_REVA, F.Cu at (118.5, 188.0)
- added R21: 10k, Resistor_SMD:R_1206_3216Metric, F.Cu at (135.5, 25.2)
- added R22: 10k, Resistor_SMD:R_1206_3216Metric, F.Cu at (135.1, 50.8)
- added R23: 10k, Resistor_SMD:R_1206_3216Metric, F.Cu at (94.6, 158.5)
- added U16: YAAJ_DCDC_StepDown_LM2596, KiCad:YAAJ_DCDC_StepDown_LM2596, F.Cu at (115.7, 158.1)
- turned U11 to 0 degrees
Connections:
- J10 pad 1: unconnected-(J10-Pin_1-Pad1) -> /A12-ZP07-B
- J10 pad 2: unconnected-(J10-Pin_2-Pad2) -> /A11-ZP07-A
- J10 pad 3: unconnected-(J10-Pin_3-Pad3) -> +5V
- J10 pad 4: unconnected-(J10-Pin_4-Pad4) -> GND
- J3 pad 1: unconnected-(J3-Pin_1-Pad1) -> +5V
- J3 pad 2: unconnected-(J3-Pin_2-Pad2) -> GND
- J5 pad 1: unconnected-(J5-Pin_1-Pad1) -> Net-(J5-Pin_1)
- J5 pad 2: unconnected-(J5-Pin_2-Pad2) -> Net-(J5-Pin_2)
- J5 pad 3: unconnected-(J5-Pin_3-Pad3) -> Net-(J5-Pin_3)
- J5 pad 4: unconnected-(J5-Pin_4-Pad4) -> Net-(J5-Pin_4)
- J5 pad 5: unconnected-(J5-Pin_5-Pad5) -> Net-(J5-Pin_5)
- J5 pad 6: unconnected-(J5-Pin_6-Pad6) -> Net-(J5-Pin_6)
- J7 pad 1: unconnected-(J7-Pin_1-Pad1) -> /A15-SM4-N02
- J7 pad 2: unconnected-(J7-Pin_2-Pad2) -> /A14-ZE-03
- J7 pad 3: unconnected-(J7-Pin_3-Pad3) -> /A13-ZE08-CH20
- J7 pad 4: unconnected-(J7-Pin_4-Pad4) -> /A12-ZP07-A
- J7 pad 5: unconnected-(J7-Pin_5-Pad5) -> /A11-ZP07-A
- U11 pad 1: unconnected-(U11-Pad1) -> Net-(J5-Pin_5)
- U11 pad 2: unconnected-(U11-Pad2) -> Net-(J5-Pin_6)
- U11 pad 3: unconnected-(U11-Pad3) -> Net-(R21-Pad1)
- U11 pad 4: unconnected-(U11-Pad4) -> +5V
- U11 pad 5: unconnected-(U11-Pad5) -> GND
- U12 pad 2: unconnected-(U12-Pad2) -> Net-(R23-Pad1)
- U12 pad 3: unconnected-(U12-Pad3) -> GND
- U12 pad 4: unconnected-(U12-Pad4) -> +5V
- U12 pad 5: unconnected-(U12-Pad5) -> Net-(J5-Pin_2)
- U12 pad 6: unconnected-(U12-Pad6) -> Net-(J5-Pin_1)
- U14 pad 1: unconnected-(U14-Pad1) -> Net-(J5-Pin_3)
- U14 pad 2: unconnected-(U14-Pad2) -> Net-(J5-Pin_4)
- U14 pad 3: unconnected-(U14-Pad3) -> Net-(R22-Pad1)
- U14 pad 4: unconnected-(U14-Pad4) -> +5V
- U14 pad 5: unconnected-(U14-Pad5) -> GND
- U9 pad 1: unconnected-(U9-Vin-Pad1) -> Net-(U16-Vin)
- U9 pad 2: unconnected-(U9-GND-Pad2) -> GND
- U9 pad 3: unconnected-(U9-GND-Pad3) -> GND
