File: uprojects/John Ottolenghi/kicadA/snifferA/snifferA.kicad_pcb (KiCad board)
At the start: 2 copper layers, 122.5 x 174 mm, 64 parts, among them J1 DHT22, J10 ZP07, J11 DCJ200-10-A-XX-K_REVA, J2 Conn_01x10, J3 CCS811_CJMCU, J4 Conn_01x08, J5 Conn_01x08, J6 Conn_02x18_Odd_Even, J7 Conn_01x08, J8 Conn_01x08, J9 Conn_01x08, U1 MQ-131-H, U10 MQ-131-L, U11 ZE-03, U12 ZE08-CH20, U13 ZP07, U14 SM4-NO2-20, U15 MQ-07, U16 YAAJ_DCDC_StepDown_LM2596, U2 MQ-135, U3 MQ-136, U4 MQ-137, U5 MQ-02, U6 MQ-04, U7 MQ-06, U8 MQ-08, U9 YAAJ_DCDC_StepDown_LM2596

Commit message: local update 2 Mar 26
Connections:
- J7 pad 4: /A12-ZP07-A -> /A12-ZP07-B
Routing:
- net Net-(R10-Pad1): track 0.00 -> 172.2 mm
- net Net-(R7-Pad1): track 0.00 -> 149.8 mm
- net Net-(R5-Pad1): track 0.00 -> 124.1 mm
- net Net-(R11-Pad1): track 0.00 -> 116.2 mm
- net /A14-ZE-03: track 0.00 -> 95.3 mm, vias 0 -> 2
- net Net-(R3-Pad1): track 0.00 -> 94.8 mm
- net Net-(R13-Pad1): track 0.00 -> 92.1 mm
- net /A11-ZP07-A: track 0.00 -> 84.7 mm
- net /A12-ZP07-B: track 0.00 -> 82.1 mm
- net Net-(R15-Pad1): track 0.00 -> 74.5 mm, vias 0 -> 2
- net Net-(R1-Pad1): track 0.00 -> 63.8 mm
- net Net-(R19-Pad1): track 0.00 -> 59.3 mm
- net Net-(J5-Pin_3): track 0.00 -> 55.5 mm
- net GND: track 0.00 -> 45.7 mm, vias 0 -> 2
- net Net-(J8-Pin_8): track 0.00 -> 43.6 mm, vias 0 -> 2
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
Commit message: Update 3 mar 2026
Parts:
- removed A1: ARDUINO_MEGA_2560_REV3_A000067, ARDUINO_MEGA_2560_REV3_A000067:ARDUINO_ARDUINO_MEGA_2560_REV3_A000067
- moved R11 4.73 mm to (57.8, 147.2)
Connections:
- J1 pad 1: unconnected-(J1-Pin_1-Pad1) -> +5V
- J1 pad 2: unconnected-(J1-Pin_2-Pad2) -> /DHT22_DATA
- J1 pad 4: unconnected-(J1-Pin_4-Pad4) -> GND
- J3 pad 3: unconnected-(J3-Pin_3-Pad3) -> /SCL
- J3 pad 4: unconnected-(J3-Pin_4-Pad4) -> /SDA
- J3 pad 5: unconnected-(J3-Pin_5-Pad5) -> /WAK
- J3 pad 6: unconnected-(J3-Pin_6-Pad6) -> /INT
- J3 pad 7: unconnected-(J3-Pin_7-Pad7) -> /RST
- J3 pad 8: unconnected-(J3-Pin_8-Pad8) -> /ADD
- J5 pad 7: unconnected-(J5-Pin_7-Pad7) -> /SDA
- J5 pad 8: unconnected-(J5-Pin_8-Pad8) -> /SCL
- J6 pad 15: unconnected-(J6-Pin_15-Pad15) -> /DHT22_DATA
- J6 pad 3: unconnected-(J6-Pin_3-Pad3) -> /ADD
- J6 pad 5: unconnected-(J6-Pin_5-Pad5) -> /RST
- J6 pad 7: unconnected-(J6-Pin_7-Pad7) -> /INT
- J6 pad 9: unconnected-(J6-Pin_9-Pad9) -> /WAK
Routing:
- net +5VP: track 0.00 -> 376.7 mm, vias 0 -> 1
- net Net-(J5-Pin_6): track 0.00 -> 144.3 mm, vias 0 -> 1
- net Net-(J5-Pin_5): track 0.00 -> 140.5 mm, vias 0 -> 3
- net Net-(J5-Pin_4): track 30.2 -> 123.8 mm, vias 0 -> 2
- net Net-(J5-Pin_2): track 0.00 -> 86.7 mm, vias 0 -> 2
- net /SDA: track 0.00 -> 83.8 mm
- net /RST: track 0.00 -> 83.7 mm, vias 0 -> 1
- net /INT: track 0.00 -> 82.8 mm, vias 0 -> 1
- net /DHT22_DATA: track 0.00 -> 82.0 mm
- net /WAK: track 0.00 -> 81.9 mm, vias 0 -> 1
- net /ADD: track 0.00 -> 81.6 mm, vias 0 -> 1
- net /SCL: track 0.00 -> 80.1 mm
- net Net-(J5-Pin_1): track 0.00 -> 67.3 mm, vias 0 -> 2
- net Net-(U16-Vin): track 0.00 -> 67.0 mm
- net /A15-SM4-N02: track 3.67 -> 70.3 mm, vias 0 -> 1
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- added copper zone on B.Cu, net +5V
- added copper zone on F.Cu, net GND

Commit message: Update 4 mar 2026
Routing:
- net Net-(J8-Pin_1): track 18.0 -> 40.8 mm, vias 0 -> 2
- net GND: track 30.8 -> 48.7 mm, vias 2 -> 9
- net Net-(J5-Pin_1): track 67.3 -> 69.6 mm
- net +5V: vias 0 -> 1

Commit message: Update 9 mar 2026
Parts:
- added R24: 4K7, Resistor_SMD:R_0603_1608Metric, F.Cu at (82.8, 110.6)
- added R25: 4K7, Resistor_SMD:R_0603_1608Metric, F.Cu at (82.8, 108.1)
- added R26: 4K7, Resistor_SMD:R_0603_1608Metric, F.Cu at (86.2, 126.0)
- added R27: 4K7, Resistor_SMD:R_0603_1608Metric, F.Cu at (88.7, 126.0)
- added R28: 4K7, Resistor_SMD:R_0603_1608Metric, F.Cu at (91.2, 126.0)
- added R29: 4K7, Resistor_SMD:R_0603_1608Metric, F.Cu at (93.8, 126.0)
