File: uprojects/John Ottolenghi/kicadA/snifferA/snifferA.kicad_pcb (KiCad board)
At the start: 2 copper layers, 122.5 x 174 mm, 66 parts, among them J1 DHT22, J10 ZP07, J11 DCJ200-10-A-XX-K_REVA, J2 Conn_01x10, J3 CCS811_CJMCU, J4 Conn_01x08, J5 Conn_01x08, J6 Conn_02x18_Odd_Even, J7 Conn_01x08, J8 Conn_01x08, J9 Conn_01x08, U1 MQ-131-H, U10 MQ-131-L, U12 ZE08-CH20, U13 ZP07, U14 SM4-NO2-20, U15 MQ-07, U16 YAAJ_DCDC_StepDown_LM2596, U2 MQ-135, U3 MQ-136, U4 MQ-137, U5 MQ-02, U6 MQ-04, U7 MQ-06, U8 MQ-08, U9 YAAJ_DCDC_StepDown_LM2596

Commit message: Update 12 mar 2026
Parts:
- removed U16, U9: YAAJ_DCDC_StepDown_LM2596, KiCad:YAAJ_DCDC_StepDown_LM2596
- added Q1: SI4403DDY-T1-GE3, MOSFET-P-20V:SO-8_MS-012_VIS, F.Cu at (141.9, 186.1)
- moved R29 8.88 mm to (84.9, 126.0)
- moved R26 5.03 mm to (91.2, 126.0)
- moved R28 4.24 mm to (87.0, 126.0)
- moved R27 0.39 mm to (89.1, 126.0)
Connections:
- J11 pad 1: Net-(U16-Vin) -> unconnected-(J11-Pad1)
- J11 pad 2: GND -> unconnected-(J11-Pad2)
- J11 pad 3: GND -> unconnected-(J11-Pad3)
- J3 pad 1: +5V -> +3.3V
- J9 pad 5: unconnected-(J9-Pin_5-Pad5) -> +3.3V
- R24 pad 1: +5V -> +3.3V
- R25 pad 1: +5V -> +3.3V
- R26 pad 1: +5V -> +3.3V
- R27 pad 1: +5V -> +3.3V
- R28 pad 1: +5V -> +3.3V
- R29 pad 1: +5V -> +3.3V
Routing:
- net +5VP: track 376.7 -> 279.2 mm
- net unconnected-(J11-Pad1): track 0.00 -> 67.0 mm
- net Net-(U16-Vin): track 67.0 -> 0.00 mm
- net +3.3V: track 0.00 -> 16.6 mm, vias 0 -> 2
- net /ADD: track 81.6 -> 89.1 mm
- net /RST: track 83.7 -> 90.6 mm
- net /INT: track 82.8 -> 89.6 mm
- net /WAK: track 81.9 -> 88.1 mm

Commit message: Update 13 mar 2026
Parts:
- removed U15: MQ-07, MQ-X:MQ
- moved U1 176.0 mm to (157.5, 200.5)
- moved U10 170.0 mm to (145.1, 176.8)
- moved R2 151.4 mm to (135.4, 167.1)
- moved R3 149.0 mm to (135.4, 189.5)
- moved R5 115.9 mm to (28.6, 192.6)
- moved U2 115.2 mm to (43.3, 199.7)
- moved U5 112.9 mm to (164.8, 165.0)
- moved U4 112.8 mm to (164.6, 129.9)
- moved C13 98.8 mm to (160.2, 81.6)
- moved R23 98.8 mm to (160.2, 84.6)
- moved U12 98.8 mm to (150.8, 80.2)
- moved J3 97.1 mm to (138.5, 120.8), turned to 0 degrees
- moved R11 96.0 mm to (153.6, 143.1), turned to -90 degrees
- moved R9 94.5 mm to (153.6, 116.6), turned to 90 degrees
- moved J7 74.8 mm to (130.6, 41.0), turned to -90 degrees
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Routing:
- net +5VP: track 279.2 -> 0.00 mm, vias 1 -> 0
- net Net-(R10-Pad1): track 172.2 -> 0.00 mm
- net Net-(R7-Pad1): track 149.8 -> 0.00 mm
- net Net-(R11-Pad1): track 137.7 -> 0.00 mm, vias 1 -> 0
- net Net-(R5-Pad1): track 124.1 -> 0.00 mm
- net Net-(R3-Pad1): track 94.8 -> 0.00 mm
- net Net-(R13-Pad1): track 92.1 -> 0.00 mm
- net /A11-ZP07-A: track 89.2 -> 0.00 mm
- net Net-(J5-Pin_2): track 86.7 -> 0.00 mm, vias 2 -> 0
- net /A12-ZP07-B: track 85.1 -> 0.00 mm, vias 1 -> 0
- net /SDA: track 87.5 -> 3.68 mm
- net /RST: track 90.6 -> 6.93 mm, vias 1 -> 0
- net /INT: track 89.6 -> 6.77 mm, vias 1 -> 0
- net /DHT22_DATA: track 82.0 -> 0.00 mm
- net /WAK: track 88.1 -> 6.22 mm, vias 1 -> 0
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- removed copper zone on B.Cu, net +5V
- removed copper zone on F.Cu, net GND
Other:
- board size 122.5 x 174 mm -> 165.9 x 191.9 mm

Commit message: local update 14 Mar 26
Parts:
- moved U14 159.0 mm to (34.0, 152.0), turned to 180 degrees
- moved R23 117.3 mm to (43.0, 80.4), turned to 180 degrees
- moved C13 117.3 mm to (43.0, 83.4), turned to 180 degrees
- moved U12 98.4 mm to (52.5, 84.8), turned to 90 degrees
- moved J7 94.1 mm to (69.6, 112.6), turned to 90 degrees
- moved R22 93.8 mm to (50.5, 67.1), turned to 0 degrees
- moved C12 92.9 mm to (50.5, 63.5), turned to 0 degrees
- moved R17 90.5 mm to (145.3, 76.4), turned to 90 degrees
- moved J2 87.8 mm to (142.2, 64.4), turned to -90 degrees
- moved R1 87.0 mm to (140.3, 93.5), turned to -90 degrees
- moved R29 82.5 mm to (59.3, 71.0), turned to 0 degrees
- moved C1 82.0 mm to (137.5, 93.6), turned to -90 degrees
- moved R28 81.9 mm to (59.3, 73.1), turned to 0 degrees
- moved R27 81.6 mm to (59.3, 75.2), turned to 0 degrees
- moved R26 81.6 mm to (59.3, 77.4), turned to 0 degrees
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Routing:
- net +3.3V: track 16.6 -> 7.30 mm, vias 2 -> 1
- net /ADD: track 7.48 -> 5.03 mm
Other:
- board size 165.9 x 191.9 mm -> 166 x 177.5 mm

Commit message: Update 13 mar 2026
Parts:
- removed C9: 0.1uF, Capacitor_SMD:C_1206_3216Metric_Pad1.33x1.80mm_HandSolder
- removed R17: 10K, Resistor_SMD:R_1206_3216Metric
- removed R18: 10k, Resistor_SMD:R_1206_3216Metric
- added J12: MICS-6814, Connector_PinSocket_2.54mm:PinSocket_1x05_P2.54mm_Vertical, F.Cu at (28.8, 195.2)
- moved Q1 87.3 mm to (166.8, 82.1)
- moved U7 31.9 mm to (173.4, 129.2)
- moved R5 30.2 mm to (65.5, 190.0)
- moved U4 23.5 mm to (173.4, 153.2)
- moved U3 18.9 mm to (33.9, 127.1)
- moved R7 17.6 mm to (47.8, 124.6)
- moved U5 12.1 mm to (173.4, 177.0)
- moved R13 6.37 mm to (59.1, 109.7)
- moved U6 6.37 mm to (45.8, 108.5)
- moved U2 6.19 mm to (56.1, 200.6)
Connections:
- J7 pad 8: Net-(J7-Pin_8) -> unconnected-(J7-Pin_8-Pad8)
Routing:
- net unconnected-(J7-Pin_8-Pad8): track 0.00 -> 21.3 mm
- net Net-(J7-Pin_8): track 21.3 -> 0.00 mm
- net Net-(R17-Pad1): track 7.66 -> 0.00 mm, vias 2 -> 0
- net (no net): track 0.00 -> 7.66 mm, vias 0 -> 2
- net /RST: track 6.93 -> 0.00 mm
- net /INT: track 6.77 -> 0.00 mm
- net /WAK: track 6.22 -> 0.00 mm
- net /ADD: track 5.03 -> 0.00 mm
Other:
- board size 166 x 177.5 mm -> 166 x 160.6 mm
- board text added: "5V"
- board text added: "CO"
- board text added: "GND"
- board text added: "NH3"
- board text added: "NO2"

Commit message: Update 17 mar 2026
Parts:
- added R17: 1M, Resistor_SMD:R_0603_1608Metric_Pad0.98x0.95mm_HandSolder, F.Cu at (92.2, 130.1)
- added R18: 1K, Resistor_SMD:R_0603_1608Metric_Pad0.98x0.95mm_HandSolder, F.Cu at (92.2, 132.6)
- added R21: 1K, Resistor_SMD:R_0603_1608Metric_Pad0.98x0.95mm_HandSolder, F.Cu at (92.2, 135.1)
- added RV1: 1M, Potentiometer_THT:Potentiometer_Vishay_T73YP_Vertical, F.Cu at (28.2, 172.7)
- added RV2: 500K, Potentiometer_THT:Potentiometer_Vishay_T73YP_Vertical, F.Cu at (28.2, 180.9)
- added RV3: 100K, Potentiometer_THT:Potentiometer_Vishay_T73YP_Vertical, F.Cu at (28.2, 189.0)
- moved R26 4.29 mm to (57.9, 73.3)
- moved R27 4.29 mm to (57.9, 71.2)
- moved R28 4.29 mm to (57.9, 69.1)
- moved R29 4.29 mm to (57.9, 66.9)
Connections:
- J12 pad 1: unconnected-(J12-Pin_1-Pad1) -> /CO
- J12 pad 2: unconnected-(J12-Pin_2-Pad2) -> /NH3
- J12 pad 3: unconnected-(J12-Pin_3-Pad3) -> /NO2
- J6 pad 27: unconnected-(J6-Pin_27-Pad27) -> /A12-ZP07-B
- J6 pad 29: unconnected-(J6-Pin_29-Pad29) -> /A11-ZP07-A
- J7 pad 2: /A14-ZE-03 -> unconnected-(J7-Pin_2-Pad2)
- J7 pad 4: /A12-ZP07-B -> unconnected-(J7-Pin_4-Pad4)
- J7 pad 5: /A11-ZP07-A -> unconnected-(J7-Pin_5-Pad5)
Routing:
- net /ADD: track 0.00 -> 166.0 mm, vias 0 -> 2
- net /RST: track 0.00 -> 160.3 mm, vias 0 -> 1
- net /INT: track 0.00 -> 152.6 mm, vias 0 -> 1
- net /WAK: track 0.00 -> 145.4 mm, vias 0 -> 1
- net /A12-ZP07-B: track 0.00 -> 142.4 mm
- net /SCL: track 3.69 -> 141.6 mm, vias 0 -> 2
- net /A11-ZP07-A: track 0.00 -> 135.6 mm
- net /SDA: track 3.68 -> 136.2 mm, vias 0 -> 2
- net Net-(J5-Pin_1): track 0.00 -> 51.8 mm
- net Net-(J5-Pin_2): track 0.00 -> 47.2 mm
- net unconnected-(J7-Pin_8-Pad8): track 21.3 -> 0.00 mm
- net Net-(J5-Pin_3): track 53.6 -> 34.9 mm
- net Net-(R23-Pad1): track 0.00 -> 8.81 mm
- net GND: track 0.34 -> 8.17 mm
- net (no net): track 7.66 -> 0.00 mm, vias 2 -> 0
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Other:
- board text added: "3.3V"
- board text added: "ADD"
- board text added: "INT"
- board text added: "RST"
- board text added: "SCL"
- board text added: "SDA"
- board text added: "WAK"

Commit message: Update 18 mar 2026
Parts:
- added D1: SS14, Diode_SMD:D_SMA, F.Cu at (149.2, 191.8)
- added J13: Conn_01x02, Connector_PinHeader_2.54mm:PinHeader_1x02_P2.54mm_Vertical, F.Cu at (154.9, 189.2)
- added R30: 1K, Resistor_SMD:R_0603_1608Metric_Pad0.98x0.95mm_HandSolder, F.Cu at (31.5, 94.0)
- added R31: 10K, Resistor_SMD:R_1206_3216Metric, F.Cu at (27.1, 109.0)
- moved Q1 137.5 mm to (31.0, 103.8)
- moved C12 76.8 mm to (52.5, 140.3)
- moved R22 76.8 mm to (52.5, 143.9)
- moved R17 71.2 mm to (37.7, 175.9), turned to 180 degrees
- moved R18 71.2 mm to (37.7, 178.4), turned to 180 degrees
- moved R21 71.2 mm to (37.7, 180.9), turned to 180 degrees
- moved R11 50.7 mm to (180.8, 189.5)
- moved R2 20.4 mm to (162.6, 166.6)
- moved R9 5.06 mm to (162.1, 111.8), turned to -90 degrees
- moved R5 1.52 mm to (65.5, 191.5)
Connections:
- J11 pad 1: unconnected-(J11-Pad1) -> Net-(D1-A)
- J11 pad 2: unconnected-(J11-Pad2) -> GND
- J11 pad 3: unconnected-(J11-Pad3) -> GND
- J6 pad 1: unconnected-(J6-Pin_1-Pad1) -> +5V
- J6 pad 2: unconnected-(J6-Pin_2-Pad2) -> +5V
- J6 pad 25: unconnected-(J6-Pin_25-Pad25) -> Net-(J6-Pin_25)
- J6 pad 35: unconnected-(J6-Pin_35-Pad35) -> GND
- J6 pad 36: unconnected-(J6-Pin_36-Pad36) -> GND
- J7 pad 5: unconnected-(J7-Pin_5-Pad5) -> /NO2
- J7 pad 6: unconnected-(J7-Pin_6-Pad6) -> /NH3
- J7 pad 8: unconnected-(J7-Pin_8-Pad8) -> /CO
- Q1 pad 1: unconnected-(Q1-Pad1) -> +5V
- Q1 pad 2: unconnected-(Q1-Pad2) -> +5V
- Q1 pad 3: unconnected-(Q1-Pad3) -> +5V
- Q1 pad 4: unconnected-(Q1-Pad4) -> Net-(Q1-Pad4)
- Q1 pad 5: unconnected-(Q1-Pad5) -> +5VP
- Q1 pad 6: unconnected-(Q1-Pad6) -> +5VP
- Q1 pad 7: unconnected-(Q1-Pad7) -> +5VP
- Q1 pad 8: unconnected-(Q1-Pad8) -> +5VP
Routing:
- net +5V: track 0.00 -> 428.5 mm, vias 0 -> 1
- net +5VP: track 0.00 -> 394.8 mm, vias 0 -> 2
- net Net-(R11-Pad1): track 0.00 -> 180.2 mm, vias 0 -> 3
- net Net-(R10-Pad1): track 0.00 -> 168.0 mm
- net /CO: track 0.00 -> 167.1 mm, vias 0 -> 1
- net /NH3: track 0.00 -> 166.4 mm, vias 0 -> 1
- net Net-(R5-Pad1): track 0.00 -> 164.7 mm, vias 0 -> 2
- net +3.3V: track 10.6 -> 175.0 mm, vias 1 -> 6
- net /NO2: track 0.00 -> 155.2 mm, vias 0 -> 1
- net Net-(R3-Pad1): track 0.00 -> 145.0 mm, vias 0 -> 3
- net Net-(R15-Pad1): track 33.3 -> 167.6 mm, vias 2 -> 4
- net Net-(J5-Pin_4): track 89.8 -> 202.2 mm, vias 2 -> 4
- net Net-(R1-Pad1): track 0.00 -> 112.0 mm, vias 0 -> 1
- net Net-(R7-Pad1): track 0.00 -> 107.2 mm, vias 0 -> 2
- net GND: track 8.17 -> 106.8 mm, vias 4 -> 25
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- added copper zone on B.Cu, net GND
Other:
- board text added: "45-MOSFET"
- board text added: "AD10 NH3"
- board text added: "AD8 CO"
- board text added: "RX2"
- board text added: "RX3"
- board text added: "TX2"
- board text added: "TX3"

Commit message: Update 19 mar 2026
Parts:
- removed R17: 1M, Resistor_SMD:R_0603_1608Metric_Pad0.98x0.95mm_HandSolder
- removed R18, R21: 1K, Resistor_SMD:R_0603_1608Metric_Pad0.98x0.95mm_HandSolder
- removed RV1: 1M, Potentiometer_THT:Potentiometer_Vishay_T73YP_Vertical
- removed RV2: 500K, Potentiometer_THT:Potentiometer_Vishay_T73YP_Vertical
- removed RV3: 100K, Potentiometer_THT:Potentiometer_Vishay_T73YP_Vertical
Routing:
- net /CO: track 167.1 -> 128.6 mm
- net +5V: track 428.5 -> 466.8 mm
- net /NH3: track 166.4 -> 131.0 mm
- net /NO2: track 155.2 -> 133.8 mm
- net Net-(R21-Pad2): track 14.3 -> 0.00 mm, vias 1 -> 0
- net GND: track 106.8 -> 117.6 mm
- net Net-(R17-Pad2): track 9.94 -> 0.00 mm
- net Net-(R18-Pad2): track 9.62 -> 0.00 mm
- net Net-(J6-Pin_25): track 32.4 -> 33.4 mm
- net /A13-ZE08-CH20: track 63.3 -> 64.1 mm
