File: uprojects/John Ottolenghi/kicadA/snifferA.Back01/snifferA.kicad_pcb (KiCad board)
At the start: 2 copper layers, 122.5 x 174 mm, 66 parts, among them J1 DHT22, J10 ZP07, J11 DCJ200-10-A-XX-K_REVA, J2 Conn_01x10, J3 CCS811_CJMCU, J4 Conn_01x08, J5 Conn_01x08, J6 Conn_02x18_Odd_Even, J7 Conn_01x08, J8 Conn_01x08, J9 Conn_01x08, U1 MQ-131-H, U10 MQ-131-L, U12 ZE08-CH20, U13 ZP07, U14 SM4-NO2-20, U15 MQ-07, U16 YAAJ_DCDC_StepDown_LM2596, U2 MQ-135, U3 MQ-136, U4 MQ-137, U5 MQ-02, U6 MQ-04, U7 MQ-06, U8 MQ-08, U9 YAAJ_DCDC_StepDown_LM2596

Commit message: Update 11 mar 2026
Parts:
- added C11: 0.1uF, Capacitor_SMD:C_1206_3216Metric_Pad1.33x1.80mm_HandSolder, F.Cu at (135.5, 28.8)
- added R21: 10k, Resistor_SMD:R_1206_3216Metric, F.Cu at (135.5, 25.2)
- added U11: ZE-03, sensors:SM4-NO2-20, F.Cu at (148.6, 37.5)
Connections:
- J5 pad 5: unconnected-(J5-Pin_5-Pad5) -> Net-(J5-Pin_5)
- J5 pad 6: unconnected-(J5-Pin_6-Pad6) -> Net-(J5-Pin_6)
Routing:
- net Net-(J5-Pin_6): track 0.00 -> 144.3 mm, vias 0 -> 1
- net Net-(J5-Pin_5): track 0.00 -> 140.5 mm, vias 0 -> 3
- net /A14-ZE-03: track 0.00 -> 98.4 mm, vias 0 -> 2
- net Net-(R21-Pad1): track 0.00 -> 15.5 mm
- net /SCL: track 83.8 -> 80.1 mm
- net /SDA: track 87.5 -> 83.8 mm
