File: uprojects/John Ottolenghi/kicadA/snifferA.Back01/snifferA.kicad_sch (KiCad schematic)
At the start: 67 parts, among them J1 DHT22, J10 ZP07, J11 DCJ200-10-A-XX-K_REVA, J2 Conn_01x10, J3 CCS811_CJMCU, J4 Conn_01x08, J5 Conn_01x08, J6 Conn_02x18_Odd_Even, J7 Conn_01x08, J8 Conn_01x08, J9 Conn_01x08, U1 MQ-131-H, U10 MQ-131-L, U12 ZE08-CH20, U13 ZP07, U14 SM4-NO2-20, U15 MQ-07, U16 YAAJ_DCDC_StepDown_LM2596, U2 MQ-135, U3 MQ-136, U4 MQ-137, U5 MQ-02, U6 MQ-04, U7 MQ-06, U8 MQ-08, U9 YAAJ_DCDC_StepDown_LM2596

Commit message: Update 11 mar 2026
Parts:
- added C11: 0.1uF, Capacitor_SMD:C_1206_3216Metric_Pad1.33x1.80mm_HandSolder, symbol Device:C_Small
- added R21: 10k, Resistor_SMD:R_1206_3216Metric, symbol Device:R_Small
- added U11: ZE-03, sensors:SM4-NO2-20, symbol sensors:SM4-NO2-20
Connections:
- net +5V: now also U11.4
- net A14-ZE-03: now also C11.2, R21.2
- net GND: now also C11.1, U11.5
- net at J5.5 (Pin_5): now also U11.1
- net at J5.6 (Pin_6): now also U11.2
- new net: R21.1, U11.3
