File: CM0/kicad/CM0_A/CM0_A.kicad_sch (KiCad schematic)
At the start: 0 parts

Commit message: Update 18 mar 2026
Other:
- added sheet CM0_Module (CM0_Module.kicad_sch)
- added sheet LCD_FPC (lcd_fpc.kicad_sch)
Changed lines of the file:
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@@
 	(generator "eeschema")
 	(generator_version "9.0")
-	(paper "A4")
+	(paper "A1")
+	(sheet
+		(at 220.98 157.48)
+		(size 81.026 124.968)
+		(exclude_from_sim no)
+		(in_bom yes)
+		(on_board yes)
+		(dnp no)
+		(fields_autoplaced yes)
+		(stroke
+			(width 0.1524)
+			(type solid)
+		)
+		(fill
+			(color 0 0 0 0.0000)
+		)
+		(property "Sheetname" "CM0_Module"
+			(at 220.98 156.7684 0)
+			(effects
+				(font
+					(size 1.27 1.27)
+				)
+				(justify left bottom)
+			)
+		)
+		(property "Sheetfile" "CM0_Module.kicad_sch"
+			(at 220.98 283.0326 0)
+			(effects
+				(font
+					(size 1.27 1.27)
+				)
+				(justify left top)
+			)
+		)
+		(pin "DSI_CK_N" output
+			(at 220.98 179.07 180)
+			(effects
+				(font
+					(size 1.27 1.27)
+				)
+				(justify left)
+			)
+		)
+		(pin "DSI_CK_P" output
+			(at 220.98 176.53 180)
+			(effects
+				(font
+					(size 1.27 1.27)
+				)
+				(justify left)
+			)
+		)
+		(pin "DSI_D0_N" output
+			(at 220.98 185.42 180)
+			(effects
+				(font
+					(size 1.27 1.27)
+				)
+				(justify left)
+			)
+		)
+		(pin "DSI_D1_N" output
+			(at 220.98 191.77 180)
+			(effects
+				(font
+					(size 1.27 1.27)
+				)
+				(justify left)
+			)
+		)
+		(pin "DSI_D1_P" output
+			(at 220.98 189.23 180)
+			(effects
+				(font
+					(size 1.27 1.27)
+				)
+				(justify left)
+			)
+		)
+		(pin "DSI_D0_P" output
+			(at 220.98 182.88 180)
+			(effects
+				(font
+					(size 1.27 1.27)
+				)
+				(justify left)
+			)
+		)
+		(instances
+			(project "CM0_A"
+				(path "/50bd9559-836c-4ff6-9873-987acf610763"
+					(page "2")
+				)
+			)
+		)
+	)
+	(sheet
+		(at 158.496 165.862)
+		(size 38.608 35.56)
+		(exclude_from_sim no)
+		(in_bom yes)
+		(on_board yes)
+		(dnp no)
+		(fields_autoplaced yes)
+		(stroke
+			(width 0.1524)
+			(type solid)
+		)
+		(fill
+			(color 0 0 0 0.0000)
+		)
+		(property "Sheetname" "LCD_FPC"
+			(at 158.496 165.1504 0)
+			(effects
+				(font
+					(size 1.27 1.27)
+				)
+				(justify left bottom)
+			)
+		)
+		(property "Sheetfile" "lcd_fpc.kicad_sch"
+			(at 158.496 202.0066 0)
+			(effects
+				(font
+					(size 1.27 1.27)
+				)
+				(justify left top)
+			)
+		)
+		(instances
+			(project "CM0_A"
+				(path "/50bd9559-836c-4ff6-9873-987acf610763"
+					(page "3")
+				)
+			)
+		)
+	)
 	(sheet_instances
 		(path "/"

Commit message: Update 23 mar 2026
Other:
- sheet CM0_Module ports: added LCD_RESET_CPU; removed none
- sheet LCD_FPC ports: added LCD_DSI_CK_N, LCD_DSI_CK_P, LCD_DSI_D0_N, LCD_DSI_D0_P, LCD_DSI_D1_N, LCD_DSI_D1_P, LCD_RESET; removed none
Changed lines of the file:
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@@
 	(generator_version "9.0")
 	(paper "A1")
+	(wire
+		(pts
+			(xy 220.98 189.23) (xy 191.77 189.23)
+		)
+		(stroke
+			(width 0)
+			(type default)
+		)
+	)
+	(wire
+		(pts
+			(xy 220.98 182.88) (xy 191.77 182.88)
+		)
+		(stroke
+			(width 0)
+			(type default)
+		)
+	)
+	(wire
+		(pts
+			(xy 220.98 196.85) (xy 191.77 196.85)
+		)
+		(stroke
+			(width 0)
+			(type default)
+		)
+	)
+	(wire
+		(pts
+			(xy 220.98 191.77) (xy 191.77 191.77)
+		)
+		(stroke
+			(width 0)
+			(type default)
+		)
+	)
+	(wire
+		(pts
+			(xy 220.98 176.53) (xy 191.77 176.53)
+		)
+		(stroke
+			(width 0)
+			(type default)
+		)
+	)
+	(wire
+		(pts
+			(xy 220.98 179.07) (xy 191.77 179.07)
+		)
+		(stroke
+			(width 0)
+			(type default)
+		)
+	)
+	(wire
+		(pts
+			(xy 191.77 185.42) (xy 220.98 185.42)
+		)
+		(stroke
+			(width 0)
+			(type default)
+		)
+	)
 	(sheet
 		(at 220.98 157.48)
@@
 			)
 		)
+		(pin "LCD_RESET_CPU" output
+			(at 220.98 196.85 180)
+			(effects
+				(font
+					(size 1.27 1.27)
+				)
+				(justify left)
+			)
+		)
 		(instances
 			(project "CM0_A"
@@
 	)
 	(sheet
-		(at 158.496 165.862)
+		(at 153.162 165.354)
 		(size 38.608 35.56)
 		(exclude_from_sim no)
@@
 		)
 		(property "Sheetname" "LCD_FPC"
-			(at 158.496 165.1504 0)
+			(at 153.162 164.6424 0)
 			(effects
 				(font
@@
 		)
 		(property "Sheetfile" "lcd_fpc.kicad_sch"
-			(at 158.496 202.0066 0)
+			(at 153.162 201.4986 0)
 			(effects
 				(font
@@
 			)
 		)
+		(pin "LCD_DSI_D0_N" input
+			(at 191.77 185.42 0)
+			(effects
+				(font
+					(size 1.27 1.27)
+				)
+				(justify right)
+			)
+		)
+		(pin "LCD_DSI_CK_N" input
+			(at 191.77 179.07 0)
+			(effects
+				(font
+					(size 1.27 1.27)
+				)
+				(justify right)
+			)
+		)
+		(pin "LCD_DSI_CK_P" input
+			(at 191.77 176.53 0)
+			(effects
+				(font
+					(size 1.27 1.27)
+				)
+				(justify right)
+			)
+		)
+		(pin "LCD_DSI_D0_P" input
+			(at 191.77 182.88 0)
+			(effects
+				(font
+					(size 1.27 1.27)
+				)
+				(justify right)
+			)
+		)
+		(pin "LCD_DSI_D1_N" input
+			(at 191.77 191.77 0)
+			(effects
+				(font
+					(size 1.27 1.27)
+				)
+				(justify right)
+			)
+		)
+		(pin "LCD_DSI_D1_P" input
+			(at 191.77 189.23 0)
+			(effects
+				(font
+					(size 1.27 1.27)
+				)
+				(justify right)
+			)
+		)
+		(pin "LCD_RESET" input
+			(at 191.77 196.85 0)
+			(effects
+				(font
+					(size 1.27 1.27)
+				)
+				(justify right)
+			)
+		)
