File: CM0/kicad/CM0_A/lcd_fpc.kicad_sch (KiCad schematic)
At the start: 2 parts, among them J1 5051104096

Commit message: Update 23 mar 2026
Connections:
- net DSI_CK_N renamed LCD_DSI_CK_N
- net DSI_CK_P renamed LCD_DSI_CK_P
- net DSI_D0_N renamed LCD_DSI_D0_N
- net DSI_D0_P renamed LCD_DSI_D0_P
- net DSI_D1_N renamed LCD_DSI_D1_N
- net DSI_D1_P renamed LCD_DSI_D1_P
Changed lines of the file:
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@@
 		)
 	)
-	(hierarchical_label "DSI_D1_N"
+	(hierarchical_label "LCD_DSI_D1_N"
 		(shape input)
 		(at 147.32 66.04 0)
@@
 		)
 	)
-	(hierarchical_label "DSI_D1_P"
+	(hierarchical_label "LCD_DSI_D1_P"
 		(shape input)
 		(at 147.32 68.58 0)
@@
 		)
 	)
-	(hierarchical_label "DSI_D0_N"
+	(hierarchical_label "LCD_DSI_D0_N"
 		(shape input)
 		(at 147.32 50.8 0)
@@
 		)
 	)
-	(hierarchical_label "DSI_CK_N"
+	(hierarchical_label "LCD_DSI_CK_N"
 		(shape input)
 		(at 147.32 58.42 0)
@@
 		)
 	)
-	(hierarchical_label "DSI_CK_P"
+	(hierarchical_label "LCD_DSI_CK_P"
 		(shape input)
 		(at 147.32 60.96 0)
@@
 		)
 	)
-	(hierarchical_label "DSI_D0_P"
+	(hierarchical_label "LCD_DSI_D0_P"
 		(shape input)
 		(at 147.32 53.34 0)
