File: CM0/kicad/CM0_A/CM0_Module.kicad_sch (KiCad schematic)
At the start: 1 part, among them U1 CM0

Commit message: Update 23 mar 2026
Parts:
- added C?: 10uF, symbol Device:C_Small
Connections:
- net GND: now reaches U1.1
- net GND: now also U1.10, U1.100, U1.103, U1.106, U1.109, U1.112, U1.115, U1.123, U1.126, U1.129, U1.13, U1.132, U1.16, U1.21, U1.24, U1.27, U1.30, U1.33, U1.34, U1.37, U1.4, U1.40, U1.45, U1.48, U1.51, U1.54, U1.57, U1.60, U1.63, U1.66, U1.69, U1.7, U1.72, U1.75, U1.78, U1.81, U1.84, U1.87, U1.90, U1.93, U1.96, U1.99, C?.2
- net +5V: now reaches U1.67
- net +5V: now also U1.68, C?.1
- net LCD_RESET renamed LCD_RESET_CPU

Commit message: Update 25 mar 2026
Parts:
- added C?: 0.1uF, symbol Device:C_Small
Connections:
- net +5V: now also C?.1
- net GND: now also C?.2
- net SD_VREF: now reaches U1.122
- net SD_DAT1: now reaches U1.124
- net SD_DAT0: now reaches U1.125
- net SD_CLK: now reaches U1.127
- net SD_CMD: now reaches U1.128
- net SD_DAT3: now reaches U1.130
- net SD_DAT2: now reaches U1.131
- net DSI_D3_P: now reaches U1.2
- net DSI_D3_N: now reaches U1.3
- net CSI_D3_P: now reaches U1.46
- net CSI_D3_N: now reaches U1.47
- net CSI_D2_P: now reaches U1.49
- net DSI_D2_P: now reaches U1.5
- net CSI_D2_N: now reaches U1.50
- net CSI_CK_P: now reaches U1.52
- net CSI_CK_N: now reaches U1.53
- net CSI_D1_P: now reaches U1.55
- net CSI_D1_N: now reaches U1.56
- net CSI_D0_P: now reaches U1.58
- net CSI_D0_N: now reaches U1.59
- net DSI_D2_N: now reaches U1.6
