File: uprojects/Stethiscope/stetho-01/stetho-01.kicad_pcb (KiCad board)
At the start: 2 copper layers, 70.9 x 66.5 mm, 2 parts, among them U1 ESP32-S3-WROOM-1-N16R8, U2 ADS1298IPAGR

Commit message: Update 06 May 2026
Other:
- board size 70.9 x 66.5 mm -> 61.9 x 57.5 mm
