File: uprojects/Stethiscope/stetho-01/stetho-01.kicad_sch (KiCad schematic)
At the start: 2 parts, among them U1 ESP32-S3-WROOM-1-N16R8, U2 ADS1298IPAGR

Commit message: Update 11 May 2026
Parts:
- added C?: 1.2nF, symbol Device:C_Small
- added R?: 1M 5%, symbol Device:R_Small
Connections:
- net RLDINV: now reaches U2.61 (RLDINV)
- net RLDINV: now also C?.2, R?.2
- net at U2.62 (RLDIN): now also U2.63 (RLDOUT), C?.1, R?.1

Commit message: Update 12 May 2026
Parts:
- added C?: 1nF, symbol Device:C_Small
- added R?: 10K 1%, symbol Device:R_Small
Connections:
- net AVDD: now reaches U2.1 (IN8N)
- net AVDD: now also U2.2 (IN8P), U2.3 (IN7N), U2.4 (IN7P), U2.5 (IN6N), U2.54 (AVDD1), U2.56 (AVDD), U2.59 (AVDD), U2.6 (IN6P), U2.7 (IN5N), U2.8 (IN5P)
- net DVDD: now reaches U2.48 (DVDD)
- net DVDD: now also U2.50 (DVDD), R?.2
- net at U2.49 (DGND): now also U2.51 (DGND)
- net at U2.52 (CLKSEL): now also R?.1
- net at U2.64 (WCT): now also U2.9 (IN4N), C?.2
- new net AGND: C?.1

Commit message: Update 13 May 2026
Parts:
- added C? (x2): 1nF, symbol Device:C_Small
Connections:
- net at U2.57 (AVSS): now also U2.58 (AVSS)
Changed lines of the file:
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@@
+	(wire
+		(pts
+			(xy 154.94 177.8) (xy 157.48 177.8)
+		)
+		(stroke
+			(width 0)
+			(type default)
+		)
+	)
 	(wire
 		(pts
@@
 	(wire
 		(pts
+			(xy 154.94 181.61) (xy 154.94 177.8)
+		)
+		(stroke
+			(width 0)
+			(type default)
+		)
+	)
+	(wire
+		(pts
 			(xy 120.65 194.31) (xy 120.65 195.58)
 		)
@@
 		(pts
 			(xy 123.19 200.66) (xy 120.65 200.66)
+		)
+		(stroke
+			(width 0)
+			(type default)
+		)
+	)
+	(wire
+		(pts
+			(xy 157.48 177.8) (xy 157.48 181.61)
 		)
 		(stroke
@@
 	)
 	(symbol
+		(lib_id "Device:C_Small")
+		(at 158.75 152.4 270)
+		(unit 1)
+		(body_style 1)
+		(exclude_from_sim no)
+		(in_bom yes)
+		(on_board yes)
+		(in_pos_files yes)
+		(dnp no)
+		(fields_autoplaced yes)
+		(property "Reference" "C?"
+			(at 158.7436 146.05 90)
+			(show_name no)
+			(do_not_autoplace no)
+			(effects
+				(font
+					(size 1.27 1.27)
+				)
+			)
+		)
+		(property "Value" "1nF"
+			(at 158.7436 148.59 90)
+			(show_name no)
+			(do_not_autoplace no)
+			(effects
+				(font
+					(size 1.27 1.27)
+				)
+			)
+		)
+		(property "Footprint" ""
+			(at 158.75 152.4 0)
+			(hide yes)
+			(show_name no)
+			(do_not_autoplace no)
+			(effects
+				(font
+					(size 1.27 1.27)
+				)
+			)
+		)
+		(property "Datasheet" ""
+			(at 158.75 152.4 0)
+			(hide yes)
+			(show_name no)
+			(do_not_autoplace no)
+			(effects
+				(font
+					(size 1.27 1.27)
+				)
+			)
+		)
+		(property "Description" "Unpolarized capacitor, small symbol"
+			(at 158.75 152.4 0)
+			(hide yes)
+			(show_name no)
+			(do_not_autoplace no)
+			(effects
+				(font
+					(size 1.27 1.27)
+				)
+			)
+		)
+		(pin "2"
+		)
+		(pin "1"
+		)
+		(instances
+			(project "stetho-01"
+				(path "/04fa24c6-1746-4cd8-a57f-0a98044e2410"
+					(reference "C?")
+					(unit 1)
+				)
+			)
+		)
+	)
+	(symbol
 		(lib_id "power:VDDA")
 		(at 214.63 191.77 0)
@@
 					(unit 1)
 				)
+			)
+		)
+	)
+	(symbol
+		(lib_id "Device:C_Small")
+		(at 158.75 158.75 270)
+		(unit 1)
+		(body_style 1)
+		(exclude_from_sim no)
+		(in_bom yes)
+		(on_board yes)
+		(in_pos_files yes)
+		(dnp no)
+		(property "Reference" "C?"
+			(at 160.02 161.544 90)
+			(show_name no)
+			(do_not_autoplace no)
+			(effects
+				(font
+					(size 1.27 1.27)
+				)
+			)
+		)
+		(property "Value" "1nF"
+			(at 156.718 161.544 90)
+			(show_name no)
+			(do_not_autoplace no)
+			(effects
+				(font
+					(size 1.27 1.27)
+				)
+			)
+		)
+		(property "Footprint" ""
+			(at 158.75 158.75 0)
+			(hide yes)
+			(show_name no)
+			(do_not_autoplace no)
+			(effects
+				(font
+					(size 1.27 1.27)
+				)
+			)
+		)
+		(property "Datasheet" ""
+			(at 158.75 158.75 0)
+			(hide yes)
+			(show_name no)
+			(do_not_autoplace no)
+			(effects
+				(font
+					(size 1.27 1.27)
+				)
+			)
+		)
+		(property "Description" "Unpolarized capacitor, small symbol"
+			(at 158.75 158.75 0)
+			(hide yes)
+			(show_name no)
+			(do_not_autoplace no)
+			(effects
+				(font
+					(size 1.27 1.27)
+				)
+			)
+		)
+		(pin "2"
+		)
+		(pin "1"
+		)
+		(instances
+			(project "stetho-01"
+				(path "/04fa24c6-1746-4cd8-a57f-0a98044e2410"
+					(reference "C?")
+					(unit 1)
+				)

Commit message: Update 13 May 2026
Parts:
- added C?: 0.1uF, symbol Device:C_Small
- added C? (x2): 1uF, symbol Device:C_Small
- added C?: 22uF, symbol Device:C_Small
- added C?: 10uF, symbol Device:C_Small
- added R?: 0, symbol Device:R_Small
- C?: value 1nF -> 1uF
- C?: value 1nF -> 0.1uF
Connections:
- net AGND: now also C?.2, C?.2, U2.20 (AVSS), U2.23 (AVSS), U2.25 (VREFN), U2.32 (AVSS), U2.53 (AVSS1), U2.57 (AVSS), U2.58 (AVSS), C?.2, C?.2, C?.2, C?.2, C?.2
- net AVDD: now also U2.19 (AVDD), U2.21 (AVDD), U2.22 (AVDD)
- net DVDD: now also R?.2
- net at C?.1: now also C?.1, U2.55 (VCAP3)
- net at U2.24 (VREFP): now also C?.1, C?.1
- net at U2.26 (VCAP4): now also C?.1
- net at U2.28 (VCAP1): now also C?.1
- net at U2.30 (VCAP2): now also C?.1
- net DGND: now reaches U2.31 (RESV1)
- net DGND: now also U2.33 (DGND), U2.49 (DGND), U2.51 (DGND)
- net at U2.46 (GPIO4): now also R?.1
- net *DRDY: now reaches U2.47 (*DRDY)
- no-connect marks 0 -> 1
Other:
- moved on the sheet: C?

Commit message: Update 2 June 2026
Parts:
- added J?: Conn_01x01, symbol Connector_Generic:Conn_01x01
Connections:
- net at U2.17 (TESTP_PACE_OUT1): now also J?.1 (Pin_1)
Changed lines of the file:
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@@
+	(wire
+		(pts
+			(xy 139.7 252.73) (xy 139.7 250.19)
+		)
+		(stroke
+			(width 0)
+			(type default)
+		)
+	)
 	(wire
 		(pts
@@
 	(wire
 		(pts
+			(xy 138.43 252.73) (xy 139.7 252.73)
+		)
+		(stroke
+			(width 0)
+			(type default)
+		)
+	)
+	(wire
+		(pts
 			(xy 120.65 198.12) (xy 120.65 200.66)
 		)
@@
 		(pts
 			(xy 177.8 177.8) (xy 177.8 181.61)
+		)
+		(stroke
+			(width 0)
+			(type default)
+		)
+	)
+	(wire
+		(pts
+			(xy 138.43 259.08) (xy 138.43 252.73)
 		)
 		(stroke
@@
 					(unit 1)
 				)
+			)
+		)
+	)
+	(symbol
+		(lib_id "Connector_Generic:Conn_01x01")
+		(at 138.43 264.16 270)
+		(unit 1)
+		(body_style 1)
+		(exclude_from_sim no)
+		(in_bom yes)
+		(on_board yes)
+		(in_pos_files yes)
+		(dnp no)
+		(property "Reference" "J?"
+			(at 137.414 266.954 90)
+			(show_name no)
+			(do_not_autoplace no)
+			(effects
+				(font
+					(size 1.27 1.27)
+				)
+				(justify left)
+			)
+		)
+		(property "Value" "Conn_01x01"
+			(at 135.89 262.89 0)
+			(show_name no)
+			(do_not_autoplace no)
+			(effects
+				(font
+					(size 1.27 1.27)
+				)
+				(justify left)
+			)
+		)
+		(property "Footprint" ""
+			(at 138.43 264.16 0)
+			(hide yes)
+			(show_name no)
+			(do_not_autoplace no)
+			(effects
+				(font
+					(size 1.27 1.27)
+				)
+			)
+		)
+		(property "Datasheet" ""
+			(at 138.43 264.16 0)
+			(hide yes)
+			(show_name no)
+			(do_not_autoplace no)
+			(effects
+				(font
+					(size 1.27 1.27)
+				)
+			)
+		)
+		(property "Description" "Generic connector, single row, 01x01, script generated (kicad-library-utils/schlib/autogen/connector/)"
+			(at 138.43 264.16 0)
+			(hide yes)
+			(show_name no)
+			(do_not_autoplace no)
+			(effects
+				(font
+					(size 1.27 1.27)
+				)
+			)
+		)
+		(pin "1"
+		)
+		(instances
+			(project "stetho-01"
+				(path "/04fa24c6-1746-4cd8-a57f-0a98044e2410"
+					(reference "J?")
+					(unit 1)
+				)
