File: uprojects/Stethiscope/stetho-01/stetho-01.kicad_sch (KiCad schematic)
At the start: 15 parts, among them U1 ESP32-S3-WROOM-1-N16R8, U2 ADS1298IPAGR

Commit message: Update 7 July 2026
Connections:
- net IN1N: now reaches U2.15 (IN1N)
- net IN1P: now reaches U2.16 (IN1P)
Other:
- note added: "documentsA/Medical/docs/doc01.html"
Changed lines of the file:
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@@
 	(generator_version "10.0")
 	(paper "A3")
+	(text "documentsA/Medical/docs/doc01.html"
+		(exclude_from_sim no)
+		(at 150.876 123.19 0)
+		(effects
+			(font
+				(size 5 5)
+				(thickness 1)
+				(bold yes)
+			)
+		)
+	)
 	(junction
 		(at 162.56 158.75)
@@
 	(wire
 		(pts
+			(xy 106.68 233.68) (xy 123.19 233.68)
+		)
+		(stroke
+			(width 0)
+			(type default)
+		)
+	)
+	(wire
+		(pts
 			(xy 177.8 256.54) (xy 177.8 250.19)
 		)
@@
 	(wire
 		(pts
+			(xy 106.68 231.14) (xy 123.19 231.14)
+		)
+		(stroke
+			(width 0)
+			(type default)
+		)
+	)
+	(wire
+		(pts
 			(xy 172.72 265.43) (xy 172.72 269.24)
 		)
@@
 		)
 	)
+	(label "IN1P"
+		(at 106.68 233.68 0)
+		(effects
+			(font
+				(size 1.27 1.27)
+				(thickness 0.1588)
+			)
+			(justify left bottom)
+		)
+	)
+	(label "IN1N"
+		(at 106.68 231.14 0)
+		(effects
+			(font
+				(size 1.27 1.27)
+				(thickness 0.1588)
+			)
+			(justify left bottom)
+		)
+	)
