File: uprojects/Adam/kicad_pcb/reband/reband.kicad_pcb (KiCad board)
At the start: 2 copper layers, 3 parts, among them U1 ESP32-C3FH4, U2 LMV324MT, U3 MAX30009ENA+T

Commit message: ROOM 25 MAY 2026 Updates
Parts:
- added AE1: AMCA31-2R450G-S1F-T3, AMCA31_2R450G_S1F_T3:ANT_AMCA31-2R450G-S1F-T3_ABR, F.Cu at (139.8, 77.7)
- added S1: EVQ-P7A01P, EVQ_P7A01P:SW_EVQ-P7A01P, F.Cu at (149.7, 85.4)
- added U4: BQ25100YFPR, BQ25100YFPR:BGA6N40P3X2_157X88X50N, F.Cu at (141.9, 92.2)
- added U5: BNO055, Package_LGA:LGA-28_5.2x3.8mm_P0.5mm, F.Cu at (133.1, 93.0)
- moved U1 7.20 mm to (142.2, 84.7)
- moved U2 5.93 mm to (133.8, 84.8)
Other:
- board outline added: 25 x 30 mm
- board text added: "ANT"
- board text added: "BATT CHARGE"
- board text added: "ESP32-C3"
- board text added: "GSR"
- board text added: "IMU"
- board text added: "OP-AMP"

Commit message: Update 26 May 2026
Parts:
- added J1: S2B-ZRLFSN, S2B_ZR_LF_SN:CONN_S2B-ZR_JST, F.Cu at (147.3, 92.0)
- added J2: USB4215-03-A, USB4215_03_A:CONN_8p94X6p5X3p16_12L_GCC, F.Cu at (130.0, 89.9)
- added U6: TCR2EF33_LMCT, TCR2EF33_LM_CT:SOT-25 SMV_TOS, F.Cu at (136.8, 81.3)
- added U7: TCR2EF18_LMCT, TCR2EF18_LM_CT:SOT-25 SMV_TOS, F.Cu at (136.7, 85.7)
- U2: value LMV324MT -> AP2112K-3.3TRG1; footprint LMV324MT:MTC14_TEX -> AP2112K_3_3TRG1:SOT_RG1_DIO
- moved U5 9.53 mm to (140.6, 98.9)
- moved U3 7.80 mm to (141.8, 90.3)
- moved U4 4.07 mm to (138.4, 90.3)
- moved U2 3.73 mm to (131.8, 81.7)
- moved U1 0.97 mm to (143.1, 84.4)
- moved AE1 0.78 mm to (139.6, 76.9)
Other:
- board text added: "CHG"
- board text removed: "BATT CHARGE"
- board text removed: "OP-AMP"

Commit message: Update 28 May 2026
Parts:
- removed U6: TCR2EF33_LMCT, TCR2EF33_LM_CT:SOT-25 SMV_TOS
- added IC1: USBLC6-2SC6, USBLC6-2SC6:SOT95P280X145-6N, B.Cu at (137.4, 90.1)
- added R1: 5.1K, Resistor_SMD:R_0402_1005Metric_Pad0.72x0.64mm_HandSolder, F.Cu at (131.1, 95.8)
- added R2: 5.1K, Resistor_SMD:R_0402_1005Metric_Pad0.72x0.64mm_HandSolder, F.Cu at (131.1, 84.1)
- added R3: 10K, Resistor_SMD:R_0402_1005Metric_Pad0.72x0.64mm_HandSolder, F.Cu at (128.1, 75.8)
- added R4: 2K7, Resistor_SMD:R_0402_1005Metric_Pad0.72x0.64mm_HandSolder, F.Cu at (127.9, 79.1)
- U2: value AP2112K-3.3TRG1 -> TLV75533PDBVR; footprint AP2112K_3_3TRG1:SOT_RG1_DIO -> TLV75533PDBVR:DBV0005A_N
- moved U2 8.79 mm to (123.7, 78.4)
- moved U4 4.53 mm to (137.0, 86.0)
- moved U7 4.45 mm to (136.9, 81.2)
- moved U3 2.18 mm to (144.0, 90.4)
Connections:
- J2 pad A1/B12: unconnected-(J2-GND-PadA1/B12) -> GND
- J2 pad A4/B9: unconnected-(J2-VBUS-PadA4/B9) -> +5V
- J2 pad A5: unconnected-(J2-CC1-PadA5) -> Net-(J2-CC1)
- J2 pad A6: unconnected-(J2-DP1-PadA6) -> /USB_D+
- J2 pad A7: unconnected-(J2-DN1-PadA7) -> /USB_D-
- J2 pad B1/A12: unconnected-(J2-GND-PadB1/A12) -> GND
- J2 pad B4/A9: unconnected-(J2-VBUS-PadB4/A9) -> +5V
- J2 pad B5: unconnected-(J2-CC2-PadB5) -> Net-(J2-CC2)
- J2 pad B6: unconnected-(J2-DP2-PadB6) -> /USB_D+
- J2 pad B7: unconnected-(J2-DN2-PadB7) -> /USB_D-
- U4 pad A2: unconnected-(U4-IN-PadA2) -> +5V
- U4 pad B2: unconnected-(U4-ISET-PadB2) -> Net-(U4-ISET)
Routing:
- net /USB_D+: track 0.00 -> 17.9 mm, vias 0 -> 1
- net /USB_D-: track 0.00 -> 16.8 mm, vias 0 -> 2
- net GND: track 0.00 -> 1.08 mm, vias 0 -> 1

Commit message: Update 28 May 2026
Parts:
- added C1: 2.2uF, Capacitor_SMD:C_0402_1005Metric_Pad0.74x0.62mm_HandSolder, F.Cu at (133.9, 84.1)
- added C2: 2.2uF, Capacitor_SMD:C_0402_1005Metric_Pad0.74x0.62mm_HandSolder, F.Cu at (129.4, 83.1)
- added C3: 2.2uF, Capacitor_SMD:C_0402_1005Metric_Pad0.74x0.62mm_HandSolder, F.Cu at (135.2, 77.6)
- added C4: 10pF, Capacitor_SMD:C_0402_1005Metric_Pad0.74x0.62mm_HandSolder, F.Cu at (143.4, 85.3)
- added C5: 10pF, Capacitor_SMD:C_0402_1005Metric_Pad0.74x0.62mm_HandSolder, F.Cu at (141.1, 85.3)
- added C6: 1uF, Capacitor_SMD:C_0402_1005Metric_Pad0.74x0.62mm_HandSolder, F.Cu at (136.4, 103.0)
- added C7: 120nF, Capacitor_SMD:C_0402_1005Metric_Pad0.74x0.62mm_HandSolder, F.Cu at (132.5, 99.2)
- added D1: LED, LED_SMD:LED_0402_1005Metric_Pad0.77x0.64mm_HandSolder, F.Cu at (138.7, 87.1)
- added E1: NN02-101, NN02_101:XCVR_NN02-101, F.Cu at (143.2, 77.3)
- added R10: 10K, Resistor_SMD:R_0402_1005Metric_Pad0.72x0.64mm_HandSolder, F.Cu at (143.6, 94.2)
- added R11: 10K, Resistor_SMD:R_0402_1005Metric_Pad0.72x0.64mm_HandSolder, F.Cu at (146.3, 94.2)
- added R5: 5K9, Resistor_SMD:R_0402_1005Metric_Pad0.72x0.64mm_HandSolder, F.Cu at (136.7, 87.8)
- added R6: 1K, Resistor_SMD:R_0402_1005Metric_Pad0.72x0.64mm_HandSolder, F.Cu at (130.2, 80.6)
- added R7: 2K7, Resistor_SMD:R_0402_1005Metric_Pad0.72x0.64mm_HandSolder, F.Cu at (138.7, 84.9)
- added R8: 4K7, Resistor_SMD:R_0402_1005Metric_Pad0.72x0.64mm_HandSolder, F.Cu at (138.3, 90.0)
- added R9: 4K7, Resistor_SMD:R_0402_1005Metric_Pad0.72x0.64mm_HandSolder, F.Cu at (138.3, 91.2)
- added Y1: ECS-400-18-33-JGN-TR3, ECS_400_18_33_JGN_TR3:XTAL_ECS-400-18-33-JGN-TR3, F.Cu at (142.1, 83.0)
- moved R3 11.0 mm to (136.4, 83.1)
- moved U2 9.67 mm to (133.1, 80.5)
- moved U3 8.42 mm to (137.1, 95.2)
- moved J1 8.19 mm to (143.1, 99.0), turned to 90 degrees
- moved R4 7.09 mm to (133.9, 82.9), turned to 180 degrees
- moved U1 5.37 mm to (143.4, 89.8)
- moved U5 4.27 mm to (136.4, 99.8)
- moved U7 1.02 mm to (137.6, 80.5)
- moved AE1 1.02 mm to (139.6, 75.9)
- moved U4 0.61 mm to (136.6, 85.5)
Connections:
- J1 pad 1: unconnected-(J1-Pad1) -> Net-(U2-IN)
- J1 pad 2: unconnected-(J1-Pad2) -> GND
- R3 pad 1: unconnected-(R3-Pad1) -> Net-(U4-TS)
- R3 pad 2: unconnected-(R3-Pad2) -> GND
- U1 pad 1: unconnected-(U1-LNA_IN-Pad1) -> Net-(U1-LNA_IN)
- U1 pad 14: unconnected-(U1-GPIO8-Pad14) -> Net-(U1-GPIO8)
- U1 pad 15: unconnected-(U1-GPIO9-Pad15) -> Net-(U1-GPIO9)
- U1 pad 29: unconnected-(U1-XTAL_N-Pad29) -> Net-(U1-XTAL_N)
- U1 pad 30: unconnected-(U1-XTAL_P-Pad30) -> Net-(U1-XTAL_P)
- U1 pad 6: unconnected-(U1-GPIO2-Pad6) -> /SDA
- U1 pad 7: unconnected-(U1-CHIP_EN-Pad7) -> /RST
- U1 pad 8: unconnected-(U1-GPIO3-Pad8) -> /SCL
- U2 pad 1: unconnected-(U2-IN-Pad1) -> Net-(U2-IN)
- U2 pad 2: unconnected-(U2-GND-Pad2) -> GND
- U2 pad 3: unconnected-(U2-EN-Pad3) -> Net-(U2-EN)
- U2 pad 5: unconnected-(U2-OUT-Pad5) -> +3.3V
- U4 pad A1: unconnected-(U4-OUT-PadA1) -> Net-(U2-IN)
- U4 pad B1: unconnected-(U4-TS-PadB1) -> Net-(U4-TS)
- U4 pad C1: unconnected-(U4-PRE-TERM-PadC1) -> Net-(U4-PRE-TERM)
- U4 pad C2: unconnected-(U4-VSS-PadC2) -> Net-(U4-VSS)
- U5 pad 10: unconnected-(U5-BL_IND-Pad10) -> GND
- U5 pad 11: unconnected-(U5-~{RESET}-Pad11) -> /RST
- U5 pad 14: unconnected-(U5-INT-Pad14) -> /BNO_INT
- U5 pad 18: unconnected-(U5-COM2-Pad18) -> GND
- U5 pad 19: unconnected-(U5-COM1-Pad19) -> /SCL
- U5 pad 2: unconnected-(U5-GND-Pad2) -> GND
- U5 pad 20: unconnected-(U5-COM0-Pad20) -> /SDA
- U5 pad 25: unconnected-(U5-GNDIO-Pad25) -> GND
- U5 pad 28: unconnected-(U5-VDDIO-Pad28) -> +3.3V
- U5 pad 3: unconnected-(U5-VDD-Pad3) -> +3.3V
- U5 pad 4: unconnected-(U5-~{BOOT_LOAD_PIN}-Pad4) -> +3.3V
- U5 pad 5: unconnected-(U5-PS1-Pad5) -> GND
- U5 pad 6: unconnected-(U5-PS0-Pad6) -> GND
- U5 pad 9: unconnected-(U5-CAP-Pad9) -> Net-(U5-CAP)
- U7 pad 1: unconnected-(U7-VIN-Pad1) -> +3.3V
- U7 pad 2: unconnected-(U7-GND-Pad2) -> GND
- U7 pad 5: unconnected-(U7-VOUT-Pad5) -> +1V8
Routing:
- net Net-(U1-XTAL_N): track 0.00 -> 6.25 mm
- net Net-(U1-XTAL_P): track 0.00 -> 4.11 mm

Commit message: Update 29 May 2026
Parts:
- removed AE1: AMCA31-2R450G-S1F-T3, AMCA31_2R450G_S1F_T3:ANT_AMCA31-2R450G-S1F-T3_ABR
- added C10: 47nF, Capacitor_SMD:C_0402_1005Metric_Pad0.74x0.62mm_HandSolder, F.Cu at (144.3, 96.6)
- added C11: 47nF, Capacitor_SMD:C_0402_1005Metric_Pad0.74x0.62mm_HandSolder, F.Cu at (136.6, 95.0)
- added C12: 47nF, Capacitor_SMD:C_0402_1005Metric_Pad0.74x0.62mm_HandSolder, F.Cu at (136.6, 93.9)
- added C13: 1uF, Capacitor_SMD:C_0402_1005Metric_Pad0.74x0.62mm_HandSolder, F.Cu at (136.6, 96.1)
- added C14: 1uF, Capacitor_SMD:C_0402_1005Metric_Pad0.74x0.62mm_HandSolder, F.Cu at (142.2, 92.6)
- added C15: 0.1uF, Capacitor_SMD:C_0402_1005Metric_Pad0.74x0.62mm_HandSolder, F.Cu at (144.9, 82.5)
- added C16: 0.1uF, Capacitor_SMD:C_0402_1005Metric_Pad0.74x0.62mm_HandSolder, B.Cu at (139.7, 86.9)
- added C17: 0.1uF, Capacitor_SMD:C_0402_1005Metric_Pad0.74x0.62mm_HandSolder, F.Cu at (118.1, 90.2)
- added C18: 0.1uF, Capacitor_SMD:C_0402_1005Metric_Pad0.74x0.62mm_HandSolder, F.Cu at (118.1, 93.9)
- added C8: 1pF, Capacitor_SMD:C_0402_1005Metric_Pad0.74x0.62mm_HandSolder, F.Cu at (144.7, 80.1)
- added C9: 47nF, Capacitor_SMD:C_0402_1005Metric_Pad0.74x0.62mm_HandSolder, F.Cu at (143.1, 96.6)
- added R12: 10K, Resistor_SMD:R_0402_1005Metric_Pad0.72x0.64mm_HandSolder, F.Cu at (137.8, 77.6)
- added S2: EVQ-P7A01P, EVQ_P7A01P:SW_EVQ-P7A01P, F.Cu at (149.2, 94.7)
- added U6: MAX30102EFD+T, MAX30102EFD_T:21-1048_F143A5&plus_1_MXM, B.Cu at (139.5, 95.3)
- moved Y1 9.80 mm to (150.1, 88.6), turned to -90 degrees
- moved R11 8.97 mm to (138.3, 90.2), turned to 180 degrees
- moved R9 8.61 mm to (141.5, 83.2), turned to -90 degrees
- moved R8 8.07 mm to (142.6, 83.2), turned to -90 degrees
- moved U3 7.75 mm to (144.7, 93.8)
- moved R10 7.43 mm to (138.3, 89.0)
- moved C5 7.10 mm to (147.8, 87.7), turned to 90 degrees
- moved C4 6.40 mm to (147.8, 90.0), turned to -90 degrees
- moved J1 2.34 mm to (143.6, 101.3)
- moved S1 2.22 mm to (148.9, 83.4)
- moved U1 1.58 mm to (143.7, 88.2), turned to -90 degrees
- moved C6 0.25 mm to (136.4, 102.7)
Connections:
- net Net-(U1-GPIO8) renamed /GPIO8
- IC1 pad 4: unconnected-(IC1-I/O2_2-Pad4) -> /D+
- IC1 pad 6: unconnected-(IC1-I/O1_2-Pad6) -> /D-
- R11 pad 1: Net-(U1-GPIO9) -> /BOOT
- S1 pad 1_1: Net-(S1-Pad1_1) -> /BOOT
- S1 pad 1_2: Net-(S1-Pad1_1) -> /BOOT
- S1 pad 2_1: Net-(S1-Pad2_1) -> GND
- S1 pad 2_2: Net-(S1-Pad2_1) -> GND
- U1 pad 10: unconnected-(U1-GPIO5/MTDI-Pad10) -> /PPG_INT
- U1 pad 11: unconnected-(U1-VDD3P3_RTC-Pad11) -> +3.3V
- U1 pad 12: unconnected-(U1-GPIO6/MTCK-Pad12) -> /BNO_INT
- U1 pad 13: unconnected-(U1-GPIO7/MTDO-Pad13) -> /1.8V_CTRL
- U1 pad 15: Net-(U1-GPIO9) -> /BOOT
- U1 pad 17: unconnected-(U1-VDD3P3_CPU-Pad17) -> +3.3V
- U1 pad 18: unconnected-(U1-VDD_SPI-Pad18) -> Net-(U1-VDD_SPI)
- U1 pad 2: VDD3P3 -> +3.3V
- U1 pad 25: unconnected-(U1-GPIO18/USB_D--Pad25) -> /D-
- U1 pad 26: unconnected-(U1-GPIO19/USB_D+-Pad26) -> /D+
- U1 pad 3: VDD3P3 -> +3.3V
- U1 pad 31: VDDA -> +3.3V
- U1 pad 32: VDDA -> +3.3V
- U1 pad 9: unconnected-(U1-GPIO4/MTMS-Pad9) -> /GSR_INT
- U3 pad A1: unconnected-(U3-EL1-PadA1) -> Net-(U3-EL1)
- U3 pad A2: unconnected-(U3-EL2A-PadA2) -> Net-(U3-EL2A)
- U3 pad B1: unconnected-(U3-EL4-PadB1) -> Net-(U3-EL4)
- U3 pad B2: unconnected-(U3-EL3A-PadB2) -> Net-(U3-EL3A)
- U3 pad C1: unconnected-(U3-AVDD-PadC1) -> +1V8
- U3 pad C2: unconnected-(U3-VREF-PadC2) -> Net-(U3-VREF)
- U3 pad C3: unconnected-(U3-AGND-PadC3) -> GND
- U3 pad D1: unconnected-(U3-DVDD-PadD1) -> +1V8
- U3 pad D2: unconnected-(U3-CSB/I2C_SEL-PadD2) -> +1V8
- U3 pad E1: unconnected-(U3-DGND-PadE1) -> GND
- U3 pad E2: unconnected-(U3-SDO/ADDR-PadE2) -> GND
- U3 pad E3: unconnected-(U3-SDI/SDA-PadE3) -> /SDA
- U3 pad E4: unconnected-(U3-SCLK/SCL-PadE4) -> /SCL
- U3 pad E5: unconnected-(U3-INT-PadE5) -> /GSR_INT
- U5 pad 10: GND -> unconnected-(U5-BL_IND-Pad10)
- U5 pad 17: unconnected-(U5-COM3-Pad17) -> GND
- U7 pad 3: unconnected-(U7-CONTROL-Pad3) -> /1.8V_CTRL
Routing:
- net /PPG_INT: track 0.00 -> 4.32 mm, vias 0 -> 1
- net Net-(U1-XTAL_P): track 4.11 -> 1.71 mm
- net Net-(U1-XTAL_N): track 6.25 -> 3.94 mm
- net Net-(U3-EL2A): track 0.00 -> 2.20 mm, vias 0 -> 1
- net Net-(U3-EL1): track 0.00 -> 1.90 mm, vias 0 -> 1
