File: uprojects/Adam/kicad_pcb/reband/reband.kicad_pcb (KiCad board)
At the start: 4 copper layers, 26.1 x 31.3 mm, 49 parts, among them IC1 USBLC6-2SC6, J1 S2B-ZRLFSN, J2 USB4215-03-A, J3 POGOB, J4 POGOB, J5 Conn_01x02, J6 Conn_01x02, U1 ESP32-C3FH4, U2 TLV75533PDBVR, U3 MAX30009ENA+T, U4 BQ25100YFPR, U5 BNO055, U6 MAX30102EFD+T, U7 TCR2EF18_LMCT, Y1 ECS-400-18-33-JGN-TR3

Commit message: Update 4 June 2026
Parts:
- added C19: 3.3pF, Capacitor_SMD:C_0402_1005Metric_Pad0.74x0.62mm_HandSolder, F.Cu at (146.1, 83.1)
- added L1: LQG15HS2N2B02D, LQG15HS2N2B02D:INDC1005X55N, F.Cu at (145.5, 81.1)
- C4, C5: value 10pF -> 27pF
- C8: value 1pF -> 3.3pF
- S1, S2: moved to B.Cu
- moved C8 1.83 mm to (146.1, 79.5), turned to 0 degrees
- moved J4 0.86 mm to (131.3, 99.9)
- moved J3 0.83 mm to (148.0, 99.9)
- moved S2 0.72 mm to (149.1, 95.4), turned to -90 degrees
- moved J6 0.49 mm to (144.4, 100.8), turned to 90 degrees
- moved J2 0.37 mm to (130.0, 89.5)
- moved R6 0.37 mm to (130.4, 80.4)
- moved R12 0.37 mm to (138.1, 77.3)
- moved U7 0.37 mm to (137.9, 80.3)
- moved U2 0.37 mm to (133.4, 80.3)
- moved C17 0.37 mm to (133.0, 77.3)
- moved C3 0.37 mm to (135.5, 77.3)
- moved S1 0.26 mm to (149.1, 83.4), turned to -90 degrees
Connections:
- C8 pad 1: GND -> Net-(C8-Pad1)
- C8 pad 2: Net-(U1-LNA_IN) -> GND
- E1 pad 1: Net-(U1-LNA_IN) -> Net-(C8-Pad1)
Routing:
- net GND: track 31.3 -> 15.5 mm, vias 45 -> 41
- net /USB_D-: track 16.8 -> 6.45 mm, vias 2 -> 1
- net /USB_D+: track 17.9 -> 7.61 mm, vias 1 -> 2
- net +5V: track 27.2 -> 22.1 mm
- net Net-(J2-CC2): track 6.28 -> 1.26 mm
- net Net-(U1-LNA_IN): track 8.96 -> 4.13 mm
- net Net-(C8-Pad1): track 0.00 -> 4.18 mm
- net /Tx0: track 16.7 -> 13.4 mm
- net Net-(C10-Pad1): track 4.00 -> 1.36 mm, vias 1 -> 0
- net +3.3V: track 47.1 -> 45.2 mm
- net Net-(C11-Pad1): track 11.0 -> 9.13 mm
- net /Rx0: track 14.1 -> 12.7 mm
- net /RST: track 57.8 -> 56.4 mm, vias 5 -> 4
- net Net-(U2-IN): track 47.3 -> 46.0 mm
- net /GSR_INT: track 20.7 -> 19.5 mm
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Other:
- board text added: "+"
- board text added: "-"
- board text added: "BATT"

Commit message: Update 5 June 2026
Parts:
- moved C5 0.36 mm to (148.1, 87.3)
- moved C4 0.36 mm to (148.1, 89.6)
- moved J3 0.33 mm to (148.0, 99.6)
- moved J4 0.33 mm to (131.3, 99.6)
Routing:
- net +3.3V: track 45.2 -> 54.9 mm, vias 9 -> 10
- net +5V: track 22.1 -> 31.0 mm
- net GND: track 15.5 -> 9.79 mm, vias 41 -> 49
- net Net-(J2-CC2): track 1.26 -> 6.24 mm
- net /Rx0: track 12.7 -> 16.0 mm
- net +1V8: track 46.9 -> 43.9 mm
- net Net-(C10-Pad1): track 1.36 -> 4.09 mm, vias 0 -> 1
- net /RST: track 56.4 -> 54.0 mm
- net Net-(C11-Pad1): track 9.13 -> 11.5 mm
- net /Tx0: track 13.4 -> 15.3 mm
- net Net-(U3-EL4): track 7.76 -> 8.64 mm
- net Net-(U2-IN): track 46.0 -> 46.6 mm
- added copper zone on In1.Cu, net GND
