File: uprojects/Andrew G/Light chaser/Light chaser.kicad_pcb (KiCad board)
At the start: 2 copper layers, 91.9 x 106.2 mm, 21 parts, among them J1 Screw_Terminal_01x02, U1 NE555P, U2 4017

Commit message: Update 7 July 2026
Parts:
- removed U1: NE555P, Package_DIP:DIP-8_W7.62mm
- added U3: NA555D, NA555D:D8, F.Cu at (88.3, 66.1)
- U2: footprint Package_DIP:CERDIP-16_W7.62mm_SideBrazed -> Package_SO:SO-16_3.9x9.9mm_P1.27mm
- moved R3 35.8 mm to (73.9, 64.5), turned to 0 degrees
- moved C1 24.7 mm to (78.4, 68.6), turned to 180 degrees
- moved C3 23.7 mm to (90.8, 52.3), turned to 180 degrees
- moved C2 18.6 mm to (76.4, 62.0), turned to 0 degrees
- moved J1 18.6 mm to (85.8, 32.7)
- moved R2 18.2 mm to (94.0, 64.4), turned to 0 degrees
- moved U2 16.8 mm to (88.2, 79.5)
- moved D1 16.1 mm to (77.2, 100.3), turned to 180 degrees
- moved R4 11.2 mm to (102.4, 100.8)
- moved R1 10.0 mm to (94.0, 62.0), turned to 0 degrees
Routing:
- net Net-(D3-A): track 245.3 -> 0.00 mm
- net Net-(D4-A): track 193.6 -> 0.00 mm
- net Net-(D2-A): track 146.6 -> 0.00 mm, vias 1 -> 0
- net Net-(D5-A): track 127.1 -> 0.00 mm
- net GND: track 82.9 -> 0.00 mm, vias 1 -> 0
- net Net-(D6-A): track 58.4 -> 0.00 mm
- net Net-(D7-A): track 55.1 -> 0.00 mm
- net Net-(D8-A): track 51.4 -> 0.00 mm
- net Net-(D9-A): track 43.8 -> 0.00 mm
- net Net-(U2-CLK): track 42.0 -> 0.00 mm, vias 1 -> 0
- net Net-(D10-K): track 35.4 -> 0.00 mm
- net Net-(D10-A): track 34.9 -> 0.00 mm
- net Net-(D11-A): track 31.6 -> 0.00 mm
- net Net-(U3-THRES): track 29.0 -> 0.00 mm
- net VCC: track 14.5 -> 0.00 mm, vias 1 -> 0
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Other:
- board size 91.9 x 106.2 mm -> 51.9 x 79.9 mm
