File: uprojects/Andrew G/Light chaser/Light chaser.kicad_sch (KiCad schematic)
At the start: 21 parts, among them J1 Screw_Terminal_01x02, U1 NE555P, U2 4017

Commit message: Update 7 July 2026
Parts:
- removed U1: NE555P, Package_DIP:DIP-8_W7.62mm, symbol Timer:NE555P
- added U3: NA555D, NA555D:D8, symbol NA555D:NA555D
- U2: footprint Package_DIP:CERDIP-16_W7.62mm_SideBrazed -> Package_SO:SO-16_3.9x9.9mm_P1.27mm
Connections:
- net GND: now also U3.1 (GND)
- net VCC: now also U3.4 (RESET), U3.8 (VCC)
- net at R1.2, R2.1: now also U3.7 (DISCH)
- net at C1.1, R2.2: now also U3.2 (TRIG), U3.6 (THRES)
- net at C2.2: now also U3.5 (CONT)
- net at R3.2, U2.14 (CLK): now also U3.3 (OUT)
Changed lines of the file:
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@@
 	)
 	(junction
+		(at 82.55 72.39)
+		(diameter 0)
+		(color 0 0 0 0)
+	)
+	(junction
+		(at 54.61 77.47)
+		(diameter 0)
+		(color 0 0 0 0)
+	)
+	(junction
 		(at 176.53 63.5)
 		(diameter 0)
@@
 	)
 	(junction
-		(at 78.74 59.69)
-		(diameter 0)
-		(color 0 0 0 0)
-	)
-	(junction
 		(at 82.55 90.17)
 		(diameter 0)
@@
 	)
 	(junction
-		(at 55.88 77.47)
+		(at 78.74 59.69)
+		(diameter 0)
+		(color 0 0 0 0)
+	)
+	(junction
+		(at 68.58 90.17)
 		(diameter 0)
 		(color 0 0 0 0)
@@
 	)
 	(junction
-		(at 82.55 72.39)
-		(diameter 0)
-		(color 0 0 0 0)
-	)
-	(junction
 		(at 67.31 90.17)
 		(diameter 0)
@@
 	(wire
 		(pts
-			(xy 52.07 77.47) (xy 55.88 77.47)
+			(xy 52.07 77.47) (xy 54.61 77.47)
 		)
 		(stroke
@@
 	(wire
 		(pts
-			(xy 67.31 90.17) (xy 82.55 90.17)
+			(xy 67.31 90.17) (xy 68.58 90.17)
 		)
 		(stroke
@@
 	(wire
 		(pts
+			(xy 68.58 90.17) (xy 82.55 90.17)
+		)
+		(stroke
+			(width 0)
+			(type default)
+		)
+	)
+	(wire
+		(pts
 			(xy 105.41 62.23) (xy 105.41 72.39)
 		)
@@
 	(wire
 		(pts
-			(xy 69.85 62.23) (xy 69.85 59.69)
+			(xy 71.12 62.23) (xy 71.12 59.69)
 		)
 		(stroke
@@
 	(wire
 		(pts
-			(xy 67.31 82.55) (xy 67.31 90.17)
-		)
-		(stroke
-			(width 0)
-			(type default)
-		)
-	)
-	(wire
-		(pts
 			(xy 151.13 58.42) (xy 144.78 58.42)
 		)
@@
 	(wire
 		(pts
-			(xy 55.88 77.47) (xy 57.15 77.47)
+			(xy 176.53 73.66) (xy 176.53 78.74)
 		)
 		(stroke
@@
 	(wire
 		(pts
-			(xy 176.53 73.66) (xy 176.53 78.74)
+			(xy 54.61 80.01) (xy 54.61 77.47)
 		)
 		(stroke
@@
 	(wire
 		(pts
-			(xy 77.47 72.39) (xy 82.55 72.39)
+			(xy 158.75 73.66) (xy 176.53 73.66)
 		)
 		(stroke
@@
 	(wire
 		(pts
-			(xy 158.75 73.66) (xy 176.53 73.66)
+			(xy 142.24 64.77) (xy 139.7 64.77)
 		)
 		(stroke
@@
 	(wire
 		(pts
-			(xy 142.24 64.77) (xy 139.7 64.77)
+			(xy 149.86 68.58) (xy 149.86 67.31)
 		)
 		(stroke
@@
 	(wire
 		(pts
-			(xy 149.86 68.58) (xy 149.86 67.31)
+			(xy 57.15 80.01) (xy 54.61 80.01)
 		)
 		(stroke
@@
 	(wire
 		(pts
-			(xy 57.15 74.93) (xy 55.88 74.93)
+			(xy 176.53 104.14) (xy 176.53 109.22)
 		)
 		(stroke
@@
 	(wire
 		(pts
-			(xy 176.53 104.14) (xy 176.53 109.22)
+			(xy 127 99.06) (xy 127 101.6)
 		)
 		(stroke
@@
 	(wire
 		(pts
-			(xy 127 99.06) (xy 127 101.6)
+			(xy 82.55 81.28) (xy 82.55 82.55)
 		)
 		(stroke
@@
 	(wire
 		(pts
-			(xy 82.55 81.28) (xy 82.55 82.55)
+			(xy 158.75 68.58) (xy 176.53 68.58)
 		)
 		(stroke
@@
 	(wire
 		(pts
-			(xy 158.75 68.58) (xy 176.53 68.58)
+			(xy 149.86 67.31) (xy 139.7 67.31)
 		)
 		(stroke
@@
 	(wire
 		(pts
-			(xy 149.86 67.31) (xy 139.7 67.31)
+			(xy 90.17 49.53) (xy 90.17 46.99)
 		)
 		(stroke
@@
 	(wire
 		(pts
-			(xy 90.17 49.53) (xy 90.17 46.99)
+			(xy 151.13 63.5) (xy 142.24 63.5)
 		)
 		(stroke
@@
 	(wire
 		(pts
-			(xy 151.13 63.5) (xy 142.24 63.5)
+			(xy 80.01 72.39) (xy 82.55 72.39)
 		)
 		(stroke
@@
 	(wire
 		(pts
+			(xy 68.58 83.82) (xy 68.58 90.17)
+		)
+		(stroke
+			(width 0)
+			(type default)
+		)
+	)
+	(wire
+		(pts
 			(xy 147.32 88.9) (xy 147.32 77.47)
 		)
@@
 	(wire
 		(pts
+			(xy 54.61 77.47) (xy 57.15 77.47)
+		)
+		(stroke
+			(width 0)
+			(type default)
+		)
+	)
+	(wire
+		(pts
 			(xy 139.7 69.85) (xy 151.13 69.85)
 		)
@@
 	(wire
 		(pts
-			(xy 55.88 74.93) (xy 55.88 77.47)
-		)
-		(stroke
-			(width 0)
-			(type default)
-		)
-	)
-	(wire
-		(pts
 			(xy 176.53 99.06) (xy 176.53 104.14)
 		)
@@
 	(wire
 		(pts
-			(xy 69.85 59.69) (xy 78.74 59.69)
+			(xy 71.12 59.69) (xy 78.74 59.69)
 		)
 		(stroke
@@
 	)
 	(symbol
+		(lib_id "NA555D:NA555D")
+		(at 30.48 68.58 0)
+		(unit 1)
+		(body_style 1)
+		(exclude_from_sim no)
+		(in_bom yes)
+		(on_board yes)
+		(in_pos_files yes)
+		(dnp no)
+		(fields_autoplaced yes)
+		(property "Reference" "U3"
+			(at 83.312 66.04 0)
+			(show_name no)
+			(do_not_autoplace no)
+			(effects
+				(font
+					(size 1.524 1.524)
+				)
+			)
+		)
+		(property "Value" "NA555D"
+			(at 83.312 68.58 0)
+			(show_name no)
+			(do_not_autoplace no)
+			(effects
+				(font
+					(size 1.524 1.524)
+				)
+			)
+		)
+		(property "Footprint" "NA555D:D8"
+			(at 30.48 68.58 0)
+			(hide yes)
+			(show_name no)
+			(do_not_autoplace no)
+			(effects
+				(font
+					(size 1.27 1.27)
+					(italic yes)
+				)
+			)
+		)
+		(property "Datasheet" "https://www.ti.com/lit/gpn/na555"
+			(at 67.31 83.566 0)
+			(hide yes)
+			(show_name no)
+			(do_not_autoplace no)
+			(effects
+				(font
+					(size 1.27 1.27)
+					(italic yes)
+				)
+			)
+		)
+		(property "Description" ""
+			(at 30.48 68.58 0)
+			(hide yes)
+			(show_name no)
+			(do_not_autoplace no)
+			(effects
+				(font
+					(size 1.27 1.27)
+				)
+			)
+		)
+		(pin "1"
+		)
+		(pin "4"
+		)
+		(pin "3"
+		)
+		(pin "2"
+		)
+		(pin "7"
+		)
+		(pin "8"
+		)
+		(pin "5"
+		)
+		(pin "6"
+		)
+		(instances
+			(project "Light chaser"
+				(path "/c022ac8d-43db-4ad9-9e1e-e953e5b1763d"
+					(reference "U3")
+					(unit 1)
+				)
+			)
+		)
+	)
+	(symbol
 		(lib_id "Device:LED")
 		(at 154.94 78.74 180)
@@
 			)
 		)
-		(property "Footprint" "Package_DIP:CERDIP-16_W7.62mm_SideBrazed"
+		(property "Footprint" "Package_SO:SO-16_3.9x9.9mm_P1.27mm"
 			(at 127 74.93 0)
 			(hide yes)
@@
 					(unit 1)
 				)
-			)
-		)
-	)
-	(symbol
-		(lib_id "Timer:NE555P")
-		(at 67.31 72.39 0)
-		(unit 1)
-		(body_style 1)
-		(exclude_from_sim no)
-		(in_bom yes)
-		(on_board yes)
-		(in_pos_files yes)
-		(dnp no)
-		(fields_autoplaced yes)
-		(property "Reference" "U1"
-			(at 80.01 65.9698 0)
-			(show_name no)
-			(do_not_autoplace no)
-			(effects
-				(font
-					(size 1.27 1.27)
-				)
-			)
-		)
-		(property "Value" "NE555P"
-			(at 80.01 68.5098 0)
-			(show_name no)
-			(do_not_autoplace no)
-			(effects
-				(font
-					(size 1.27 1.27)
-				)
-			)
-		)
-		(property "Footprint" "Package_DIP:DIP-8_W7.62mm"
-			(at 67.31 96.52 0)
-			(hide yes)
-			(show_name no)
-			(do_not_autoplace no)
-			(effects
-				(font
-					(size 1.27 1.27)
-				)
-			)
-		)
-		(property "Datasheet" "http://www.ti.com/lit/ds/symlink/ne555.pdf"
-			(at 67.31 99.06 0)
-			(hide yes)
-			(show_name no)
-			(do_not_autoplace no)
-			(effects
-				(font
-					(size 1.27 1.27)
-				)
-			)
-		)
-		(property "Description" "Precision Timers, 555 compatible, PDIP-8"
-			(at 67.31 93.98 0)
-			(hide yes)
-			(show_name no)
-			(do_not_autoplace no)
-			(effects
-				(font
-					(size 1.27 1.27)
-				)
-			)
-		)
-		(pin "1"
-		)
-		(pin "4"
-		)
-		(pin "5"
-		)
-		(pin "2"
-		)
-		(pin "8"
-		)
-		(pin "7"
-		)
-		(pin "3"
-		)
-		(pin "6"
-		)
-		(instances
-			(project "Light chaser"
-				(path "/c022ac8d-43db-4ad9-9e1e-e953e5b1763d"
-					(reference "U1")
-					(unit 1)
-				)
